Commit message: Make URDF for flashlight and LED

File: subt_example/urdf/flashlight.urdf.xacro (robot description, xacro)
@@ -1,17 +1,74 @@
 <?xml version="1.0"?>
 <robot xmlns:xacro="http://ros.org/wiki/xacro" name="flashlight">
-  <xacro:macro name="flashlight" params="flashlight_prefix">
-    <include>
-      <uri>model://flashlight</uri>
-    </include>
-    <joint name="joint" type="fixed">
-  		<parent link="base_link"/>
-  		<child link="flashlight_model::handle"/>
-    </joint>
-		<!--<gazebo>
-      <plugin name="${flashlight_prefix}_flashlight_control" filename="libdummy.so">
-        <service_name>${flash_light_prefix}_flashlight/switch</service_name>
-      </plugin>
-		</gazebo>-->
+  <xacro:macro name="flashlight" params="flashlight_prefix parent_link *pose">
+    <gazebo>
+      <model name='${flashlight_prefix}_flashlight_model'>
+        <xacro:insert_block name="pose"/>
+        <link name='handle'>
+          <pose>0 0 0.075 0 0 0</pose>
+          <collision name='collision'>
+            <geometry>
+              <cylinder>
+                <radius>0.025</radius>
+                <length>0.15</length>
+              </cylinder>
+            </geometry>
+          </collision>
+          <visual name='visual'>
+            <geometry>
+              <cylinder>
+                <radius>0.025</radius>
+                <length>0.15</length>
+              </cylinder>
+            </geometry>
+          </visual>
+        </link>
+        <link name='light_source'>
+          <pose>0 0 0.15 0 0 0</pose>
+          <light name='lamp' type='spot'>
+            <pose>0 0 0.0 0 3.14159 0</pose>
+            <attenuation>
+              <range>50</range>
+              <linear>0.05</linear>
+            </attenuation>
+            <diffuse>1 1 1 1</diffuse>
+            <specular>1 1 1 1</specular>
+            <spot>
+              <inner_angle>1</inner_angle>
+              <outer_angle>1.1</outer_angle>
+              <falloff>1</falloff>
+            </spot>
+            <direction>0 0 -1</direction>
+          </light>
+          <visual name='lamp'>
+            <geometry>
+              <sphere>
+                <radius>0.025</radius>
+              </sphere>
+            </geometry>
+            <transparency>0</transparency>
+            <material>
+              <ambient>1 1 1 1</ambient>
+              <diffuse>1 1 1 1</diffuse>
+              <specular>1 1 1 1</specular>
+              <emissive>1 1 1 1</emissive>
+            </material>
+          </visual>
+        </link>
+        <joint name='joint' type='fixed'>
+          <parent>handle</parent>
+          <child>light_source</child>
+        </joint>
+        <!--
+        <plugin?
+        -->
+      </model>
+    </gazebo>
+    <gazebo>
+      <joint name='${flashlight_prefix}_flashlight_joint' type='fixed'>
+        <parent>${parent_link}</parent>
+        <child>${flashlight_prefix}_flashlight_model::handle</child>
+      </joint>
+    </gazebo>
 	</xacro:macro>
 </robot>

Commit message: Improve the tunnel appearance

File: subt_example/urdf/flashlight.urdf.xacro (robot description, xacro)
@@ -22,4 +22,7 @@
               </cylinder>
             </geometry>
+            <material>
+              <ambient>0 0 0 1</ambient>
+            </material>
           </visual>
         </link>

File: subt_example/urdf/husky_equipments.urdf.xacro (robot description, xacro)
@@ -7,5 +7,5 @@
   </xacro:flashlight>
   <xacro:flashlight flashlight_prefix="downward" parent_link="base_link">
-    <pose>0.4 0 0.4 0 ${M_PI*0.75} 0</pose>
+    <pose>0.4 0 0.4 0 ${M_PI*0.6} 0</pose>
   </xacro:flashlight>
   <xacro:flashlight flashlight_prefix="left" parent_link="base_link">

File: subt_example/urdf/jackal_equipments.urdf.xacro (robot description, xacro)
@@ -8,5 +8,5 @@
   </xacro:flashlight>
   <xacro:flashlight flashlight_prefix="downward" parent_link="base_link">
-    <pose>0.2 0 0.25 0 ${M_PI*0.75} 0</pose>
+    <pose>0.2 0 0.25 0 ${M_PI*0.6} 0</pose>
   </xacro:flashlight>
   <xacro:flashlight flashlight_prefix="left" parent_link="base_link">
