Commit message: Implement LED light plugin

File: subt_example/urdf/husky_equipments.urdf.xacro (robot description, xacro)
@@ -5,19 +5,61 @@
   <xacro:flashlight flashlight_prefix="right" parent_link="base_link">
     <pose>0.3 -0.3 0.3 0 ${M_PI*0.5} ${-M_PI*0.1}</pose>
+    <block>
+      <duration>1</duration>
+      <interval>0</interval>
+      <color>1 1 1</color>
+    </block>
   </xacro:flashlight>
   <xacro:flashlight flashlight_prefix="downward" parent_link="base_link">
     <pose>0.4 0 0.4 0 ${M_PI*0.6} 0</pose>
+    <block>
+      <duration>1</duration>
+      <interval>0</interval>
+      <color>1 1 1</color>
+    </block>
   </xacro:flashlight>
   <xacro:flashlight flashlight_prefix="left" parent_link="base_link">
     <pose>0.3 0.3 0.3 0 ${M_PI*0.5} ${M_PI*0.1}</pose>
+    <block>
+      <duration>1</duration>
+      <interval>0</interval>
+      <color>1 1 1</color>
+    </block>
   </xacro:flashlight>
   <xacro:led led_prefix="right" parent_link="base_link" color="1 0 0">
     <pose>-0.3 -0.3 0.3 0 0 0</pose>
+    <params>
+      <duration>0.5</duration>
+      <interval>0.5</interval>
+      <color>1 0.8 0</color>
+    </params>
   </xacro:led>
   <xacro:led led_prefix="center" parent_link="base_link" color="0 1 0">
     <pose>-0.3 0 0.3 0 0 0</pose>
+    <params>
+      <block>
+        <duration>0.25</duration>
+        <interval>0</interval>
+        <color>1 0 0</color>
+      </block>
+      <block>
+        <duration>0.25</duration>
+        <interval>0</interval>
+        <color>0 1 0</color>
+      </block>
+      <block>
+        <duration>0.25</duration>
+        <interval>0</interval>
+        <color>0 0 1</color>
+      </block>
+    </params>
   </xacro:led>
   <xacro:led led_prefix="left" parent_link="base_link" color="0 0 1">
     <pose>-0.3 0.3 0.3 0 0 0</pose>
+    <params>
+      <duration>0.5</duration>
+      <interval>0.5</interval>
+      <color>1 0.8 0</color>
+    </params>
   </xacro:led>
 </robot>

File: subt_example/urdf/jackal_equipments.urdf.xacro (robot description, xacro)
@@ -6,19 +6,61 @@
   <xacro:flashlight flashlight_prefix="right" parent_link="base_link">
     <pose>0.0 -0.2 0.2 0 ${M_PI*0.5} ${-M_PI*0.1}</pose>
+    <block>
+      <duration>1</duration>
+      <interval>0</interval>
+      <color>1 1 1</color>
+    </block>
   </xacro:flashlight>
   <xacro:flashlight flashlight_prefix="downward" parent_link="base_link">
     <pose>0.2 0 0.25 0 ${M_PI*0.6} 0</pose>
+    <block>
+      <duration>1</duration>
+      <interval>0</interval>
+      <color>1 1 1</color>
+    </block>
   </xacro:flashlight>
   <xacro:flashlight flashlight_prefix="left" parent_link="base_link">
     <pose>0.0 0.2 0.2 0 ${M_PI*0.5} ${M_PI*0.1}</pose>
+    <block>
+      <duration>1</duration>
+      <interval>0</interval>
+      <color>1 1 1</color>
+    </block>
   </xacro:flashlight>
   <xacro:led led_prefix="right" parent_link="base_link" color="1 0 0">
     <pose>-0.2 -0.2 0.25 0 0 0</pose>
+    <params>
+      <duration>0.5</duration>
+      <interval>0.5</interval>
+      <color>1 0.8 0</color>
+    </params>
   </xacro:led>
   <xacro:led led_prefix="center" parent_link="base_link" color="0 1 0">
     <pose>-0.2 0 0.25 0 0 0</pose>
+    <params>
+      <block>
+        <duration>0.25</duration>
+        <interval>0</interval>
+        <color>1 0 0</color>
+      </block>
+      <block>
+        <duration>0.25</duration>
+        <interval>0</interval>
+        <color>0 1 0</color>
+      </block>
+      <block>
+        <duration>0.25</duration>
+        <interval>0</interval>
+        <color>0 0 1</color>
+      </block>
+    </params>
   </xacro:led>
   <xacro:led led_prefix="left" parent_link="base_link" color="0 0 1">
     <pose>-0.2 0.2 0.25 0 0 0</pose>
+    <params>
+      <duration>0.5</duration>
+      <interval>0.5</interval>
+      <color>1 0.8 0</color>
+    </params>
   </xacro:led>
 </robot>

File: subt_gazebo/urdf/flashlight.urdf.xacro (robot description, xacro)
@@ -1,7 +1,7 @@
 <?xml version="1.0"?>
 <robot xmlns:xacro="http://ros.org/wiki/xacro" name="flashlight">
-  <xacro:macro name="flashlight" params="flashlight_prefix parent_link *pose">
+  <xacro:macro name="flashlight" params="flashlight_prefix parent_link *pose **plugin_params">
     <gazebo>
-      <model name='${flashlight_prefix}_flashlight_model'>
+      <model name='${flashlight_prefix}_flashlight'>
         <xacro:insert_block name="pose"/>
         <link name='handle'>
@@ -63,7 +63,11 @@
           <child>light_source</child>
         </joint>
-        <!--
-        <plugin?
-        -->
+        <plugin name='light_control' filename='libRosLedPlugin.so'>
+          <service_name>flashlight_switch</service_name>
+          <light>
+            <id>light_source/lamp</id>
+            <xacro:insert_block name="plugin_params"/>
+          </light>
+        </plugin>
       </model>
     </gazebo>
@@ -71,5 +75,5 @@
       <joint name='${flashlight_prefix}_flashlight_joint' type='fixed'>
         <parent>${parent_link}</parent>
-        <child>${flashlight_prefix}_flashlight_model::handle</child>
+        <child>${flashlight_prefix}_flashlight::handle</child>
       </joint>
     </gazebo>

File: subt_gazebo/urdf/led.urdf.xacro (robot description, xacro)
@@ -1,7 +1,7 @@
 <?xml version="1.0"?>
 <robot xmlns:xacro="http://ros.org/wiki/xacro" name="flashlight">
-  <xacro:macro name="led" params="led_prefix parent_link color *pose">
+  <xacro:macro name="led" params="led_prefix parent_link color *pose **plugin_params">
     <gazebo>
-      <model name='${led_prefix}_led_model'>
+      <model name='${led_prefix}_led'>
         <xacro:insert_block name='pose'/>
         <link name='led_body'>
@@ -13,5 +13,5 @@
             </geometry>
           </collision>
-          <visual name='visual'>
+          <visual name='marker'>
             <geometry>
               <sphere>
@@ -26,5 +26,5 @@
             </material>
           </visual>
-          <light name='light' type='point'>
+          <light name='marker' type='point'>
             <pose>0 0 0 0 0 0</pose>
             <attenuation>
@@ -36,7 +36,11 @@
           </light>
         </link>
-        <!--
-        <plugin?
-        -->
+        <plugin name='light_control' filename='libRosLedPlugin.so'>
+          <service_name>led_switch</service_name>
+          <light>
+            <id>led_body/marker</id>
+            <xacro:insert_block name="plugin_params"/>
+          </light>
+        </plugin>
       </model>
     </gazebo>
@@ -44,5 +48,5 @@
       <joint name='${led_prefix}_led_joint' type='fixed'>
         <parent>${parent_link}</parent>
-        <child>${led_prefix}_led_model::led_body</child>
+        <child>${led_prefix}_led::led_body</child>
       </joint>
     </gazebo>

Commit message: Add lights on Iris

File: subt_example/urdf/husky_equipments.urdf.xacro (robot description, xacro)
@@ -1,4 +1,5 @@
 <?xml version="1.0"?>
 <robot xmlns:xacro="http://ros.org/wiki/xacro" name="lights">
+  <xacro:property name="M_PI" value="3.14159"/>
   <xacro:include filename="$(find subt_gazebo)/urdf/flashlight.urdf.xacro" />
   <xacro:include filename="$(find subt_gazebo)/urdf/led.urdf.xacro" />

File: subt_example/urdf/iris_with_sensors.xacro (robot description, xacro)
@@ -32,3 +32,4 @@
     <origin xyz="0.0 0.0 0.0" rpy="0.0 0.0 0.0" />
   </xacro:odometry_plugin_macro>
+  <xacro:include filename="$(find subt_example)/urdf/iris_equipments.urdf.xacro" />
 </robot>

Commit message: Update config and light settings

File: subt_example/urdf/husky_equipments.urdf.xacro (robot description, xacro)
@@ -6,49 +6,60 @@
   <xacro:flashlight flashlight_prefix="right" parent_link="base_link">
     <pose>0.3 -0.3 0.3 0 ${M_PI*0.5} ${-M_PI*0.1}</pose>
-    <block>
-      <duration>1</duration>
-      <interval>0</interval>
-      <color>1 1 1</color>
-    </block>
+    <params>
+      <enable>false</enable>
+      <block>
+        <duration>1</duration>
+        <interval>0</interval>
+        <color>1 1 1</color>
+      </block>
+    </params>
   </xacro:flashlight>
   <xacro:flashlight flashlight_prefix="downward" parent_link="base_link">
     <pose>0.4 0 0.4 0 ${M_PI*0.6} 0</pose>
-    <block>
-      <duration>1</duration>
-      <interval>0</interval>
-      <color>1 1 1</color>
-    </block>
+    <params>
+      <enable>false</enable>
+      <block>
+        <duration>1</duration>
+        <interval>0</interval>
+        <color>1 1 1</color>
+      </block>
+    </params>
   </xacro:flashlight>
   <xacro:flashlight flashlight_prefix="left" parent_link="base_link">
     <pose>0.3 0.3 0.3 0 ${M_PI*0.5} ${M_PI*0.1}</pose>
-    <block>
-      <duration>1</duration>
-      <interval>0</interval>
-      <color>1 1 1</color>
-    </block>
+    <params>
+      <enable>false</enable>
+      <block>
+        <duration>1</duration>
+        <interval>0</interval>
+        <color>1 1 1</color>
+      </block>
+    </params>
   </xacro:flashlight>
-  <xacro:led led_prefix="right" parent_link="base_link" color="1 0 0">
+  <xacro:led led_prefix="right" parent_link="base_link">
     <pose>-0.3 -0.3 0.3 0 0 0</pose>
     <params>
-      <duration>0.5</duration>
-      <interval>0.5</interval>
+      <enable>false</enable>
+      <duration>0.3</duration>
+      <interval>0.3</interval>
       <color>1 0.8 0</color>
     </params>
   </xacro:led>
-  <xacro:led led_prefix="center" parent_link="base_link" color="0 1 0">
+  <xacro:led led_prefix="center" parent_link="base_link">
     <pose>-0.3 0 0.3 0 0 0</pose>
     <params>
+      <enable>false</enable>
       <block>
-        <duration>0.25</duration>
+        <duration>0.2</duration>
         <interval>0</interval>
         <color>1 0 0</color>
       </block>
       <block>
-        <duration>0.25</duration>
+        <duration>0.2</duration>
         <interval>0</interval>
         <color>0 1 0</color>
       </block>
       <block>
-        <duration>0.25</duration>
+        <duration>0.2</duration>
         <interval>0</interval>
         <color>0 0 1</color>
@@ -56,9 +67,10 @@
     </params>
   </xacro:led>
-  <xacro:led led_prefix="left" parent_link="base_link" color="0 0 1">
+  <xacro:led led_prefix="left" parent_link="base_link">
     <pose>-0.3 0.3 0.3 0 0 0</pose>
     <params>
-      <duration>0.5</duration>
-      <interval>0.5</interval>
+      <enable>false</enable>
+      <duration>0.3</duration>
+      <interval>0.3</interval>
       <color>1 0.8 0</color>
     </params>

File: subt_example/urdf/iris_equipments.urdf.xacro (robot description, xacro)
@@ -7,4 +7,5 @@
     <pose>0 0 0.1 0 ${M_PI/3*2} 0</pose>
     <block>
+      <enable>false</enable>
       <duration>1</duration>
       <interval>0</interval>
@@ -12,19 +13,29 @@
     </block>
   </xacro:flashlight>
-  <xacro:led led_prefix="center" parent_link="${namespace}/base_link" color="0 1 0">
+  <xacro:led led_prefix="right" parent_link="${namespace}/base_link">
+    <pose>-0.05 -0.05 0.05 0 0 0</pose>
+    <params>
+      <enable>false</enable>
+      <duration>0.3</duration>
+      <interval>0.3</interval>
+      <color>1 0.8 0</color>
+    </params>
+  </xacro:led>
+  <xacro:led led_prefix="center" parent_link="${namespace}/base_link">
     <pose>0 0 -0.05 0 0 0</pose>
     <params>
+      <enable>false</enable>
       <block>
-        <duration>0.25</duration>
+        <duration>0.2</duration>
         <interval>0</interval>
         <color>1 0 0</color>
       </block>
       <block>
-        <duration>0.25</duration>
+        <duration>0.2</duration>
         <interval>0</interval>
         <color>0 1 0</color>
       </block>
       <block>
-        <duration>0.25</duration>
+        <duration>0.2</duration>
         <interval>0</interval>
         <color>0 0 1</color>
@@ -32,3 +43,12 @@
     </params>
   </xacro:led>
+  <xacro:led led_prefix="left" parent_link="${namespace}/base_link">
+    <pose>-0.05 0.05 0.05 0 0 0</pose>
+    <params>
+      <enable>false</enable>
+      <duration>0.3</duration>
+      <interval>0.3</interval>
+      <color>1 0.8 0</color>
+    </params>
+  </xacro:led>
 </robot>

File: subt_example/urdf/jackal_equipments.urdf.xacro (robot description, xacro)
@@ -6,49 +6,60 @@
   <xacro:flashlight flashlight_prefix="right" parent_link="base_link">
     <pose>0.0 -0.2 0.2 0 ${M_PI*0.5} ${-M_PI*0.1}</pose>
-    <block>
-      <duration>1</duration>
-      <interval>0</interval>
-      <color>1 1 1</color>
-    </block>
+    <params>
+      <enable>false</enable>
+      <block>
+        <duration>1</duration>
+        <interval>0</interval>
+        <color>1 1 1</color>
+      </block>
+    </params>
   </xacro:flashlight>
   <xacro:flashlight flashlight_prefix="downward" parent_link="base_link">
     <pose>0.2 0 0.25 0 ${M_PI*0.6} 0</pose>
-    <block>
-      <duration>1</duration>
-      <interval>0</interval>
-      <color>1 1 1</color>
-    </block>
+    <params>
+      <enable>false</enable>
+      <block>
+        <duration>1</duration>
+        <interval>0</interval>
+        <color>1 1 1</color>
+      </block>
+    </params>
   </xacro:flashlight>
   <xacro:flashlight flashlight_prefix="left" parent_link="base_link">
     <pose>0.0 0.2 0.2 0 ${M_PI*0.5} ${M_PI*0.1}</pose>
-    <block>
-      <duration>1</duration>
-      <interval>0</interval>
-      <color>1 1 1</color>
-    </block>
+    <params>
+      <enable>false</enable>
+      <block>
+        <duration>1</duration>
+        <interval>0</interval>
+        <color>1 1 1</color>
+      </block>
+    </params>
   </xacro:flashlight>
-  <xacro:led led_prefix="right" parent_link="base_link" color="1 0 0">
+  <xacro:led led_prefix="right" parent_link="base_link">
     <pose>-0.2 -0.2 0.25 0 0 0</pose>
     <params>
-      <duration>0.5</duration>
-      <interval>0.5</interval>
+      <enable>false</enable>
+      <duration>0.3</duration>
+      <interval>0.3</interval>
       <color>1 0.8 0</color>
     </params>
   </xacro:led>
-  <xacro:led led_prefix="center" parent_link="base_link" color="0 1 0">
+  <xacro:led led_prefix="center" parent_link="base_link">
     <pose>-0.2 0 0.25 0 0 0</pose>
     <params>
+      <enable>false</enable>
       <block>
-        <duration>0.25</duration>
+        <duration>0.2</duration>
         <interval>0</interval>
         <color>1 0 0</color>
       </block>
       <block>
-        <duration>0.25</duration>
+        <duration>0.2</duration>
         <interval>0</interval>
         <color>0 1 0</color>
       </block>
       <block>
-        <duration>0.25</duration>
+        <duration>0.2</duration>
         <interval>0</interval>
         <color>0 0 1</color>
@@ -56,9 +67,10 @@
     </params>
   </xacro:led>
-  <xacro:led led_prefix="left" parent_link="base_link" color="0 0 1">
+  <xacro:led led_prefix="left" parent_link="base_link">
     <pose>-0.2 0.2 0.25 0 0 0</pose>
     <params>
-      <duration>0.5</duration>
-      <interval>0.5</interval>
+      <enable>false</enable>
+      <duration>0.3</duration>
+      <interval>0.3</interval>
       <color>1 0.8 0</color>
     </params>

File: subt_gazebo/urdf/flashlight.urdf.xacro (robot description, xacro)
@@ -1,5 +1,5 @@
 <?xml version="1.0"?>
 <robot xmlns:xacro="http://ros.org/wiki/xacro" name="flashlight">
-  <xacro:macro name="flashlight" params="flashlight_prefix parent_link *pose **plugin_params">
+  <xacro:macro name="flashlight" params="flashlight_prefix parent_link default_color:='0 0 0' *pose **plugin_params">
     <gazebo>
       <model name='${flashlight_prefix}_flashlight'>
@@ -57,6 +57,6 @@
               <linear>0.05</linear>
             </attenuation>
-            <diffuse>1 1 1 1</diffuse>
-            <specular>1 1 1 1</specular>
+            <diffuse>${default_color} 1</diffuse>
+            <specular>${default_color} 1</specular>
             <spot>
               <inner_angle>1</inner_angle>
@@ -77,5 +77,5 @@
               <diffuse>1 1 1 1</diffuse>
               <specular>1 1 1 1</specular>
-              <emissive>1 1 1 1</emissive>
+              <emissive>${default_color} 1</emissive>
             </material>
           </visual>

File: subt_gazebo/urdf/led.urdf.xacro (robot description, xacro)
@@ -1,5 +1,5 @@
 <?xml version="1.0"?>
 <robot xmlns:xacro="http://ros.org/wiki/xacro" name="flashlight">
-  <xacro:macro name="led" params="led_prefix parent_link color *pose **plugin_params">
+  <xacro:macro name="led" params="led_prefix parent_link default_color:='0 0 0' *pose **plugin_params">
     <gazebo>
       <model name='${led_prefix}_led'>
@@ -37,5 +37,5 @@
               <diffuse>1 1 1 1</diffuse>
               <specular>1 1 1 1</specular>
-              <emissive>${color} 1</emissive>
+              <emissive>${default_color} 1</emissive>
             </material>
           </visual>
@@ -46,6 +46,6 @@
               <linear>0.10</linear>
             </attenuation>
-            <diffuse>${color} 1</diffuse>
-            <specular>${color} 1</specular>
+            <diffuse>${default_color} 1</diffuse>
+            <specular>${default_color} 1</specular>
           </light>
         </link>
