Commit message: Adding a magnetometer, pressure sensor and two cameras to Iris.

File: subt_example/urdf/iris_with_sensors.xacro (robot description, xacro)
@@ -32,3 +32,43 @@
     <origin xyz="0.0 0.0 0.0" rpy="0.0 0.0 0.0" />
   </xacro:odometry_plugin_macro>
+  <!-- Mount a magnetometer. -->
+  <xacro:default_magnetometer namespace="${namespace}" parent_link="${namespace}/base_link" />
+  <!-- Mount a pressure sensor. -->
+  <xacro:default_pressure_sensor namespace="${namespace}" parent_link="${namespace}/base_link" />
+  <!-- Front camera. -->
+  <xacro:camera_macro
+    namespace="${namespace}"
+    parent_link="${namespace}/base_link"
+    camera_suffix="front"
+    frame_rate="30"
+    horizontal_fov="2"
+    image_width="752"
+    image_height="480"
+    image_format="L8"
+    min_distance="0.02"
+    max_distance="50"
+    noise_mean="0.0"
+    noise_stddev="0.007"
+    enable_visual="false">
+    <box size="0.02 0.05 0.05" />
+    <origin xyz="0.1 0 0" rpy="0 0 0" />
+  </xacro:camera_macro>
+  <!-- Lower camera. -->
+  <xacro:camera_macro
+    namespace="${namespace}"
+    parent_link="${namespace}/base_link"
+    camera_suffix="lower"
+    frame_rate="30"
+    horizontal_fov="2"
+    image_width="752"
+    image_height="480"
+    image_format="L8"
+    min_distance="0.02"
+    max_distance="50"
+    noise_mean="0.0"
+    noise_stddev="0.007"
+    enable_visual="false">
+    <box size="0.02 0.05 0.05" />
+    <origin xyz="0 0 -0.07" rpy="0 1.57 0" />
+  </xacro:camera_macro>
 </robot>
