Commit message: Add plugin for LEDs

File: x1_description/urdf/led.urdf.xacro (robot description, xacro)
@@ -1,5 +1,5 @@
 <?xml version="1.0"?>
 <robot xmlns:xacro="http://ros.org/wiki/xacro" name="led">
-  <xacro:macro name="led" params="led_prefix *joint_pose">
+  <xacro:macro name="led" params="led_prefix xyz rpy **plugin_params">
     <link name="${led_prefix}_led_link">
       <visual name="marker">
@@ -9,41 +9,58 @@
         </geometry>
       </visual>
-<!--
-      <gazebo>
-        <light name="marker" type='point'>
-          <pose>0 0 0 0 0 0</pose>
-          <attenuation>
-            <range>50</range>
-            <linear>0.05</linear>
-          </attenuation>
-          <diffuse>1 1 1 1</diffuse>
-          <specular>1 1 1 1</specular>
-          <spot>
-            <inner_angle>2</inner_angle>
-            <outer_angle>2.1</outer_angle>
-            <falloff>1</falloff>
-          </spot>
-          <direction>1 0 0</direction>
-        </light>
-      </gazebo>-->
     </link>
-<!--
-    <gazebo>
-      <plugin name='light_control' filename='libRosFlashLightPlugin.so'>
-        <service_name>enable</service_name>
-        <light>
-          <id>${led_prefix}_led_link/marker</id>
-          <enable>false</enable>
-          <duration>1</duration>
-          <interval>0</interval>
-          <color>1 1 1</color>
-        </light>
-      </plugin>
-    </gazebo>-->
     <joint name="${led_prefix}_led" type="fixed">
       <parent link="base_link"/>
       <child link="${led_prefix}_led_link"/>
-      <xacro:insert_block name="joint_pose"/>
+      <origin xyz="${xyz}" rpy="${rpy}"/>
     </joint>
+    <gazebo>
+      <model name="${led_prefix}_led_lamp">
+        <pose>${xyz} ${rpy}</pose>
+        <link name="body">
+          <pose>0 0 0.0005 0 0 0</pose>
+          <light name='light_source' type='point'>
+            <pose>0 0 0 0 0 0</pose>
+            <attenuation>
+              <range>0.20</range>
+              <linear>0.10</linear>
+            </attenuation>
+            <diffuse>0 0 0 1</diffuse>
+            <specular>0 0 0 1</specular>
+          </light>
+          <visual name="light_source">
+            <geometry>
+              <mesh>
+                <uri>package://x1_description/meshes/led_lamp.dae</uri>
+              </mesh>
+            </geometry>
+            <transparency>1</transparency>
+            <material>
+              <ambient>1 1 1 1</ambient>
+              <diffuse>1 1 1 1</diffuse>
+              <specular>1 1 1 1</specular>
+              <emissive>0 0 0 1</emissive>
+            </material>
+          </visual>
+        </link>
+        <plugin name='light_control' filename='libRosFlashLightPlugin.so'>
+          <service_name>enable</service_name>
+          <light>
+            <id>body/light_source</id>
+            <xacro:insert_block name="plugin_params"/>
+            <enable>false</enable>
+            <duration>1</duration>
+            <interval>0</interval>
+            <color>1 1 1</color>
+          </light>
+        </plugin>
+      </model>
+    </gazebo>
+    <gazebo>
+      <joint name="${led_prefix}_led" type="fixed">
+        <parent>base_link</parent>
+        <child>${led_prefix}_led_lamp::body</child>
+      </joint>
+    </gazebo>
   </xacro:macro>
 </robot>

File: x1_description/urdf/x1.urdf.xacro (robot description, xacro)
@@ -126,24 +126,66 @@
     xyz="0.461459  -0.216803 0.124431" rpy="0 0 3.1416" />
    <!-- LEDs -->
-  <xacro:led led_prefix="rear_left">
-    <origin xyz="-0.42493 -0.13619 0.209188" rpy="0 1.573 3.1416" />
-  </xacro:led>
-  <xacro:led led_prefix="rear_center">
-    <origin xyz="-0.42493 0 0.209188" rpy="0 1.573 3.1416" />
-  </xacro:led>
-  <xacro:led led_prefix="rear_right">
-    <origin xyz="-0.42493 0.13619 0.209188" rpy="0 1.573 3.1416" />
-  </xacro:led>
-  <xacro:led led_prefix="left_lateral_rear">
-    <origin xyz="0.066047 -0.212211 0.209188" rpy="0 1.573 -1.539" />
-  </xacro:led>
-  <xacro:led led_prefix="left_lateral_front">
-    <origin xyz="-0.066047 -0.212211 0.209188" rpy="0 1.573 -1.539" />
-  </xacro:led>
-  <xacro:led led_prefix="right_lateral_rear">
-    <origin xyz="0.066047 0.212211 0.209188" rpy="0 1.573 1.539" />
-  </xacro:led>
-  <xacro:led led_prefix="right_lateral_front">
-    <origin xyz="-0.066047 0.212211 0.209188" rpy="0 1.573 1.539" />
+  <xacro:led led_prefix="rear_right" xyz="-0.42493 -0.13619 0.209188" rpy="0 1.573 3.1416">
+    <plugin_params>
+      <block>
+        <duration>0.2</duration>
+        <interval>0.2</interval>
+        <color>0 1 0</color>
+      </block>
+    </plugin_params>
+  </xacro:led>
+  <xacro:led led_prefix="rear_center" xyz="-0.42493 0 0.209188" rpy="0 1.573 3.1416">
+    <plugin_params>
+      <block>
+        <duration>0.2</duration>
+        <interval>0.2</interval>
+        <color>1 1 0</color>
+      </block>
+    </plugin_params>
+  </xacro:led>
+  <xacro:led led_prefix="rear_left" xyz="-0.42493 0.13619 0.209188" rpy="0 1.573 3.1416">
+    <plugin_params>
+      <block>
+        <duration>0.2</duration>
+        <interval>0.2</interval>
+        <color>1 0 0</color>
+      </block>
+    </plugin_params>
+  </xacro:led>
+  <xacro:led led_prefix="right_lateral_front" xyz="0.066047 -0.212211 0.209188" rpy="0 1.573 -1.539">
+    <plugin_params>
+      <block>
+        <duration>0.2</duration>
+        <interval>0.2</interval>
+        <color>0 1 0</color>
+      </block>
+    </plugin_params>
+  </xacro:led>
+  <xacro:led led_prefix="right_lateral_rear" xyz="-0.066047 -0.212211 0.209188" rpy="0 1.573 -1.539">
+    <plugin_params>
+      <block>
+        <duration>0.1</duration>
+        <interval>0.1</interval>
+        <color>0 1 0</color>
+      </block>
+    </plugin_params>
+  </xacro:led>
+  <xacro:led led_prefix="left_lateral_front" xyz="0.066047 0.212211 0.209188" rpy="0 1.573 1.539">
+    <plugin_params>
+      <block>
+        <duration>0.2</duration>
+        <interval>0.2</interval>
+        <color>1 0 0</color>
+      </block>
+    </plugin_params>
+  </xacro:led>
+  <xacro:led led_prefix="left_lateral_rear" xyz="-0.066047 0.212211 0.209188" rpy="0 1.573 1.539">
+    <plugin_params>
+      <block>
+        <duration>0.1</duration>
+        <interval>0.1</interval>
+        <color>1 0 0</color>
+      </block>
+    </plugin_params>
   </xacro:led>
   <xacro:if value="$(arg laser_enabled)">
