Commit message: Add plugin for headlights

File: x1_description/urdf/headlight.urdf.xacro (robot description, xacro)
@@ -1,5 +1,5 @@
 <?xml version="1.0"?>
 <robot xmlns:xacro="http://ros.org/wiki/xacro" name="headlight">
-  <xacro:macro name="headlight" params="headlight_prefix *joint_pose">
+  <xacro:macro name="headlight" params="headlight_prefix xyz rpy">
     <link name="${headlight_prefix}_headlight_link">
       <visual>
@@ -13,6 +13,59 @@
       <parent link="base_link"/>
       <child link="${headlight_prefix}_headlight_link"/>
-      <xacro:insert_block name="joint_pose"/>
+      <origin xyz="${xyz}" rpy="${rpy}"/>
     </joint>
+    <gazebo>
+      <model name="${headlight_prefix}_headlight_lamp">
+        <pose>${xyz} ${rpy}</pose>
+        <link name="body">
+          <pose>-0.0005 0 0 0 0 0</pose>
+          <light name="light_source" type="spot">
+            <pose>-0.025 0 0.06 0 1.573 0</pose>
+            <attenuation>
+              <range>50</range>
+              <linear>0.05</linear>
+            </attenuation>
+            <diffuse>0 0 0 1</diffuse>
+            <specular>0 0 0 1</specular>
+            <spot>
+              <inner_angle>1</inner_angle>
+              <outer_angle>1.1</outer_angle>
+              <falloff>1</falloff>
+            </spot>
+            <direction>0 0 -1</direction>
+          </light>
+          <visual name="light_source">
+            <geometry>
+              <mesh>
+                <uri>package://x1_description/meshes/headlight_lamp.dae</uri>
+              </mesh>
+            </geometry>
+            <transparency>1</transparency>
+            <material>
+              <ambient>1 1 1 1</ambient>
+              <diffuse>1 1 1 1</diffuse>
+              <specular>1 1 1 1</specular>
+              <emissive>0 0 0 1</emissive>
+            </material>
+          </visual>
+        </link>
+        <plugin name='light_control' filename='libRosFlashLightPlugin.so'>
+          <service_name>enable</service_name>
+          <light>
+            <id>body/light_source</id>
+            <enable>false</enable>
+            <duration>1</duration>
+            <interval>0</interval>
+            <color>1 1 1</color>
+          </light>
+        </plugin>
+      </model>
+    </gazebo>
+    <gazebo>
+      <joint name="${headlight_prefix}_headlight" type="fixed">
+        <parent>base_link</parent>
+        <child>${headlight_prefix}_headlight_lamp::body</child>
+      </joint>
+    </gazebo>
   </xacro:macro>
 </robot>

File: x1_description/urdf/led.urdf.xacro (robot description, xacro)
@@ -3,5 +3,5 @@
   <xacro:macro name="led" params="led_prefix *joint_pose">
     <link name="${led_prefix}_led_link">
-      <visual>
+      <visual name="marker">
         <origin xyz="0 0 0" rpy="0 0 0" />
         <geometry>
@@ -9,5 +9,36 @@
         </geometry>
       </visual>
+<!--
+      <gazebo>
+        <light name="marker" type='point'>
+          <pose>0 0 0 0 0 0</pose>
+          <attenuation>
+            <range>50</range>
+            <linear>0.05</linear>
+          </attenuation>
+          <diffuse>1 1 1 1</diffuse>
+          <specular>1 1 1 1</specular>
+          <spot>
+            <inner_angle>2</inner_angle>
+            <outer_angle>2.1</outer_angle>
+            <falloff>1</falloff>
+          </spot>
+          <direction>1 0 0</direction>
+        </light>
+      </gazebo>-->
     </link>
+<!--
+    <gazebo>
+      <plugin name='light_control' filename='libRosFlashLightPlugin.so'>
+        <service_name>enable</service_name>
+        <light>
+          <id>${led_prefix}_led_link/marker</id>
+          <enable>false</enable>
+          <duration>1</duration>
+          <interval>0</interval>
+          <color>1 1 1</color>
+        </light>
+      </plugin>
+    </gazebo>-->
     <joint name="${led_prefix}_led" type="fixed">
       <parent link="base_link"/>

File: x1_description/urdf/x1.urdf.xacro (robot description, xacro)
@@ -117,16 +117,12 @@
   <xacro:x1_decorate />
   <!-- Head lights -->
-  <xacro:headlight headlight_prefix="right">
-    <origin xyz="0.461459  0.216803 0.124431" rpy="0 0 3.1416" />
-  </xacro:headlight>
-  <xacro:headlight headlight_prefix="center_right">
-    <origin xyz="0.485766 0.0844 0.124431" rpy="0 0 3.1416" />
-  </xacro:headlight>
-  <xacro:headlight headlight_prefix="center_left">
-    <origin xyz="0.485766 -0.0844 0.124431" rpy="0 0 3.1416" />
-  </xacro:headlight>
-  <xacro:headlight headlight_prefix="left">
-    <origin xyz="0.461459  -0.216803 0.124431" rpy="0 0 3.1416" />
-  </xacro:headlight>
+  <xacro:headlight headlight_prefix="right"
+    xyz="0.461459  0.216803 0.124431" rpy="0 0 3.1416" />
+  <xacro:headlight headlight_prefix="center_right"
+    xyz="0.485766 0.0844 0.124431" rpy="0 0 3.1416" />
+  <xacro:headlight headlight_prefix="center_left"
+    xyz="0.485766 -0.0844 0.124431" rpy="0 0 3.1416" />
+  <xacro:headlight headlight_prefix="left"
+    xyz="0.461459  -0.216803 0.124431" rpy="0 0 3.1416" />
    <!-- LEDs -->
   <xacro:led led_prefix="rear_left">

Commit message: Replace Husky in the team with X1

File: x1_description/urdf/headlight.urdf.xacro (robot description, xacro)
@@ -16,10 +16,10 @@
     </joint>
     <gazebo>
-      <model name="${headlight_prefix}_headlight_lamp">
+      <model name="${headlight_prefix}_headlight">
         <pose>${xyz} ${rpy}</pose>
         <link name="body">
           <pose>-0.0005 0 0 0 0 0</pose>
           <light name="light_source" type="spot">
-            <pose>-0.025 0 0.06 0 1.573 0</pose>
+            <pose>-0.025 0 0.055 0 1.573 0</pose>
             <attenuation>
               <range>50</range>
@@ -65,5 +65,5 @@
       <joint name="${headlight_prefix}_headlight" type="fixed">
         <parent>base_link</parent>
-        <child>${headlight_prefix}_headlight_lamp::body</child>
+        <child>${headlight_prefix}_headlight::body</child>
       </joint>
     </gazebo>

File: x1_description/urdf/led.urdf.xacro (robot description, xacro)
@@ -16,5 +16,5 @@
     </joint>
     <gazebo>
-      <model name="${led_prefix}_led_lamp">
+      <model name="${led_prefix}_led">
         <pose>${xyz} ${rpy}</pose>
         <link name="body">
@@ -60,5 +60,5 @@
       <joint name="${led_prefix}_led" type="fixed">
         <parent>base_link</parent>
-        <child>${led_prefix}_led_lamp::body</child>
+        <child>${led_prefix}_led::body</child>
       </joint>
     </gazebo>

File: x1_description/urdf/x1.urdf.xacro (robot description, xacro)
@@ -30,4 +30,5 @@
   <xacro:property name="x1_bumper_extend" value="$(optenv X1_FORWARD_BUMPER_EXTEND 0)" />
   <xacro:arg name="robot_namespace" default="/" />
+  <xacro:arg name="tfpre" default="x0_tf" />
   <xacro:arg name="urdf_extras" default="empty.urdf" />
   <!-- Included URDF/XACRO Files -->
@@ -117,11 +118,11 @@
   <xacro:x1_decorate />
   <!-- Head lights -->
+  <xacro:headlight headlight_prefix="left"
+    xyz="0.461459  0.216803 0.124431" rpy="0 0 3.1416" />
+  <xacro:headlight headlight_prefix="center_left"
+    xyz="0.485766 0.0844 0.124431" rpy="0 0 3.1416" />
+  <xacro:headlight headlight_prefix="center_right"
+    xyz="0.485766 -0.0844 0.124431" rpy="0 0 3.1416" />
   <xacro:headlight headlight_prefix="right"
-    xyz="0.461459  0.216803 0.124431" rpy="0 0 3.1416" />
-  <xacro:headlight headlight_prefix="center_right"
-    xyz="0.485766 0.0844 0.124431" rpy="0 0 3.1416" />
-  <xacro:headlight headlight_prefix="center_left"
-    xyz="0.485766 -0.0844 0.124431" rpy="0 0 3.1416" />
-  <xacro:headlight headlight_prefix="left"
     xyz="0.461459  -0.216803 0.124431" rpy="0 0 3.1416" />
    <!-- LEDs -->
@@ -129,16 +130,26 @@
     <plugin_params>
       <block>
-        <duration>0.2</duration>
-        <interval>0.2</interval>
+        <duration>0.3</duration>
+        <interval>0.3</interval>
+        <color>1 0.8</color>
+      </block>
+    </plugin_params>
+  </xacro:led>
+  <xacro:led led_prefix="rear_center" xyz="-0.42493 0 0.209188" rpy="0 1.573 3.1416">
+    <plugin_params>
+      <block>
+        <duration>0.1</duration>
+        <interval>0</interval>
+        <color>1 0 0</color>
+      </block>
+      <block>
+        <duration>0.1</duration>
+        <interval>0</interval>
         <color>0 1 0</color>
       </block>
-    </plugin_params>
-  </xacro:led>
-  <xacro:led led_prefix="rear_center" xyz="-0.42493 0 0.209188" rpy="0 1.573 3.1416">
-    <plugin_params>
-      <block>
-        <duration>0.2</duration>
-        <interval>0.2</interval>
-        <color>1 1 0</color>
+      <block>
+        <duration>0.1</duration>
+        <interval>0</interval>
+        <color>0 0 1</color>
       </block>
     </plugin_params>
@@ -147,7 +158,7 @@
     <plugin_params>
       <block>
-        <duration>0.2</duration>
-        <interval>0.2</interval>
-        <color>1 0 0</color>
+        <duration>0.3</duration>
+        <interval>0.3</interval>
+        <color>1 0.8</color>
       </block>
     </plugin_params>
@@ -156,7 +167,7 @@
     <plugin_params>
       <block>
-        <duration>0.2</duration>
-        <interval>0.2</interval>
-        <color>0 1 0</color>
+        <duration>0.3</duration>
+        <interval>0.3</interval>
+        <color>1 0.8</color>
       </block>
     </plugin_params>
@@ -165,7 +176,7 @@
     <plugin_params>
       <block>
-        <duration>0.1</duration>
-        <interval>0.1</interval>
-        <color>0 1 0</color>
+        <duration>0.3</duration>
+        <interval>0.3</interval>
+        <color>1 0.8</color>
       </block>
     </plugin_params>
@@ -174,7 +185,7 @@
     <plugin_params>
       <block>
-        <duration>0.2</duration>
-        <interval>0.2</interval>
-        <color>1 0 0</color>
+        <duration>0.3</duration>
+        <interval>0.3</interval>
+        <color>1 0.8</color>
       </block>
     </plugin_params>
@@ -183,7 +194,7 @@
     <plugin_params>
       <block>
-        <duration>0.1</duration>
-        <interval>0.1</interval>
-        <color>1 0 0</color>
+        <duration>0.3</duration>
+        <interval>0.3</interval>
+        <color>1 0.8</color>
       </block>
     </plugin_params>
@@ -218,4 +229,5 @@
       <robotNamespace>$(arg robot_namespace)</robotNamespace>
       <updateRate>50.0</updateRate>
+      <frameId>$(arg tfpre)base_link</frameId>
       <bodyName>base_link</bodyName>
       <topicName>imu/data</topicName>
@@ -233,5 +245,5 @@
       <updateRate>40</updateRate>
       <bodyName>base_link</bodyName>
-      <frameId>base_link</frameId>
+      <frameId>$(arg tfpre)base_link</frameId>
       <topicName>navsat/fix</topicName>
       <velocityTopicName>navsat/vel</velocityTopicName>

Commit message: Add dummy intertial info to light models of X1

File: x1_description/urdf/headlight.urdf.xacro (robot description, xacro)
@@ -9,4 +9,13 @@
         </geometry>
       </visual>
+      <inertial>
+        <origin xyz="0 0 0" rpy="0 0 0"/>
+        <mass value="0.000001" />
+        <inertia
+          ixx="0.001"
+          ixy="0.0" iyy="0.001"
+          ixz="0.0" iyz="0.0" izz="0.001"
+        />
+      </inertial>
     </link>
     <joint name="${headlight_prefix}_headlight" type="fixed">
@@ -49,4 +58,13 @@
             </material>
           </visual>
+          <inertial>
+            <origin xyz="0 0 0" rpy="0 0 0"/>
+            <mass>0.000001</mass>
+            <inertia>
+              <ixx>0.001</ixx>
+              <ixy>0.0</ixy><iyy>0.001</iyy>
+              <ixz>0.0</ixz><iyz>0.0</iyz><izz>0.001</izz>
+            </inertia>
+          </inertial>
         </link>
         <plugin name='light_control' filename='libRosFlashLightPlugin.so'>

File: x1_description/urdf/led.urdf.xacro (robot description, xacro)
@@ -9,4 +9,13 @@
         </geometry>
       </visual>
+      <inertial>
+        <origin xyz="0 0 0" rpy="0 0 0"/>
+        <mass value="0.000001" />
+        <inertia
+          ixx="0.001"
+          ixy="0.0" iyy="0.001"
+          ixz="0.0" iyz="0.0" izz="0.001"
+        />
+      </inertial>
     </link>
     <joint name="${led_prefix}_led" type="fixed">
@@ -43,4 +52,13 @@
             </material>
           </visual>
+          <inertial>
+            <origin xyz="0 0 0" rpy="0 0 0"/>
+            <mass>0.000001</mass>
+            <inertia>
+              <ixx>0.001</ixx>
+              <ixy>0.0</ixy><iyy>0.001</iyy>
+              <ixz>0.0</ixz><iyz>0.0</iyz><izz>0.001</izz>
+            </inertia>
+          </inertial>
         </link>
         <plugin name='light_control' filename='libRosFlashLightPlugin.so'>
