Commit message: Prefix X1 links with the robot's namespace

File: x1_description/urdf/decorations.urdf.xacro (robot description, xacro)
@@ -24,12 +24,12 @@
   <xacro:macro name="x1_decorate">
     <!-- Spawn X1 chassis -->
-    <link name="top_chassis_link">
+    <link name="${namespace}/top_chassis_link">
     </link>
     <!-- Attach chassis to the robot -->
     <joint name="top_chassis_joint" type="fixed">
-      <parent link="base_link" />
-      <child link="top_chassis_link" />
+      <parent link="${namespace}/base_link" />
+      <child link="${namespace}/top_chassis_link" />
     </joint>
-    <link name="top_plate_link">
+    <link name="${namespace}/top_plate_link">
       <visual>
         <origin xyz="0 0 0" rpy="0 0 0" />
@@ -53,22 +53,22 @@
     <!-- Attach top plate -->
     <joint name="top_plate_joint" type="fixed">
-      <parent link="base_link" />
-      <child link="top_plate_link"/>
+      <parent link="${namespace}/base_link" />
+      <child link="${namespace}/top_plate_link"/>
       <origin xyz="0.0812 0 0.245" rpy="0 0 0"/>
     </joint>
     <!-- Top plate front link -->
     <joint name="top_plate_front_joint" type="fixed">
-      <parent link="top_plate_link" />
-      <child link="top_plate_front_link"/>
+      <parent link="${namespace}/top_plate_link" />
+      <child link="${namespace}/top_plate_front_link"/>
       <origin xyz="0.36367 0 0.00639" rpy="0 0 0"/>
     </joint>
     <!-- Top plate rear link-->
     <joint name="top_plate_rear_joint" type="fixed">
-      <parent link="top_plate_link" />
-      <child link="top_plate_rear_link"/>
+      <parent link="${namespace}/top_plate_link" />
+      <child link="${namespace}/top_plate_rear_link"/>
       <origin xyz="-0.36633 0 0.00639" rpy="0 0 0"/>
     </joint>
-    <link name="top_plate_front_link"/>
-    <link name="top_plate_rear_link"/>
+    <link name="${namespace}/top_plate_front_link"/>
+    <link name="${namespace}/top_plate_rear_link"/>
   </xacro:macro>
 </robot>

File: x1_description/urdf/headlight.urdf.xacro (robot description, xacro)
@@ -2,5 +2,5 @@
 <robot xmlns:xacro="http://ros.org/wiki/xacro" name="headlight">
   <xacro:macro name="headlight" params="headlight_prefix xyz rpy">
-    <link name="${headlight_prefix}_headlight_link">
+    <link name="${namespace}/${headlight_prefix}_headlight_link">
       <visual>
         <origin xyz="0 0 0" rpy="0 0 0" />
@@ -20,6 +20,6 @@
     </link>
     <joint name="${headlight_prefix}_headlight" type="fixed">
-      <parent link="base_link"/>
-      <child link="${headlight_prefix}_headlight_link"/>
+      <parent link="${namespace}/base_link"/>
+      <child link="${namespace}/${headlight_prefix}_headlight_link"/>
       <origin xyz="${xyz}" rpy="${rpy}"/>
     </joint>
@@ -90,5 +90,5 @@
     <gazebo>
       <joint name="${headlight_prefix}_headlight" type="fixed">
-        <parent>base_link</parent>
+        <parent>${namespace}/base_link</parent>
         <child>${headlight_prefix}_headlight::body</child>
       </joint>

File: x1_description/urdf/led.urdf.xacro (robot description, xacro)
@@ -2,5 +2,5 @@
 <robot xmlns:xacro="http://ros.org/wiki/xacro" name="led">
   <xacro:macro name="led" params="led_prefix xyz rpy **plugin_params">
-    <link name="${led_prefix}_led_link">
+    <link name="${namespace}/${led_prefix}_led_link">
       <visual name="marker">
         <origin xyz="0 0 0" rpy="0 0 0" />
@@ -20,6 +20,6 @@
     </link>
     <joint name="${led_prefix}_led" type="fixed">
-      <parent link="base_link"/>
-      <child link="${led_prefix}_led_link"/>
+      <parent link="${namespace}/base_link"/>
+      <child link="${namespace}/${led_prefix}_led_link"/>
       <origin xyz="${xyz}" rpy="${rpy}"/>
     </joint>
@@ -85,5 +85,5 @@
     <gazebo>
       <joint name="${led_prefix}_led" type="fixed">
-        <parent>base_link</parent>
+        <parent>${namespace}/base_link</parent>
         <child>${led_prefix}_led::body</child>
       </joint>

File: x1_description/urdf/wheel.urdf.xacro (robot description, xacro)
@@ -23,5 +23,5 @@
 <robot xmlns:xacro="http://ros.org/wiki/xacro" name="x1_wheel">
 	<xacro:macro name="x1_wheel" params="wheel_prefix *joint_pose">
-		<link name="${wheel_prefix}_wheel_link">
+		<link name="${namespace}/${wheel_prefix}_wheel_link">
 			<inertial>
 				<mass value="2.637" />
@@ -42,5 +42,5 @@
 			</collision>
 		</link>
-		<gazebo reference="${wheel_prefix}_wheel_link">
+		<gazebo reference="${namespace}/${wheel_prefix}_wheel_link">
 			<mu1 value="1.0"/>
 			<mu2 value="1.0"/>
@@ -50,6 +50,6 @@
 		</gazebo>
 		<joint name="${wheel_prefix}_wheel" type="continuous">
-			<parent link="base_link"/>
-			<child link="${wheel_prefix}_wheel_link"/>
+			<parent link="${namespace}/base_link"/>
+			<child link="${namespace}/${wheel_prefix}_wheel_link"/>
 			<xacro:insert_block name="joint_pose"/>
 			<axis xyz="0 1 0" rpy="0 0 0" />

File: x1_description/urdf/x1.urdf.xacro (robot description, xacro)
@@ -29,7 +29,8 @@
   <xacro:arg name="kinect_rpy" default="$(optenv X1_KINECT_RPY 0 0.18 3.14)" />
   <xacro:property name="x1_bumper_extend" value="$(optenv X1_FORWARD_BUMPER_EXTEND 0)" />
-  <xacro:arg name="robot_namespace" default="/" />
+  <xacro:arg name="robot_namespace" default="" />
   <xacro:arg name="tfpre" default="x0_tf" />
   <xacro:arg name="urdf_extras" default="empty.urdf" />
+  <xacro:property name="namespace" value="$(arg robot_namespace)" />
   <!-- Included URDF/XACRO Files -->
   <xacro:include filename="$(find x1_description)/urdf/decorations.urdf.xacro" />
@@ -53,5 +54,5 @@
   <xacro:property name="wheel_radius" value="0.1651" />
   <!-- Base link is the center of the robot's bottom plate -->
-  <link name="base_link">
+  <link name="${namespace}/base_link">
     <visual>
       <origin xyz="0 0 0" rpy="0 0 3.1416" />
@@ -74,12 +75,12 @@
   </link>
   <!-- Base footprint is on the ground under the robot -->
-  <link name="base_footprint"/>
+  <link name="${namespace}/base_footprint"/>
   <joint name="base_footprint_joint" type="fixed">
     <origin xyz="0 0 ${wheel_vertical_offset - wheel_radius}" rpy="0 0 0" />
-    <parent link="base_link" />
-    <child link="base_footprint" />
+    <parent link="${namespace}/base_link" />
+    <child link="${namespace}/base_footprint" />
   </joint>
   <!-- Interial link stores the robot's inertial information -->
-  <link name="inertial_link">
+  <link name="${namespace}/inertial_link">
     <inertial>
       <mass value="46.034" />
@@ -90,16 +91,16 @@
   <joint name="inertial_joint" type="fixed">
     <origin xyz="0 0 0" rpy="0 0 0" />
-    <parent link="base_link" />
-    <child link="inertial_link" />
+    <parent link="${namespace}/base_link" />
+    <child link="${namespace}/inertial_link" />
   </joint>
   <!-- IMU Link is the standard mounting position for the UM6 IMU.-->
   <!-- Can be modified with environment variables in /etc/ros/setup.bash -->
-  <link name="imu_link"/>
+  <link name="${namespace}/imu_link"/>
   <joint name="imu_joint" type="fixed">
     <origin xyz="$(optenv X1_IMU_XYZ 0.19 0 0.149)" rpy="$(optenv X1_IMU_RPY 0 -1.5708 3.1416)" />
-    <parent link="base_link" />
-    <child link="imu_link" />
+    <parent link="${namespace}/base_link" />
+    <child link="${namespace}/imu_link" />
   </joint>
-  <gazebo reference="imu_link">
+  <gazebo reference="${namespace}/imu_link">
   </gazebo>
   <!-- X1 wheel macros -->
@@ -202,9 +203,9 @@
   <xacro:if value="$(arg laser_enabled)">
     <sick_lms1xx_mount prefix="base"/>
-    <sick_lms1xx frame="base_laser" topic="scan" robot_namespace="$(arg robot_namespace)"/>
+    <sick_lms1xx frame="base_laser" topic="scan" robot_namespace="${namespace}"/>
     <joint name="laser_mount_joint" type="fixed">
       <origin xyz="$(arg laser_xyz)" rpy="$(arg laser_rpy)" />
-      <parent link="top_plate_link" />
-      <child link="base_laser_mount" />
+      <parent link="${namespace}/top_plate_link" />
+      <child link="${namespace}/base_laser_mount" />
     </joint>
   </xacro:if>
@@ -215,20 +216,21 @@
     <joint name="kinect_frame_joint" type="fixed">
       <origin xyz="$(arg kinect_xyz)" rpy="$(arg kinect_rpy)" />
-      <parent link="sensor_arch_mount_link"/>
-      <child link="camera_link"/>
+      <parent link="${namespace}/sensor_arch_mount_link"/>
+      <child link="${namespace}/camera_link"/>
     </joint>
-    <xacro:kinect_camera prefix="camera" robot_namespace="$(arg robot_namespace)"/>
+    <xacro:kinect_camera prefix="camera" robot_namespace="${namespace}"/>
   </xacro:if>
   <gazebo>
     <plugin name="gazebo_ros_control" filename="libgazebo_ros_control.so">
-      <robotNamespace>$(arg robot_namespace)</robotNamespace>
+      <robotNamespace>${namespace}/</robotNamespace>
     </plugin>
   </gazebo>
   <gazebo>
     <plugin name="imu_controller" filename="libhector_gazebo_ros_imu.so">
-      <robotNamespace>$(arg robot_namespace)</robotNamespace>
+      <robotNamespace>${namespace}/</robotNamespace>
       <updateRate>50.0</updateRate>
-      <frameId>$(arg tfpre)base_link</frameId>
-      <bodyName>base_link</bodyName>
+      <!--TODO: The frame id and body name need the namespace-->
+      <frameId>${namespace}/base_link</frameId>
+      <bodyName>${namespace}/base_link</bodyName>
       <topicName>imu/data</topicName>
       <accelDrift>0.005 0.005 0.005</accelDrift>
@@ -242,8 +244,8 @@
   <gazebo>
     <plugin name="gps_controller" filename="libhector_gazebo_ros_gps.so">
-      <robotNamespace>$(arg robot_namespace)</robotNamespace>
+      <robotNamespace>${namespace}/</robotNamespace>
       <updateRate>40</updateRate>
-      <bodyName>base_link</bodyName>
-      <frameId>$(arg tfpre)base_link</frameId>
+      <bodyName>${namespace}/base_link</bodyName>
+      <frameId>${namespace}/base_link</frameId>
       <topicName>navsat/fix</topicName>
       <velocityTopicName>navsat/vel</velocityTopicName>
