Commit message: Rotate the model.

File: x1_description/urdf/x1.urdf.xacro (robot description, xacro)
@@ -54,5 +54,5 @@
   <link name="base_link">
     <visual>
-      <origin xyz="0 0 0" rpy="0 0 0" />
+      <origin xyz="0 0 0" rpy="0 0 3.1416" />
       <geometry>
         <mesh filename="package://x1_description/meshes/chassis.dae" />
@@ -118,24 +118,24 @@
   <!-- Head lights -->
   <xacro:headlight headlight_prefix="right">
-    <origin xyz="-0.461459  0.216803 0.124431" rpy="0 0 0" />
+    <origin xyz="0.461459  0.216803 0.124431" rpy="0 0 3.1416" />
   </xacro:headlight>
   <xacro:headlight headlight_prefix="center_right">
-    <origin xyz="-0.485766 0.0844 0.124431" rpy="0 0 0" />
+    <origin xyz="0.485766 0.0844 0.124431" rpy="0 0 3.1416" />
   </xacro:headlight>
   <xacro:headlight headlight_prefix="center_left">
-    <origin xyz="-0.485766 -0.0844 0.124431" rpy="0 0 0" />
+    <origin xyz="0.485766 -0.0844 0.124431" rpy="0 0 3.1416" />
   </xacro:headlight>
   <xacro:headlight headlight_prefix="left">
-    <origin xyz="-0.461459  -0.216803 0.124431" rpy="0 0 0" />
+    <origin xyz="0.461459  -0.216803 0.124431" rpy="0 0 3.1416" />
   </xacro:headlight>
    <!-- LEDs -->
   <xacro:led led_prefix="rear_left">
-    <origin xyz="0.42493 -0.13619 0.209188" rpy="0 1.573 0" />
+    <origin xyz="-0.42493 -0.13619 0.209188" rpy="0 1.573 3.1416" />
   </xacro:led>
   <xacro:led led_prefix="rear_center">
-    <origin xyz="0.42493 0 0.209188" rpy="0 1.573 0" />
+    <origin xyz="-0.42493 0 0.209188" rpy="0 1.573 3.1416" />
   </xacro:led>
   <xacro:led led_prefix="rear_right">
-    <origin xyz="0.42493 0.13619 0.209188" rpy="0 1.573 0" />
+    <origin xyz="-0.42493 0.13619 0.209188" rpy="0 1.573 3.1416" />
   </xacro:led>
   <xacro:led led_prefix="left_lateral_rear">

Commit message: Remove unused 'laser_enabled' and 'kinect_enabled' parameters.

File: x1_description/urdf/x1.urdf.xacro (robot description, xacro)
@@ -22,10 +22,4 @@
 -->
 <robot name="x1" xmlns:xacro="http://ros.org/wiki/xacro">
-  <xacro:arg name="laser_enabled" default="false" />
-  <xacro:arg name="laser_xyz" default="$(optenv X1_LMS1XX_XYZ 0.2206 0.0 0.00635)" />
-  <xacro:arg name="laser_rpy" default="$(optenv X1_LMS1XX_RPY 0.0 0.0 0.0)" />
-  <xacro:arg name="kinect_enabled" default="false" />
-  <xacro:arg name="kinect_xyz" default="$(optenv X1_KINECT_XYZ 0 0 0)" />
-  <xacro:arg name="kinect_rpy" default="$(optenv X1_KINECT_RPY 0 0.18 3.14)" />
   <xacro:property name="x1_bumper_extend" value="$(optenv X1_FORWARD_BUMPER_EXTEND 0)" />
   <xacro:arg name="robot_namespace" default="" />
@@ -240,24 +234,4 @@
     <hd_camera_and_mount />
   </xacro:if>
-  <xacro:if value="$(arg laser_enabled)">
-    <sick_lms1xx_mount prefix="base"/>
-    <sick_lms1xx frame="base_laser" topic="scan" robot_namespace="${namespace}"/>
-    <joint name="laser_mount_joint" type="fixed">
-      <origin xyz="$(arg laser_xyz)" rpy="$(arg laser_rpy)" />
-      <parent link="${namespace}/top_plate_link" />
-      <child link="${namespace}/base_laser_mount" />
-    </joint>
-  </xacro:if>
-  <xacro:if value="$(arg kinect_enabled)">
-    <xacro:sensor_arch prefix="" parent="top_plate_link">
-      <origin xyz="-0.35 0 0.51" rpy="0 0 -3.14"/>
-    </xacro:sensor_arch>
-    <joint name="kinect_frame_joint" type="fixed">
-      <origin xyz="$(arg kinect_xyz)" rpy="$(arg kinect_rpy)" />
-      <parent link="${namespace}/sensor_arch_mount_link"/>
-      <child link="${namespace}/camera_link"/>
-    </joint>
-    <xacro:kinect_camera prefix="camera" robot_namespace="${namespace}"/>
-  </xacro:if>
   <gazebo>
     <plugin name="gazebo_ros_control" filename="libgazebo_ros_control.so">
