Commit message: Unify topic names.

File: x1_description/urdf/sensors.urdf.xacro (robot description, xacro)
@@ -79,5 +79,5 @@
       <child link="${namespace}/front_camera_mount" />
     </joint>
-    <pointgrey_flea3 frame="${namespace}/front_camera" name="front"
+    <pointgrey_flea3 frame="${namespace}/front_camera" name="camera_front"
       camera_x="0.0754" camera_y="0.029" camera_z="0.029"
       camera_mass="0.085" hfov="1.0471975512" fps="20" width="320" height="240"
@@ -97,5 +97,5 @@
       <child link="${namespace}/front_camera_mount" />
     </joint>
-    <pointgrey_flea3 frame="${namespace}/front_camera" name="front"
+    <pointgrey_flea3 frame="${namespace}/front_camera" name="camera_front"
       camera_x="0.0754" camera_y="0.029" camera_z="0.029"
       camera_mass="0.085" hfov="1.0471975512" fps="20" width="1280" height="960"

File: x2_description/urdf/accessories.urdf.xacro (robot description, xacro)
@@ -54,5 +54,5 @@
       <child link="${namespace}/front_camera_mount" />
     </joint>
-    <pointgrey_flea3 frame="${namespace}/front_camera" name="front"
+    <pointgrey_flea3 frame="${namespace}/front_camera" name="camera_front"
       camera_x="0.0754" camera_y="0.029" camera_z="0.029"
       camera_mass="0.085" hfov="1.0471975512" fps="20" width="320" height="240"
@@ -72,5 +72,5 @@
       <child link="${namespace}/front_camera_mount" />
     </joint>
-    <pointgrey_flea3 frame="${namespace}/front_camera" name="front"
+    <pointgrey_flea3 frame="${namespace}/front_camera" name="camera_front"
       camera_x="0.0754" camera_y="0.029" camera_z="0.029"
       camera_mass="0.085" hfov="1.0471975512" fps="20" width="1280" height="960"

File: x3_description/urdf/x3_base.xacro (robot description, xacro)
@@ -5,5 +5,5 @@
   <xacro:include filename="$(find x3_description)/urdf/x3.xacro" />
   <!-- Instantiate a controller. -->
-  <xacro:controller_plugin_macro namespace="${namespace}" imu_sub_topic="imu" />
+  <xacro:controller_plugin_macro namespace="${namespace}" imu_sub_topic="imu/data" />
   <gazebo>
     <enable_wind>true</enable_wind>

File: x3_description/urdf/x3_with_sensors.xacro (robot description, xacro)
@@ -39,5 +39,21 @@
   <xacro:default_pressure_sensor namespace="${namespace}" parent_link="${namespace}/base_link" />
   <!-- Mount an ADIS16448 IMU. -->
-  <xacro:default_imu namespace="${namespace}" parent_link="${namespace}/base_link" />
+  <xacro:imu_plugin_macro
+    namespace="${namespace}"
+    imu_suffix=""
+    parent_link="${namespace}/base_link"
+    imu_topic="imu/data"
+    mass_imu_sensor="0.015"
+    gyroscope_noise_density="0.0003394"
+    gyroscope_random_walk="0.000038785"
+    gyroscope_bias_correlation_time="1000.0"
+    gyroscope_turn_on_bias_sigma="0.0087"
+    accelerometer_noise_density="0.004"
+    accelerometer_random_walk="0.006"
+    accelerometer_bias_correlation_time="300.0"
+    accelerometer_turn_on_bias_sigma="0.1960">
+    <inertia ixx="0.00001" ixy="0.0" ixz="0.0" iyy="0.00001" iyz="0.0" izz="0.00001" />
+    <origin xyz="0 0 0" rpy="0 0 0" />
+  </xacro:imu_plugin_macro>
   <!-- Sensor configuration #1
          * QVGA camera

File: x4_description/urdf/x4_base.xacro (robot description, xacro)
@@ -21,5 +21,5 @@
   <xacro:include filename="$(find x4_description)/urdf/x4.xacro" />
   <!-- Instantiate a controller. -->
-  <xacro:controller_plugin_macro namespace="${namespace}" imu_sub_topic="imu" />
+  <xacro:controller_plugin_macro namespace="${namespace}" imu_sub_topic="imu/data" />
   <gazebo>
     <enable_wind>true</enable_wind>

File: x4_description/urdf/x4_with_sensors.xacro (robot description, xacro)
@@ -40,5 +40,21 @@
   <xacro:default_pressure_sensor namespace="${namespace}" parent_link="${namespace}/base_link" />
   <!-- Mount an ADIS16448 IMU. -->
-  <xacro:default_imu namespace="${namespace}" parent_link="${namespace}/base_link" />
+  <xacro:imu_plugin_macro
+    namespace="${namespace}"
+    imu_suffix=""
+    parent_link="${namespace}/base_link"
+    imu_topic="imu/data"
+    mass_imu_sensor="0.015"
+    gyroscope_noise_density="0.0003394"
+    gyroscope_random_walk="0.000038785"
+    gyroscope_bias_correlation_time="1000.0"
+    gyroscope_turn_on_bias_sigma="0.0087"
+    accelerometer_noise_density="0.004"
+    accelerometer_random_walk="0.006"
+    accelerometer_bias_correlation_time="300.0"
+    accelerometer_turn_on_bias_sigma="0.1960">
+    <inertia ixx="0.00001" ixy="0.0" ixz="0.0" iyy="0.00001" iyz="0.0" izz="0.00001" />
+    <origin xyz="0 0 0" rpy="0 0 0" />
+  </xacro:imu_plugin_macro>
   <!-- Sensor configuration #1
          * HD camera

Commit message: added new robot configuration with two cameras

File: x1_description/urdf/sensors.urdf.xacro (robot description, xacro)
@@ -107,3 +107,37 @@
     </joint>
   </xacro:macro>
+  <xacro:macro name="two_hd_cameras_and_mount">
+    <camera_mount prefix="front_R"
+                  tilt="0.0"/>
+    <joint name="front_camera_mount_joint_R" type="fixed">
+      <origin xyz="0 0 0" rpy="0 0 0" />
+      <parent link="${namespace}/top_plate_front_link" />
+      <child link="${namespace}/front_R_camera_mount" />
+    </joint>
+    <pointgrey_flea3 frame="${namespace}/front_camera_R" name="camera_front_R"
+      camera_x="0.0754" camera_y="0.029" camera_z="0.029"
+      camera_mass="0.085" hfov="1.0471975512" fps="20" width="1280" height="960"
+      near="0.01" />
+    <joint name="front_camera_bracket_joint_R" type="fixed">
+      <origin xyz="0.020 -0.1 0.0245" rpy="0 0 0" />
+      <parent link="${namespace}/front_R_camera_beam" />
+      <child link="${namespace}/front_camera_R" />
+    </joint>
+    <camera_mount prefix="front_L"
+                  tilt="0.0"/>
+    <joint name="front_camera_mount_joint_L" type="fixed">
+      <origin xyz="0 0 0" rpy="0 0 0" />
+      <parent link="${namespace}/top_plate_front_link" />
+      <child link="${namespace}/front_L_camera_mount" />
+    </joint>
+    <pointgrey_flea3 frame="${namespace}/front_camera_L" name="camera_front_L"
+      camera_x="0.0754" camera_y="0.029" camera_z="0.029"
+      camera_mass="0.085" hfov="1.0471975512" fps="20" width="1280" height="960"
+      near="0.01" />
+    <joint name="front_camera_bracket_joint_L" type="fixed">
+      <origin xyz="0.020 0.1 0.0245" rpy="0 0 0" />
+      <parent link="${namespace}/front_L_camera_beam" />
+      <child link="${namespace}/front_camera_L" />
+    </joint>
+  </xacro:macro>
 </robot>

File: x1_description/urdf/x1.urdf.xacro (robot description, xacro)
@@ -234,4 +234,11 @@
     <hd_camera_and_mount />
   </xacro:if>
+  <!-- Sensor configuration #5
+         * two HD cameras
+         * IMU
+  -->
+  <xacro:if value="$(optenv X1_SENSOR_CONFIG_5 0)">
+    <two_hd_cameras_and_mount />
+  </xacro:if>
   <gazebo>
     <plugin name="gazebo_ros_control" filename="libgazebo_ros_control.so">

File: x2_description/urdf/accessories.urdf.xacro (robot description, xacro)
@@ -82,4 +82,38 @@
     </joint>
   </xacro:macro>
+  <xacro:macro name="two_hd_cameras_and_mount">
+    <camera_mount prefix="front_R"
+                  tilt="0.0"/>
+    <joint name="front_camera_mount_joint_R" type="fixed">
+      <origin xyz="0 0 0" rpy="0 0 0" />
+      <parent link="${namespace}/front_mount" />
+      <child link="${namespace}/front_R_camera_mount" />
+    </joint>
+    <pointgrey_flea3 frame="${namespace}/front_camera_R" name="camera_front_R"
+      camera_x="0.0754" camera_y="0.029" camera_z="0.029"
+      camera_mass="0.085" hfov="1.0471975512" fps="20" width="1280" height="960"
+      near="0.01" />
+    <joint name="front_camera_bracket_joint_R" type="fixed">
+      <origin xyz="0.020 -0.1 0.0245" rpy="0 0 0" />
+      <parent link="${namespace}/front_R_camera_beam" />
+      <child link="${namespace}/front_camera_R" />
+    </joint>
+    <camera_mount prefix="front_L"
+                  tilt="0.0"/>
+    <joint name="front_camera_mount_joint_L" type="fixed">
+      <origin xyz="0 0 0" rpy="0 0 0" />
+      <parent link="${namespace}/front_mount" />
+      <child link="${namespace}/front_L_camera_mount" />
+    </joint>
+    <pointgrey_flea3 frame="${namespace}/front_camera_L" name="camera_front_L"
+      camera_x="0.0754" camera_y="0.029" camera_z="0.029"
+      camera_mass="0.085" hfov="1.0471975512" fps="20" width="1280" height="960"
+      near="0.01" />
+    <joint name="front_camera_bracket_joint_L" type="fixed">
+      <origin xyz="0.020 0.1 0.0245" rpy="0 0 0" />
+      <parent link="${namespace}/front_L_camera_beam" />
+      <child link="${namespace}/front_camera_L" />
+    </joint>
+  </xacro:macro>
   <!-- Sensor configuration #1
          * 2D short range lidar
@@ -118,3 +152,10 @@
     <hd_camera_and_mount />
   </xacro:if>
+  <!-- Sensor configuration #5
+         * two HD cameras
+         * IMU
+  -->
+  <xacro:if value="$(optenv X2_SENSOR_CONFIG_5 0)">
+    <two_hd_cameras_and_mount />
+  </xacro:if>
 </robot>

File: x4_description/urdf/x4_with_sensors.xacro (robot description, xacro)
@@ -176,3 +176,44 @@
     </joint>
   </xacro:if>
+  <!-- Sensor configuration #5
+         * HD camera
+         * HD camera
+         * IMU
+  -->
+  <xacro:if value="$(optenv X4_SENSOR_CONFIG_5 0)">
+    <xacro:camera_macro
+      namespace="${namespace}"
+      parent_link="${namespace}/base_link"
+      camera_suffix="front_R"
+      frame_rate="20"
+      horizontal_fov="2"
+      image_width="1280"
+      image_height="960"
+      image_format="R8G8B8"
+      min_distance="0.02"
+      max_distance="100"
+      noise_mean="0.0"
+      noise_stddev="0.007"
+      enable_visual="true">
+      <box size="0.02 0.05 0.05" />
+      <origin xyz="0.125 -0.07 -0.08" rpy="0 0 0" />
+    </xacro:camera_macro>
+    <xacro:camera_macro
+      namespace="${namespace}"
+      parent_link="${namespace}/base_link"
+      camera_suffix="front_L"
+      frame_rate="20"
+      horizontal_fov="2"
+      image_width="1280"
+      image_height="960"
+      image_format="R8G8B8"
+      min_distance="0.02"
+      max_distance="100"
+      noise_mean="0.0"
+      noise_stddev="0.007"
+      enable_visual="true">
+      <box size="0.02 0.05 0.05" />
+      <origin xyz="0.125 0.07 -0.08" rpy="0 0 0" />
+    </xacro:camera_macro>
+  </xacro:if>
 </robot>
