Commit message: X4 mesh and texture and new collision.

File: x4_description/urdf/x4.xacro (robot description, xacro)
@@ -23,6 +23,6 @@
   <xacro:property name="mesh_file" value="package://x4_description/meshes/x4.dae" />
   <xacro:property name="mass" value="3.42" /> <!-- [kg] -->
-  <xacro:property name="body_width" value="0.2" /> <!-- [m] -->
-  <xacro:property name="body_height" value="0.234" /> <!-- [m] -->
+  <xacro:property name="body_width" value="0.3" /> <!-- [m] -->
+  <xacro:property name="body_height" value="0.25" /> <!-- [m] -->
   <xacro:property name="mass_rotor" value="0.005" /> <!-- [kg] -->
   <xacro:property name="arm_length" value="0.2895" /> <!-- [m] -->
