Commit message: Initial sensor configuration for X4.

File: x4_description/urdf/x4_base.xacro (robot description, xacro)
@@ -22,15 +22,3 @@
   <!-- Instantiate a controller. -->
   <xacro:controller_plugin_macro namespace="${namespace}" imu_sub_topic="imu" />
-  <!-- Mount an ADIS16448 IMU. -->
-  <xacro:default_imu namespace="${namespace}" parent_link="${namespace}/base_link" />
-  <xacro:if value="$(arg enable_ground_truth)">
-    <xacro:ground_truth_imu_and_odometry namespace="${namespace}" parent_link="${namespace}/base_link" />
-  </xacro:if>
-  <xacro:if value="$(arg enable_logging)">
-    <!-- Instantiate a logger -->
-    <xacro:bag_plugin_macro
-      namespace="${namespace}"
-      bag_file="$(arg log_file)"
-      rotor_velocity_slowdown_sim="${rotor_velocity_slowdown_sim}" />
-  </xacro:if>
 </robot>

File: x4_description/urdf/x4_with_sensors.xacro (robot description, xacro)
@@ -37,39 +37,92 @@
   <!-- Mount a pressure sensor. -->
   <xacro:default_pressure_sensor namespace="${namespace}" parent_link="${namespace}/base_link" />
-  <!-- Front camera. -->
-  <xacro:camera_macro
-    namespace="${namespace}"
-    parent_link="${namespace}/base_link"
-    camera_suffix="front"
-    frame_rate="30"
-    horizontal_fov="2"
-    image_width="752"
-    image_height="480"
-    image_format="L8"
-    min_distance="0.02"
-    max_distance="50"
-    noise_mean="0.0"
-    noise_stddev="0.007"
-    enable_visual="false">
-    <box size="0.02 0.05 0.05" />
-    <origin xyz="0.1 0 0" rpy="0 0 0" />
-  </xacro:camera_macro>
-  <!-- Lower camera. -->
-  <xacro:camera_macro
-    namespace="${namespace}"
-    parent_link="${namespace}/base_link"
-    camera_suffix="lower"
-    frame_rate="30"
-    horizontal_fov="2"
-    image_width="752"
-    image_height="480"
-    image_format="L8"
-    min_distance="0.02"
-    max_distance="50"
-    noise_mean="0.0"
-    noise_stddev="0.007"
-    enable_visual="false">
-    <box size="0.02 0.05 0.05" />
-    <origin xyz="0 0 -0.07" rpy="0 1.57 0" />
-  </xacro:camera_macro>
+  <!-- Mount an ADIS16448 IMU. -->
+  <xacro:default_imu namespace="${namespace}" parent_link="${namespace}/base_link" />
+  <!-- Sensor configuration #1
+         * HD camera
+         * IMU
+  -->
+  <xacro:if value="$(optenv X4_SENSOR_CONFIG_1 0)">
+    <xacro:camera_macro
+      namespace="${namespace}"
+      parent_link="${namespace}/base_link"
+      camera_suffix="front"
+      frame_rate="30"
+      horizontal_fov="2"
+      image_width="1280"
+      image_height="960"
+      image_format="R8G8B8"
+      min_distance="0.02"
+      max_distance="50"
+      noise_mean="0.0"
+      noise_stddev="0.007"
+      enable_visual="true">
+      <box size="0.02 0.05 0.05" />
+      <origin xyz="0.1 0 0" rpy="0 0 0" />
+    </xacro:camera_macro>
+  </xacro:if>
+  <!-- Sensor configuration #2
+         * VGA RGBD camera
+         * IMU
+  -->
+  <xacro:if value="$(optenv X4_SENSOR_CONFIG_2 0)">
+    <xacro:rgbd_camera
+       name="${namespace}/rgbd_camera"
+       width="640"
+       height="480"
+    />
+    <joint name="rgbd_camera_mount_joint" type="fixed">
+      <origin xyz="0.05 0 -0.05" rpy="0 0.2618 0" />
+      <parent link="${namespace}/base_link" />
+      <child link="${namespace}/rgbd_camera_link" />
+    </joint>
+  </xacro:if>
+  <!-- Sensor configuration #3
+         * QVGA camera
+         * 2D short range lidar
+         * IMU
+  -->
+  <xacro:if value="$(optenv X4_SENSOR_CONFIG_3 0)">
+    <xacro:camera_macro
+      namespace="${namespace}"
+      parent_link="${namespace}/base_link"
+      camera_suffix="front"
+      frame_rate="30"
+      horizontal_fov="2"
+      image_width="320"
+      image_height="240"
+      image_format="R8G8B8"
+      min_distance="0.02"
+      max_distance="50"
+      noise_mean="0.0"
+      noise_stddev="0.007"
+      enable_visual="true">
+      <box size="0.02 0.05 0.05" />
+      <origin xyz="0.1 0 0" rpy="0 0 0" />
+    </xacro:camera_macro>
+  </xacro:if>
+  <!-- Sensor configuration #4
+         * HD camera
+         * 2D mid range lidar
+         * IMU
+  -->
+  <xacro:if value="$(optenv X4_SENSOR_CONFIG_4 0)">
+    <xacro:camera_macro
+      namespace="${namespace}"
+      parent_link="${namespace}/base_link"
+      camera_suffix="front"
+      frame_rate="30"
+      horizontal_fov="2"
+      image_width="1280"
+      image_height="960"
+      image_format="R8G8B8"
+      min_distance="0.02"
+      max_distance="50"
+      noise_mean="0.0"
+      noise_stddev="0.007"
+      enable_visual="true">
+      <box size="0.02 0.05 0.05" />
+      <origin xyz="0.1 0 0" rpy="0 0 0" />
+    </xacro:camera_macro>
+  </xacro:if>
 </robot>
