Commit message: Specify lighter mass for lights

File: subt_gazebo/urdf/flashlight.urdf.xacro (robot description, xacro)
@@ -7,4 +7,7 @@
         <link name='handle'>
           <pose>0 0 0.05 0 0 0</pose>
+          <inertia>
+            <mass>0.001</mass>
+          </inertia>
           <collision name='collision'>
             <geometry>
@@ -29,4 +32,7 @@
         <link name='light_source'>
           <pose>0 0 0.10 0 0 0</pose>
+          <inertia>
+            <mass>0.001</mass>
+          </inertia>
           <light name='lamp' type='spot'>
             <pose>0 0 0.0 0 3.14159 0</pose>

File: subt_gazebo/urdf/led.urdf.xacro (robot description, xacro)
@@ -6,4 +6,7 @@
         <xacro:insert_block name='pose'/>
         <link name='led_body'>
+          <inertia>
+            <mass>0.00001</mass>
+          </inertia>
           <collision name='collision'>
             <geometry>

Commit message: Fix intertial element in light urdf files

File: subt_gazebo/urdf/flashlight.urdf.xacro (robot description, xacro)
@@ -6,13 +6,21 @@
         <xacro:insert_block name="pose"/>
         <link name='handle'>
-          <pose>0 0 0.05 0 0 0</pose>
-          <inertia>
-            <mass>0.001</mass>
-          </inertia>
+          <pose>0 0 0.025 0 0 0</pose>
+          <inertial>
+            <mass>0.025</mass>
+            <inertia>
+              <ixx>1.0e-05</ixx>
+              <ixy>0</ixy>
+              <ixz>0</ixz>
+              <iyy>1.0e-05</iyy>
+              <iyz>0</iyz>
+              <izz>1.0e-05</izz>
+            </inertia>
+          </inertial>
           <collision name='collision'>
             <geometry>
               <cylinder>
                 <radius>0.025</radius>
-                <length>0.15</length>
+                <length>0.05</length>
               </cylinder>
             </geometry>
@@ -22,5 +30,5 @@
               <cylinder>
                 <radius>0.025</radius>
-                <length>0.10</length>
+                <length>0.05</length>
               </cylinder>
             </geometry>
@@ -31,8 +39,16 @@
         </link>
         <link name='light_source'>
-          <pose>0 0 0.10 0 0 0</pose>
-          <inertia>
-            <mass>0.001</mass>
-          </inertia>
+          <pose>0 0 0.05 0 0 0</pose>
+          <inertial>
+            <mass>0.025</mass>
+            <inertia>
+              <ixx>1.0e-05</ixx>
+              <ixy>0</ixy>
+              <ixz>0</ixz>
+              <iyy>1.0e-05</iyy>
+              <iyz>0</iyz>
+              <izz>1.0e-05</izz>
+            </inertia>
+          </inertial>
           <light name='lamp' type='spot'>
             <pose>0 0 0.0 0 3.14159 0</pose>

File: subt_gazebo/urdf/led.urdf.xacro (robot description, xacro)
@@ -6,8 +6,18 @@
         <xacro:insert_block name='pose'/>
         <link name='led_body'>
-          <inertia>
+          <inertial>
+            <pose>0 0 0 0 0 0</pose>
             <mass>0.00001</mass>
-          </inertia>
+            <inertia>
+              <ixx>1.0e-05</ixx>
+              <ixy>0</ixy>
+              <ixz>0</ixz>
+              <iyy>1.0e-05</iyy>
+              <iyz>0</iyz>
+              <izz>1.0e-05</izz>
+            </inertia>
+          </inertial>
           <collision name='collision'>
+            <pose>0 0 0 0 0 0</pose>
             <geometry>
               <sphere>
@@ -17,4 +27,5 @@
           </collision>
           <visual name='marker'>
+            <pose>0 0 0 0 0 0</pose>
             <geometry>
               <sphere>

Commit message: Tweak lights.

File: subt_gazebo/urdf/flashlight.urdf.xacro (robot description, xacro)
@@ -1,5 +1,5 @@
 <?xml version="1.0"?>
 <robot xmlns:xacro="http://www.ros.org/wiki/xacro" name="flashlight">
-  <xacro:macro name="flashlight" params="flashlight_prefix parent_link default_color:='0 0 0' *pose **plugin_params">
+  <xacro:macro name="flashlight" params="flashlight_prefix parent_link default_color:='0.8 0.8 0.5' *pose **plugin_params">
     <gazebo>
       <model name='${flashlight_prefix}_flashlight'>
@@ -54,6 +54,8 @@
             <pose>0 0 0.0 0 3.14159 0</pose>
             <attenuation>
-              <range>50</range>
-              <linear>0.05</linear>
+              <range>15</range>
+              <linear>0</linear>
+              <constant>0.1</constant>
+              <quadratic>0.01</quadratic>
             </attenuation>
             <diffuse>${default_color} 1</diffuse>

File: subt_gazebo/urdf/led.urdf.xacro (robot description, xacro)
@@ -43,6 +43,8 @@
             <pose>0 0 0 0 0 0</pose>
             <attenuation>
-              <range>0.20</range>
+              <range>1</range>
+              <constant>0.5</constant>
               <linear>0.10</linear>
+              <quadratic>0.5</quadratic>
             </attenuation>
             <diffuse>${default_color} 1</diffuse>

File: x1_description/urdf/headlight.urdf.xacro (robot description, xacro)
@@ -33,8 +33,10 @@
             <attenuation>
               <range>50</range>
-              <linear>0.05</linear>
+              <linear>0</linear>
+              <constant>0.1</constant>
+              <quadratic>0.0025</quadratic>
             </attenuation>
-            <diffuse>0 0 0 1</diffuse>
-            <specular>0 0 0 1</specular>
+            <diffuse>0.8 0.8 0.5 1</diffuse>
+            <specular>0.8 0.8 0.5 1</specular>
             <spot>
               <inner_angle>1</inner_angle>

File: x1_description/urdf/led.urdf.xacro (robot description, xacro)
@@ -32,6 +32,8 @@
             <pose>0 0 0 0 0 0</pose>
             <attenuation>
-              <range>0.20</range>
+              <range>2.0</range>
+              <constant>0.5</constant>
               <linear>0.10</linear>
+              <quadratic>0.5</quadratic>
             </attenuation>
             <diffuse>0 0 0 1</diffuse>

File: x2_description/urdf/x2.urdf.xacro (robot description, xacro)
@@ -105,9 +105,11 @@
             <pose>-0.025 0 0.055 0 1.573 0</pose>
             <attenuation>
-              <range>50</range>
-              <linear>0.05</linear>
+              <range>25</range>
+              <linear>0</linear>
+              <constant>0.1</constant>
+              <quadratic>0.005</quadratic>
             </attenuation>
-            <diffuse>0 0 0 1</diffuse>
-            <specular>0 0 0 1</specular>
+            <diffuse>0.8 0.8 0.5 1</diffuse>
+            <specular>0.8 0.8 0.5 1</specular>
             <spot>
               <inner_angle>1</inner_angle>
@@ -191,6 +193,8 @@
             <pose>0 0 0 0 0 0</pose>
             <attenuation>
-              <range>0.20</range>
+              <range>2.0</range>
+              <constant>0.5</constant>
               <linear>0.10</linear>
+              <quadratic>0.5</quadratic>
             </attenuation>
             <diffuse>0 0 0 1</diffuse>

Commit message: Tweaking drones to stay still.

File: subt_gazebo/urdf/flashlight.urdf.xacro (robot description, xacro)
@@ -8,5 +8,5 @@
           <pose>0 0 0.025 0 0 0</pose>
           <inertial>
-            <mass>0.025</mass>
+            <mass>0.0025</mass>
             <inertia>
               <ixx>1.0e-05</ixx>
@@ -41,5 +41,5 @@
           <pose>0 0 0.05 0 0 0</pose>
           <inertial>
-            <mass>0.025</mass>
+            <mass>0.0025</mass>
             <inertia>
               <ixx>1.0e-05</ixx>
