Commit message: Adding lights.

File: x2_description/urdf/x2.urdf.xacro (robot description, xacro)
@@ -62,9 +62,140 @@
     </transmission>
   </xacro:macro>
+  <xacro:macro name="headlight" params="headlight_prefix xyz rpy">
+    <link name="${headlight_prefix}_headlight_link">
+      <visual>
+        <origin xyz="0 0 0" rpy="0 0 0" />
+        <geometry>
+          <mesh filename="package://x2_description/meshes/headlight.dae" />
+        </geometry>
+      </visual>
+    </link>
+    <joint name="${headlight_prefix}_headlight" type="fixed">
+      <parent link="base_link"/>
+      <child link="${headlight_prefix}_headlight_link"/>
+      <origin xyz="${xyz}" rpy="${rpy}"/>
+    </joint>
+    <gazebo>
+      <model name="${headlight_prefix}_headlight">
+        <pose>${xyz} ${rpy}</pose>
+        <link name="body">
+          <pose>-0.0005 0 0 0 0 0</pose>
+          <light name="light_source" type="spot">
+            <pose>-0.025 0 0.055 0 1.573 0</pose>
+            <attenuation>
+              <range>50</range>
+              <linear>0.05</linear>
+            </attenuation>
+            <diffuse>0 0 0 1</diffuse>
+            <specular>0 0 0 1</specular>
+            <spot>
+              <inner_angle>1</inner_angle>
+              <outer_angle>1.1</outer_angle>
+              <falloff>1</falloff>
+            </spot>
+            <direction>0 0 -1</direction>
+          </light>
+          <visual name="light_source">
+            <geometry>
+              <mesh>
+                <uri>package://x2_description/meshes/headlight_lamp.dae</uri>
+              </mesh>
+            </geometry>
+            <transparency>1</transparency>
+            <material>
+              <ambient>1 1 1 1</ambient>
+              <diffuse>1 1 1 1</diffuse>
+              <specular>1 1 1 1</specular>
+              <emissive>0 0 0 1</emissive>
+            </material>
+          </visual>
+        </link>
+        <plugin name='light_control' filename='libRosFlashLightPlugin.so'>
+          <service_name>enable</service_name>
+          <light>
+            <id>body/light_source</id>
+            <enable>false</enable>
+            <duration>1</duration>
+            <interval>0</interval>
+            <color>1 1 1</color>
+          </light>
+        </plugin>
+      </model>
+    </gazebo>
+    <gazebo>
+      <joint name="${headlight_prefix}_headlight" type="fixed">
+        <parent>base_link</parent>
+        <child>${headlight_prefix}_headlight::body</child>
+      </joint>
+    </gazebo>
+  </xacro:macro>
+  <xacro:macro name="led" params="led_prefix xyz rpy **plugin_params">
+    <link name="${led_prefix}_led_link">
+      <visual name="marker">
+        <origin xyz="0 0 0" rpy="0 0 0" />
+        <geometry>
+          <mesh filename="package://x2_description/meshes/led.dae" />
+        </geometry>
+      </visual>
+    </link>
+    <joint name="${led_prefix}_led" type="fixed">
+      <parent link="base_link"/>
+      <child link="${led_prefix}_led_link"/>
+      <origin xyz="${xyz}" rpy="${rpy}"/>
+    </joint>
+    <gazebo>
+      <model name="${led_prefix}_led">
+        <pose>${xyz} ${rpy}</pose>
+        <link name="body">
+          <pose>0 0 0.0005 0 0 0</pose>
+          <light name='light_source' type='point'>
+            <pose>0 0 0 0 0 0</pose>
+            <attenuation>
+              <range>0.20</range>
+              <linear>0.10</linear>
+            </attenuation>
+            <diffuse>0 0 0 1</diffuse>
+            <specular>0 0 0 1</specular>
+          </light>
+          <visual name="light_source">
+            <geometry>
+              <mesh>
+                <uri>package://x2_description/meshes/led_lamp.dae</uri>
+              </mesh>
+            </geometry>
+            <transparency>1</transparency>
+            <material>
+              <ambient>1 1 1 1</ambient>
+              <diffuse>1 1 1 1</diffuse>
+              <specular>1 1 1 1</specular>
+              <emissive>0 0 0 1</emissive>
+            </material>
+          </visual>
+        </link>
+        <plugin name='light_control' filename='libRosFlashLightPlugin.so'>
+          <service_name>enable</service_name>
+          <light>
+            <id>body/light_source</id>
+            <xacro:insert_block name="plugin_params"/>
+            <enable>false</enable>
+            <duration>1</duration>
+            <interval>0</interval>
+            <color>1 1 1</color>
+          </light>
+        </plugin>
+      </model>
+    </gazebo>
+    <gazebo>
+      <joint name="${led_prefix}_led" type="fixed">
+        <parent>base_link</parent>
+        <child>${led_prefix}_led::body</child>
+      </joint>
+    </gazebo>
+  </xacro:macro>
   <xacro:wheel prefix="front_left">
     <origin xyz="${wheelbase/2} ${track/2} ${wheel_vertical_offset}" rpy="0 0 0" />
   </xacro:wheel>
   <xacro:wheel prefix="front_right">
-    <origin xyz="${wheelbase/2} ${-track/2} ${wheel_vertical_offset}" rpy="0 0 0" />
+    <origin xyz="${wheelbase/2} ${-track/2} ${wheel_vertical_offset}" rpy="0 0 3.14159" />
   </xacro:wheel>
   <xacro:wheel prefix="rear_left">
@@ -72,6 +203,31 @@
   </xacro:wheel>
   <xacro:wheel prefix="rear_right">
-    <origin xyz="${-wheelbase/2} ${-track/2} ${wheel_vertical_offset}" rpy="0 0 0" />
+    <origin xyz="${-wheelbase/2} ${-track/2} ${wheel_vertical_offset}" rpy="0 0 3.14159" />
   </xacro:wheel>
+  <!-- Head lights -->
+  <xacro:headlight headlight_prefix="left"
+    xyz="-0.214809 0.149719 0.118767" rpy="0 0 0" />
+<!--
+  <xacro:headlight headlight_prefix="center_left"
+    xyz="0.485766 0.0844 0.124431" rpy="0 0 3.1416" />
+  <xacro:headlight headlight_prefix="center_right"
+    xyz="0.485766 -0.0844 0.124431" rpy="0 0 3.1416" />
+  <xacro:headlight headlight_prefix="right"
+    xyz="0.461459  -0.216803 0.124431" rpy="0 0 3.1416" />
+X: -118.767mm
+Y: 149.719mm
+Y: -214.809mm
+Spotlight Right
+X: 118.767mm
+Y: 149.719mm
+Y: -214.809mm
+Spotlight Center Right
+X: 41.302mm
+Y: 149.719mm
+Y: -222.897mm
+Spotlight Center Left
+X: -41.302mm
+Y: 149.719mm
+Y: -222.897mm -->
   <link name="base_link"></link>
   <joint name="base_link_joint" type="fixed">

Commit message: Adding lights.

File: x2_description/urdf/x2.urdf.xacro (robot description, xacro)
@@ -17,10 +17,55 @@
   <material name="yellow"><color rgba="0.8 0.8 0.0 1.0" /></material>
   <material name="black"><color rgba="0.15 0.15 0.15 1.0" /></material>
-  <xacro:macro name="wheel" params="prefix *joint_pose">
+  <xacro:macro name="left_wheel" params="prefix *joint_pose">
     <link name="${prefix}_wheel_link">
       <visual>
         <origin xyz="0 0 0" rpy="${PI/2} 0 0"/>
         <geometry>
-          <mesh filename="package://x2_description/meshes/x2_wheel.dae"/>
+          <mesh filename="package://x2_description/meshes/x2_wheel_left.dae"/>
+        </geometry>
+        <material name="black" />
+      </visual>
+      <collision>
+        <origin xyz="0 0 0" rpy="${PI/2} 0 0"/>
+        <geometry>
+          <cylinder radius="${wheel_radius}" length="${wheel_width}"/>
+        </geometry>
+      </collision>
+      <inertial>
+        <origin xyz="0 0 0" rpy="0 0 0"/>
+        <mass value="0.477"/>
+        <inertia
+          ixx="0.0013" ixy="0" ixz="0"
+          iyy="0.0024" iyz="0"
+          izz="0.0013"/>
+      </inertial>
+    </link>
+    <gazebo reference="${prefix}_wheel_link">
+      <material>Gazebo/DarkGrey</material>
+    </gazebo>
+    <joint name="${prefix}_wheel" type="continuous">
+      <parent link="chassis_link"/>
+      <child link="${prefix}_wheel_link" />
+      <xacro:insert_block name="joint_pose" />
+      <axis xyz="0 1 0" />
+    </joint>
+    <!-- In reality, X2 has only two motors, one per side. However, it's more
+         straightforward for Gazebo to simulate as if there's an actuator per wheel. -->
+    <transmission name="${prefix}_wheel_trans">
+      <type>transmission_interface/SimpleTransmission</type>
+      <joint name="${prefix}_wheel">
+        <hardwareInterface>hardware_interface/VelocityJointInterface</hardwareInterface>
+      </joint>
+      <actuator name="${prefix}_actuator">
+        <mechanicalReduction>1</mechanicalReduction>
+      </actuator>
+    </transmission>
+  </xacro:macro>
+  <xacro:macro name="right_wheel" params="prefix *joint_pose">
+    <link name="${prefix}_wheel_link">
+      <visual>
+        <origin xyz="0 0 0" rpy="${PI/2} 0 0"/>
+        <geometry>
+          <mesh filename="package://x2_description/meshes/x2_wheel_right.dae"/>
         </geometry>
         <material name="black" />
@@ -193,41 +238,63 @@
     </gazebo>
   </xacro:macro>
-  <xacro:wheel prefix="front_left">
+  <xacro:left_wheel prefix="front_left">
     <origin xyz="${wheelbase/2} ${track/2} ${wheel_vertical_offset}" rpy="0 0 0" />
-  </xacro:wheel>
-  <xacro:wheel prefix="front_right">
-    <origin xyz="${wheelbase/2} ${-track/2} ${wheel_vertical_offset}" rpy="0 0 3.14159" />
-  </xacro:wheel>
-  <xacro:wheel prefix="rear_left">
+  </xacro:left_wheel>
+  <xacro:right_wheel prefix="front_right">
+    <origin xyz="${wheelbase/2} ${-track/2} ${wheel_vertical_offset}" rpy="0 0 0" />
+  </xacro:right_wheel>
+  <xacro:left_wheel prefix="rear_left">
     <origin xyz="${-wheelbase/2} ${track/2} ${wheel_vertical_offset}" rpy="0 0 0" />
-  </xacro:wheel>
-  <xacro:wheel prefix="rear_right">
-    <origin xyz="${-wheelbase/2} ${-track/2} ${wheel_vertical_offset}" rpy="0 0 3.14159" />
-  </xacro:wheel>
+  </xacro:left_wheel>
+  <xacro:right_wheel prefix="rear_right">
+    <origin xyz="${-wheelbase/2} ${-track/2} ${wheel_vertical_offset}" rpy="0 0 0" />
+  </xacro:right_wheel>
   <!-- Head lights -->
   <xacro:headlight headlight_prefix="left"
-    xyz="-0.214809 0.149719 0.118767" rpy="0 0 0" />
-<!--
-  <xacro:headlight headlight_prefix="center_left"
-    xyz="0.485766 0.0844 0.124431" rpy="0 0 3.1416" />
-  <xacro:headlight headlight_prefix="center_right"
-    xyz="0.485766 -0.0844 0.124431" rpy="0 0 3.1416" />
+    xyz="0.22 0.145 ${footprint_vertical_offset+0.15}" rpy="0 0 ${PI}" />
   <xacro:headlight headlight_prefix="right"
-    xyz="0.461459  -0.216803 0.124431" rpy="0 0 3.1416" />
-X: -118.767mm
-Y: 149.719mm
-Y: -214.809mm
-Spotlight Right
-X: 118.767mm
-Y: 149.719mm
-Y: -214.809mm
-Spotlight Center Right
-X: 41.302mm
-Y: 149.719mm
-Y: -222.897mm
-Spotlight Center Left
-X: -41.302mm
-Y: 149.719mm
-Y: -222.897mm -->
+    xyz="0.22 -0.145 ${footprint_vertical_offset+0.15}" rpy="0 0 ${PI}" />
+  <xacro:headlight headlight_prefix="front_left"
+    xyz="0.22 0.05 ${footprint_vertical_offset+0.15}" rpy="0 0 ${PI}" />
+  <xacro:headlight headlight_prefix="front_right"
+    xyz="0.22 -0.05 ${footprint_vertical_offset+0.15}" rpy="0 0 ${PI}" />
+  <!-- LED's -->
+  <xacro:led led_prefix="rear_center" xyz="${-0.127-wheelbase/2} 0 0.165" rpy="0 1.573 3.1416">
+    <plugin_params>
+      <block>
+        <duration>0.1</duration>
+        <interval>0</interval>
+        <color>1 0 0</color>
+      </block>
+      <block>
+        <duration>0.1</duration>
+        <interval>0</interval>
+        <color>0 1 0</color>
+      </block>
+      <block>
+        <duration>0.1</duration>
+        <interval>0</interval>
+        <color>0 0 1</color>
+      </block>
+    </plugin_params>
+  </xacro:led>
+  <xacro:led led_prefix="right_lateral" xyz="0 ${-track/2} 0.15" rpy="0 1.573 -1.539">
+    <plugin_params>
+      <block>
+        <duration>0.3</duration>
+        <interval>0.3</interval>
+        <color>1 0.8</color>
+      </block>
+    </plugin_params>
+  </xacro:led>
+  <xacro:led led_prefix="left_lateral" xyz="0 ${track/2} 0.15" rpy="0 1.573 1.539">
+    <plugin_params>
+      <block>
+        <duration>0.3</duration>
+        <interval>0.3</interval>
+        <color>1 0.8</color>
+      </block>
+    </plugin_params>
+  </xacro:led>
   <link name="base_link"></link>
   <joint name="base_link_joint" type="fixed">
@@ -238,5 +305,5 @@
   <link name="chassis_link">
     <visual>
-      <origin xyz="0 0 ${footprint_vertical_offset}" rpy="${PI/2} 0 ${PI/2}"/>
+      <origin xyz="0 0 ${footprint_vertical_offset}" rpy="${PI/2} 0 ${-PI/2}"/>
       <geometry>
         <mesh filename="package://x2_description/meshes/x2_chassis.dae"/>

Commit message: Add dummy inertial info to light models of X2

File: x2_description/urdf/x2.urdf.xacro (robot description, xacro)
@@ -117,4 +117,13 @@
         </geometry>
       </visual>
+      <inertial>
+        <origin xyz="0 0 0" rpy="0 0 0"/>
+        <mass value="0.000001" />
+        <inertia
+          ixx="0.001"
+          ixy="0.0" iyy="0.001"
+          ixz="0.0" iyz="0.0" izz="0.001"
+        />
+      </inertial>
     </link>
     <joint name="${headlight_prefix}_headlight" type="fixed">
@@ -157,4 +166,13 @@
             </material>
           </visual>
+          <inertial>
+            <origin xyz="0 0 0" rpy="0 0 0"/>
+            <mass>0.000001</mass>
+            <inertia>
+              <ixx>0.001</ixx>
+              <ixy>0.0</ixy><iyy>0.001</iyy>
+              <ixz>0.0</ixz><iyz>0.0</iyz><izz>0.001</izz>
+            </inertia>
+          </inertial>
         </link>
         <plugin name='light_control' filename='libRosFlashLightPlugin.so'>
@@ -185,4 +203,13 @@
         </geometry>
       </visual>
+      <inertial>
+        <origin xyz="0 0 0" rpy="0 0 0"/>
+        <mass value="0.000001" />
+        <inertia
+          ixx="0.001"
+          ixy="0.0" iyy="0.001"
+          ixz="0.0" iyz="0.0" izz="0.001"
+        />
+      </inertial>
     </link>
     <joint name="${led_prefix}_led" type="fixed">
@@ -219,4 +246,13 @@
             </material>
           </visual>
+          <inertial>
+            <origin xyz="0 0 0" rpy="0 0 0"/>
+            <mass>0.000001</mass>
+            <inertia>
+              <ixx>0.001</ixx>
+              <ixy>0.0</ixy><iyy>0.001</iyy>
+              <ixz>0.0</ixz><iyz>0.0</iyz><izz>0.001</izz>
+            </inertia>
+          </inertial>
         </link>
         <plugin name='light_control' filename='libRosFlashLightPlugin.so'>
@@ -328,5 +364,5 @@
         iyy="0.3922" iyz="-0.0009"
         izz="0.4485"/>
-      </inertial>
+    </inertial>
   </link>
   <!-- TODO: Make this internal_imu_link or something, and use a mixed-in xacro

Commit message: Tweak in x2.urdf.xacro

File: x2_description/urdf/x2.urdf.xacro (robot description, xacro)
@@ -19,10 +19,10 @@
   <material name="yellow"><color rgba="0.8 0.8 0.0 1.0" /></material>
   <material name="black"><color rgba="0.15 0.15 0.15 1.0" /></material>
-  <xacro:macro name="left_wheel" params="prefix *joint_pose">
+  <xacro:macro name="wheel_common" params="prefix left_or_right *joint_pose">
     <link name="${prefix}_wheel_link">
       <visual>
         <origin xyz="0 0 0" rpy="${PI/2} 0 0"/>
         <geometry>
-          <mesh filename="package://x2_description/meshes/x2_wheel_left.dae"/>
+          <mesh filename="package://x2_description/meshes/x2_wheel_${left_or_right}.dae"/>
         </geometry>
         <material name="black" />
@@ -64,48 +64,13 @@
     </transmission>
   </xacro:macro>
+  <xacro:macro name="left_wheel" params="prefix *joint_pose">
+    <xacro:wheel_common prefix="${prefix}" left_or_right="left">
+      <xacro:insert_block name="joint_pose" />
+    </xacro:wheel_common>
+  </xacro:macro>
   <xacro:macro name="right_wheel" params="prefix *joint_pose">
-    <link name="${prefix}_wheel_link">
-      <visual>
-        <origin xyz="0 0 0" rpy="${PI/2} 0 0"/>
-        <geometry>
-          <mesh filename="package://x2_description/meshes/x2_wheel_right.dae"/>
-        </geometry>
-        <material name="black" />
-      </visual>
-      <collision>
-        <origin xyz="0 0 0" rpy="${PI/2} 0 0"/>
-        <geometry>
-          <cylinder radius="${wheel_radius}" length="${wheel_width}"/>
-        </geometry>
-      </collision>
-      <inertial>
-        <origin xyz="0 0 0" rpy="0 0 0"/>
-        <mass value="0.477"/>
-        <inertia
-          ixx="0.0013" ixy="0" ixz="0"
-          iyy="0.0024" iyz="0"
-          izz="0.0013"/>
-      </inertial>
-    </link>
-    <gazebo reference="${prefix}_wheel_link">
-      <material>Gazebo/DarkGrey</material>
-    </gazebo>
-    <joint name="${prefix}_wheel" type="continuous">
-      <parent link="chassis_link"/>
-      <child link="${prefix}_wheel_link" />
+    <xacro:wheel_common prefix="${prefix}" left_or_right="right">
       <xacro:insert_block name="joint_pose" />
-      <axis xyz="0 1 0" />
-    </joint>
-    <!-- In reality, X2 has only two motors, one per side. However, it's more
-         straightforward for Gazebo to simulate as if there's an actuator per wheel. -->
-    <transmission name="${prefix}_wheel_trans">
-      <type>transmission_interface/SimpleTransmission</type>
-      <joint name="${prefix}_wheel">
-        <hardwareInterface>hardware_interface/VelocityJointInterface</hardwareInterface>
-      </joint>
-      <actuator name="${prefix}_actuator">
-        <mechanicalReduction>1</mechanicalReduction>
-      </actuator>
-    </transmission>
+    </xacro:wheel_common>
   </xacro:macro>
   <xacro:macro name="headlight" params="headlight_prefix xyz rpy">

Commit message: Prefix X2 links with the robot's namespace

File: x2_description/urdf/x2.urdf.xacro (robot description, xacro)
@@ -3,4 +3,5 @@
   <xacro:arg name="robot_namespace" default="/" />
   <xacro:arg name="tfpre" default="" />
+  <xacro:property name="namespace" value="$(arg robot_namespace)" />
   <xacro:property name="PI" value="3.1415926535897931" />
   <xacro:property name="wheelbase" value="0.262" />
@@ -20,5 +21,5 @@
   <material name="black"><color rgba="0.15 0.15 0.15 1.0" /></material>
   <xacro:macro name="wheel_common" params="prefix left_or_right *joint_pose">
-    <link name="${prefix}_wheel_link">
+    <link name="${namespace}/${prefix}_wheel_link">
       <visual>
         <origin xyz="0 0 0" rpy="${PI/2} 0 0"/>
@@ -43,10 +44,10 @@
       </inertial>
     </link>
-    <gazebo reference="${prefix}_wheel_link">
+    <gazebo reference="${namespace}/${prefix}_wheel_link">
       <material>Gazebo/DarkGrey</material>
     </gazebo>
     <joint name="${prefix}_wheel" type="continuous">
-      <parent link="chassis_link"/>
-      <child link="${prefix}_wheel_link" />
+      <parent link="${namespace}/chassis_link"/>
+      <child link="${namespace}/${prefix}_wheel_link" />
       <xacro:insert_block name="joint_pose" />
       <axis xyz="0 1 0" />
@@ -75,5 +76,5 @@
   </xacro:macro>
   <xacro:macro name="headlight" params="headlight_prefix xyz rpy">
-    <link name="${headlight_prefix}_headlight_link">
+    <link name="${namespace}/${headlight_prefix}_headlight_link">
       <visual>
         <origin xyz="0 0 0" rpy="0 0 0" />
@@ -93,6 +94,6 @@
     </link>
     <joint name="${headlight_prefix}_headlight" type="fixed">
-      <parent link="base_link"/>
-      <child link="${headlight_prefix}_headlight_link"/>
+      <parent link="${namespace}/base_link"/>
+      <child link="${namespace}/${headlight_prefix}_headlight_link"/>
       <origin xyz="${xyz}" rpy="${rpy}"/>
     </joint>
@@ -163,5 +164,5 @@
     <gazebo>
       <joint name="${headlight_prefix}_headlight" type="fixed">
-        <parent>base_link</parent>
+        <parent>${namespace}/base_link</parent>
         <child>${headlight_prefix}_headlight::body</child>
       </joint>
@@ -169,5 +170,5 @@
   </xacro:macro>
   <xacro:macro name="led" params="led_prefix xyz rpy **plugin_params">
-    <link name="${led_prefix}_led_link">
+    <link name="${namespace}/${led_prefix}_led_link">
       <visual name="marker">
         <origin xyz="0 0 0" rpy="0 0 0" />
@@ -187,6 +188,6 @@
     </link>
     <joint name="${led_prefix}_led" type="fixed">
-      <parent link="base_link"/>
-      <child link="${led_prefix}_led_link"/>
+      <parent link="${namespace}/base_link"/>
+      <child link="${namespace}/${led_prefix}_led_link"/>
       <origin xyz="${xyz}" rpy="${rpy}"/>
     </joint>
@@ -252,5 +253,5 @@
     <gazebo>
       <joint name="${led_prefix}_led" type="fixed">
-        <parent>base_link</parent>
+        <parent>${namespace}/base_link</parent>
         <child>${led_prefix}_led::body</child>
       </joint>
@@ -316,11 +317,11 @@
     </plugin_params>
   </xacro:led>
-  <link name="base_link"></link>
+  <link name="${namespace}/base_link"></link>
   <joint name="base_link_joint" type="fixed">
     <origin xyz="0 0 0" rpy="0 0 0" />
-    <parent link="base_link"/>
-    <child link="chassis_link" />
-  </joint>
-  <link name="chassis_link">
+    <parent link="${namespace}/base_link"/>
+    <child link="${namespace}/chassis_link" />
+  </joint>
+  <link name="${namespace}/chassis_link">
     <visual>
       <origin xyz="0 0 ${footprint_vertical_offset}" rpy="${PI/2} 0 ${-PI/2}"/>
@@ -351,5 +352,5 @@
        always points to the "active" IMU. When an upgrade IMU is connected, the
        internal_imu_link should remain, but imu_link should point to the upgrade one. -->
-  <link name="imu_link">
+  <link name="${namespace}/imu_link">
     <inertial>
       <mass value="0.001"/>
@@ -359,9 +360,9 @@
   </link>
   <joint name="imu_joint" type="fixed">
-    <parent link="chassis_link" />
-    <child link="imu_link" />
-  </joint>
-  <!-- TODO: Same note as applies to imu_link -->
-  <link name="navsat_link">
+    <parent link="${namespace}/chassis_link" />
+    <child link="${namespace}/imu_link" />
+  </joint>
+  <!-- TODO: Same note as applies to ${namespace}/imu_link -->
+  <link name="${namespace}/navsat_link">
     <visual>
       <geometry>
@@ -373,24 +374,24 @@
   </link>
   <joint name="navsat_joint" type="fixed">
-    <parent link="chassis_link" />
-    <child link="navsat_link" />
+    <parent link="${namespace}/chassis_link" />
+    <child link="${namespace}/navsat_link" />
     <origin xyz="-0.180 0.126 0.1815" />
   </joint>
-  <link name="mid_mount"></link>
+  <link name="${namespace}/mid_mount"></link>
   <joint name="mid_mount_joint" type="fixed">
-    <parent link="chassis_link" />
-    <child link="mid_mount" />
+    <parent link="${namespace}/chassis_link" />
+    <child link="${namespace}/mid_mount" />
     <origin xyz="0 0 ${chassis_height}" />
   </joint>
-  <link name="rear_mount"></link>
+  <link name="${namespace}/rear_mount"></link>
   <joint name="rear_mount_joint" type="fixed">
-    <parent link="mid_mount" />
-    <child link="rear_mount" />
+    <parent link="${namespace}/mid_mount" />
+    <child link="${namespace}/rear_mount" />
     <origin xyz="${-mount_spacing} 0 0" />
   </joint>
-  <link name="front_mount"></link>
+  <link name="${namespace}/front_mount"></link>
   <joint name="front_mount_joint" type="fixed">
-    <parent link="mid_mount" />
-    <child link="front_mount" />
+    <parent link="${namespace}/mid_mount" />
+    <child link="${namespace}/front_mount" />
     <origin xyz="${mount_spacing} 0 0" />
   </joint>
