Commit message: Clean macros.

File: subt_sensors/urdf/planar_lidar.urdf.xacro (robot description, xacro)
@@ -13,7 +13,8 @@
 -->
 <robot xmlns:xacro="http://www.ros.org/wiki/xacro">
-  <xacro:macro name="planar_short_range_lidar" params="frame:=laser topic:=scan sample_size:=720 update_rate:=30
+  <xacro:macro name="planar_lidar" params="frame:=laser topic:=scan sample_size:=720 update_rate:=30
                min_angle:=-2.35619 max_angle:=2.35619 min_range:=0.1 max_range:=30.0 robot_namespace:=/
-               x:=0 y:=0 z:=0" >
+               x:=0 y:=0 z:=0
+               mesh:=package://subt_sensors/meshes/hokuyo.dae">
     <link name="${frame}">
       <inertial>
@@ -26,5 +27,5 @@
         <geometry>
           <!-- Origin of this mesh is the focal point of the LIDAR. -->
-          <mesh filename="package://subt_sensors/meshes/hokuyo.dae" />
+          <mesh filename="${mesh}" />
         </geometry>
       </visual>
@@ -47,11 +48,11 @@
               <samples>${sample_size}</samples>
               <resolution>1</resolution>
-              <max_angle>2.0944</max_angle> <!-- 120 Degree -->
-              <min_angle>-2.0944</min_angle> <!-- -120 Degree -->
+              <max_angle>${min_angle}</max_angle>
+              <min_angle>${max_angle}</min_angle>
             </horizontal>
           </scan>
           <range>
-            <min>0.10</min>
-            <max>5.0</max>
+            <min>${min_range}</min>
+            <max>${max_range}</max>
             <resolution>0.01</resolution>
           </range>

File: x2_description/urdf/accessories.urdf.xacro (robot description, xacro)
@@ -1,87 +1,78 @@
 <?xml version="1.0"?>
 <robot xmlns:xacro="http://www.ros.org/wiki/xacro">
-  <!--
-    As you add to this URDF, please be aware that both the robot and
-    simulation include it. You must retain compatibility with all of
-    the following launch files:
-    jackal_viz/launch/view_model.launch
-    jackal_gazebo/launch/jackal_world.launch
-    jackal_base/launch/base.launch
-  -->
   <!-- Macros to generate standoffs for offset payload mounting. -->
   <xacro:include filename="$(find jackal_description)/urdf/accessories/standoffs.urdf.xacro" />
   <!-- This optional plate mounts both the upgraded GPS and the Velodyne 3D LIDAR. -->
   <xacro:include filename="$(find jackal_description)/urdf/accessories/bridge_plate.urdf.xacro" />
-  <!-- If enabled, generate the LASER payload (by default, a SICK LMS111). -->
-  <!--<xacro:include filename="$(find jackal_description)/urdf/accessories/sick_lms1xx_mount.urdf.xacro" />
-  <xacro:if value="$(optenv JACKAL_LASER 0)">
-    <sick_lms1xx_mount prefix="$(optenv JACKAL_LASER_MOUNT front)"
-                       topic="$(optenv JACKAL_LASER_TOPIC front/scan)"/>
-    <joint name="$(optenv JACKAL_LASER_MOUNT front)_laser_mount_joint" type="fixed">
-      <origin xyz="$(optenv JACKAL_LASER_OFFSET 0 0 0)"
-              rpy="$(optenv JACKAL_LASER_RPY 0 0 0)" />
-      <parent link="$(optenv JACKAL_LASER_MOUNT front)_mount" />
-      <child link="$(optenv JACKAL_LASER_MOUNT front)_laser_mount" />
-    </joint>
-  </xacro:if>
--->
-  <xacro:include filename="$(find x2_description)/urdf/short_range_laser_mount.urdf.xacro" />
-  <xacro:include filename="$(find x2_description)/urdf/mid_range_laser_mount.urdf.xacro" />
+  <xacro:include filename="$(find x2_description)/urdf/laser_mount.urdf.xacro" />
+  <xacro:include filename="$(find subt_sensors)/urdf/planar_lidar.urdf.xacro" />
   <xacro:include filename="$(find x2_description)/urdf/camera_mount.urdf.xacro" />
   <xacro:include filename="$(find pointgrey_camera_description)/urdf/pointgrey_flea3.urdf.xacro" />
   <xacro:macro name="planar_short_range_lidar_and_mount">
-    <short_range_laser_mount prefix="$(optenv JACKAL_LASER_MOUNT front)"
-                       topic="$(optenv JACKAL_LASER_TOPIC front/scan)"/>
-    <joint name="$(optenv JACKAL_LASER_MOUNT front)_laser_mount_joint" type="fixed">
-      <origin xyz="$(optenv JACKAL_LASER_OFFSET 0 0 0)"
-              rpy="$(optenv JACKAL_LASER_RPY 0 0 0)" />
-      <parent link="$(optenv JACKAL_LASER_MOUNT front)_mount" />
-      <child link="$(optenv JACKAL_LASER_MOUNT front)_laser_mount" />
+    <laser_mount prefix="front"/>
+    <planar_lidar
+      frame="front_laser"
+      topic="front_scan"
+      mesh="package://subt_sensors/meshes/hokuyo.dae"
+      min_angle="2.3562"
+      max_angle="-2.3562"
+      min_range="0.1"
+      max_range="5"
+    />
+    <joint name="front_laser_mount_joint" type="fixed">
+      <origin xyz="0 0 0" rpy="0 0 0" />
+      <parent link="front_mount" />
+      <child link="front_laser_mount" />
     </joint>
   </xacro:macro>
   <xacro:macro name="planar_mid_range_lidar_and_mount">
-    <mid_range_laser_mount prefix="$(optenv JACKAL_LASER_MOUNT front)"
-                       topic="$(optenv JACKAL_LASER_TOPIC front/scan)"/>
-    <joint name="$(optenv JACKAL_LASER_MOUNT front)_laser_mount_joint" type="fixed">
-      <origin xyz="$(optenv JACKAL_LASER_OFFSET 0 0 0)"
-              rpy="$(optenv JACKAL_LASER_RPY 0 0 0)" />
-      <parent link="$(optenv JACKAL_LASER_MOUNT front)_mount" />
-      <child link="$(optenv JACKAL_LASER_MOUNT front)_laser_mount" />
+    <laser_mount prefix="front"/>
+    <planar_lidar
+      frame="front_laser"
+      topic="front_scan"
+      mesh="package://subt_sensors/meshes/sick-lms1xx.dae"
+      min_angle="2.3562"
+      max_angle="-2.3562"
+      min_range="0.1"
+      max_range="30"
+    />
+    <joint name="front_laser_mount_joint" type="fixed">
+      <origin xyz="0 0 0" rpy="0 0 0" />
+      <parent link="front_mount" />
+      <child link="front_laser_mount" />
     </joint>
   </xacro:macro>
   <xacro:macro name="qvga_camera_and_mount">
-    <camera_mount prefix="$(optenv JACKAL_FLEA3_MOUNT front)"
-                       tilt="$(optenv JACKAL_FLEA3_TILT 0.5236)"/>
-    <joint name="$(optenv JACKAL_FLEA3_MOUNT front)_camera_mount_joint" type="fixed">
-      <origin xyz="$(optenv JACKAL_FLEA3_OFFSET 0 0 0)"
-              rpy="$(optenv JACKAL_FLEA3_RPY 0 0 0)" />
-      <parent link="$(optenv JACKAL_FLEA3_MOUNT front)_mount" />
-      <child link="$(optenv JACKAL_FLEA3_MOUNT front)_camera_mount" />
+    <camera_mount prefix="front"
+                  tilt="0.5236"/>
+    <joint name="front_camera_mount_joint" type="fixed">
+      <origin xyz="0 0 0" rpy="0 0 0" />
+      <parent link="front_mount" />
+      <child link="front_camera_mount" />
     </joint>
-    <pointgrey_flea3 frame="$(optenv JACKAL_FLEA3_MOUNT front)_camera" name="$(optenv JACKAL_FLEA3_NAME front)"
+    <pointgrey_flea3 frame="front_camera" name="front"
       camera_x="0.0754" camera_y="0.029" camera_z="0.029"
       camera_mass="0.085" hfov="1.0471975512" fps="30" width="320" height="240"/>
-    <joint name="$(optenv JACKAL_FLEA3_MOUNT front)_camera_bracket_joint" type="fixed">
+    <joint name="front_camera_bracket_joint" type="fixed">
       <origin xyz="0.020 0 0.0245" rpy="0 0 0" />
-      <parent link="$(optenv JACKAL_FLEA3_MOUNT front)_camera_beam" />
-      <child link="$(optenv JACKAL_FLEA3_MOUNT front)_camera" />
+      <parent link="front_camera_beam" />
+      <child link="front_camera" />
     </joint>
   </xacro:macro>
   <xacro:macro name="hd_camera_and_mount">
-    <camera_mount prefix="$(optenv JACKAL_FLEA3_MOUNT front)"
-                       tilt="$(optenv JACKAL_FLEA3_TILT 0.5236)"/>
-    <joint name="$(optenv JACKAL_FLEA3_MOUNT front)_camera_mount_joint" type="fixed">
-      <origin xyz="$(optenv JACKAL_FLEA3_OFFSET 0 0 0)"
-              rpy="$(optenv JACKAL_FLEA3_RPY 0 0 0)" />
-      <parent link="$(optenv JACKAL_FLEA3_MOUNT front)_mount" />
-      <child link="$(optenv JACKAL_FLEA3_MOUNT front)_camera_mount" />
+    <camera_mount prefix="front"
+                  tilt="0.5236"/>
+    <joint name="front_camera_mount_joint" type="fixed">
+      <origin xyz="0 0 0" rpy="0 0 0" />
+      <parent link="front_mount" />
+      <child link="front_camera_mount" />
     </joint>
-    <pointgrey_flea3 frame="$(optenv JACKAL_FLEA3_MOUNT front)_camera" name="$(optenv JACKAL_FLEA3_NAME front)"
+    <pointgrey_flea3 frame="front_camera" name="front"
       camera_x="0.0754" camera_y="0.029" camera_z="0.029"
       camera_mass="0.085" hfov="1.0471975512" fps="30" width="1280" height="960"/>
-    <joint name="$(optenv JACKAL_FLEA3_MOUNT front)_camera_bracket_joint" type="fixed">
+    <joint name="front_camera_bracket_joint" type="fixed">
       <origin xyz="0.020 0 0.0245" rpy="0 0 0" />
-      <parent link="$(optenv JACKAL_FLEA3_MOUNT front)_camera_beam" />
-      <child link="$(optenv JACKAL_FLEA3_MOUNT front)_camera" />
+      <parent link="front_camera_beam" />
+      <child link="front_camera" />
     </joint>
   </xacro:macro>
@@ -89,4 +80,5 @@
          * 2D short range lidar
          * QVGA camera
+         * IMU
   -->
   <xacro:if value="$(optenv X2_SENSOR_CONFIG_1 0)">
@@ -97,4 +89,5 @@
          * 2D short range lidar
          * HD camera
+         * IMU
   -->
   <xacro:if value="$(optenv X2_SENSOR_CONFIG_2 0)">
@@ -105,4 +98,5 @@
          * 2D mid range lidar
          * QVGA camera
+         * IMU
   -->
   <xacro:if value="$(optenv X2_SENSOR_CONFIG_3 0)">
@@ -113,4 +107,5 @@
          * 2D mid range lidar
          * HD camera
+         * IMU
   -->
   <xacro:if value="$(optenv X2_SENSOR_CONFIG_4 0)">
@@ -118,84 +113,3 @@
     <hd_camera_and_mount />
   </xacro:if>
-  <!-- If enabled, generate the upgraded Navsat payload (a Novatel Smart6). -->
-  <xacro:include filename="$(find jackal_description)/urdf/accessories/novatel_smart6.urdf.xacro" />
-  <xacro:if value="$(optenv JACKAL_NAVSAT 0)">
-    <bridge_plate mount="$(optenv JACKAL_NAVSAT_MOUNT rear)"
-                  height="$(optenv JACKAL_NAVSAT_HEIGHT 0.1)" />
-    <novatel_smart6 prefix="$(optenv JACKAL_NAVSAT_MOUNT rear)"/>
-    <joint name="$(optenv JACKAL_NAVSAT_MOUNT rear)_navsat_joint" type="fixed">
-      <origin xyz="0 0 0" rpy="0 0 0" />
-      <parent link="$(optenv JACKAL_NAVSAT_MOUNT rear)_bridge" />
-      <child link="$(optenv JACKAL_NAVSAT_MOUNT rear)_navsat" />
-    </joint>
-  </xacro:if>
-  <!-- Common camera mounts and accessory URDFs. -->
-  <xacro:include filename="$(find jackal_description)/urdf/accessories/camera_mount.urdf.xacro" />
-  <xacro:include filename="$(find pointgrey_camera_description)/urdf/pointgrey_flea3.urdf.xacro" />
-  <!-- If enabled, generate the flea3 camera payload with a tilt of 30 degrees. -->
-  <xacro:if value="$(optenv JACKAL_FLEA3 0)">
-    <camera_mount prefix="$(optenv JACKAL_FLEA3_MOUNT front)"
-                       tilt="$(optenv JACKAL_FLEA3_TILT 0.5236)"/>
-    <joint name="$(optenv JACKAL_FLEA3_MOUNT front)_camera_mount_joint" type="fixed">
-      <origin xyz="$(optenv JACKAL_FLEA3_OFFSET 0 0 0)"
-              rpy="$(optenv JACKAL_FLEA3_RPY 0 0 0)" />
-      <parent link="$(optenv JACKAL_FLEA3_MOUNT front)_mount" />
-      <child link="$(optenv JACKAL_FLEA3_MOUNT front)_camera_mount" />
-    </joint>
-    <pointgrey_flea3 frame="$(optenv JACKAL_FLEA3_MOUNT front)_camera" name="$(optenv JACKAL_FLEA3_NAME front)"
-      camera_x="0.0754" camera_y="0.029" camera_z="0.029"
-      camera_mass="0.085" hfov="1.0471975512" fps="60" width="640" height="512"/>
-    <joint name="$(optenv JACKAL_FLEA3_MOUNT front)_camera_bracket_joint" type="fixed">
-      <origin xyz="0.020 0 0.0245" rpy="0 0 0" />
-      <parent link="$(optenv JACKAL_FLEA3_MOUNT front)_camera_beam" />
-      <child link="$(optenv JACKAL_FLEA3_MOUNT front)_camera" />
-    </joint>
-  </xacro:if>
-  <xacro:include filename="$(find jackal_description)/urdf/accessories/stereo_camera_mount.urdf.xacro" />
-  <!-- If enabled, generates a pair of flea3 cameras for stereo vision with a tilt of 30 degrees. -->
-  <xacro:if value="$(optenv JACKAL_STEREO_FLEA3 0)">
-    <stereo_camera_mount prefix="$(optenv JACKAL_FLEA3_MOUNT front)"
-                       tilt="$(optenv JACKAL_FLEA3_TILT 0.5236)"/>
-    <joint name="$(optenv JACKAL_FLEA3_MOUNT front)_stereo_camera_mount_joint" type="fixed">
-      <origin xyz="$(optenv JACKAL_FLEA3_OFFSET 0 0 0)"
-              rpy="$(optenv JACKAL_FLEA3_RPY 0 0 0)" />
-      <parent link="$(optenv JACKAL_FLEA3_MOUNT front)_mount" />
-      <child link="$(optenv JACKAL_FLEA3_MOUNT front)_stereo_camera_mount" />
-    </joint>
-    <pointgrey_flea3 frame="$(optenv JACKAL_FLEA3_MOUNT front)_left_camera" name="$(optenv JACKAL_FLEA3_LEFT_NAME front/left)"
-      camera_x="0.0754" camera_y="0.029" camera_z="0.029"
-      camera_mass="0.085" hfov="1.0471975512" fps="60" width="640" height="512"/>
-    <joint name="$(optenv JACKAL_FLEA3_MOUNT front)_left_stereo_camera_bracket_joint" type="fixed">
-      <origin xyz="0.015 $(optenv JACKAL_STEREO_SEPERATION 0.16) 0.0599" rpy="0 0 0" />
-      <parent link="$(optenv JACKAL_FLEA3_MOUNT front)_stereo_camera_beam" />
-      <child link="$(optenv JACKAL_FLEA3_MOUNT front)_left_camera" />
-    </joint>
-    <pointgrey_flea3 frame="$(optenv JACKAL_FLEA3_MOUNT front)_right_camera" name="$(optenv JACKAL_FLEA3_RIGHT_NAME front/right)"
-      camera_x="0.0754" camera_y="0.029" camera_z="0.029"
-      camera_mass="0.085" hfov="1.0471975512" fps="60" width="640" height="512"/>
-    <joint name="$(optenv JACKAL_FLEA3_MOUNT front)_right_stereo_camera_bracket_joint" type="fixed">
-      <origin xyz="0.015 -$(optenv JACKAL_STEREO_SEPERATION 0.16) 0.0599" rpy="0 0 0" />
-      <parent link="$(optenv JACKAL_FLEA3_MOUNT front)_stereo_camera_beam" />
-      <child link="$(optenv JACKAL_FLEA3_MOUNT front)_right_camera" />
-    </joint>
-  </xacro:if>
-  <!-- If enabled, generate the bumblebee2 camera payload with a tilt of 0 degrees. -->
-  <xacro:include filename="$(find pointgrey_camera_description)/urdf/pointgrey_bumblebee2.urdf.xacro" />
-  <!-- If enabled, generate the bumblebee2 camera payload with a tilt of 0 degrees. -->
-  <xacro:if value="$(optenv JACKAL_BB2 0)">
-    <camera_mount prefix="$(optenv JACKAL_BB2_MOUNT front)"
-                        tilt="$(optenv JACKAL_BB2_TILT 0)"/>
-    <joint name="$(optenv JACKAL_BB2_MOUNT front)_camera_mount_joint" type="fixed">
-      <origin xyz="$(optenv JACKAL_BB2_OFFSET 0 0 0)"
-              rpy="$(optenv JACKAL_BB2_RPY 0 0 0)" />
-      <parent link="$(optenv JACKAL_BB2_MOUNT front)_mount" />
-      <child link="$(optenv JACKAL_BB2_MOUNT front)_camera_mount" />
-    </joint>
-    <BB2-08S2C-38 frame="$(optenv JACKAL_BB2_MOUNT front)_camera" name="$(optenv JACKAL_BB2_NAME front)" />
-    <joint name="$(optenv JACKAL_BB2_MOUNT front)_camera_bracket_joint" type="fixed">
-      <origin xyz="0.007 0 0.02450" rpy="0 0 0" />
-      <parent link="$(optenv JACKAL_BB2_MOUNT front)_camera_beam" />
-      <child link="$(optenv JACKAL_BB2_MOUNT front)_camera" />
-    </joint>
-  </xacro:if>
 </robot>

File: x2_description/urdf/laser_mount.urdf.xacro (robot description, xacro)
@@ -26,9 +26,6 @@
 -->
 <robot xmlns:xacro="http://ros.org/wiki/xacro">
-  <xacro:include filename="$(find subt_sensors)/urdf/2d_short_range_lidar.urdf.xacro" />
-  <xacro:macro name="short_range_laser_mount" params="prefix topic
-    x:=0 y:=0 z:=0">
-    <planar_short_range_lidar frame="${prefix}_laser" topic="${topic}"
-      x="${x}" y="${y}" z="${z}"/>
+  <xacro:include filename="$(find subt_sensors)/urdf/planar_lidar.urdf.xacro" />
+  <xacro:macro name="laser_mount" params="prefix x:=0 y:=0 z:=0">
     <link name="${prefix}_laser_mount">
       <visual>
