Commit message: Sensor configurations for X1.

File: subt_sensors/urdf/planar_lidar.urdf.xacro (robot description, xacro)
@@ -13,9 +13,30 @@
 -->
 <robot xmlns:xacro="http://www.ros.org/wiki/xacro">
-  <xacro:macro name="planar_lidar" params="frame:=laser topic:=scan sample_size:=720 update_rate:=30
-               min_angle:=-2.35619 max_angle:=2.35619 min_range:=0.1 max_range:=30.0 robot_namespace:=/
-               x:=0 y:=0 z:=0
-               mesh:=package://subt_sensors/meshes/hokuyo.dae">
-    <link name="${frame}">
+  <!-- Macro to insert a 2D scanning LIDAR with ROS integration.
+    name: Name of the link associated to the sensor.
+    topic: ROS topic name where the laser scan is published.
+    samples: number of samples during scan.
+    update_rate: frequency to publish output, hz.
+    min_angle: the horizontal angle that the scan begins at.
+    max_angle: the angle that the scan ends at.
+    min_range: minimum distance for an object to be detected by laser.
+    max_range: maximum distance for an object to be detected by laser.
+    robot_namespace: The robot namespace.
+    mesh: The laser mesh.
+    noise_stddev: Standard deviation of gaussian noise applied to output.
+  -->
+  <xacro:macro name="planar_lidar"
+               params="name:=laser
+                       update_rate:=30
+                       samples:=720
+                       min_angle:=-2.35619
+                       max_angle:=2.35619
+                       min_range:=0.1
+                       max_range:=30.0
+                       noise_stddev:=0.01
+                       robot_namespace:=/
+                       topic:=scan
+                       mesh:=package://subt_sensors/meshes/hokuyo.dae">
+    <link name="${name}">
       <inertial>
         <mass value="1e-5" />
@@ -37,14 +58,12 @@
       </collision>
     </link>
-    <gazebo reference="${frame}">
+    <gazebo reference="${name}">
       <turnGravityOff>false</turnGravityOff>
-      <sensor type="gpu_ray" name="${frame}">
-        <pose>${x} ${y} ${z} 0 0 0</pose>
-        <visualize>false</visualize>
+      <sensor type="gpu_ray" name="${name}">
         <update_rate>${update_rate}</update_rate>
         <ray>
           <scan>
             <horizontal>
-              <samples>${sample_size}</samples>
+              <samples>${samples}</samples>
               <resolution>1</resolution>
               <max_angle>${min_angle}</max_angle>
@@ -60,10 +79,10 @@
             <type>gaussian</type>
             <mean>0.0</mean>
-            <stddev>0.001</stddev>
+            <stddev>${noise_stddev}</stddev>
           </noise>
         </ray>
-       <plugin name="gazebo_ros_2d_short_range_lidar" filename="libgazebo_ros_gpu_laser.so">
+       <plugin name="gazebo_ros_planar_lidar" filename="libgazebo_ros_gpu_laser.so">
           <topicName>${topic}</topicName>
-          <frameName>${frame}</frameName>
+          <frameName>${name}</frameName>
           <robotNamespace>${robot_namespace}</robotNamespace>
         </plugin>

File: x1_description/urdf/decorations.urdf.xacro (robot description, xacro)
@@ -61,5 +61,5 @@
       <parent link="${namespace}/top_plate_link" />
       <child link="${namespace}/top_plate_front_link"/>
-      <origin xyz="0.36367 0 0.00639" rpy="0 0 0"/>
+      <origin xyz="0.24 0 0.00639" rpy="0 0 0"/>
     </joint>
     <!-- Top plate rear link-->

File: x1_description/urdf/sensors.urdf.xacro (robot description, xacro)
@@ -2,12 +2,9 @@
 <robot xmlns:xacro="http://www.ros.org/wiki/xacro">
   <xacro:property name="namespace" value="$(arg robot_namespace)" />
-  <!-- Macros to generate standoffs for offset payload mounting. -->
-  <xacro:include filename="$(find jackal_description)/urdf/accessories/standoffs.urdf.xacro" />
-  <!-- This optional plate mounts both the upgraded GPS and the Velodyne 3D LIDAR. -->
-  <xacro:include filename="$(find jackal_description)/urdf/accessories/bridge_plate.urdf.xacro" />
   <xacro:include filename="$(find x2_description)/urdf/laser_mount.urdf.xacro" />
   <xacro:include filename="$(find subt_sensors)/urdf/planar_lidar.urdf.xacro" />
   <xacro:include filename="$(find x2_description)/urdf/camera_mount.urdf.xacro" />
   <xacro:include filename="$(find pointgrey_camera_description)/urdf/pointgrey_flea3.urdf.xacro" />
+  <xacro:include filename="$(find subt_sensors)/urdf/3d_lidar.urdf.xacro" />
   <xacro:macro name="planar_short_range_lidar_and_mount">
     <laser_mount prefix="front"/>
@@ -23,5 +20,5 @@
     <joint name="front_laser_mount_joint" type="fixed">
       <origin xyz="0 0 0" rpy="0 0 0" />
-      <parent link="${namespace}/front_mount" />
+      <parent link="${namespace}/top_plate_front_link" />
       <child link="front_laser_mount" />
     </joint>
@@ -40,5 +37,30 @@
     <joint name="front_laser_mount_joint" type="fixed">
       <origin xyz="0 0 0" rpy="0 0 0" />
-      <parent link="${namespace}/front_mount" />
+      <parent link="${namespace}/top_plate_front_link" />
+      <child link="front_laser_mount" />
+    </joint>
+  </xacro:macro>
+  <xacro:macro name="velodyne_mid_range_lidar_and_mount">
+    <laser_mount prefix="front"/>
+    <velodyne_lidar
+      name="front_laser"
+      topic="${namespace}/points"
+    />
+    <joint name="front_laser_mount_joint" type="fixed">
+      <origin xyz="0 0 0" rpy="0 0 0" />
+      <parent link="${namespace}/top_plate_link" />
+      <child link="front_laser_mount" />
+    </joint>
+  </xacro:macro>
+  <xacro:macro name="velodyne_long_range_lidar_and_mount">
+    <laser_mount prefix="front"/>
+    <velodyne_lidar
+      name="front_laser"
+      topic="${namespace}/points"
+      max_range="300"
+    />
+    <joint name="front_laser_mount_joint" type="fixed">
+      <origin xyz="0 0 0" rpy="0 0 0" />
+      <parent link="${namespace}/top_plate_link" />
       <child link="front_laser_mount" />
     </joint>
@@ -49,5 +71,5 @@
     <joint name="front_camera_mount_joint" type="fixed">
       <origin xyz="0 0 0" rpy="0 0 0" />
-      <parent link="${namespace}/front_mount" />
+      <parent link="${namespace}/top_plate_front_link" />
       <child link="front_camera_mount" />
     </joint>
@@ -67,5 +89,5 @@
     <joint name="front_camera_mount_joint" type="fixed">
       <origin xyz="0 0 0" rpy="0 0 0" />
-      <parent link="${namespace}/front_mount" />
+      <parent link="${namespace}/top_plate_front_link" />
       <child link="front_camera_mount" />
     </joint>
@@ -80,39 +102,3 @@
     </joint>
   </xacro:macro>
-  <!-- Sensor configuration #1
-         * 2D short range lidar
-         * QVGA camera
-         * IMU
-  -->
-  <xacro:if value="$(optenv X2_SENSOR_CONFIG_1 0)">
-    <planar_short_range_lidar_and_mount />
-    <qvga_camera_and_mount />
-  </xacro:if>
-  <!-- Sensor configuration #2
-         * 2D short range lidar
-         * HD camera
-         * IMU
-  -->
-  <xacro:if value="$(optenv X2_SENSOR_CONFIG_2 0)">
-    <planar_short_range_lidar_and_mount />
-    <hd_camera_and_mount />
-  </xacro:if>
-  <!-- Sensor configuration #3
-         * 2D mid range lidar
-         * QVGA camera
-         * IMU
-  -->
-  <xacro:if value="$(optenv X2_SENSOR_CONFIG_3 0)">
-    <planar_mid_range_lidar_and_mount />
-    <qvga_camera_and_mount />
-  </xacro:if>
-  <!-- Sensor configuration #4
-         * 2D mid range lidar
-         * HD camera
-         * IMU
-  -->
-  <xacro:if value="$(optenv X2_SENSOR_CONFIG_4 0)">
-    <planar_mid_range_lidar_and_mount />
-    <hd_camera_and_mount />
-  </xacro:if>
 </robot>

File: x1_description/urdf/x1.urdf.xacro (robot description, xacro)
@@ -201,4 +201,41 @@
     </plugin_params>
   </xacro:led>
+  <xacro:include filename="$(find x1_description)/urdf/sensors.urdf.xacro" />
+  <!-- Sensor configuration #1
+         * 2D short range lidar
+         * QVGA camera
+         * IMU
+  -->
+  <xacro:if value="$(optenv X1_SENSOR_CONFIG_1 0)">
+    <planar_short_range_lidar_and_mount />
+    <qvga_camera_and_mount />
+  </xacro:if>
+  <!-- Sensor configuration #2
+         * 2D short range lidar
+         * HD camera
+         * IMU
+  -->
+  <xacro:if value="$(optenv X1_SENSOR_CONFIG_2 0)">
+    <planar_short_range_lidar_and_mount />
+    <hd_camera_and_mount />
+  </xacro:if>
+  <!-- Sensor configuration #3
+         * 3D mid range lidar
+         * QVGA camera
+         * IMU
+  -->
+  <xacro:if value="$(optenv X1_SENSOR_CONFIG_3 0)">
+    <velodyne_mid_range_lidar_and_mount />
+    <qvga_camera_and_mount />
+  </xacro:if>
+  <!-- Sensor configuration #4
+         * 3D long range lidar
+         * HD camera
+         * IMU
+  -->
+  <xacro:if value="$(optenv X1_SENSOR_CONFIG_4 0)">
+    <velodyne_long_range_lidar_and_mount />
+    <hd_camera_and_mount />
+  </xacro:if>
   <xacro:if value="$(arg laser_enabled)">
     <sick_lms1xx_mount prefix="base"/>
