Commit message: More namespace and tweaking.

File: subt_sensors/urdf/3d_lidar.urdf.xacro (robot description, xacro)
@@ -46,11 +46,9 @@
                                              topic:=points">
     <link name="${name}">
-      <visual name="${name}_visual">>
+      <visual name="${name}_top_visual">
+        <origin xyz="0 0 0" rpy="0 0 1.5707" />
         <geometry>
-          <cylinder radius="0.025" length="0.1" />
+          <mesh filename="model://velodyne_hdl32/meshes/velodyne_top.dae" />
         </geometry>
-        <material name="${name}_visual_material">
-          <color rgba="0.5 1.0 0.5 1.0" />
-        </material>
       </visual>
     </link>

File: x1_description/urdf/sensors.urdf.xacro (robot description, xacro)
@@ -10,5 +10,5 @@
     <laser_mount prefix="front"/>
     <planar_lidar
-      name="front_laser"
+      name="${namespace}/front_laser"
       topic="${namespace}/front_scan"
       mesh="package://subt_sensors/meshes/hokuyo.dae"
@@ -21,5 +21,5 @@
       <origin xyz="0 0 0" rpy="0 0 0" />
       <parent link="${namespace}/top_plate_front_link" />
-      <child link="front_laser_mount" />
+      <child link="${namespace}/front_laser_mount" />
     </joint>
   </xacro:macro>
@@ -27,5 +27,5 @@
     <laser_mount prefix="front"/>
     <planar_lidar
-      name="front_laser"
+      name="${namespace}/front_laser"
       topic="${namespace}/front_scan"
       mesh="package://subt_sensors/meshes/sick-lms1xx.dae"
@@ -38,5 +38,5 @@
       <origin xyz="0 0 0" rpy="0 0 0" />
       <parent link="${namespace}/top_plate_front_link" />
-      <child link="front_laser_mount" />
+      <child link="${namespace}/front_laser_mount" />
     </joint>
   </xacro:macro>
@@ -44,5 +44,5 @@
     <laser_mount prefix="front"/>
     <velodyne_lidar
-      name="front_laser"
+      name="${namespace}/front_laser"
       topic="${namespace}/points"
     />
@@ -50,5 +50,5 @@
       <origin xyz="0 0 0" rpy="0 0 0" />
       <parent link="${namespace}/top_plate_link" />
-      <child link="front_laser_mount" />
+      <child link="${namespace}/front_laser_mount" />
     </joint>
   </xacro:macro>
@@ -56,5 +56,5 @@
     <laser_mount prefix="front"/>
     <velodyne_lidar
-      name="front_laser"
+      name="${namespace}/front_laser"
       topic="${namespace}/points"
       max_range="300"
@@ -63,5 +63,5 @@
       <origin xyz="0 0 0" rpy="0 0 0" />
       <parent link="${namespace}/top_plate_link" />
-      <child link="front_laser_mount" />
+      <child link="${namespace}/front_laser_mount" />
     </joint>
   </xacro:macro>
@@ -72,7 +72,7 @@
       <origin xyz="0 0 0" rpy="0 0 0" />
       <parent link="${namespace}/top_plate_front_link" />
-      <child link="front_camera_mount" />
+      <child link="${namespace}/front_camera_mount" />
     </joint>
-    <pointgrey_flea3 frame="front_camera" name="front"
+    <pointgrey_flea3 frame="${namespace}/front_camera" name="front"
       camera_x="0.0754" camera_y="0.029" camera_z="0.029"
       camera_mass="0.085" hfov="1.0471975512" fps="30" width="320" height="240"
@@ -80,6 +80,6 @@
     <joint name="front_camera_bracket_joint" type="fixed">
       <origin xyz="0.020 0 0.0245" rpy="0 0 0" />
-      <parent link="front_camera_beam" />
-      <child link="front_camera" />
+      <parent link="${namespace}/front_camera_beam" />
+      <child link="${namespace}/front_camera" />
     </joint>
   </xacro:macro>
@@ -90,7 +90,7 @@
       <origin xyz="0 0 0" rpy="0 0 0" />
       <parent link="${namespace}/top_plate_front_link" />
-      <child link="front_camera_mount" />
+      <child link="${namespace}/front_camera_mount" />
     </joint>
-    <pointgrey_flea3 frame="front_camera" name="front"
+    <pointgrey_flea3 frame="${namespace}/front_camera" name="front"
       camera_x="0.0754" camera_y="0.029" camera_z="0.029"
       camera_mass="0.085" hfov="1.0471975512" fps="30" width="1280" height="960"
@@ -98,6 +98,6 @@
     <joint name="front_camera_bracket_joint" type="fixed">
       <origin xyz="0.020 0 0.0245" rpy="0 0 0" />
-      <parent link="front_camera_beam" />
-      <child link="front_camera" />
+      <parent link="${namespace}/front_camera_beam" />
+      <child link="${namespace}/front_camera" />
     </joint>
   </xacro:macro>

File: x2_description/urdf/accessories.urdf.xacro (robot description, xacro)
@@ -13,5 +13,5 @@
     <laser_mount prefix="front"/>
     <planar_lidar
-      name="front_laser"
+      name="${namespace}/front_laser"
       topic="${namespace}/front_scan"
       mesh="package://subt_sensors/meshes/hokuyo.dae"
@@ -24,5 +24,5 @@
       <origin xyz="0 0 0" rpy="0 0 0" />
       <parent link="${namespace}/front_mount" />
-      <child link="front_laser_mount" />
+      <child link="${namespace}/front_laser_mount" />
     </joint>
   </xacro:macro>
@@ -30,5 +30,5 @@
     <laser_mount prefix="front"/>
     <planar_lidar
-      name="front_laser"
+      name="${namespace}/front_laser"
       topic="${namespace}/front_scan"
       mesh="package://subt_sensors/meshes/sick-lms1xx.dae"
@@ -41,5 +41,5 @@
       <origin xyz="0 0 0" rpy="0 0 0" />
       <parent link="${namespace}/front_mount" />
-      <child link="front_laser_mount" />
+      <child link="${namespace}/front_laser_mount" />
     </joint>
   </xacro:macro>
@@ -50,7 +50,7 @@
       <origin xyz="0 0 0" rpy="0 0 0" />
       <parent link="${namespace}/front_mount" />
-      <child link="front_camera_mount" />
+      <child link="${namespace}/front_camera_mount" />
     </joint>
-    <pointgrey_flea3 frame="front_camera" name="front"
+    <pointgrey_flea3 frame="${namespace}/front_camera" name="front"
       camera_x="0.0754" camera_y="0.029" camera_z="0.029"
       camera_mass="0.085" hfov="1.0471975512" fps="30" width="320" height="240"
@@ -58,6 +58,6 @@
     <joint name="front_camera_bracket_joint" type="fixed">
       <origin xyz="0.020 0 0.0245" rpy="0 0 0" />
-      <parent link="front_camera_beam" />
-      <child link="front_camera" />
+      <parent link="${namespace}/front_camera_beam" />
+      <child link="${namespace}/front_camera" />
     </joint>
   </xacro:macro>
@@ -68,7 +68,7 @@
       <origin xyz="0 0 0" rpy="0 0 0" />
       <parent link="${namespace}/front_mount" />
-      <child link="front_camera_mount" />
+      <child link="${namespace}/front_camera_mount" />
     </joint>
-    <pointgrey_flea3 frame="front_camera" name="front"
+    <pointgrey_flea3 frame="${namespace}/front_camera" name="front"
       camera_x="0.0754" camera_y="0.029" camera_z="0.029"
       camera_mass="0.085" hfov="1.0471975512" fps="30" width="1280" height="960"
@@ -76,6 +76,6 @@
     <joint name="front_camera_bracket_joint" type="fixed">
       <origin xyz="0.020 0 0.0245" rpy="0 0 0" />
-      <parent link="front_camera_beam" />
-      <child link="front_camera" />
+      <parent link="${namespace}/front_camera_beam" />
+      <child link="${namespace}/front_camera" />
     </joint>
   </xacro:macro>

File: x2_description/urdf/camera_mount.urdf.xacro (robot description, xacro)
@@ -1,5 +1,7 @@
+<?xml version="1.0"?>
 <robot xmlns:xacro="http://ros.org/wiki/xacro">
+  <xacro:property name="namespace" value="$(arg robot_namespace)" />
   <xacro:macro name="camera_mount" params="prefix tilt:=0">
-    <link name="${prefix}_camera_mount">
+    <link name="${namespace}/${prefix}_camera_mount">
       <visual>
         <origin xyz="0 0 0" rpy="1.5707 0 1.5707" />
@@ -10,5 +12,5 @@
       </visual>
     </link>
-    <link name="${prefix}_camera_beam">
+    <link name="${namespace}/${prefix}_camera_beam">
       <visual>
         <origin xyz="0 0 0" rpy="0 0 1.5707" />
@@ -21,11 +23,11 @@
     <joint name="${prefix}_camera_pivot_joint" type="fixed">
       <origin xyz="0.102 0 0.008" rpy="0 ${tilt} 0" />
-      <parent link="${prefix}_camera_mount" />
-      <child link="${prefix}_camera_beam" />
+      <parent link="${namespace}/${prefix}_camera_mount" />
+      <child link="${namespace}/${prefix}_camera_beam" />
     </joint>
-    <gazebo reference="${prefix}_camera_beam">
+    <gazebo reference="${namespace}/${prefix}_camera_beam">
       <material>Gazebo/DarkGrey</material>
     </gazebo>
-    <gazebo reference="${prefix}_camera_mount">
+    <gazebo reference="${namespace}/${prefix}_camera_mount">
       <material>Gazebo/DarkGrey</material>
     </gazebo>

File: x2_description/urdf/laser_mount.urdf.xacro (robot description, xacro)
@@ -26,7 +26,8 @@
 -->
 <robot xmlns:xacro="http://ros.org/wiki/xacro">
+  <xacro:property name="namespace" value="$(arg robot_namespace)" />
   <xacro:include filename="$(find subt_sensors)/urdf/planar_lidar.urdf.xacro" />
   <xacro:macro name="laser_mount" params="prefix x:=0 y:=0 z:=0">
-    <link name="${prefix}_laser_mount">
+    <link name="${namespace}/${prefix}_laser_mount">
       <visual>
         <origin xyz="${x} ${y} ${z}" rpy="0 0 0" />
@@ -41,8 +42,8 @@
       <!-- This offset is from the base of the bracket to the LIDAR's focal point. -->
       <origin xyz="0 0 0.149" rpy="0 0 0" />
-      <parent link="${prefix}_laser_mount" />
-      <child link="${prefix}_laser" />
+      <parent link="${namespace}/${prefix}_laser_mount" />
+      <child link="${namespace}/${prefix}_laser" />
     </joint>
-    <gazebo reference="${prefix}_laser_mount">
+    <gazebo reference="${namespace}/${prefix}_laser_mount">
       <material>Gazebo/DarkGrey</material>
     </gazebo>

Commit message: No mesh

File: subt_sensors/urdf/3d_lidar.urdf.xacro (robot description, xacro)
@@ -46,9 +46,13 @@
                                              topic:=points">
     <link name="${name}">
-      <visual name="${name}_top_visual">
-        <origin xyz="0 0 0" rpy="0 0 1.5707" />
+      <visual name="${name}_visual">>
         <geometry>
-          <mesh filename="model://velodyne_hdl32/meshes/velodyne_top.dae" />
+          <mesh>
+            <cylinder radius="0.025" length="0.1" />
+          </mesh>
         </geometry>
+        <material name="${name}_visual_material">
+          <color rgba="0.5 1.0 0.5 1.0" />
+        </material>
       </visual>
     </link>

Commit message: No mesh

File: subt_sensors/urdf/3d_lidar.urdf.xacro (robot description, xacro)
@@ -48,7 +48,5 @@
       <visual name="${name}_visual">>
         <geometry>
-          <mesh>
-            <cylinder radius="0.025" length="0.1" />
-          </mesh>
+          <cylinder radius="0.025" length="0.1" />
         </geometry>
         <material name="${name}_visual_material">
