Commit message: Use spotlight meshes.
This also creates a new package called `subt_description` to hold some common urdf files and meshes. `flashlight.urdf.xacro` and `led.urdf.xacro` have been moved there from `subt_gazebo`.

File: subt_description/urdf/flashlight.urdf.xacro (robot description, xacro)
@@ -1,43 +1,32 @@
 <?xml version="1.0"?>
 <robot xmlns:xacro="http://www.ros.org/wiki/xacro" name="flashlight">
-  <xacro:macro name="flashlight" params="flashlight_prefix parent_link default_color:='0.8 0.8 0.5' *pose **plugin_params">
+  <xacro:macro name="flashlight" params="flashlight_prefix parent_link xyz rpy default_color:='0.8 0.8 0.5' **plugin_params">
+    <link name="${namespace}/${flashlight_prefix}_flashlight_link">
+      <visual>
+        <origin xyz="-0.065 0.0 0" rpy="0 0 -1.57" />
+        <geometry>
+          <mesh filename="package://subt_description/meshes/spotlight.dae" scale="0.01 0.01 0.01"/>
+        </geometry>
+      </visual>
+      <inertial>
+        <origin xyz="0 0 0" rpy="0 0 0"/>
+        <mass value="0.000001" />
+        <inertia
+          ixx="0.001"
+          ixy="0.0" iyy="0.001"
+          ixz="0.0" iyz="0.0" izz="0.001"
+        />
+      </inertial>
+    </link>
+    <joint name="${flashlight_prefix}_flashlight" type="fixed">
+      <parent link="${parent_link}"/>
+      <child link="${namespace}/${flashlight_prefix}_flashlight_link"/>
+      <origin xyz="${xyz}" rpy="${rpy}"/>
+    </joint>
     <gazebo>
       <model name='${flashlight_prefix}_flashlight'>
-        <xacro:insert_block name="pose"/>
-        <link name='handle'>
-          <pose>0 0 0.025 0 0 0</pose>
-          <inertial>
-            <mass>0.0025</mass>
-            <inertia>
-              <ixx>1.0e-05</ixx>
-              <ixy>0</ixy>
-              <ixz>0</ixz>
-              <iyy>1.0e-05</iyy>
-              <iyz>0</iyz>
-              <izz>1.0e-05</izz>
-            </inertia>
-          </inertial>
-          <collision name='collision'>
-            <geometry>
-              <cylinder>
-                <radius>0.025</radius>
-                <length>0.05</length>
-              </cylinder>
-            </geometry>
-          </collision>
-          <visual name='visual'>
-            <geometry>
-              <cylinder>
-                <radius>0.025</radius>
-                <length>0.05</length>
-              </cylinder>
-            </geometry>
-            <material>
-              <ambient>0 0 0 1</ambient>
-            </material>
-          </visual>
-        </link>
+        <pose>${xyz} ${rpy}</pose>
         <link name='light_source'>
-          <pose>0 0 0.05 0 0 0</pose>
+          <pose>0 0 0.0 0.01 ${M_PI/2} 0</pose>
           <inertial>
             <mass>0.0025</mass>
@@ -52,5 +41,5 @@
           </inertial>
           <light name='lamp' type='spot'>
-            <pose>0 0 0.0 0 3.14159 0</pose>
+            <pose>0 0 0.0 0 ${M_PI} 0</pose>
             <attenuation>
               <range>15</range>
@@ -70,9 +59,13 @@
           <visual name='lamp'>
             <geometry>
-              <sphere>
-                <radius>0.020</radius>
-              </sphere>
+              <cylinder>
+                <radius>0.019</radius>
+                <length>0.005</length>
+              </cylinder>
+              <!--<sphere>-->
+              <!--  <radius>0.020</radius>-->
+              <!--</sphere>-->
             </geometry>
-            <transparency>0</transparency>
+            <transparency>0.0</transparency>
             <material>
               <ambient>1 1 1 1</ambient>
@@ -89,8 +82,4 @@
           </visual>
         </link>
-        <joint name='joint' type='fixed'>
-          <parent>handle</parent>
-          <child>light_source</child>
-        </joint>
         <plugin name='light_control' filename='libRosFlashLightPlugin.so'>
           <service_name>enable</service_name>
@@ -109,5 +98,5 @@
       <joint name='${flashlight_prefix}_flashlight_joint' type='fixed'>
         <parent>${parent_link}</parent>
-        <child>${flashlight_prefix}_flashlight::handle</child>
+        <child>${flashlight_prefix}_flashlight::light_source</child>
       </joint>
     </gazebo>

File: subt_description/urdf/led.urdf.xacro (robot description, xacro)
@@ -1,11 +1,32 @@
 <?xml version="1.0"?>
 <robot xmlns:xacro="http://www.ros.org/wiki/xacro" name="flashlight">
-  <xacro:macro name="led" params="led_prefix parent_link default_color:='0 0 0' *pose **plugin_params">
+  <xacro:macro name="led" params="led_prefix parent_link xyz rpy default_color:='0 0 0'  **plugin_params">
+    <link name="${namespace}/${led_prefix}_led_link">
+      <visual name="marker">
+        <origin xyz="0 0 0" rpy="0 0 0" />
+        <geometry>
+          <mesh filename="package://subt_description/meshes/led.dae" />
+        </geometry>
+      </visual>
+      <inertial>
+        <origin xyz="0 0 0" rpy="0 0 0"/>
+        <mass value="0.000001" />
+        <inertia
+          ixx="0.001"
+          ixy="0.0" iyy="0.001"
+          ixz="0.0" iyz="0.0" izz="0.001"
+          />
+      </inertial>
+    </link>
+    <joint name="${led_prefix}_led" type="fixed">
+      <parent link="${parent_link}"/>
+      <child link="${namespace}/${led_prefix}_led_link"/>
+      <origin xyz="${xyz}" rpy="${rpy}"/>
+    </joint>
     <gazebo>
       <model name='${led_prefix}_led'>
-        <xacro:insert_block name='pose'/>
+        <pose>${xyz} ${rpy}</pose>
         <link name='led_body'>
           <inertial>
-            <pose>0 0 0 0 0 0</pose>
             <mass>0.00001</mass>
             <inertia>
@@ -18,19 +39,12 @@
             </inertia>
           </inertial>
-          <collision name='collision'>
-            <pose>0 0 0 0 0 0</pose>
+          <visual name='marker'>
+            <pose>0 0 0.008 0 0 0</pose>
             <geometry>
               <sphere>
-                <radius>0.025</radius>
+                <radius>0.015</radius>
               </sphere>
             </geometry>
-          </collision>
-          <visual name='marker'>
-            <pose>0 0 0 0 0 0</pose>
-            <geometry>
-              <sphere>
-                <radius>0.025</radius>
-              </sphere>
-            </geometry>
+            <transparency>1</transparency>
             <material>
               <ambient>1 1 1 1</ambient>
@@ -47,5 +61,5 @@
           </visual>
           <light name='marker' type='point'>
-            <pose>0 0 0 0 0 0</pose>
+            <pose>0 0 0 0 ${M_PI} 0</pose>
             <attenuation>
               <range>1</range>

File: x3_description/urdf/x3_equipments.urdf.xacro (robot description, xacro)
@@ -4,18 +4,29 @@
   <xacro:include filename="$(find subt_gazebo)/urdf/flashlight.urdf.xacro" />
   <xacro:include filename="$(find subt_gazebo)/urdf/led.urdf.xacro" />
-  <xacro:flashlight flashlight_prefix="right" parent_link="${namespace}/base_link">
-    <pose>-0.02 -0.07 0.05 0 ${M_PI*0.4} ${-M_PI*0.1}</pose>
+  <xacro:flashlight
+    flashlight_prefix="right"
+    parent_link="${namespace}/base_link"
+    xyz="-0.0 -0.08 0.05"
+    rpy="0.0 -0.06 -0.3">
     <params></params>
   </xacro:flashlight>
-  <xacro:flashlight flashlight_prefix="downward" parent_link="${namespace}/base_link">
-    <pose>0 0 0.1 0 ${M_PI/3*2} 0</pose>
+  <xacro:flashlight
+    flashlight_prefix="downward"
+    parent_link="${namespace}/base_link"
+    xyz="0.02 0 0.075"
+    rpy="0 0.2 0">
     <params></params>
   </xacro:flashlight>
-  <xacro:flashlight flashlight_prefix="left" parent_link="${namespace}/base_link">
-    <pose>-0.02 0.07 0.05 0 ${M_PI*0.4} ${M_PI*0.1}</pose>
+  <xacro:flashlight
+    flashlight_prefix="left"
+    parent_link="${namespace}/base_link"
+    xyz="0 0.08 0.05"
+    rpy="0 -0.06 0.3">
     <params></params>
   </xacro:flashlight>
-  <xacro:led led_prefix="right" parent_link="${namespace}/base_link">
-    <pose>-0.05 -0.05 0.05 0 0 0</pose>
+  <xacro:led led_prefix="right"
+    parent_link="${namespace}/base_link"
+    xyz="-0.08 -0.035 0.04"
+    rpy="${M_PI/3} 0 -0.1">
     <params>
       <duration>0.3</duration>
@@ -26,6 +37,8 @@
     </params>
   </xacro:led>
-  <xacro:led led_prefix="center" parent_link="${namespace}/base_link">
-    <pose>-0.1 0 0.05 0 0 0</pose>
+  <xacro:led led_prefix="center"
+    parent_link="${namespace}/base_link"
+    xyz="-0.07 0 0.065"
+    rpy="0 0 0">
     <params>
       <block>
@@ -46,6 +59,8 @@
     </params>
   </xacro:led>
-  <xacro:led led_prefix="left" parent_link="${namespace}/base_link">
-    <pose>-0.05 0.05 0.05 0 0 0</pose>
+  <xacro:led led_prefix="left"
+    parent_link="${namespace}/base_link"
+    xyz="-0.08 0.037 0.04"
+    rpy="${-M_PI/3} 0 0.2">
     <params>
       <duration>0.3</duration>

File: x4_description/urdf/x4_equipments.urdf.xacro (robot description, xacro)
@@ -4,18 +4,29 @@
   <xacro:include filename="$(find subt_gazebo)/urdf/flashlight.urdf.xacro" />
   <xacro:include filename="$(find subt_gazebo)/urdf/led.urdf.xacro" />
-  <xacro:flashlight flashlight_prefix="right" parent_link="${namespace}/base_link">
-    <pose>-0.02 -0.1 0.05 0 ${M_PI*0.4} ${-M_PI*0.1}</pose>
+  <xacro:flashlight
+    flashlight_prefix="right"
+    parent_link="${namespace}/base_link"
+    xyz="-0.01 -0.11 0.07"
+    rpy="0.0 -0.06 -0.3">
     <params></params>
   </xacro:flashlight>
-  <xacro:flashlight flashlight_prefix="downward" parent_link="${namespace}/base_link">
-    <pose>0.05 0 0.1 0 ${M_PI/3*2} 0</pose>
+  <xacro:flashlight
+    flashlight_prefix="downward"
+    parent_link="${namespace}/base_link"
+    xyz="0.02 0 0.09"
+    rpy="0 0.2 0">
     <params></params>
   </xacro:flashlight>
-  <xacro:flashlight flashlight_prefix="left" parent_link="${namespace}/base_link">
-    <pose>-0.02 0.1 0.05 0 ${M_PI*0.4} ${M_PI*0.1}</pose>
+  <xacro:flashlight
+    flashlight_prefix="left"
+    parent_link="${namespace}/base_link"
+    xyz="-0.01 0.11 0.07"
+    rpy="0 -0.06 0.3">
     <params></params>
   </xacro:flashlight>
-  <xacro:led led_prefix="right" parent_link="${namespace}/base_link">
-    <pose>-0.05 -0.08 0.05 0 0 0</pose>
+  <xacro:led led_prefix="right"
+    parent_link="${namespace}/base_link"
+    xyz="-0.09 -0.059 0.059"
+    rpy="${M_PI/4} 0 -0.2">
     <params>
       <duration>0.3</duration>
@@ -26,6 +37,8 @@
     </params>
   </xacro:led>
-  <xacro:led led_prefix="center" parent_link="${namespace}/base_link">
-    <pose>-0.13 0 0.05 0 0 0</pose>
+  <xacro:led led_prefix="center"
+    parent_link="${namespace}/base_link"
+    xyz="-0.10 0 0.077"
+    rpy="0 -0.1 0">
     <params>
       <block>
@@ -46,6 +59,8 @@
     </params>
   </xacro:led>
-  <xacro:led led_prefix="left" parent_link="${namespace}/base_link">
-    <pose>-0.05 0.08 0.05 0 0 0</pose>
+  <xacro:led led_prefix="left"
+    parent_link="${namespace}/base_link"
+    xyz="-0.09 0.059 0.059"
+    rpy="${-M_PI/4} 0 0.2">
     <params>
       <duration>0.3</duration>
