Commit message: update x3 and x4 inertias

File: subt_description/urdf/led.urdf.xacro (robot description, xacro)
@@ -31,10 +31,10 @@
             <mass>0.00001</mass>
             <inertia>
-              <ixx>1.0e-05</ixx>
+              <ixx>1.0e-08</ixx>
               <ixy>0</ixy>
               <ixz>0</ixz>
-              <iyy>1.0e-05</iyy>
+              <iyy>1.0e-08</iyy>
               <iyz>0</iyz>
-              <izz>1.0e-05</izz>
+              <izz>1.0e-08</izz>
             </inertia>
           </inertial>

File: x3_description/urdf/x3_with_sensors.xacro (robot description, xacro)
@@ -29,5 +29,5 @@
     image_scale="">
     <!-- [kg m^2] [kg m^2] [kg m^2] [kg m^2] [kg m^2] [kg m^2] -->
-    <inertia ixx="0.00001" ixy="0.0" ixz="0.0" iyy="0.00001" iyz="0.0" izz="0.00001" />
+    <inertia ixx="0.0000005" ixy="0.0" ixz="0.0" iyy="0.0000005" iyz="0.0" izz="0.0000005" />
     <origin xyz="0.0 0.0 0.0" rpy="0.0 0.0 0.0" />
   </xacro:odometry_plugin_macro>

File: x4_description/urdf/x4_with_sensors.xacro (robot description, xacro)
@@ -31,5 +31,5 @@
     image_scale="">
     <!-- [kg m^2] [kg m^2] [kg m^2] [kg m^2] [kg m^2] [kg m^2] -->
-    <inertia ixx="0.00001" ixy="0.0" ixz="0.0" iyy="0.00001" iyz="0.0" izz="0.00001" />
+    <inertia ixx="0.0000005" ixy="0.0" ixz="0.0" iyy="0.0000005" iyz="0.0" izz="0.0000005" />
     <origin xyz="0.0 0.0 0.0" rpy="0.0 0.0 0.0" />
   </xacro:odometry_plugin_macro>

Commit message: tweaks

File: subt_description/urdf/led.urdf.xacro (robot description, xacro)
@@ -29,12 +29,12 @@
         <link name='led_body'>
           <inertial>
-            <mass>0.00001</mass>
+            <mass>0.001</mass>
             <inertia>
-              <ixx>1.0e-08</ixx>
+              <ixx>1.0e-06</ixx>
               <ixy>0</ixy>
               <ixz>0</ixz>
-              <iyy>1.0e-08</iyy>
+              <iyy>1.0e-06</iyy>
               <iyz>0</iyz>
-              <izz>1.0e-08</izz>
+              <izz>1.0e-06</izz>
             </inertia>
           </inertial>

File: x3_description/urdf/x3_with_sensors.xacro (robot description, xacro)
@@ -13,5 +13,5 @@
     parent_frame_id="world"
     child_frame_id="${namespace}/odometry_sensor1"
-    mass_odometry_sensor="0.00001"
+    mass_odometry_sensor="0.001"
     measurement_divisor="1"
     measurement_delay="0"
@@ -29,5 +29,5 @@
     image_scale="">
     <!-- [kg m^2] [kg m^2] [kg m^2] [kg m^2] [kg m^2] [kg m^2] -->
-    <inertia ixx="0.0000005" ixy="0.0" ixz="0.0" iyy="0.0000005" iyz="0.0" izz="0.0000005" />
+    <inertia ixx="0.00001" ixy="0.0" ixz="0.0" iyy="0.00001" iyz="0.0" izz="0.00001" />
     <origin xyz="0.0 0.0 0.0" rpy="0.0 0.0 0.0" />
   </xacro:odometry_plugin_macro>

File: x4_description/urdf/x4_with_sensors.xacro (robot description, xacro)
@@ -15,5 +15,5 @@
     parent_frame_id="world"
     child_frame_id="${namespace}/odometry_sensor1"
-    mass_odometry_sensor="0.00001"
+    mass_odometry_sensor="0.001"
     measurement_divisor="1"
     measurement_delay="0"
@@ -31,5 +31,5 @@
     image_scale="">
     <!-- [kg m^2] [kg m^2] [kg m^2] [kg m^2] [kg m^2] [kg m^2] -->
-    <inertia ixx="0.0000005" ixy="0.0" ixz="0.0" iyy="0.0000005" iyz="0.0" izz="0.0000005" />
+    <inertia ixx="0.00001" ixy="0.0" ixz="0.0" iyy="0.00001" iyz="0.0" izz="0.00001" />
     <origin xyz="0.0 0.0 0.0" rpy="0.0 0.0 0.0" />
   </xacro:odometry_plugin_macro>
