Commit message: Rviz config

File: x3_description/urdf/x3_base.xacro (robot description, xacro)
@@ -6,20 +6,8 @@
   <!-- Instantiate a controller. -->
   <xacro:controller_plugin_macro namespace="${namespace}" imu_sub_topic="imu" />
-  <xacro:if value="$(arg enable_mavlink_interface)">
-    <!-- Instantiate mavlink telemetry interface. -->
-    <xacro:default_mavlink_interface namespace="${namespace}" imu_sub_topic="imu" rotor_count="4" />
-  </xacro:if>
-  <!-- Mount an ADIS16448 IMU. -->
-  <xacro:default_imu namespace="${namespace}" parent_link="${namespace}/base_link" />
+  <!--
   <xacro:if value="$(arg enable_ground_truth)">
     <xacro:ground_truth_imu_and_odometry namespace="${namespace}" parent_link="${namespace}/base_link" />
   </xacro:if>
-  <xacro:if value="$(arg enable_logging)">
-    <!-- Instantiate a logger -->
-    <xacro:bag_plugin_macro
-      namespace="${namespace}"
-      bag_file="$(arg log_file)"
-      rotor_velocity_slowdown_sim="${rotor_velocity_slowdown_sim}"
-      wait_to_record_bag="$(arg wait_to_record_bag)" />
-  </xacro:if>
+  -->
 </robot>

File: x3_description/urdf/x3_with_sensors.xacro (robot description, xacro)
@@ -32,11 +32,45 @@
     <origin xyz="0.0 0.0 0.0" rpy="0.0 0.0 0.0" />
   </xacro:odometry_plugin_macro>
+  <!--
+  <joint name="odometry_joint" type="fixed">
+    <origin xyz="0 0 0" rpy="0 0 0" />
+    <parent link="${namespace}/base_link" />
+    <child link="${namespace}/odometry_sensor1_link" />
+  </joint>
+-->
   <xacro:include filename="$(find x3_description)/urdf/x3_equipments.urdf.xacro" />
   <!-- Mount a magnetometer. -->
   <xacro:default_magnetometer namespace="${namespace}" parent_link="${namespace}/base_link" />
+  <!--
+  <joint name="magnetometer_joint" type="fixed">
+    <origin xyz="0 0 0" rpy="0 0 0" />
+    <parent link="${namespace}/base_link" />
+    <child link="${namespace}/magnetometer_link" />
+  </joint>
+  -->
   <!-- Mount a pressure sensor. -->
   <xacro:default_pressure_sensor namespace="${namespace}" parent_link="${namespace}/base_link" />
-  <!-- Front camera. -->
-  <xacro:camera_macro
+  <!--
+  <joint name="pressure_joint" type="fixed">
+    <origin xyz="0 0 0" rpy="0 0 0" />
+    <parent link="${namespace}/base_link" />
+    <child link="${namespace}/pressure_sensor_link" />
+  </joint>
+  -->
+  <!-- Mount an ADIS16448 IMU. -->
+  <xacro:default_imu namespace="${namespace}" parent_link="${namespace}/base_link" />
+  <!--
+  <joint name="imu_fixed_caguero_joint" type="fixed">
+    <origin xyz="0 0 0" rpy="0 0 0" />
+    <parent link="${namespace}/base_link" />
+    <child link="${namespace}/imu_link" />
+  </joint>
+  -->
+  <!-- Sensor configuration #1
+         * QVGA camera
+         * IMU
+  -->
+  <xacro:if value="$(optenv X3_SENSOR_CONFIG_1 0)">
+    <xacro:camera_macro
     namespace="${namespace}"
     parent_link="${namespace}/base_link"
@@ -44,7 +78,7 @@
     frame_rate="30"
     horizontal_fov="2"
-    image_width="752"
-    image_height="480"
-    image_format="L8"
+    image_width="320"
+    image_height="240"
+    image_format="R8G8B8"
     min_distance="0.02"
     max_distance="50"
@@ -55,21 +89,25 @@
     <origin xyz="0.1 0 0" rpy="0 0 0" />
   </xacro:camera_macro>
-  <!-- Lower camera. -->
-  <xacro:camera_macro
-    namespace="${namespace}"
-    parent_link="${namespace}/base_link"
-    camera_suffix="lower"
-    frame_rate="30"
-    horizontal_fov="2"
-    image_width="752"
-    image_height="480"
-    image_format="L8"
-    min_distance="0.02"
-    max_distance="50"
-    noise_mean="0.0"
-    noise_stddev="0.007"
-    enable_visual="false">
-    <box size="0.02 0.05 0.05" />
-    <origin xyz="0 0 -0.07" rpy="0 1.57 0" />
-  </xacro:camera_macro>
+  </xacro:if>
+  <!-- Sensor configuration #2
+         * HD camera
+         * IMU
+  -->
+  <xacro:if value="$(optenv X3_SENSOR_CONFIG_2 0)">
+    <hd_camera_and_mount />
+  </xacro:if>
+  <!-- Sensor configuration #3
+         * QVGA RGBD camera
+         * IMU
+  -->
+  <xacro:if value="$(optenv X3_SENSOR_CONFIG_3 0)">
+    <qvga_camera_and_mount />
+  </xacro:if>
+  <!-- Sensor configuration #4
+         * VGA RGBD camera
+         * IMU
+  -->
+  <xacro:if value="$(optenv X3_SENSOR_CONFIG_4 0)">
+    <hd_camera_and_mount />
+  </xacro:if>
 </robot>

Commit message: Cameras, RGBD and Rviz.

File: x3_description/urdf/x3_base.xacro (robot description, xacro)
@@ -6,8 +6,3 @@
   <!-- Instantiate a controller. -->
   <xacro:controller_plugin_macro namespace="${namespace}" imu_sub_topic="imu" />
-  <!--
-  <xacro:if value="$(arg enable_ground_truth)">
-    <xacro:ground_truth_imu_and_odometry namespace="${namespace}" parent_link="${namespace}/base_link" />
-  </xacro:if>
-  -->
 </robot>

File: x3_description/urdf/x3_with_sensors.xacro (robot description, xacro)
@@ -32,39 +32,12 @@
     <origin xyz="0.0 0.0 0.0" rpy="0.0 0.0 0.0" />
   </xacro:odometry_plugin_macro>
-  <!--
-  <joint name="odometry_joint" type="fixed">
-    <origin xyz="0 0 0" rpy="0 0 0" />
-    <parent link="${namespace}/base_link" />
-    <child link="${namespace}/odometry_sensor1_link" />
-  </joint>
--->
   <xacro:include filename="$(find x3_description)/urdf/x3_equipments.urdf.xacro" />
+  <xacro:include filename="$(find subt_sensors)/urdf/rgbd_camera.urdf.xacro" />
   <!-- Mount a magnetometer. -->
   <xacro:default_magnetometer namespace="${namespace}" parent_link="${namespace}/base_link" />
-  <!--
-  <joint name="magnetometer_joint" type="fixed">
-    <origin xyz="0 0 0" rpy="0 0 0" />
-    <parent link="${namespace}/base_link" />
-    <child link="${namespace}/magnetometer_link" />
-  </joint>
-  -->
   <!-- Mount a pressure sensor. -->
   <xacro:default_pressure_sensor namespace="${namespace}" parent_link="${namespace}/base_link" />
-  <!--
-  <joint name="pressure_joint" type="fixed">
-    <origin xyz="0 0 0" rpy="0 0 0" />
-    <parent link="${namespace}/base_link" />
-    <child link="${namespace}/pressure_sensor_link" />
-  </joint>
-  -->
   <!-- Mount an ADIS16448 IMU. -->
   <xacro:default_imu namespace="${namespace}" parent_link="${namespace}/base_link" />
-  <!--
-  <joint name="imu_fixed_caguero_joint" type="fixed">
-    <origin xyz="0 0 0" rpy="0 0 0" />
-    <parent link="${namespace}/base_link" />
-    <child link="${namespace}/imu_link" />
-  </joint>
-  -->
   <!-- Sensor configuration #1
          * QVGA camera
@@ -73,20 +46,20 @@
   <xacro:if value="$(optenv X3_SENSOR_CONFIG_1 0)">
     <xacro:camera_macro
-    namespace="${namespace}"
-    parent_link="${namespace}/base_link"
-    camera_suffix="front"
-    frame_rate="30"
-    horizontal_fov="2"
-    image_width="320"
-    image_height="240"
-    image_format="R8G8B8"
-    min_distance="0.02"
-    max_distance="50"
-    noise_mean="0.0"
-    noise_stddev="0.007"
-    enable_visual="false">
-    <box size="0.02 0.05 0.05" />
-    <origin xyz="0.1 0 0" rpy="0 0 0" />
-  </xacro:camera_macro>
+      namespace="${namespace}"
+      parent_link="${namespace}/base_link"
+      camera_suffix="front"
+      frame_rate="30"
+      horizontal_fov="2"
+      image_width="320"
+      image_height="240"
+      image_format="R8G8B8"
+      min_distance="0.02"
+      max_distance="50"
+      noise_mean="0.0"
+      noise_stddev="0.007"
+      enable_visual="true">
+      <box size="0.02 0.05 0.05" />
+      <origin xyz="0.1 0 0" rpy="0 0 0" />
+    </xacro:camera_macro>
   </xacro:if>
   <!-- Sensor configuration #2
@@ -95,5 +68,21 @@
   -->
   <xacro:if value="$(optenv X3_SENSOR_CONFIG_2 0)">
-    <hd_camera_and_mount />
+    <xacro:camera_macro
+      namespace="${namespace}"
+      parent_link="${namespace}/base_link"
+      camera_suffix="front"
+      frame_rate="30"
+      horizontal_fov="2"
+      image_width="1280"
+      image_height="960"
+      image_format="R8G8B8"
+      min_distance="0.02"
+      max_distance="50"
+      noise_mean="0.0"
+      noise_stddev="0.007"
+      enable_visual="true">
+      <box size="0.02 0.05 0.05" />
+      <origin xyz="0.1 0 0" rpy="0 0 0" />
+    </xacro:camera_macro>
   </xacro:if>
   <!-- Sensor configuration #3
@@ -102,5 +91,14 @@
   -->
   <xacro:if value="$(optenv X3_SENSOR_CONFIG_3 0)">
-    <qvga_camera_and_mount />
+    <xacro:rgbd_camera
+       name="${namespace}/rgbd_camera"
+       width="320"
+       height="240"
+    />
+    <joint name="rgbd_camera_mount_joint" type="fixed">
+      <origin xyz="0.05 0 -0.05" rpy="0 0.2618 0" />
+      <parent link="${namespace}/base_link" />
+      <child link="${namespace}/rgbd_camera_link" />
+    </joint>
   </xacro:if>
   <!-- Sensor configuration #4
@@ -109,5 +107,14 @@
   -->
   <xacro:if value="$(optenv X3_SENSOR_CONFIG_4 0)">
-    <hd_camera_and_mount />
+    <xacro:rgbd_camera
+       name="${namespace}/rgbd_camera"
+       width="640"
+       height="480"
+    />
+    <joint name="rgbd_camera_mount_joint" type="fixed">
+      <origin xyz="0.05 0 -0.05" rpy="0 0.2618 0" />
+      <parent link="${namespace}/base_link" />
+      <child link="${namespace}/rgbd_camera_link" />
+    </joint>
   </xacro:if>
 </robot>

Commit message: check sdf for either an all_joints tag or joint tags with named joints, skipping fixed joints. test with x3 and x4 models

File: x3_description/urdf/x3_base.xacro (robot description, xacro)
@@ -7,4 +7,7 @@
   <xacro:controller_plugin_macro namespace="${namespace}" imu_sub_topic="imu" />
   <gazebo>
+    <plugin name="${namespace}_joint_motion_timer" filename="libJointMotionTimerPlugin.so">
+      <all_joints/>
+    </plugin>
     <plugin name="${namespace}_joint_state_publisher" filename="libgazebo_ros_joint_state_publisher.so">
       <robotNamespace>${namespace}/fixed</robotNamespace>

File: x4_description/urdf/x4_base.xacro (robot description, xacro)
@@ -23,4 +23,12 @@
   <xacro:controller_plugin_macro namespace="${namespace}" imu_sub_topic="imu" />
   <gazebo>
+    <plugin name="${namespace}_joint_motion_timer" filename="libJointMotionTimerPlugin.so">
+      <joint>X4/rotor_0_joint</joint>
+      <joint>X4/rotor_1_joint</joint>
+      <joint>X4/rotor_2_joint</joint>
+      <joint>X4/rotor_3_joint</joint>
+      <joint>X4/rotor_4_joint</joint>
+      <joint>X4/rotor_5_joint</joint>
+    </plugin>
     <plugin name="${namespace}_joint_state_publisher" filename="libgazebo_ros_joint_state_publisher.so">
       <robotNamespace>${namespace}/fixed</robotNamespace>
