Commit message: Rename husky_migration -> husky_migration_sensor_config_1

File: submitted_models/husky_migration_sensor_config_1/urdf/robot_from_sdf.xacro (robot description, xacro)
@@ -24,5 +24,5 @@
       <origin xyz='0.0812 0 0.245' rpy='0 -0 0'/>
       <geometry>
-        <mesh filename='package://husky_migration/meshes/top_plate.dae' scale='1 1 1'/>
+        <mesh filename='package://husky_migration_sensor_config_1/meshes/top_plate.dae' scale='1 1 1'/>
       </geometry>
     </collision>
@@ -48,5 +48,5 @@
       <origin xyz='0 0 0' rpy='0 -0 0'/>
       <geometry>
-        <mesh filename='package://husky_migration/meshes/base_link.dae' scale='1 1 1'/>
+        <mesh filename='package://husky_migration_sensor_config_1/meshes/base_link.dae' scale='1 1 1'/>
       </geometry>
     </visual>
@@ -54,5 +54,5 @@
       <origin xyz='0.48 0 0.091' rpy='0 -0 0'/>
       <geometry>
-        <mesh filename='package://husky_migration/meshes/bumper.dae' scale='1 1 1'/>
+        <mesh filename='package://husky_migration_sensor_config_1/meshes/bumper.dae' scale='1 1 1'/>
       </geometry>
     </visual>
@@ -60,5 +60,5 @@
       <origin xyz='-0.48 0 0.091' rpy='0 -0 3.14159'/>
       <geometry>
-        <mesh filename='package://husky_migration/meshes/bumper.dae' scale='1 1 1'/>
+        <mesh filename='package://husky_migration_sensor_config_1/meshes/bumper.dae' scale='1 1 1'/>
       </geometry>
     </visual>
@@ -66,5 +66,5 @@
       <origin xyz='0 0 0' rpy='0 -0 0'/>
       <geometry>
-        <mesh filename='package://husky_migration/meshes/top_chassis.dae' scale='1 1 1'/>
+        <mesh filename='package://husky_migration_sensor_config_1/meshes/top_chassis.dae' scale='1 1 1'/>
       </geometry>
     </visual>
@@ -72,5 +72,5 @@
       <origin xyz='0.0812 0 0.245' rpy='0 -0 0'/>
       <geometry>
-        <mesh filename='package://husky_migration/meshes/top_plate.dae' scale='1 1 1'/>
+        <mesh filename='package://husky_migration_sensor_config_1/meshes/top_plate.dae' scale='1 1 1'/>
       </geometry>
     </visual>
@@ -78,5 +78,5 @@
       <origin xyz='0.3018 0 0.25135' rpy='0 0 -1.5708'/>
       <geometry>
-        <mesh filename='package://husky_migration/meshes/lms1xx_mount.dae' scale='1 1 1'/>
+        <mesh filename='package://husky_migration_sensor_config_1/meshes/lms1xx_mount.dae' scale='1 1 1'/>
       </geometry>
     </visual>
@@ -84,5 +84,5 @@
       <origin xyz='0.337 0 0.30795' rpy='3.14159 -0 0'/>
       <geometry>
-        <mesh filename='package://husky_migration/meshes/sick-lms1xx.dae' scale='1 1 1'/>
+        <mesh filename='package://husky_migration_sensor_config_1/meshes/sick-lms1xx.dae' scale='1 1 1'/>
       </geometry>
     </visual>
@@ -90,5 +90,5 @@
       <origin xyz='0.272 0 0.245' rpy='0 -0 0'/>
       <geometry>
-        <mesh filename='package://husky_migration/meshes/user_rail.dae' scale='1 1 1'/>
+        <mesh filename='package://husky_migration_sensor_config_1/meshes/user_rail.dae' scale='1 1 1'/>
       </geometry>
     </visual>
@@ -117,5 +117,5 @@
       <origin xyz='0 0 0' rpy='0 -0 0'/>
       <geometry>
-        <mesh filename='package://husky_migration/meshes/wheel.dae' scale='1 1 1'/>
+        <mesh filename='package://husky_migration_sensor_config_1/meshes/wheel.dae' scale='1 1 1'/>
       </geometry>
     </visual>
@@ -136,5 +136,5 @@
       <origin xyz='0 0 0' rpy='0 -0 0'/>
       <geometry>
-        <mesh filename='package://husky_migration/meshes/wheel.dae' scale='1 1 1'/>
+        <mesh filename='package://husky_migration_sensor_config_1/meshes/wheel.dae' scale='1 1 1'/>
       </geometry>
     </visual>
@@ -155,5 +155,5 @@
       <origin xyz='0 0 0' rpy='0 -0 0'/>
       <geometry>
-        <mesh filename='package://husky_migration/meshes/wheel.dae' scale='1 1 1'/>
+        <mesh filename='package://husky_migration_sensor_config_1/meshes/wheel.dae' scale='1 1 1'/>
       </geometry>
     </visual>
@@ -174,5 +174,5 @@
       <origin xyz='0 0 0' rpy='0 -0 0'/>
       <geometry>
-        <mesh filename='package://husky_migration/meshes/wheel.dae' scale='1 1 1'/>
+        <mesh filename='package://husky_migration_sensor_config_1/meshes/wheel.dae' scale='1 1 1'/>
       </geometry>
     </visual>
