Commit message: Solution of not working robotmodels in rviz

File: submitted_models/sophisticated_engineering_x2_sensor_config_8/urdf/x2_from_sdf.xacro (robot description, xacro)
@@ -1,6 +1,6 @@
 <?xml version='1.0' encoding='utf-8'?>
-<robot name='X2' xmlns:xacro='http://ros.org/wiki/xacro'>
-  <xacro:arg name='name' default='X2'/>
-  <xacro:property name='robot_namespace' value='$(arg name)'/>
+<robot name="X2" xmlns:xacro="http://ros.org/wiki/xacro">
+  <xacro:arg name="name" default="X2"/>
+  <xacro:property name="robot_namespace" value="$(arg name)"/>
   <link name='${robot_namespace}/base_link'>
     <inertial>
@@ -18,5 +18,5 @@
       <origin xyz='0 0 -0.0655' rpy='1.5708 0 -1.5708'/>
       <geometry>
-        <mesh filename='package://meshes/x2_chassis.dae' scale='1 1 1'/>
+        <mesh filename='package://x2_description/meshes/x2_chassis.dae' scale='1 1 1'/>
       </geometry>
     </visual>
@@ -30,5 +30,5 @@
       <origin xyz='0.22 0.05 0.0845' rpy='0 0 -3.14159'/>
       <geometry>
-        <mesh filename='package://meshes/headlight.dae' scale='1 1 1'/>
+        <mesh filename='package://x2_description/meshes/headlight.dae' scale='1 1 1'/>
       </geometry>
     </visual>
@@ -36,5 +36,5 @@
       <origin xyz='0.22 0.145 0.0845' rpy='0 0 -3.14159'/>
       <geometry>
-        <mesh filename='package://meshes/headlight.dae' scale='1 1 1'/>
+        <mesh filename='package://x2_description/meshes/headlight.dae' scale='1 1 1'/>
       </geometry>
     </visual>
@@ -42,5 +42,5 @@
       <origin xyz='0.22 -0.05 0.0845' rpy='0 0 -3.14159'/>
       <geometry>
-        <mesh filename='package://meshes/headlight.dae' scale='1 1 1'/>
+        <mesh filename='package://x2_description/meshes/headlight.dae' scale='1 1 1'/>
       </geometry>
     </visual>
@@ -48,39 +48,13 @@
       <origin xyz='0.22 -0.145 0.0845' rpy='0 0 -3.14159'/>
       <geometry>
-        <mesh filename='package://meshes/headlight.dae' scale='1 1 1'/>
-      </geometry>
-    </visual>
-    <visual name='camera_left_visual'>
-      <origin xyz='0.23 0.1 0.19' rpy='0 -0 0'/>
-      <geometry>
-        <box size='0.02 0.02 0.02'/>
-      </geometry>
-    </visual>
-    <visual name='camera_right_visual'>
-      <origin xyz='0.23 -0.1 0.19' rpy='0 -0 0'/>
-      <geometry>
-        <box size='0.02 0.02 0.02'/>
+        <mesh filename='package://x2_description/meshes/headlight.dae' scale='1 1 1'/>
       </geometry>
     </visual>
   </link>
-  <sensor name='imu_sensor' update_rate='50'>
-    <parent link='base_link'/>
+  <sensor name='imu_sensor' update_rate='1000'>
+    <parent link='${robot_namespace}/base_link'/>
     <origin xyz='0 0 0' rpy='0 -0 0'/>
   </sensor>
-  <sensor name='camera_front_left' update_rate='20'>
-    <parent link='base_link'/>
-    <origin xyz='0.23 0.1 0.19' rpy='0 -0 0'/>
-    <camera>
-      <image width='1280' height='960' format='R8G8B8' hfov='2' near='0.01' far='300' />
-    </camera>
-  </sensor>
-  <sensor name='camera_front_right' update_rate='20'>
-    <parent link='base_link'/>
-    <origin xyz='0.23 -0.1 0.19' rpy='0 -0 0'/>
-    <camera>
-      <image width='1280' height='960' format='R8G8B8' hfov='2' near='0.01' far='300' />
-    </camera>
-  </sensor>
-  <link name='front_left_wheel'>
+  <link name='${robot_namespace}/front_left_wheel'>
     <inertial>
       <origin xyz='0 0 0' rpy='0 -0 0'/>
@@ -97,9 +71,9 @@
       <origin xyz='0 0 0' rpy='1.5708 -0 0'/>
       <geometry>
-        <mesh filename='package://meshes/x2_wheel_left.dae' scale='1 1 1'/>
+        <mesh filename='package://x2_description/meshes/x2_wheel_left.dae' scale='1 1 1'/>
       </geometry>
     </visual>
   </link>
-  <link name='front_right_wheel'>
+  <link name='${robot_namespace}/front_right_wheel'>
     <inertial>
       <origin xyz='0 0 0' rpy='0 -0 0'/>
@@ -116,9 +90,9 @@
       <origin xyz='0 0 0' rpy='1.5708 -0 0'/>
       <geometry>
-        <mesh filename='package://meshes/x2_wheel_right.dae' scale='1 1 1'/>
+        <mesh filename='package://x2_description/meshes/x2_wheel_right.dae' scale='1 1 1'/>
       </geometry>
     </visual>
   </link>
-  <link name='rear_left_wheel'>
+  <link name='${robot_namespace}/rear_left_wheel'>
     <inertial>
       <origin xyz='0 0 0' rpy='0 -0 0'/>
@@ -135,9 +109,9 @@
       <origin xyz='0 0 0' rpy='1.5708 -0 0'/>
       <geometry>
-        <mesh filename='package://meshes/x2_wheel_left.dae' scale='1 1 1'/>
+        <mesh filename='package://x2_description/meshes/x2_wheel_left.dae' scale='1 1 1'/>
       </geometry>
     </visual>
   </link>
-  <link name='rear_right_wheel'>
+  <link name='${robot_namespace}/rear_right_wheel'>
     <inertial>
       <origin xyz='0 0 0' rpy='0 -0 0'/>
@@ -154,5 +128,5 @@
       <origin xyz='0 0 0' rpy='1.5708 -0 0'/>
       <geometry>
-        <mesh filename='package://meshes/x2_wheel_right.dae' scale='1 1 1'/>
+        <mesh filename='package://x2_description/meshes/x2_wheel_right.dae' scale='1 1 1'/>
       </geometry>
     </visual>
@@ -160,6 +134,6 @@
   <joint name='front_left_wheel_joint' type='revolute'>
     <origin xyz='0.131 0.187795 0.0345' rpy='0 -0 0'/>
-    <parent link='base_link'/>
-    <child link='front_left_wheel'/>
+    <parent link='${robot_namespace}/base_link'/>
+    <child link='${robot_namespace}/front_left_wheel'/>
     <axis xyz='0 1 0'/>
     <limit lower='-1e+16' upper='1e+16' effort='-1' velocity='-1'/>
@@ -167,6 +141,6 @@
   <joint name='rear_left_wheel_joint' type='revolute'>
     <origin xyz='-0.131 0.187795 0.0345' rpy='0 -0 0'/>
-    <parent link='base_link'/>
-    <child link='rear_left_wheel'/>
+    <parent link='${robot_namespace}/base_link'/>
+    <child link='${robot_namespace}/rear_left_wheel'/>
     <axis xyz='0 1 0'/>
     <limit lower='-1.79769e+308' upper='1.79769e+308' effort='-1' velocity='-1'/>
@@ -174,6 +148,6 @@
   <joint name='rear_right_wheel_joint' type='revolute'>
     <origin xyz='-0.131 -0.187795 0.0345' rpy='0 -0 0'/>
-    <parent link='base_link'/>
-    <child link='rear_right_wheel'/>
+    <parent link='${robot_namespace}/base_link'/>
+    <child link='${robot_namespace}/rear_right_wheel'/>
     <axis xyz='0 1 0'/>
     <limit lower='-1.79769e+308' upper='1.79769e+308' effort='-1' velocity='-1'/>
@@ -181,6 +155,6 @@
   <joint name='front_right_wheel_joint' type='revolute'>
     <origin xyz='0.131 -0.187795 0.0345' rpy='0 -0 0'/>
-    <parent link='base_link'/>
-    <child link='front_right_wheel'/>
+    <parent link='${robot_namespace}/base_link'/>
+    <child link='${robot_namespace}/front_right_wheel'/>
     <axis xyz='0 1 0'/>
     <limit lower='-1.79769e+308' upper='1.79769e+308' effort='-1' velocity='-1'/>
