Commit message: fixed joints. missing {name}

File: submitted_models/ssci_x2_sensor_config_8/urdf/model.xacro (robot description, xacro)
@@ -64,9 +64,9 @@
   </link>
   <sensor name='imu_sensor' update_rate='50'>
-    <parent link='base_link'/>
+    <parent link='{name}/base_link'/>
     <origin xyz='0 0 0' rpy='0 -0 0'/>
   </sensor>
   <sensor name='camera_front' update_rate='20'>
-    <parent link='base_link'/>
+    <parent link='{name}/base_link'/>
     <origin xyz='0.23 0 0.19' rpy='0 -0 0'/>
     <camera>
@@ -75,9 +75,9 @@
   </sensor>
   <sensor name='top_laser' update_rate='50'>
-    <parent link='base_link'/>
+    <parent link='{name}/base_link'/>
     <origin xyz='0 0 0.1' rpy='0 1.57 0'/>
   </sensor>
   <sensor name='front_laser' update_rate='15'>
-    <parent link='base_link'/>
+    <parent link='{name}/base_link'/>
     <origin xyz='0.08 0 0.394' rpy='0 -0 0'/>
   </sensor>
@@ -160,6 +160,6 @@
   <joint name='front_left_wheel_joint' type='revolute'>
     <origin xyz='0.131 0.187795 0.0345' rpy='0 -0 0'/>
-    <parent link='base_link'/>
-    <child link='front_left_wheel'/>
+    <parent link='{name}/base_link'/>
+    <child link='{name}/front_left_wheel'/>
     <axis xyz='0 1 0'/>
     <limit lower='-1e+16' upper='1e+16' effort='-1' velocity='-1'/>
@@ -167,6 +167,6 @@
   <joint name='rear_left_wheel_joint' type='revolute'>
     <origin xyz='-0.131 0.187795 0.0345' rpy='0 -0 0'/>
-    <parent link='base_link'/>
-    <child link='rear_left_wheel'/>
+    <parent link='{name}/base_link'/>
+    <child link='{name}/rear_left_wheel'/>
     <axis xyz='0 1 0'/>
     <limit lower='-1.79769e+308' upper='1.79769e+308' effort='-1' velocity='-1'/>
@@ -174,6 +174,6 @@
   <joint name='rear_right_wheel_joint' type='revolute'>
     <origin xyz='-0.131 -0.187795 0.0345' rpy='0 -0 0'/>
-    <parent link='base_link'/>
-    <child link='rear_right_wheel'/>
+    <parent link='{name}/base_link'/>
+    <child link='{name}/rear_right_wheel'/>
     <axis xyz='0 1 0'/>
     <limit lower='-1.79769e+308' upper='1.79769e+308' effort='-1' velocity='-1'/>
@@ -181,6 +181,6 @@
   <joint name='front_right_wheel_joint' type='revolute'>
     <origin xyz='0.131 -0.187795 0.0345' rpy='0 -0 0'/>
-    <parent link='base_link'/>
-    <child link='front_right_wheel'/>
+    <parent link='{name}/base_link'/>
+    <child link='{name}/front_right_wheel'/>
     <axis xyz='0 1 0'/>
     <limit lower='-1.79769e+308' upper='1.79769e+308' effort='-1' velocity='-1'/>

Commit message: Fixed the xacro file

File: submitted_models/ssci_x2_sensor_config_8/urdf/model.xacro (robot description, xacro)
@@ -1,6 +1,7 @@
 <?xml version='1.0' encoding='utf-8'?>
-<robot name='X2'>
-  <xacro:arg name="name" default="X3"/>
-  <link name='{name}/base_link'>
+<robot name="X2" xmlns:xacro="http://ros.org/wiki/xacro">
+  <xacro:arg name="name" default="X2"/>
+  <xacro:property name="robot_namespace" value="$(arg name)"/>
+  <link name='${robot_namespace}/base_link'>
     <inertial>
       <origin xyz='0.011999 0.002 0.066996' rpy='0 -0 0'/>
@@ -63,10 +64,10 @@
     </visual>
   </link>
-  <sensor name='imu_sensor' update_rate='50'>
-    <parent link='base_link'/>
+  <sensor name='imu_sensor' update_rate='1000'>
+    <parent link='${robot_namespace}/base_link'/>
     <origin xyz='0 0 0' rpy='0 -0 0'/>
   </sensor>
   <sensor name='camera_front' update_rate='20'>
-    <parent link='base_link'/>
+    <parent link='${robot_namespace}/base_link'/>
     <origin xyz='0.23 0 0.19' rpy='0 -0 0'/>
     <camera>
@@ -75,12 +76,12 @@
   </sensor>
   <sensor name='top_laser' update_rate='50'>
-    <parent link='base_link'/>
+    <parent link='${robot_namespace}/base_link'/>
     <origin xyz='0 0 0.1' rpy='0 1.57 0'/>
   </sensor>
   <sensor name='front_laser' update_rate='15'>
-    <parent link='base_link'/>
+    <parent link='${robot_namespace}/base_link'/>
     <origin xyz='0.08 0 0.394' rpy='0 -0 0'/>
   </sensor>
-  <link name='{name}/front_left_wheel'>
+  <link name='${robot_namespace}/front_left_wheel'>
     <inertial>
       <origin xyz='0 0 0' rpy='0 -0 0'/>
@@ -101,5 +102,5 @@
     </visual>
   </link>
-  <link name='{name}/front_right_wheel'>
+  <link name='${robot_namespace}/front_right_wheel'>
     <inertial>
       <origin xyz='0 0 0' rpy='0 -0 0'/>
@@ -120,5 +121,5 @@
     </visual>
   </link>
-  <link name='{name}/rear_left_wheel'>
+  <link name='${robot_namespace}/rear_left_wheel'>
     <inertial>
       <origin xyz='0 0 0' rpy='0 -0 0'/>
@@ -139,5 +140,5 @@
     </visual>
   </link>
-  <link name='{name}/rear_right_wheel'>
+  <link name='${robot_namespace}/rear_right_wheel'>
     <inertial>
       <origin xyz='0 0 0' rpy='0 -0 0'/>
@@ -160,6 +161,6 @@
   <joint name='front_left_wheel_joint' type='revolute'>
     <origin xyz='0.131 0.187795 0.0345' rpy='0 -0 0'/>
-    <parent link='base_link'/>
-    <child link='front_left_wheel'/>
+    <parent link='${robot_namespace}/base_link'/>
+    <child link='${robot_namespace}/front_left_wheel'/>
     <axis xyz='0 1 0'/>
     <limit lower='-1e+16' upper='1e+16' effort='-1' velocity='-1'/>
@@ -167,6 +168,6 @@
   <joint name='rear_left_wheel_joint' type='revolute'>
     <origin xyz='-0.131 0.187795 0.0345' rpy='0 -0 0'/>
-    <parent link='base_link'/>
-    <child link='rear_left_wheel'/>
+    <parent link='${robot_namespace}/base_link'/>
+    <child link='${robot_namespace}/rear_left_wheel'/>
     <axis xyz='0 1 0'/>
     <limit lower='-1.79769e+308' upper='1.79769e+308' effort='-1' velocity='-1'/>
@@ -174,6 +175,6 @@
   <joint name='rear_right_wheel_joint' type='revolute'>
     <origin xyz='-0.131 -0.187795 0.0345' rpy='0 -0 0'/>
-    <parent link='base_link'/>
-    <child link='rear_right_wheel'/>
+    <parent link='${robot_namespace}/base_link'/>
+    <child link='${robot_namespace}/rear_right_wheel'/>
     <axis xyz='0 1 0'/>
     <limit lower='-1.79769e+308' upper='1.79769e+308' effort='-1' velocity='-1'/>
@@ -181,6 +182,6 @@
   <joint name='front_right_wheel_joint' type='revolute'>
     <origin xyz='0.131 -0.187795 0.0345' rpy='0 -0 0'/>
-    <parent link='base_link'/>
-    <child link='front_right_wheel'/>
+    <parent link='${robot_namespace}/base_link'/>
+    <child link='${robot_namespace}/front_right_wheel'/>
     <axis xyz='0 1 0'/>
     <limit lower='-1.79769e+308' upper='1.79769e+308' effort='-1' velocity='-1'/>

Commit message: Add package paths to meshes in xacro file

File: submitted_models/ssci_x2_sensor_config_8/urdf/model.xacro (robot description, xacro)
@@ -18,5 +18,5 @@
       <origin xyz='0 0 -0.0655' rpy='1.5708 0 -1.5708'/>
       <geometry>
-        <mesh filename='meshes/x2_chassis.dae' scale='1 1 1'/>
+        <mesh filename='package://ssci_x2_sensor_config_8/meshes/x2_chassis.dae' scale='1 1 1'/>
       </geometry>
     </visual>
@@ -30,5 +30,5 @@
       <origin xyz='0.22 0.05 0.0845' rpy='0 0 -3.14159'/>
       <geometry>
-        <mesh filename='meshes/headlight.dae' scale='1 1 1'/>
+        <mesh filename='package://ssci_x2_sensor_config_8/meshes/headlight.dae' scale='1 1 1'/>
       </geometry>
     </visual>
@@ -36,5 +36,5 @@
       <origin xyz='0.22 0.145 0.0845' rpy='0 0 -3.14159'/>
       <geometry>
-        <mesh filename='meshes/headlight.dae' scale='1 1 1'/>
+        <mesh filename='package://ssci_x2_sensor_config_8/meshes/headlight.dae' scale='1 1 1'/>
       </geometry>
     </visual>
@@ -42,5 +42,5 @@
       <origin xyz='0.22 -0.05 0.0845' rpy='0 0 -3.14159'/>
       <geometry>
-        <mesh filename='meshes/headlight.dae' scale='1 1 1'/>
+        <mesh filename='package://ssci_x2_sensor_config_8/meshes/headlight.dae' scale='1 1 1'/>
       </geometry>
     </visual>
@@ -48,5 +48,5 @@
       <origin xyz='0.22 -0.145 0.0845' rpy='0 0 -3.14159'/>
       <geometry>
-        <mesh filename='meshes/headlight.dae' scale='1 1 1'/>
+        <mesh filename='package://ssci_x2_sensor_config_8/meshes/headlight.dae' scale='1 1 1'/>
       </geometry>
     </visual>
@@ -98,5 +98,5 @@
       <origin xyz='0 0 0' rpy='1.5708 -0 0'/>
       <geometry>
-        <mesh filename='meshes/x2_wheel_left.dae' scale='1 1 1'/>
+        <mesh filename='package://ssci_x2_sensor_config_8/meshes/x2_wheel_left.dae' scale='1 1 1'/>
       </geometry>
     </visual>
@@ -117,5 +117,5 @@
       <origin xyz='0 0 0' rpy='1.5708 -0 0'/>
       <geometry>
-        <mesh filename='meshes/x2_wheel_right.dae' scale='1 1 1'/>
+        <mesh filename='package://ssci_x2_sensor_config_8/meshes/x2_wheel_right.dae' scale='1 1 1'/>
       </geometry>
     </visual>
@@ -136,5 +136,5 @@
       <origin xyz='0 0 0' rpy='1.5708 -0 0'/>
       <geometry>
-        <mesh filename='meshes/x2_wheel_left.dae' scale='1 1 1'/>
+        <mesh filename='package://ssci_x2_sensor_config_8/meshes/x2_wheel_left.dae' scale='1 1 1'/>
       </geometry>
     </visual>
@@ -155,5 +155,5 @@
       <origin xyz='0 0 0' rpy='1.5708 -0 0'/>
       <geometry>
-        <mesh filename='meshes/x2_wheel_right.dae' scale='1 1 1'/>
+        <mesh filename='package://ssci_x2_sensor_config_8/meshes/x2_wheel_right.dae' scale='1 1 1'/>
       </geometry>
     </visual>
