Commit message: Fixed reference of name on xacro file

File: submitted_models/ssci_x4_sensor_config_8/urdf/model.xacro (robot description, xacro)
@@ -2,5 +2,6 @@
 <robot name="X4" xmlns:xacro="http://ros.org/wiki/xacro">
   <xacro:arg name="name" default="X4"/>
-  <link name='{name}/base_link'>
+  <xacro:property name="name" value="$(arg name)"/>
+  <link name='${name}/base_link'>
     <inertial>
       <origin xyz='0 0 0' rpy='0 -0 0'/>
@@ -88,17 +89,17 @@
   </link>
   <sensor name='imu_sensor' update_rate='250'>
-    <parent link='{name}/base_link'/>
+    <parent link='${name}/base_link'/>
     <origin xyz='0 0 0' rpy='0 -0 0'/>
   </sensor>
   <sensor name='air_pressure' update_rate='20'>
-    <parent link='{name}/base_link'/>
+    <parent link='${name}/base_link'/>
     <origin xyz='0 0 0' rpy='0 -0 0'/>
   </sensor>
   <sensor name='magnetometer' update_rate='20'>
-    <parent link='{name}/base_link'/>
+    <parent link='${name}/base_link'/>
     <origin xyz='0 0 0' rpy='0 -0 0'/>
   </sensor>
   <sensor name='camera_front' update_rate='20'>
-    <parent link='{name}/base_link'/>
+    <parent link='${name}/base_link'/>
     <origin xyz='0.1 0 -0.08' rpy='0 -0 0'/>
     <camera>
@@ -107,8 +108,8 @@
   </sensor>
   <sensor name='front_laser' update_rate='15'>
-    <parent link='{name}/base_link'/>
+    <parent link='${name}/base_link'/>
     <origin xyz='0.08 0 0.394' rpy='0 -0 0'/>
   </sensor>
-  <link name='{name}/rotor_0'>
+  <link name='${name}/rotor_0'>
     <inertial>
       <origin xyz='0 0 0' rpy='0 -0 0'/>
@@ -129,5 +130,5 @@
     </visual>
   </link>
-  <link name='{name}/rotor_1'>
+  <link name='${name}/rotor_1'>
     <inertial>
       <origin xyz='0 0 0' rpy='0 -0 0'/>
@@ -148,5 +149,5 @@
     </visual>
   </link>
-  <link name='{name}/rotor_2'>
+  <link name='${name}/rotor_2'>
     <inertial>
       <origin xyz='0 0 0' rpy='0 -0 0'/>
@@ -167,5 +168,5 @@
     </visual>
   </link>
-  <link name='{name}/rotor_3'>
+  <link name='${name}/rotor_3'>
     <inertial>
       <origin xyz='0 0 0' rpy='0 -0 0'/>
@@ -186,5 +187,5 @@
     </visual>
   </link>
-  <link name='{name}/rotor_4'>
+  <link name='${name}/rotor_4'>
     <inertial>
       <origin xyz='0 0 0' rpy='-0 -0 -0'/>
@@ -205,5 +206,5 @@
     </visual>
   </link>
-  <link name='{name}/rotor_5'>
+  <link name='${name}/rotor_5'>
     <inertial>
       <origin xyz='0 0 0' rpy='0 -0 0'/>
@@ -226,6 +227,6 @@
   <joint name='rotor_0_joint' type='revolute'>
     <origin xyz='0.247 0.1506 0.028' rpy='0.087267 0 0.523599'/>
-    <parent link='{name}/base_link'/>
-    <child link='{name}/rotor_0'/>
+    <parent link='${name}/base_link'/>
+    <child link='${name}/rotor_0'/>
     <dynamics damping='0' friction='0' />
     <axis xyz='0.118748 -0.118521 0.985826'/>
@@ -234,6 +235,6 @@
   <joint name='rotor_1_joint' type='revolute'>
     <origin xyz='-0.00067 0.28929 0.028' rpy='0 -0.087267 0'/>
-    <parent link='{name}/base_link'/>
-    <child link='{name}/rotor_1'/>
+    <parent link='${name}/base_link'/>
+    <child link='${name}/rotor_1'/>
     <dynamics damping='0' friction='0' />
     <axis xyz='-0.173649 0 0.984808'/>
@@ -242,6 +243,6 @@
   <joint name='rotor_2_joint' type='revolute'>
     <origin xyz='-0.2501 0.1454 0.028' rpy='0.087267 -0 2.61799'/>
-    <parent link='{name}/base_link'/>
-    <child link='{name}/rotor_2'/>
+    <parent link='${name}/base_link'/>
+    <child link='${name}/rotor_2'/>
     <dynamics damping='0' friction='0' />
     <axis xyz='-0.031923 0.031863 0.998983'/>
@@ -250,6 +251,6 @@
   <joint name='rotor_3_joint' type='revolute'>
     <origin xyz='-0.2501 -0.1454 0.028' rpy='-0.087267 -0 -2.61799'/>
-    <parent link='{name}/base_link'/>
-    <child link='{name}/rotor_3'/>
+    <parent link='${name}/base_link'/>
+    <child link='${name}/rotor_3'/>
     <dynamics damping='0' friction='0' />
     <axis xyz='-0.031923 -0.031863 0.998983'/>
@@ -258,6 +259,6 @@
   <joint name='rotor_4_joint' type='revolute'>
     <origin xyz='-0.00067 -0.28929 0.028' rpy='-0 0.087267 -3.14159'/>
-    <parent link='{name}/base_link'/>
-    <child link='{name}/rotor_4'/>
+    <parent link='${name}/base_link'/>
+    <child link='${name}/rotor_4'/>
     <dynamics damping='0' friction='0' />
     <axis xyz='-0 -0 1'/>
@@ -266,6 +267,6 @@
   <joint name='rotor_5_joint' type='revolute'>
     <origin xyz='0.247 -0.1506 0.028' rpy='-0.087267 0 -0.523599'/>
-    <parent link='{name}/base_link'/>
-    <child link='{name}/rotor_5'/>
+    <parent link='${name}/base_link'/>
+    <child link='${name}/rotor_5'/>
     <dynamics damping='0' friction='0' />
     <axis xyz='0.118748 0.118521 0.985826'/>

Commit message: Fixed meshes path

File: submitted_models/ssci_x4_sensor_config_8/urdf/model.xacro (robot description, xacro)
@@ -18,5 +18,5 @@
       <origin xyz='0 0 0' rpy='0 -0 0'/>
       <geometry>
-        <mesh filename='meshes/x4.dae' scale='1 1 1'/>
+        <mesh filename='package://ssci_x4_sensor_config_8/meshes/x4.dae' scale='1 1 1'/>
       </geometry>
     </visual>
@@ -24,5 +24,5 @@
       <origin xyz='-0.1 0 0.077' rpy='0 -0.1 0'/>
       <geometry>
-        <mesh filename='meshes/led.dae' scale='1 1 1'/>
+        <mesh filename='package://ssci_x4_sensor_config_8/meshes/led.dae' scale='1 1 1'/>
       </geometry>
     </visual>
@@ -30,5 +30,5 @@
       <origin xyz='-0.09 0.059 0.059' rpy='-0.785397 -0 0.2'/>
       <geometry>
-        <mesh filename='meshes/led.dae' scale='1 1 1'/>
+        <mesh filename='package://ssci_x4_sensor_config_8/meshes/led.dae' scale='1 1 1'/>
       </geometry>
     </visual>
@@ -36,5 +36,5 @@
       <origin xyz='-0.09 -0.059 0.059' rpy='0.785397 -0 -0.2'/>
       <geometry>
-        <mesh filename='meshes/led.dae' scale='1 1 1'/>
+        <mesh filename='package://ssci_x4_sensor_config_8/meshes/led.dae' scale='1 1 1'/>
       </geometry>
     </visual>
@@ -42,5 +42,5 @@
       <origin xyz='-0.043704 0 0.102914' rpy='-0.2 0.000158 -1.57002'/>
       <geometry>
-        <mesh filename='meshes/spotlight.dae' scale='0.01 0.01 0.01'/>
+        <mesh filename='package://ssci_x4_sensor_config_8/meshes/spotlight.dae' scale='0.01 0.01 0.01'/>
       </geometry>
     </visual>
@@ -48,5 +48,5 @@
       <origin xyz='-0.071985 0.090826 0.066102' rpy='0.06 -4.8e-05 -1.27'/>
       <geometry>
-        <mesh filename='meshes/spotlight.dae' scale='0.01 0.01 0.01'/>
+        <mesh filename='package://ssci_x4_sensor_config_8/meshes/spotlight.dae' scale='0.01 0.01 0.01'/>
       </geometry>
     </visual>
@@ -54,5 +54,5 @@
       <origin xyz='-0.071985 -0.090826 0.066102' rpy='0.06 -4.8e-05 -1.87'/>
       <geometry>
-        <mesh filename='meshes/spotlight.dae' scale='0.01 0.01 0.01'/>
+        <mesh filename='package://ssci_x4_sensor_config_8/meshes/spotlight.dae' scale='0.01 0.01 0.01'/>
       </geometry>
     </visual>
@@ -126,5 +126,5 @@
       <origin xyz='0 0 0' rpy='0 -0 0'/>
       <geometry>
-        <mesh filename='meshes/neo11_propeller_ccw.dae' scale='1 1 1'/>
+        <mesh filename='package://ssci_x4_sensor_config_8/meshes/neo11_propeller_ccw.dae' scale='1 1 1'/>
       </geometry>
     </visual>
@@ -145,5 +145,5 @@
       <origin xyz='0 0 0' rpy='0 -0 0'/>
       <geometry>
-        <mesh filename='meshes/neo11_propeller_cw.dae' scale='1 1 1'/>
+        <mesh filename='package://ssci_x4_sensor_config_8/meshes/neo11_propeller_cw.dae' scale='1 1 1'/>
       </geometry>
     </visual>
@@ -164,5 +164,5 @@
       <origin xyz='0 0 0' rpy='0 -0 0'/>
       <geometry>
-        <mesh filename='meshes/neo11_propeller_ccw.dae' scale='1 1 1'/>
+        <mesh filename='package://ssci_x4_sensor_config_8/meshes/neo11_propeller_ccw.dae' scale='1 1 1'/>
       </geometry>
     </visual>
@@ -183,5 +183,5 @@
       <origin xyz='0 0 0' rpy='0 -0 0'/>
       <geometry>
-        <mesh filename='meshes/neo11_propeller_cw.dae' scale='1 1 1'/>
+        <mesh filename='package://ssci_x4_sensor_config_8/meshes/neo11_propeller_cw.dae' scale='1 1 1'/>
       </geometry>
     </visual>
@@ -202,5 +202,5 @@
       <origin xyz='0 0 0' rpy='-0 -0 -0'/>
       <geometry>
-        <mesh filename='meshes/neo11_propeller_ccw.dae' scale='1 1 1'/>
+        <mesh filename='package://ssci_x4_sensor_config_8/meshes/neo11_propeller_ccw.dae' scale='1 1 1'/>
       </geometry>
     </visual>
@@ -221,5 +221,5 @@
       <origin xyz='0 0 0' rpy='0 -0 0'/>
       <geometry>
-        <mesh filename='meshes/neo11_propeller_cw.dae' scale='1 1 1'/>
+        <mesh filename='package://ssci_x4_sensor_config_8/meshes/neo11_propeller_cw.dae' scale='1 1 1'/>
       </geometry>
     </visual>
