Commit message: PR review - FIXUP relative path ins robot_from_sdf.urdf

File: submitted_models/robotika_x2_sensor_config_1/urdf/robot_from_sdf.urdf (robot description, URDF)
Before this commit: robot ROBOTIKA_X2, 5 links, 4 joints
Links:
- link base_link: geometry collision box size=0.42 0.31 0.184; visual box size=0.02 0.02 0.02
- link front_left_wheel: geometry collision cylinder length=0.04 radius=0.098; visual mesh filename=package:meshes/x2_wheel_left.dae scale=1 1 1
- link front_right_wheel: geometry collision cylinder length=0.04 radius=0.098; visual mesh filename=package:meshes/x2_wheel_right.dae scale=1 1 1
- link rear_left_wheel: geometry collision cylinder length=0.04 radius=0.098; visual mesh filename=package:meshes/x2_wheel_left.dae scale=1 1 1
- link rear_right_wheel: geometry collision cylinder length=0.04 radius=0.098; visual mesh filename=package:meshes/x2_wheel_right.dae scale=1 1 1

Commit message: PR review - Backed out changeset: cc289d215a00

File: submitted_models/robotika_x2_sensor_config_1/urdf/robot_from_sdf.urdf (robot description, URDF)
Before this commit: robot ROBOTIKA_X2, 5 links, 4 joints
Links:
- link base_link: geometry collision box size=0.42 0.31 0.184; visual box size=0.02 0.02 0.02
- link front_left_wheel: geometry collision cylinder length=0.04 radius=0.098; visual mesh filename=package://robotika_x2_sensor_config_1/meshes/x2_wheel_left.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 scale=1 1 1
- link front_right_wheel: geometry collision cylinder length=0.04 radius=0.098; visual mesh filename=package://robotika_x2_sensor_config_1/meshes/x2_wheel_right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 scale=1 1 1
- link rear_left_wheel: geometry collision cylinder length=0.04 radius=0.098; visual mesh filename=package://robotika_x2_sensor_config_1/meshes/x2_wheel_left.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 scale=1 1 1
- link rear_right_wheel: geometry collision cylinder length=0.04 radius=0.098; visual mesh filename=package://robotika_x2_sensor_config_1/meshes/x2_wheel_right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 scale=1 1 1
