Commit message: Fix for robotmodel in rviz

File: submitted_models/sophisticated_engineering_x4_sensor_config_9/urdf/x4_from_sdf.xacro (robot description, xacro)
@@ -1,6 +1,6 @@
 <?xml version='1.0' encoding='utf-8'?>
-<robot name='X4' xmlns:xacro='http://ros.org/wiki/xacro'>
-  <xacro:arg name='name' default='X4'/>
-  <xacro:property name='robot_namespace' value='$(arg name)'/>
+<robot name="X4" xmlns:xacro="http://ros.org/wiki/xacro">
+  <xacro:arg name="name" default="X4"/>
+  <xacro:property name="robot_namespace" value="$(arg name)"/>
   <link name='${robot_namespace}/base_link'>
     <inertial>
@@ -18,83 +18,13 @@
       <origin xyz='0 0 0' rpy='0 -0 0'/>
       <geometry>
-        <mesh filename='package://meshes/x4.dae' scale='1 1 1'/>
-      </geometry>
-    </visual>
-    <visual name='marker_visual_1'>
-      <origin xyz='-0.1 0 0.077' rpy='0 -0.1 0'/>
-      <geometry>
-        <mesh filename='package://meshes/led.dae' scale='1 1 1'/>
-      </geometry>
-    </visual>
-    <visual name='marker_visual_2'>
-      <origin xyz='-0.09 0.059 0.059' rpy='-0.785397 -0 0.2'/>
-      <geometry>
-        <mesh filename='package://meshes/led.dae' scale='1 1 1'/>
-      </geometry>
-    </visual>
-    <visual name='marker_visual_3'>
-      <origin xyz='-0.09 -0.059 0.059' rpy='0.785397 -0 -0.2'/>
-      <geometry>
-        <mesh filename='package://meshes/led.dae' scale='1 1 1'/>
-      </geometry>
-    </visual>
-    <visual name='downward_flashlight_visual'>
-      <origin xyz='-0.043704 0 0.102914' rpy='-0.2 0.000158 -1.57002'/>
-      <geometry>
-        <mesh filename='package://meshes/spotlight.dae' scale='0.01 0.01 0.01'/>
-      </geometry>
-    </visual>
-    <visual name='left_flashlight_visual'>
-      <origin xyz='-0.071985 0.090826 0.066102' rpy='0.06 -4.8e-05 -1.27'/>
-      <geometry>
-        <mesh filename='package://meshes/spotlight.dae' scale='0.01 0.01 0.01'/>
-      </geometry>
-    </visual>
-    <visual name='right_flashlight_visual'>
-      <origin xyz='-0.071985 -0.090826 0.066102' rpy='0.06 -4.8e-05 -1.87'/>
-      <geometry>
-        <mesh filename='package://meshes/spotlight.dae' scale='0.01 0.01 0.01'/>
-      </geometry>
-    </visual>
-    <visual name='camera_visual_right'>
-      <origin xyz='0.26 -0.15 -0.04' rpy='0 -0 0'/>
-      <geometry>
-        <box size='0.02 0.02 0.02'/>
-      </geometry>
-    </visual>
-    <visual name='camera_visual_left'>
-      <origin xyz='0.26 0.15 -0.04' rpy='0 -0 0'/>
-      <geometry>
-        <box size='0.02 0.02 0.02'/>
+        <mesh filename='package://x4_description/meshes/x4.dae' scale='1 1 1'/>
       </geometry>
     </visual>
   </link>
-  <sensor name='imu_sensor' update_rate='250'>
-    <parent link='base_link'/>
+  <sensor name='imu_sensor' update_rate='1000'>
+    <parent link='${robot_namespace}/base_link'/>
     <origin xyz='0 0 0' rpy='0 -0 0'/>
   </sensor>
-  <sensor name='air_pressure' update_rate='20'>
-    <parent link='base_link'/>
-    <origin xyz='0 0 0' rpy='0 -0 0'/>
-  </sensor>
-  <sensor name='magnetometer' update_rate='20'>
-    <parent link='base_link'/>
-    <origin xyz='0 0 0' rpy='0 -0 0'/>
-  </sensor>
-  <sensor name='camera_front_right' update_rate='20'>
-    <parent link='base_link'/>
-    <origin xyz='0.26 -0.15 -0.04' rpy='0 -0 0'/>
-    <camera>
-      <image width='1280' height='960' format='R8G8B8' hfov='2' near='0.02' far='300' />
-    </camera>
-  </sensor>
-  <sensor name='camera_front_left' update_rate='20'>
-    <parent link='base_link'/>
-    <origin xyz='0.26 0.15 -0.04' rpy='0 -0 0'/>
-    <camera>
-      <image width='1280' height='960' format='R8G8B8' hfov='2' near='0.02' far='300' />
-    </camera>
-  </sensor>
-  <link name='rotor_0'>
+  <link name='${robot_namespace}/rotor_0'>
     <inertial>
       <origin xyz='0 0 0' rpy='0 -0 0'/>
@@ -111,9 +41,9 @@
       <origin xyz='0 0 0' rpy='0 -0 0'/>
       <geometry>
-        <mesh filename='package://meshes/neo11_propeller_ccw.dae' scale='1 1 1'/>
+        <mesh filename='package://x4_description/meshes/neo11_propeller_ccw.dae' scale='1 1 1'/>
       </geometry>
     </visual>
   </link>
-  <link name='rotor_1'>
+  <link name='${robot_namespace}/rotor_1'>
     <inertial>
       <origin xyz='0 0 0' rpy='0 -0 0'/>
@@ -130,9 +60,9 @@
       <origin xyz='0 0 0' rpy='0 -0 0'/>
       <geometry>
-        <mesh filename='package://meshes/neo11_propeller_cw.dae' scale='1 1 1'/>
+        <mesh filename='package://x4_description/meshes/neo11_propeller_cw.dae' scale='1 1 1'/>
       </geometry>
     </visual>
   </link>
-  <link name='rotor_2'>
+  <link name='${robot_namespace}/rotor_2'>
     <inertial>
       <origin xyz='0 0 0' rpy='0 -0 0'/>
@@ -149,9 +79,9 @@
       <origin xyz='0 0 0' rpy='0 -0 0'/>
       <geometry>
-        <mesh filename='package://meshes/neo11_propeller_ccw.dae' scale='1 1 1'/>
+        <mesh filename='package://x4_description/meshes/neo11_propeller_ccw.dae' scale='1 1 1'/>
       </geometry>
     </visual>
   </link>
-  <link name='rotor_3'>
+  <link name='${robot_namespace}/rotor_3'>
     <inertial>
       <origin xyz='0 0 0' rpy='0 -0 0'/>
@@ -168,9 +98,9 @@
       <origin xyz='0 0 0' rpy='0 -0 0'/>
       <geometry>
-        <mesh filename='package://meshes/neo11_propeller_cw.dae' scale='1 1 1'/>
+        <mesh filename='package://x4_description/meshes/neo11_propeller_cw.dae' scale='1 1 1'/>
       </geometry>
     </visual>
   </link>
-  <link name='rotor_4'>
+  <link name='${robot_namespace}/rotor_4'>
     <inertial>
       <origin xyz='0 0 0' rpy='-0 -0 -0'/>
@@ -187,9 +117,9 @@
       <origin xyz='0 0 0' rpy='-0 -0 -0'/>
       <geometry>
-        <mesh filename='package://meshes/neo11_propeller_ccw.dae' scale='1 1 1'/>
+        <mesh filename='package://x4_description/meshes/neo11_propeller_ccw.dae' scale='1 1 1'/>
       </geometry>
     </visual>
   </link>
-  <link name='rotor_5'>
+  <link name='${robot_namespace}/rotor_5'>
     <inertial>
       <origin xyz='0 0 0' rpy='0 -0 0'/>
@@ -206,5 +136,5 @@
       <origin xyz='0 0 0' rpy='0 -0 0'/>
       <geometry>
-        <mesh filename='package://meshes/neo11_propeller_cw.dae' scale='1 1 1'/>
+        <mesh filename='package://x4_description/meshes/neo11_propeller_cw.dae' scale='1 1 1'/>
       </geometry>
     </visual>
@@ -212,38 +142,38 @@
   <joint name='rotor_0_joint' type='revolute'>
     <origin xyz='0.247 0.1506 0.028' rpy='0.087267 0 0.523599'/>
-    <parent link='base_link'/>
-    <child link='rotor_0'/>
+    <parent link='${robot_namespace}/base_link'/>
+    <child link='${robot_namespace}/rotor_0'/>
     <dynamics damping='0' friction='0' />
-    <axis xyz='0.118748 -0.118521 0.985826'/>
+    <axis xyz='0 1e-06 1'/>
     <limit lower='-1e+16' upper='1e+16' effort='-1' velocity='-1'/>
   </joint>
   <joint name='rotor_1_joint' type='revolute'>
     <origin xyz='-0.00067 0.28929 0.028' rpy='0 -0.087267 0'/>
-    <parent link='base_link'/>
-    <child link='rotor_1'/>
+    <parent link='${robot_namespace}/base_link'/>
+    <child link='${robot_namespace}/rotor_1'/>
     <dynamics damping='0' friction='0' />
-    <axis xyz='-0.173649 0 0.984808'/>
+    <axis xyz='0 0 1'/>
     <limit lower='-1e+16' upper='1e+16' effort='-1' velocity='-1'/>
   </joint>
   <joint name='rotor_2_joint' type='revolute'>
     <origin xyz='-0.2501 0.1454 0.028' rpy='0.087267 -0 2.61799'/>
-    <parent link='base_link'/>
-    <child link='rotor_2'/>
+    <parent link='${robot_namespace}/base_link'/>
+    <child link='${robot_namespace}/rotor_2'/>
     <dynamics damping='0' friction='0' />
-    <axis xyz='-0.031923 0.031863 0.998983'/>
+    <axis xyz='0 1e-06 1'/>
     <limit lower='-1e+16' upper='1e+16' effort='-1' velocity='-1'/>
   </joint>
   <joint name='rotor_3_joint' type='revolute'>
     <origin xyz='-0.2501 -0.1454 0.028' rpy='-0.087267 -0 -2.61799'/>
-    <parent link='base_link'/>
-    <child link='rotor_3'/>
+    <parent link='${robot_namespace}/base_link'/>
+    <child link='${robot_namespace}/rotor_3'/>
     <dynamics damping='0' friction='0' />
-    <axis xyz='-0.031923 -0.031863 0.998983'/>
+    <axis xyz='0 -1e-06 1'/>
     <limit lower='-1e+16' upper='1e+16' effort='-1' velocity='-1'/>
   </joint>
   <joint name='rotor_4_joint' type='revolute'>
     <origin xyz='-0.00067 -0.28929 0.028' rpy='-0 0.087267 -3.14159'/>
-    <parent link='base_link'/>
-    <child link='rotor_4'/>
+    <parent link='${robot_namespace}/base_link'/>
+    <child link='${robot_namespace}/rotor_4'/>
     <dynamics damping='0' friction='0' />
     <axis xyz='-0 -0 1'/>
@@ -252,8 +182,8 @@
   <joint name='rotor_5_joint' type='revolute'>
     <origin xyz='0.247 -0.1506 0.028' rpy='-0.087267 0 -0.523599'/>
-    <parent link='base_link'/>
-    <child link='rotor_5'/>
+    <parent link='${robot_namespace}/base_link'/>
+    <child link='${robot_namespace}/rotor_5'/>
     <dynamics damping='0' friction='0' />
-    <axis xyz='0.118748 0.118521 0.985826'/>
+    <axis xyz='0 -1e-06 1'/>
     <limit lower='-1e+16' upper='1e+16' effort='-1' velocity='-1'/>
   </joint>

Commit message: Changes made as requested: Added Gas-Sensor, Updated lights to cast shadows and propellers not to cast shadows

File: submitted_models/sophisticated_engineering_x4_sensor_config_9/urdf/x4_from_sdf.xacro (robot description, xacro)
@@ -18,12 +18,82 @@
       <origin xyz='0 0 0' rpy='0 -0 0'/>
       <geometry>
-        <mesh filename='package://x4_description/meshes/x4.dae' scale='1 1 1'/>
-      </geometry>
-    </visual>
-  </link>
-  <sensor name='imu_sensor' update_rate='1000'>
+        <mesh filename='package://sophisticated_engineering_x4_sensor_config_9/meshes/x4.dae' scale='1 1 1'/>
+      </geometry>
+    </visual>
+    <visual name='marker_visual_1'>
+      <origin xyz='-0.1 0 0.077' rpy='0 -0.1 0'/>
+      <geometry>
+        <mesh filename='package://sophisticated_engineering_x4_sensor_config_9/meshes/led.dae' scale='1 1 1'/>
+      </geometry>
+    </visual>
+    <visual name='marker_visual_2'>
+      <origin xyz='-0.09 0.059 0.059' rpy='-0.785397 -0 0.2'/>
+      <geometry>
+        <mesh filename='package://sophisticated_engineering_x4_sensor_config_9/meshes/led.dae' scale='1 1 1'/>
+      </geometry>
+    </visual>
+    <visual name='marker_visual_3'>
+      <origin xyz='-0.09 -0.059 0.059' rpy='0.785397 -0 -0.2'/>
+      <geometry>
+        <mesh filename='package://sophisticated_engineering_x4_sensor_config_9/meshes/led.dae' scale='1 1 1'/>
+      </geometry>
+    </visual>
+    <visual name='downward_flashlight_visual'>
+      <origin xyz='-0.043704 0 0.102914' rpy='-0.2 0.000158 -1.57002'/>
+      <geometry>
+        <mesh filename='package://sophisticated_engineering_x4_sensor_config_9/meshes/spotlight.dae' scale='0.01 0.01 0.01'/>
+      </geometry>
+    </visual>
+    <visual name='left_flashlight_visual'>
+      <origin xyz='-0.071985 0.090826 0.066102' rpy='0.06 -4.8e-05 -1.27'/>
+      <geometry>
+        <mesh filename='package://sophisticated_engineering_x4_sensor_config_9/meshes/spotlight.dae' scale='0.01 0.01 0.01'/>
+      </geometry>
+    </visual>
+    <visual name='right_flashlight_visual'>
+      <origin xyz='-0.071985 -0.090826 0.066102' rpy='0.06 -4.8e-05 -1.87'/>
+      <geometry>
+        <mesh filename='package://sophisticated_engineering_x4_sensor_config_9/meshes/spotlight.dae' scale='0.01 0.01 0.01'/>
+      </geometry>
+    </visual>
+    <visual name='camera_visual_right'>
+      <origin xyz='0.26 -0.15 -0.04' rpy='0 -0 0'/>
+      <geometry>
+        <box size='0.02 0.02 0.02'/>
+      </geometry>
+    </visual>
+    <visual name='camera_visual_left'>
+      <origin xyz='0.26 0.15 -0.04' rpy='0 -0 0'/>
+      <geometry>
+        <box size='0.02 0.02 0.02'/>
+      </geometry>
+    </visual>
+  </link>
+  <sensor name='imu_sensor' update_rate='250'>
     <parent link='${robot_namespace}/base_link'/>
     <origin xyz='0 0 0' rpy='0 -0 0'/>
   </sensor>
+  <sensor name='air_pressure' update_rate='20'>
+    <parent link='${robot_namespace}/base_link'/>
+    <origin xyz='0 0 0' rpy='0 -0 0'/>
+  </sensor>
+  <sensor name='magnetometer' update_rate='20'>
+    <parent link='${robot_namespace}/base_link'/>
+    <origin xyz='0 0 0' rpy='0 -0 0'/>
+  </sensor>
+  <sensor name='camera_front_right' update_rate='20'>
+    <parent link='${robot_namespace}/base_link'/>
+    <origin xyz='0.26 -0.15 -0.04' rpy='0 -0 0'/>
+    <camera>
+      <image width='1280' height='960' format='R8G8B8' hfov='2' near='0.02' far='300' />
+    </camera>
+  </sensor>
+  <sensor name='camera_front_left' update_rate='20'>
+    <parent link='${robot_namespace}/base_link'/>
+    <origin xyz='0.26 0.15 -0.04' rpy='0 -0 0'/>
+    <camera>
+      <image width='1280' height='960' format='R8G8B8' hfov='2' near='0.02' far='300' />
+    </camera>
+  </sensor>
   <link name='${robot_namespace}/rotor_0'>
     <inertial>
@@ -41,5 +111,5 @@
       <origin xyz='0 0 0' rpy='0 -0 0'/>
       <geometry>
-        <mesh filename='package://x4_description/meshes/neo11_propeller_ccw.dae' scale='1 1 1'/>
+        <mesh filename='package://sophisticated_engineering_x4_sensor_config_9/meshes/neo11_propeller_ccw.dae' scale='1 1 1'/>
       </geometry>
     </visual>
@@ -60,5 +130,5 @@
       <origin xyz='0 0 0' rpy='0 -0 0'/>
       <geometry>
-        <mesh filename='package://x4_description/meshes/neo11_propeller_cw.dae' scale='1 1 1'/>
+        <mesh filename='package://sophisticated_engineering_x4_sensor_config_9/meshes/neo11_propeller_cw.dae' scale='1 1 1'/>
       </geometry>
     </visual>
@@ -79,5 +149,5 @@
       <origin xyz='0 0 0' rpy='0 -0 0'/>
       <geometry>
-        <mesh filename='package://x4_description/meshes/neo11_propeller_ccw.dae' scale='1 1 1'/>
+        <mesh filename='package://sophisticated_engineering_x4_sensor_config_9/meshes/neo11_propeller_ccw.dae' scale='1 1 1'/>
       </geometry>
     </visual>
@@ -98,5 +168,5 @@
       <origin xyz='0 0 0' rpy='0 -0 0'/>
       <geometry>
-        <mesh filename='package://x4_description/meshes/neo11_propeller_cw.dae' scale='1 1 1'/>
+        <mesh filename='package://sophisticated_engineering_x4_sensor_config_9/meshes/neo11_propeller_cw.dae' scale='1 1 1'/>
       </geometry>
     </visual>
@@ -117,5 +187,5 @@
       <origin xyz='0 0 0' rpy='-0 -0 -0'/>
       <geometry>
-        <mesh filename='package://x4_description/meshes/neo11_propeller_ccw.dae' scale='1 1 1'/>
+        <mesh filename='package://sophisticated_engineering_x4_sensor_config_9/meshes/neo11_propeller_ccw.dae' scale='1 1 1'/>
       </geometry>
     </visual>
@@ -136,5 +206,5 @@
       <origin xyz='0 0 0' rpy='0 -0 0'/>
       <geometry>
-        <mesh filename='package://x4_description/meshes/neo11_propeller_cw.dae' scale='1 1 1'/>
+        <mesh filename='package://sophisticated_engineering_x4_sensor_config_9/meshes/neo11_propeller_cw.dae' scale='1 1 1'/>
       </geometry>
     </visual>
@@ -145,5 +215,5 @@
     <child link='${robot_namespace}/rotor_0'/>
     <dynamics damping='0' friction='0' />
-    <axis xyz='0 1e-06 1'/>
+    <axis xyz='0.118748 -0.118521 0.985826'/>
     <limit lower='-1e+16' upper='1e+16' effort='-1' velocity='-1'/>
   </joint>
@@ -153,5 +223,5 @@
     <child link='${robot_namespace}/rotor_1'/>
     <dynamics damping='0' friction='0' />
-    <axis xyz='0 0 1'/>
+    <axis xyz='-0.173649 0 0.984808'/>
     <limit lower='-1e+16' upper='1e+16' effort='-1' velocity='-1'/>
   </joint>
@@ -161,5 +231,5 @@
     <child link='${robot_namespace}/rotor_2'/>
     <dynamics damping='0' friction='0' />
-    <axis xyz='0 1e-06 1'/>
+    <axis xyz='-0.031923 0.031863 0.998983'/>
     <limit lower='-1e+16' upper='1e+16' effort='-1' velocity='-1'/>
   </joint>
@@ -169,5 +239,5 @@
     <child link='${robot_namespace}/rotor_3'/>
     <dynamics damping='0' friction='0' />
-    <axis xyz='0 -1e-06 1'/>
+    <axis xyz='-0.031923 -0.031863 0.998983'/>
     <limit lower='-1e+16' upper='1e+16' effort='-1' velocity='-1'/>
   </joint>
@@ -185,5 +255,5 @@
     <child link='${robot_namespace}/rotor_5'/>
     <dynamics damping='0' friction='0' />
-    <axis xyz='0 -1e-06 1'/>
+    <axis xyz='0.118748 0.118521 0.985826'/>
     <limit lower='-1e+16' upper='1e+16' effort='-1' velocity='-1'/>
   </joint>
