Commit message: Updating internal references from 8 -> 1

File: submitted_models/ssci_x2_sensor_config_1/urdf/model.xacro (robot description, xacro)
@@ -18,5 +18,5 @@
       <origin xyz='0 0 -0.0655' rpy='1.5708 0 -1.5708'/>
       <geometry>
-        <mesh filename='package://ssci_x2_sensor_config_8/meshes/x2_chassis.dae' scale='1 1 1'/>
+        <mesh filename='package://ssci_x2_sensor_config_1/meshes/x2_chassis.dae' scale='1 1 1'/>
       </geometry>
     </visual>
@@ -30,5 +30,5 @@
       <origin xyz='0.22 0.05 0.0845' rpy='0 0 -3.14159'/>
       <geometry>
-        <mesh filename='package://ssci_x2_sensor_config_8/meshes/headlight.dae' scale='1 1 1'/>
+        <mesh filename='package://ssci_x2_sensor_config_1/meshes/headlight.dae' scale='1 1 1'/>
       </geometry>
     </visual>
@@ -36,5 +36,5 @@
       <origin xyz='0.22 0.145 0.0845' rpy='0 0 -3.14159'/>
       <geometry>
-        <mesh filename='package://ssci_x2_sensor_config_8/meshes/headlight.dae' scale='1 1 1'/>
+        <mesh filename='package://ssci_x2_sensor_config_1/meshes/headlight.dae' scale='1 1 1'/>
       </geometry>
     </visual>
@@ -42,5 +42,5 @@
       <origin xyz='0.22 -0.05 0.0845' rpy='0 0 -3.14159'/>
       <geometry>
-        <mesh filename='package://ssci_x2_sensor_config_8/meshes/headlight.dae' scale='1 1 1'/>
+        <mesh filename='package://ssci_x2_sensor_config_1/meshes/headlight.dae' scale='1 1 1'/>
       </geometry>
     </visual>
@@ -48,5 +48,5 @@
       <origin xyz='0.22 -0.145 0.0845' rpy='0 0 -3.14159'/>
       <geometry>
-        <mesh filename='package://ssci_x2_sensor_config_8/meshes/headlight.dae' scale='1 1 1'/>
+        <mesh filename='package://ssci_x2_sensor_config_1/meshes/headlight.dae' scale='1 1 1'/>
       </geometry>
     </visual>
@@ -98,5 +98,5 @@
       <origin xyz='0 0 0' rpy='1.5708 -0 0'/>
       <geometry>
-        <mesh filename='package://ssci_x2_sensor_config_8/meshes/x2_wheel_left.dae' scale='1 1 1'/>
+        <mesh filename='package://ssci_x2_sensor_config_1/meshes/x2_wheel_left.dae' scale='1 1 1'/>
       </geometry>
     </visual>
@@ -117,5 +117,5 @@
       <origin xyz='0 0 0' rpy='1.5708 -0 0'/>
       <geometry>
-        <mesh filename='package://ssci_x2_sensor_config_8/meshes/x2_wheel_right.dae' scale='1 1 1'/>
+        <mesh filename='package://ssci_x2_sensor_config_1/meshes/x2_wheel_right.dae' scale='1 1 1'/>
       </geometry>
     </visual>
@@ -136,5 +136,5 @@
       <origin xyz='0 0 0' rpy='1.5708 -0 0'/>
       <geometry>
-        <mesh filename='package://ssci_x2_sensor_config_8/meshes/x2_wheel_left.dae' scale='1 1 1'/>
+        <mesh filename='package://ssci_x2_sensor_config_1/meshes/x2_wheel_left.dae' scale='1 1 1'/>
       </geometry>
     </visual>
@@ -155,5 +155,5 @@
       <origin xyz='0 0 0' rpy='1.5708 -0 0'/>
       <geometry>
-        <mesh filename='package://ssci_x2_sensor_config_8/meshes/x2_wheel_right.dae' scale='1 1 1'/>
+        <mesh filename='package://ssci_x2_sensor_config_1/meshes/x2_wheel_right.dae' scale='1 1 1'/>
       </geometry>
     </visual>
