Commit message: changed config number from 8 to 1

File: submitted_models/sophisticated_engineering_x2_sensor_config_1/urdf/x2_from_sdf.xacro (robot description, xacro)
@@ -18,5 +18,5 @@
       <origin xyz='0 0 -0.0655' rpy='1.5708 0 -1.5708'/>
       <geometry>
-        <mesh filename='package://x2_description/meshes/x2_chassis.dae' scale='1 1 1'/>
+        <mesh filename='package://sophisticated_engineering_x2_sensor_config_1/meshes/x2_chassis.dae' scale='1 1 1'/>
       </geometry>
     </visual>
@@ -30,5 +30,5 @@
       <origin xyz='0.22 0.05 0.0845' rpy='0 0 -3.14159'/>
       <geometry>
-        <mesh filename='package://x2_description/meshes/headlight.dae' scale='1 1 1'/>
+        <mesh filename='package://sophisticated_engineering_x2_sensor_config_1/meshes/headlight.dae' scale='1 1 1'/>
       </geometry>
     </visual>
@@ -36,5 +36,5 @@
       <origin xyz='0.22 0.145 0.0845' rpy='0 0 -3.14159'/>
       <geometry>
-        <mesh filename='package://x2_description/meshes/headlight.dae' scale='1 1 1'/>
+        <mesh filename='package://sophisticated_engineering_x2_sensor_config_1/meshes/headlight.dae' scale='1 1 1'/>
       </geometry>
     </visual>
@@ -42,5 +42,5 @@
       <origin xyz='0.22 -0.05 0.0845' rpy='0 0 -3.14159'/>
       <geometry>
-        <mesh filename='package://x2_description/meshes/headlight.dae' scale='1 1 1'/>
+        <mesh filename='package://sophisticated_engineering_x2_sensor_config_1/meshes/headlight.dae' scale='1 1 1'/>
       </geometry>
     </visual>
@@ -48,5 +48,5 @@
       <origin xyz='0.22 -0.145 0.0845' rpy='0 0 -3.14159'/>
       <geometry>
-        <mesh filename='package://x2_description/meshes/headlight.dae' scale='1 1 1'/>
+        <mesh filename='package://sophisticated_engineering_x2_sensor_config_1/meshes/headlight.dae' scale='1 1 1'/>
       </geometry>
     </visual>
@@ -71,5 +71,5 @@
       <origin xyz='0 0 0' rpy='1.5708 -0 0'/>
       <geometry>
-        <mesh filename='package://x2_description/meshes/x2_wheel_left.dae' scale='1 1 1'/>
+        <mesh filename='package://sophisticated_engineering_x2_sensor_config_1/meshes/x2_wheel_left.dae' scale='1 1 1'/>
       </geometry>
     </visual>
@@ -90,5 +90,5 @@
       <origin xyz='0 0 0' rpy='1.5708 -0 0'/>
       <geometry>
-        <mesh filename='package://x2_description/meshes/x2_wheel_right.dae' scale='1 1 1'/>
+        <mesh filename='package://sophisticated_engineering_x2_sensor_config_1/meshes/x2_wheel_right.dae' scale='1 1 1'/>
       </geometry>
     </visual>
@@ -109,5 +109,5 @@
       <origin xyz='0 0 0' rpy='1.5708 -0 0'/>
       <geometry>
-        <mesh filename='package://x2_description/meshes/x2_wheel_left.dae' scale='1 1 1'/>
+        <mesh filename='package://sophisticated_engineering_x2_sensor_config_1/meshes/x2_wheel_left.dae' scale='1 1 1'/>
       </geometry>
     </visual>
@@ -128,5 +128,5 @@
       <origin xyz='0 0 0' rpy='1.5708 -0 0'/>
       <geometry>
-        <mesh filename='package://x2_description/meshes/x2_wheel_right.dae' scale='1 1 1'/>
+        <mesh filename='package://sophisticated_engineering_x2_sensor_config_1/meshes/x2_wheel_right.dae' scale='1 1 1'/>
       </geometry>
     </visual>
