Commit message: changed config number from 9 to 1; replaced thumbnails

File: submitted_models/sophisticated_engineering_x4_sensor_config_1/urdf/x4_from_sdf.xacro (robot description, xacro)
@@ -18,5 +18,5 @@
       <origin xyz='0 0 0' rpy='0 -0 0'/>
       <geometry>
-        <mesh filename='package://sophisticated_engineering_x4_sensor_config_9/meshes/x4.dae' scale='1 1 1'/>
+        <mesh filename='package://sophisticated_engineering_x4_sensor_config_1/meshes/x4.dae' scale='1 1 1'/>
       </geometry>
     </visual>
@@ -24,5 +24,5 @@
       <origin xyz='-0.1 0 0.077' rpy='0 -0.1 0'/>
       <geometry>
-        <mesh filename='package://sophisticated_engineering_x4_sensor_config_9/meshes/led.dae' scale='1 1 1'/>
+        <mesh filename='package://sophisticated_engineering_x4_sensor_config_1/meshes/led.dae' scale='1 1 1'/>
       </geometry>
     </visual>
@@ -30,5 +30,5 @@
       <origin xyz='-0.09 0.059 0.059' rpy='-0.785397 -0 0.2'/>
       <geometry>
-        <mesh filename='package://sophisticated_engineering_x4_sensor_config_9/meshes/led.dae' scale='1 1 1'/>
+        <mesh filename='package://sophisticated_engineering_x4_sensor_config_1/meshes/led.dae' scale='1 1 1'/>
       </geometry>
     </visual>
@@ -36,5 +36,5 @@
       <origin xyz='-0.09 -0.059 0.059' rpy='0.785397 -0 -0.2'/>
       <geometry>
-        <mesh filename='package://sophisticated_engineering_x4_sensor_config_9/meshes/led.dae' scale='1 1 1'/>
+        <mesh filename='package://sophisticated_engineering_x4_sensor_config_1/meshes/led.dae' scale='1 1 1'/>
       </geometry>
     </visual>
@@ -42,5 +42,5 @@
       <origin xyz='-0.043704 0 0.102914' rpy='-0.2 0.000158 -1.57002'/>
       <geometry>
-        <mesh filename='package://sophisticated_engineering_x4_sensor_config_9/meshes/spotlight.dae' scale='0.01 0.01 0.01'/>
+        <mesh filename='package://sophisticated_engineering_x4_sensor_config_1/meshes/spotlight.dae' scale='0.01 0.01 0.01'/>
       </geometry>
     </visual>
@@ -48,5 +48,5 @@
       <origin xyz='-0.071985 0.090826 0.066102' rpy='0.06 -4.8e-05 -1.27'/>
       <geometry>
-        <mesh filename='package://sophisticated_engineering_x4_sensor_config_9/meshes/spotlight.dae' scale='0.01 0.01 0.01'/>
+        <mesh filename='package://sophisticated_engineering_x4_sensor_config_1/meshes/spotlight.dae' scale='0.01 0.01 0.01'/>
       </geometry>
     </visual>
@@ -54,5 +54,5 @@
       <origin xyz='-0.071985 -0.090826 0.066102' rpy='0.06 -4.8e-05 -1.87'/>
       <geometry>
-        <mesh filename='package://sophisticated_engineering_x4_sensor_config_9/meshes/spotlight.dae' scale='0.01 0.01 0.01'/>
+        <mesh filename='package://sophisticated_engineering_x4_sensor_config_1/meshes/spotlight.dae' scale='0.01 0.01 0.01'/>
       </geometry>
     </visual>
@@ -111,5 +111,5 @@
       <origin xyz='0 0 0' rpy='0 -0 0'/>
       <geometry>
-        <mesh filename='package://sophisticated_engineering_x4_sensor_config_9/meshes/neo11_propeller_ccw.dae' scale='1 1 1'/>
+        <mesh filename='package://sophisticated_engineering_x4_sensor_config_1/meshes/neo11_propeller_ccw.dae' scale='1 1 1'/>
       </geometry>
     </visual>
@@ -130,5 +130,5 @@
       <origin xyz='0 0 0' rpy='0 -0 0'/>
       <geometry>
-        <mesh filename='package://sophisticated_engineering_x4_sensor_config_9/meshes/neo11_propeller_cw.dae' scale='1 1 1'/>
+        <mesh filename='package://sophisticated_engineering_x4_sensor_config_1/meshes/neo11_propeller_cw.dae' scale='1 1 1'/>
       </geometry>
     </visual>
@@ -149,5 +149,5 @@
       <origin xyz='0 0 0' rpy='0 -0 0'/>
       <geometry>
-        <mesh filename='package://sophisticated_engineering_x4_sensor_config_9/meshes/neo11_propeller_ccw.dae' scale='1 1 1'/>
+        <mesh filename='package://sophisticated_engineering_x4_sensor_config_1/meshes/neo11_propeller_ccw.dae' scale='1 1 1'/>
       </geometry>
     </visual>
@@ -168,5 +168,5 @@
       <origin xyz='0 0 0' rpy='0 -0 0'/>
       <geometry>
-        <mesh filename='package://sophisticated_engineering_x4_sensor_config_9/meshes/neo11_propeller_cw.dae' scale='1 1 1'/>
+        <mesh filename='package://sophisticated_engineering_x4_sensor_config_1/meshes/neo11_propeller_cw.dae' scale='1 1 1'/>
       </geometry>
     </visual>
@@ -187,5 +187,5 @@
       <origin xyz='0 0 0' rpy='-0 -0 -0'/>
       <geometry>
-        <mesh filename='package://sophisticated_engineering_x4_sensor_config_9/meshes/neo11_propeller_ccw.dae' scale='1 1 1'/>
+        <mesh filename='package://sophisticated_engineering_x4_sensor_config_1/meshes/neo11_propeller_ccw.dae' scale='1 1 1'/>
       </geometry>
     </visual>
@@ -206,5 +206,5 @@
       <origin xyz='0 0 0' rpy='0 -0 0'/>
       <geometry>
-        <mesh filename='package://sophisticated_engineering_x4_sensor_config_9/meshes/neo11_propeller_cw.dae' scale='1 1 1'/>
+        <mesh filename='package://sophisticated_engineering_x4_sensor_config_1/meshes/neo11_propeller_cw.dae' scale='1 1 1'/>
       </geometry>
     </visual>
