Commit message: added a file

File: submitted_models/marble_husky_sensor_config_1/urdf/husky_custom.orig.urdf (robot description, URDF)
Before this commit: robot husky, 29 links, 28 joints
Links:
- removed link arch
- removed link base_footprint
- removed link camera/camera_color_frame
- removed link camera/camera_color_optical_frame
- removed link camera/camera_depth_frame
- removed link camera/camera_depth_optical_frame
- removed link camera/camera_ir2_frame
- removed link camera/camera_ir2_optical_frame
- removed link camera/camera_ir_frame
- removed link camera/camera_ir_optical_frame
- removed link camera/camera_link
- removed link evo_64px_frame
- removed link evo_64px_link
- removed link front_bumper_link
- removed link husky_custom/flashlight_flashlight_link
- removed link husky_custom/overhead_light_led_link
- removed link imu_link
- removed link inertial_link
- removed link rear_bumper_link
- removed link top_chassis_link
- removed link top_plate_link
- removed link user_rail_link
- removed link velodyne
- removed link velodyne_base_link
- added link pan_gimbal_link, mass 0.1; collision cylinder length=0.045 radius=0.014; visual cylinder length=0.045 radius=0.014
- added link tilt_gimbal_link, mass 0.1; collision cylinder length=0.045 radius=0.014; visual box size=0.025 0.13 0.007
- link base_link: mass None -> 46.064; geometry collision box size=0.0078 0.13 0.0192; collision box size=0.0078 0.13 0.0192
- link front_left_wheel_link: geometry collision cylinder length=0.1143 radius=0.1651; visual mesh filename=meshes/wheel.dae scale=1 1 1
- link front_right_wheel_link: geometry collision cylinder length=0.1143 radius=0.1651; visual mesh filename=meshes/wheel.dae scale=1 1 1
- link rear_left_wheel_link: geometry collision cylinder length=0.1143 radius=0.1651; visual mesh filename=meshes/wheel.dae scale=1 1 1
- link rear_right_wheel_link: geometry collision cylinder length=0.1143 radius=0.1651; visual mesh filename=meshes/wheel.dae scale=1 1 1
Joints:
- removed joint base_footprint_joint
- removed joint camera/color_joint
- removed joint camera/color_optical_joint
- removed joint camera/depth_joint
- removed joint camera/depth_optical_joint
- removed joint camera/ired1_joint
- removed joint camera/ired1_optical_joint
- removed joint camera/ired2_joint
- removed joint camera/ired2_optical_joint
- removed joint camera/realsense_joint
- removed joint evo_64px_joint
- removed joint evo_64px_virtual_joint
- removed joint flashlight_flashlight
- removed joint front_bumper
- removed joint front_left_wheel
- removed joint front_right_wheel
- removed joint imu_joint
- removed joint inertial_joint
- removed joint overhead_light_led
- removed joint rear_bumper
- removed joint rear_left_wheel
- removed joint rear_right_wheel
- removed joint top_chassis_joint
- removed joint top_plate_joint
- removed joint top_plate_link_to_arch
- removed joint user_rail
- removed joint velodyne_base_mount_joint
- removed joint velodyne_base_scan_joint
- added joint front_left_wheel_joint: type revolute, parent base_link, child front_left_wheel_link, origin xyz=0.256 0.2854 0.03282 rpy=0 -0 0, axis 0 1 0, limit lower=-1e+16 upper=1e+16 effort=-1 velocity=-1
- added joint front_right_wheel_joint: type revolute, parent base_link, child front_right_wheel_link, origin xyz=0.256 -0.2854 0.03282 rpy=0 -0 0, axis 0 1 0, limit lower=-1e+16 upper=1e+16 effort=-1 velocity=-1
- added joint pan_gimbal_joint: type revolute, parent base_link, child pan_gimbal_link, origin xyz=0.424 0 0.427 rpy=0 -0 0, axis 0 0 1, limit lower=-1e+16 upper=1e+16 effort=-1 velocity=-1
- added joint rear_left_wheel_joint: type revolute, parent base_link, child rear_left_wheel_link, origin xyz=-0.256 0.2854 0.03282 rpy=0 -0 0, axis 0 1 0, limit lower=-1e+16 upper=1e+16 effort=-1 velocity=-1
- added joint rear_right_wheel_joint: type revolute, parent base_link, child rear_right_wheel_link, origin xyz=-0.256 -0.2854 0.03282 rpy=0 -0 0, axis 0 1 0, limit lower=-1e+16 upper=1e+16 effort=-1 velocity=-1
- added joint tilt_gimbal_joint: type revolute, parent pan_gimbal_link, child tilt_gimbal_link, origin xyz=0.424 0 0.46 rpy=0 -0 0, axis 0 1 0, limit lower=-2.79253 upper=2.79253 effort=-1 velocity=-1
