Commit message: Added the xacro file for rviz

File: submitted_models/marble_husky_sensor_config_1/urdf/robot_from_sdf.xacro (robot description, xacro)
@@ -10,7 +10,13 @@
     </inertial>
     <collision name='base_link_collision'>
-      <origin xyz='0 0 0.061875' rpy='0 -0 0'/>
-      <geometry>
-        <box size='0.9874 0.5709 0.12375'/>
+      <origin xyz='0 0 0.12' rpy='0 -0 0'/>
+      <geometry>
+        <box size='0.9874 0.5709 0.05'/>
+      </geometry>
+    </collision>
+    <collision name='base_link_collision_bottom'>
+      <origin xyz='0 0 0.046' rpy='0 -0 0'/>
+      <geometry>
+        <box size='0.8 0.5709 0.095'/>
       </geometry>
     </collision>
@@ -21,44 +27,62 @@
       </geometry>
     </collision>
+    <collision name='base_link_fixed_joint_lump__camera/camera_link_collision_1'>
+      <origin xyz='0 0 0.05' rpy='0 -0 0'/>
+      <geometry>
+        <box size='0.0078 0.13 0.0192'/>
+      </geometry>
+    </collision>
     <collision name='base_link_fixed_joint_lump__camera/camera_link_collision_2'>
-      <origin xyz='0.488 0 0.272' rpy='0 -0 0'/>
+      <origin xyz='0.478 0 0.285' rpy='0 -0 0'/>
       <geometry>
         <box size='0.0078 0.13 0.0192'/>
       </geometry>
     </collision>
-    <collision name='base_link_fixed_joint_lump__top_plate_link_collision_3'>
-      <origin xyz='0.0812 0 0.245' rpy='0 -0 0'/>
-      <geometry>
-        <mesh filename='package://costar_husky_sensor_config_1/meshes/top_plate.dae' scale='1 1 1'/>
-      </geometry>
-    </collision>
-    <collision name='base_link_fixed_joint_lump__top_plate_link_collision_4'>
-      <origin xyz='0.0812 0 0.245' rpy='0 -0 0'/>
-      <geometry>
-        <box size='0.32 0.41 0.09'/>
-      </geometry>
-    </collision>
-    <collision name='base_link_fixed_joint_lump__velodyne_base_link_collision_5'>
-      <origin xyz='0.0012 0 0.71415' rpy='0 -0 0'/>
+    <collision name='base_link_fixed_joint_lump__camera/camera_link_collision_3'>
+      <origin xyz='0.473 0 0.26' rpy='0 0.5236 0'/>
+      <geometry>
+        <box size='0.0078 0.13 0.0192'/>
+      </geometry>
+    </collision>
+    <collision name='base_link_fixed_joint_lump__velodyne_base_link_collision_6'>
+      <origin xyz='0.424 0 0.327' rpy='0 -0 0'/>
       <geometry>
         <cylinder radius='0.0516' length='0.0717'/>
       </geometry>
     </collision>
+    <collision name='base_link_fixed_joint_lump__velodyne_gimbal_plate_base_link_collision_7'>
+      <origin xyz='0.424 0 0.4' rpy='0 -0 0'/>
+      <geometry>
+        <box size='0.1 0.1 0.01'/>
+      </geometry>
+    </collision>
+    <collision name='base_link_fixed_joint_lump__sensor_tower_8'>
+      <origin xyz='0.374 0 0.215' rpy='0 -0 0'/>
+      <geometry>
+        <box size='0.2 0.25 0.225'/>
+      </geometry>
+    </collision>
+    <collision name='base_link_fixed_joint_lump__computer_block_9'>
+      <origin xyz='0.05 0 0.185' rpy='0 -0 0'/>
+      <geometry>
+        <box size='0.3 0.355 0.175'/>
+      </geometry>
+    </collision>
     <visual name='base_link_visual'>
       <origin xyz='0 0 0' rpy='0 -0 0'/>
       <geometry>
-        <mesh filename='package://costar_husky_sensor_config_1/meshes/base_link.dae' scale='1 1 1'/>
+        <mesh filename='package://marble_husky_sensor_config_1/meshes/base_link.dae' scale='1 1 1'/>
       </geometry>
     </visual>
     <visual name='base_link_fixed_joint_lump__camera/camera_link_visual_1'>
-      <origin xyz='0.438 0 0.272' rpy='0 -0 0'/>
-      <geometry>
-        <mesh filename='package://costar_husky_sensor_config_1/meshes/realsense.dae'/>
-      </geometry>
-    </visual>
-    <visual name='base_link_fixed_joint_lump__cliff_sensor_link_visual_2'>
-      <origin xyz='0.435 0 0.235' rpy='-2.35619 -0 -1.5708'/>
-      <geometry>
-        <cylinder radius='0.005' length='0.02'/>
+      <origin xyz='0.478 0 0.26' rpy='0 0.5236 0'/>
+      <geometry>
+        <mesh filename='package://marble_husky_sensor_config_1/meshes/realsense.dae' scale='1 1 1'/>
+      </geometry>
+    </visual>
+    <visual name='base_link_fixed_joint_lump__camera/camera_link_visual_2'>
+      <origin xyz='0.478 0 0.285' rpy='0 -0 0'/>
+      <geometry>
+        <mesh filename='package://marble_husky_sensor_config_1/meshes/realsense.dae' scale='1 1 1'/>
       </geometry>
     </visual>
@@ -66,5 +90,5 @@
       <origin xyz='0.48 0 0.091' rpy='0 -0 0'/>
       <geometry>
-        <mesh filename='package://costar_husky_sensor_config_1/meshes/bumper.dae' scale='1 1 1'/>
+        <mesh filename='package://marble_husky_sensor_config_1/meshes/bumper.dae' scale='1 1 1'/>
       </geometry>
     </visual>
@@ -72,5 +96,5 @@
       <origin xyz='-0.48 0 0.091' rpy='0 -0 3.14159'/>
       <geometry>
-        <mesh filename='package://costar_husky_sensor_config_1/meshes/bumper.dae' scale='1 1 1'/>
+        <mesh filename='package://marble_husky_sensor_config_1/meshes/bumper.dae' scale='1 1 1'/>
       </geometry>
     </visual>
@@ -78,44 +102,23 @@
       <origin xyz='0 0 0' rpy='0 -0 0'/>
       <geometry>
-        <mesh filename='package://costar_husky_sensor_config_1/meshes/top_chassis.dae' scale='1 1 1'/>
-      </geometry>
-    </visual>
-    <visual name='base_link_fixed_joint_lump__top_plate_link_visual_6'>
-      <origin xyz='0.0812 0 0.245' rpy='0 -0 0'/>
-      <geometry>
-        <mesh filename='package://costar_husky_sensor_config_1/meshes/top_plate.dae' scale='1 1 1'/>
-      </geometry>
-    </visual>
-    <visual name='base_link_fixed_joint_lump__arch_visual_7'>
-      <origin xyz='0.0012 0 0.251' rpy='0 -0 0'/>
-      <geometry>
-        <mesh filename='package://costar_husky_sensor_config_1/meshes/jpl04_arch_nosensor.stl' scale='1 1 1'/>
-      </geometry>
-      <material name="black">
-        <color rgba="0.15 0.15 0.15 1"/>
-      </material>
-    </visual>
-    <visual name='base_link_fixed_joint_lump__marker_visual_9'>
-      <origin xyz='0.0012 0 2.251' rpy='0 -0 0'/>
-      <geometry>
-        <sphere radius='0.0001'/>
+        <mesh filename='package://marble_husky_sensor_config_1/meshes/top_chassis.dae' scale='1 1 1'/>
       </geometry>
     </visual>
     <visual name='base_link_fixed_joint_lump__velodyne_base_link_visual_10'>
-      <origin xyz='0.0012 0 0.6783' rpy='0 -0 0'/>
-      <geometry>
-        <mesh filename='package://costar_husky_sensor_config_1/meshes/VLP16_base_1.dae' scale='1 1 1'/>
+      <origin xyz='0.424 0 0.327' rpy='0 -0 0'/>
+      <geometry>
+        <mesh filename='package://marble_husky_sensor_config_1/meshes/VLP16_base_1.dae' scale='1 1 1'/>
       </geometry>
     </visual>
     <visual name='base_link_fixed_joint_lump__velodyne_base_link_visual_11'>
-      <origin xyz='0.0012 0 0.6783' rpy='0 -0 0'/>
-      <geometry>
-        <mesh filename='package://costar_husky_sensor_config_1/meshes/VLP16_base_2.dae' scale='1 1 1'/>
+      <origin xyz='0.424 0 0.327' rpy='0 -0 0'/>
+      <geometry>
+        <mesh filename='package://marble_husky_sensor_config_1/meshes/VLP16_base_2.dae' scale='1 1 1'/>
       </geometry>
     </visual>
     <visual name='base_link_fixed_joint_lump__velodyne_visual_12'>
-      <origin xyz='0.0012 0 0.6783' rpy='0 -0 0'/>
-      <geometry>
-        <mesh filename='package://costar_husky_sensor_config_1/meshes/VLP16_scan.dae' scale='1 1 1'/>
+      <origin xyz='0.424 0 0.327' rpy='0 -0 0'/>
+      <geometry>
+        <mesh filename='package://marble_husky_sensor_config_1/meshes/VLP16_scan.dae' scale='1 1 1'/>
       </geometry>
     </visual>
@@ -123,35 +126,53 @@
       <origin xyz='0.272 0 0.245' rpy='0 -0 0'/>
       <geometry>
-        <mesh filename='package://costar_husky_sensor_config_1/meshes/user_rail.dae' scale='1 1 1'/>
-      </geometry>
-    </visual>
-    <visual name='flashlight_flashlight_light_source_lamp_viz_visual'>
-      <origin xyz='0.415 0.08 0.02' rpy='3.14159 1.57079 -0.001593'/>
-      <geometry>
-        <cylinder radius='0.019' length='0.005'/>
-      </geometry>
-    </visual>
-  </link>
-  <sensor name='camera_front' update_rate='10'>
-    <parent link='${robot_namespace}/base_link'/>
-    <origin xyz='0.438 0 0.272' rpy='0 -0 0'/>
+        <mesh filename='package://marble_husky_sensor_config_1/meshes/user_rail.dae' scale='1 1 1'/>
+      </geometry>
+    </visual>
+    <visual name='base_link_fixed_joint_lump__planar_lidar_link_visual_14'>
+      <origin xyz='0.474 0 0.127' rpy='0 -0 0'/>
+      <geometry>
+        <cylinder radius='0.045' length='0.05'/>
+      </geometry>
+    </visual>
+    <visual name='base_link_fixed_joint_lump__velodyne_gimbal_plate_15'>
+      <origin xyz='0.424 0 0.4' rpy='0 -0 0'/>
+      <geometry>
+        <box size='0.12 0.12 0.01'/>
+      </geometry>
+    </visual>
+    <visual name='base_link_fixed_joint_lump__sensor_tower_16'>
+      <origin xyz='0.374 0 0.215' rpy='0 -0 0'/>
+      <geometry>
+        <box size='0.2 0.25 0.225'/>
+      </geometry>
+    </visual>
+    <visual name='base_link_fixed_joint_lump__computer_block_17'>
+      <origin xyz='0.05 0 0.185' rpy='0 -0 0'/>
+      <geometry>
+        <box size='0.3 0.355 0.175'/>
+      </geometry>
+    </visual>
+  </link>
+  <sensor name='camera_front' update_rate='30'>
+    <parent link='${robot_namespace}/base_link'/>
+    <origin xyz='0.468 0 0.36' rpy='0 -0 0'/>
     <camera>
-      <image width='320' height='240' format='R8G8B8' hfov='1.047' near='0.01' far='300' />
+      <image width='1280' height='720' format='R8G8B8' hfov='1.5184' near='0.01' far='300' />
     </camera>
   </sensor>
-  <sensor name='front_cliff_laser' update_rate='10'>
-    <parent link='${robot_namespace}/base_link'/>
-    <origin xyz='0.435 0 0.235' rpy='-3.14159 -0.785398 3.14159'/>
-    <ray>
-      <horizontal samples='1' resolution='1' min_angle='3.141592653589793' max_angle='3.141592653589793' />
-    </ray>
-  </sensor>
-  <sensor name='front_laser' update_rate='10'>
-    <parent link='${robot_namespace}/base_link'/>
-    <origin xyz='0.0012 0 0.716' rpy='0 -0 0'/>
-    <ray>
-      <horizontal samples='440' resolution='1' min_angle='-3.14159' max_angle='3.14159' />
-      <vertical samples='16' resolution='1' min_angle='-0.261799' max_angle='0.261799' />
-    </ray>
+  <sensor name='camera_down' update_rate='30'>
+    <parent link='${robot_namespace}/base_link'/>
+    <origin xyz='0.473 0 0.335' rpy='0 0.5236 0'/>
+    <camera>
+      <image width='1280' height='720' format='R8G8B8' hfov='1.5184' near='0.01' far='300' />
+    </camera>
+  </sensor>
+  <sensor name='planar_laser' update_rate='10'>
+    <parent link='${robot_namespace}/base_link'/>
+    <origin xyz='0.474 0 0.127' rpy='0 -0 0'/>
+  </sensor>
+  <sensor name='front_laser' update_rate='20'>
+    <parent link='${robot_namespace}/base_link'/>
+    <origin xyz='0.424 0 0.402' rpy='0 -0 0'/>
   </sensor>
   <sensor name='imu_sensor' update_rate='50'>
@@ -166,5 +187,5 @@
     </inertial>
     <collision name='front_left_wheel_link_collision'>
-      <origin xyz='0 0 0' rpy='1.57079 -0 0'/>
+      <origin xyz='0 0 0' rpy='1.5708 -0 0'/>
       <geometry>
         <cylinder radius='0.1651' length='0.1143'/>
@@ -174,5 +195,5 @@
       <origin xyz='0 0 0' rpy='0 -0 0'/>
       <geometry>
-        <mesh filename='package://costar_husky_sensor_config_1/meshes/wheel.dae' scale='1 1 1'/>
+        <mesh filename='package://marble_husky_sensor_config_1/meshes/wheel.dae' scale='1 1 1'/>
       </geometry>
     </visual>
@@ -185,5 +206,5 @@
     </inertial>
     <collision name='front_right_wheel_link_collision'>
-      <origin xyz='0 0 0' rpy='1.57079 -0 0'/>
+      <origin xyz='0 0 0' rpy='1.5708 -0 0'/>
       <geometry>
         <cylinder radius='0.1651' length='0.1143'/>
@@ -193,5 +214,5 @@
       <origin xyz='0 0 0' rpy='0 -0 0'/>
       <geometry>
-        <mesh filename='package://costar_husky_sensor_config_1/meshes/wheel.dae' scale='1 1 1'/>
+        <mesh filename='package://marble_husky_sensor_config_1/meshes/wheel.dae' scale='1 1 1'/>
       </geometry>
     </visual>
@@ -204,5 +225,5 @@
     </inertial>
     <collision name='rear_left_wheel_link_collision'>
-      <origin xyz='0 0 0' rpy='1.57079 -0 0'/>
+      <origin xyz='0 0 0' rpy='1.5708 -0 0'/>
       <geometry>
         <cylinder radius='0.1651' length='0.1143'/>
@@ -212,5 +233,5 @@
       <origin xyz='0 0 0' rpy='0 -0 0'/>
       <geometry>
-        <mesh filename='package://costar_husky_sensor_config_1/meshes/wheel.dae' scale='1 1 1'/>
+        <mesh filename='package://marble_husky_sensor_config_1/meshes/wheel.dae' scale='1 1 1'/>
       </geometry>
     </visual>
@@ -223,5 +244,5 @@
     </inertial>
     <collision name='rear_right_wheel_link_collision'>
-      <origin xyz='0 0 0' rpy='1.57079 -0 0'/>
+      <origin xyz='0 0 0' rpy='1.5708 -0 0'/>
       <geometry>
         <cylinder radius='0.1651' length='0.1143'/>
@@ -231,8 +252,77 @@
       <origin xyz='0 0 0' rpy='0 -0 0'/>
       <geometry>
-        <mesh filename='package://costar_husky_sensor_config_1/meshes/wheel.dae' scale='1 1 1'/>
-      </geometry>
-    </visual>
-  </link>
+        <mesh filename='package://marble_husky_sensor_config_1/meshes/wheel.dae' scale='1 1 1'/>
+      </geometry>
+    </visual>
+  </link>
+  <link name='${robot_namespace}/pan_gimbal_link'>
+    <inertial>
+      <origin xyz='0 0 0' rpy='0 -0 0'/>
+      <mass value='0.1'/>
+      <inertia ixx='1' ixy='0' ixz='0' iyy='1' iyz='0' izz='1'/>
+    </inertial>
+    <collision name='pan_gimbal_link_collision'>
+      <origin xyz='0 0 0' rpy='0 -0 0'/>
+      <geometry>
+        <cylinder radius='0.014' length='0.045'/>
+      </geometry>
+    </collision>
+    <visual name='pan_gimbal_link_visual'>
+      <origin xyz='0 0 0' rpy='0 -0 0'/>
+      <geometry>
+        <cylinder radius='0.014' length='0.045'/>
+      </geometry>
+    </visual>
+  </link>
+  <link name='${robot_namespace}/tilt_gimbal_link'>
+    <inertial>
+      <origin xyz='0 0 0' rpy='1.5708 -0 0'/>
+      <mass value='0.1'/>
+      <inertia ixx='1' ixy='0' ixz='0' iyy='1' iyz='0' izz='1'/>
+    </inertial>
+    <collision name='tilt_gimbal_link_collision'>
+      <origin xyz='0 0 0' rpy='1.5708 -0 0'/>
+      <geometry>
+        <cylinder radius='0.014' length='0.045'/>
+      </geometry>
+    </collision>
+    <visual name='tilt_gimbal_link_visual'>
+      <origin xyz='0 0 0' rpy='1.5708 -0 0'/>
+      <geometry>
+        <cylinder radius='0.014' length='0.045'/>
+      </geometry>
+    </visual>
+    <visual name='tilt_gimbal_link_fixed_joint_lump__camera/camera_link_visual_0'>
+      <origin xyz='0 0 0.03' rpy='0 -0 0'/>
+      <geometry>
+        <mesh filename='package://marble_husky_sensor_config_1/meshes/realsense.dae' scale='1 1 1'/>
+      </geometry>
+    </visual>
+    <visual name='tilt_gimbal_link_fixed_joint_lump_bot_camera_plate_link_visual_1'>
+      <origin xyz='0 0 0.017' rpy='0 -0 0'/>
+      <geometry>
+        <box size='0.025 0.13 0.007'/>
+      </geometry>
+    </visual>
+    <visual name='tilt_gimbal_link_fixed_joint_lump_bot_camera_plate_link_visual_2'>
+      <origin xyz='0 0 0.042' rpy='0 -0 0'/>
+      <geometry>
+        <box size='0.025 0.13 0.007'/>
+      </geometry>
+    </visual>
+    <visual name='flashlight_flashlight_light_source_lamp_viz_visual'>
+      <origin xyz='0 0 0.065' rpy='-0 1.3208 3.14'/>
+      <geometry>
+        <cylinder radius='0.019' length='0.005'/>
+      </geometry>
+    </visual>
+  </link>
+  <sensor name='camera_pan_tilt' update_rate='30'>
+    <parent link='${robot_namespace}/tilt_gimbal_link'/>
+    <origin xyz='0 0 0.03' rpy='0 -0 0'/>
+    <camera>
+      <image width='1280' height='720' format='R8G8B8' hfov='1.5184' near='0.01' far='300' />
+    </camera>
+  </sensor>
   <joint name='front_left_wheel_joint' type='revolute'>
     <origin xyz='0.256 0.2854 0.03282' rpy='0 -0 0'/>
@@ -267,3 +357,19 @@
     <limit lower='-1e+16' upper='1e+16' effort='-1' velocity='-1'/>
   </joint>
+  <joint name='pan_gimbal_joint' type='revolute'>
+    <origin xyz='0.424 0 0.427' rpy='0 -0 0'/>
+    <parent link='${robot_namespace}/base_link'/>
+    <child link='${robot_namespace}/pan_gimbal_link'/>
+    <dynamics damping='0' friction='0' />
+    <axis xyz='0 0 1'/>
+    <limit lower='-1e+16' upper='1e+16' effort='-1' velocity='-1'/>
+  </joint>
+  <joint name='tilt_gimbal_joint' type='revolute'>
+    <origin xyz='0.424 0 0.46' rpy='0 -0 0'/>
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
Commit message: Updated xacro/urdf file

File: submitted_models/marble_husky_sensor_config_1/urdf/robot_from_sdf.xacro (robot description, xacro)
@@ -138,5 +138,5 @@
       <origin xyz='0.424 0 0.4' rpy='0 -0 0'/>
       <geometry>
-        <box size='0.12 0.12 0.01'/>
+        <box size='0.06 0.06 0.01'/>
       </geometry>
     </visual>
@@ -174,7 +174,7 @@
   <sensor name='front_laser' update_rate='20'>
     <parent link='${robot_namespace}/base_link'/>
-    <origin xyz='0.424 0 0.402' rpy='0 -0 0'/>
-  </sensor>
-  <sensor name='imu_sensor' update_rate='50'>
+    <origin xyz='0.424 0 0.387' rpy='0 -0 0'/>
+  </sensor>
+  <sensor name='imu_sensor' update_rate='250'>
     <parent link='${robot_namespace}/base_link'/>
     <origin xyz='0 0 0' rpy='0 -0 0'/>
