Commit message: Fix renames from config_1 to config_2

File: submitted_models/robotika_x2_sensor_config_2/urdf/robot_from_sdf.urdf (robot description, URDF)
Before this commit: robot ROBOTIKA_X2, 5 links, 4 joints
Links:
- link base_link: geometry collision box size=0.42 0.31 0.184; visual box size=0.02 0.02 0.02
- link front_left_wheel: geometry collision cylinder length=0.04 radius=0.098; visual mesh filename=package://robotika_x2_sensor_config_2/meshes/x2_wheel_left.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 scale=1 1 1
- link front_right_wheel: geometry collision cylinder length=0.04 radius=0.098; visual mesh filename=package://robotika_x2_sensor_config_2/meshes/x2_wheel_right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 scale=1 1 1
- link rear_left_wheel: geometry collision cylinder length=0.04 radius=0.098; visual mesh filename=package://robotika_x2_sensor_config_2/meshes/x2_wheel_left.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 scale=1 1 1
- link rear_right_wheel: geometry collision cylinder length=0.04 radius=0.098; visual mesh filename=package://robotika_x2_sensor_config_2/meshes/x2_wheel_right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 scale=1 1 1

File: submitted_models/robotika_x2_sensor_config_2/urdf/robot_from_sdf.xacro (robot description, xacro)
@@ -20,5 +20,5 @@
       <origin rpy="1.5708 0 -1.5708" xyz="0 0 -0.0655"/>
       <geometry>
-        <mesh filename="package://robotika_x2_sensor_config_1/meshes/x2_chassis.dae" scale="1 1 1"/>
+        <mesh filename="package://robotika_x2_sensor_config_2/meshes/x2_chassis.dae" scale="1 1 1"/>
       </geometry>
     </visual>
@@ -32,5 +32,5 @@
       <origin rpy="0 0 -3.14159" xyz="0.22 0.05 0.0845"/>
       <geometry>
-        <mesh filename="package://robotika_x2_sensor_config_1/meshes/headlight.dae" scale="1 1 1"/>
+        <mesh filename="package://robotika_x2_sensor_config_2/meshes/headlight.dae" scale="1 1 1"/>
       </geometry>
     </visual>
@@ -38,5 +38,5 @@
       <origin rpy="0 0 -3.14159" xyz="0.22 0.145 0.0845"/>
       <geometry>
-        <mesh filename="package://robotika_x2_sensor_config_1/meshes/headlight.dae" scale="1 1 1"/>
+        <mesh filename="package://robotika_x2_sensor_config_2/meshes/headlight.dae" scale="1 1 1"/>
       </geometry>
     </visual>
@@ -44,5 +44,5 @@
       <origin rpy="0 0 -3.14159" xyz="0.22 -0.05 0.0845"/>
       <geometry>
-        <mesh filename="package://robotika_x2_sensor_config_1/meshes/headlight.dae" scale="1 1 1"/>
+        <mesh filename="package://robotika_x2_sensor_config_2/meshes/headlight.dae" scale="1 1 1"/>
       </geometry>
     </visual>
@@ -50,5 +50,5 @@
       <origin rpy="0 0 -3.14159" xyz="0.22 -0.145 0.0845"/>
       <geometry>
-        <mesh filename="package://robotika_x2_sensor_config_1/meshes/headlight.dae" scale="1 1 1"/>
+        <mesh filename="package://robotika_x2_sensor_config_2/meshes/headlight.dae" scale="1 1 1"/>
       </geometry>
     </visual>
@@ -96,5 +96,5 @@
       <origin rpy="1.5708 -0 0" xyz="0 0 0"/>
       <geometry>
-        <mesh filename="package://robotika_x2_sensor_config_1/meshes/x2_wheel_left.dae" scale="1 1 1"/>
+        <mesh filename="package://robotika_x2_sensor_config_2/meshes/x2_wheel_left.dae" scale="1 1 1"/>
       </geometry>
     </visual>
@@ -115,5 +115,5 @@
       <origin rpy="1.5708 -0 0" xyz="0 0 0"/>
       <geometry>
-        <mesh filename="package://robotika_x2_sensor_config_1/meshes/x2_wheel_right.dae" scale="1 1 1"/>
+        <mesh filename="package://robotika_x2_sensor_config_2/meshes/x2_wheel_right.dae" scale="1 1 1"/>
       </geometry>
     </visual>
@@ -134,5 +134,5 @@
       <origin rpy="1.5708 -0 0" xyz="0 0 0"/>
       <geometry>
-        <mesh filename="package://robotika_x2_sensor_config_1/meshes/x2_wheel_left.dae" scale="1 1 1"/>
+        <mesh filename="package://robotika_x2_sensor_config_2/meshes/x2_wheel_left.dae" scale="1 1 1"/>
       </geometry>
     </visual>
@@ -153,5 +153,5 @@
       <origin rpy="1.5708 -0 0" xyz="0 0 0"/>
       <geometry>
-        <mesh filename="package://robotika_x2_sensor_config_1/meshes/x2_wheel_right.dae" scale="1 1 1"/>
+        <mesh filename="package://robotika_x2_sensor_config_2/meshes/x2_wheel_right.dae" scale="1 1 1"/>
       </geometry>
     </visual>
