Commit message: cleanup files for renaming

File: submitted_models/cerberus_anymal_sensor_config_1/urdf/robot_from_sdf.xacro (robot description, xacro)
@@ -1,5 +1,6 @@
 <?xml version='1.0' encoding='utf-8'?>
-<robot name='anymal' xmlns:xacro='http://ros.org/wiki/xacro'>
-  <xacro:arg name="name" default="cerberus_anymal_sensor_config_1"/>
+<robot name='anymal_b' xmlns:xacro='http://ros.org/wiki/xacro'>
+  <xacro:arg name="name" default="cerberus_anymal_b_sensor_config_1"/>
+  <xacro:property name="robot_description_package" value="cerberus_anymal_b_sensor_config_1"/>
   <xacro:property name="robot_namespace" value="$(arg name)"/>
   <link name='${robot_namespace}/base'>
@@ -84,5 +85,5 @@
       <origin xyz='0 0 0' rpy='0 -0 0'/>
       <geometry>
-        <mesh filename='meshes/anymal_base.dae' scale='0.001 0.001 0.001'/>
+        <mesh filename='package://${robot_description_package}/meshes/anymal_base.dae' scale='0.001 0.001 0.001'/>
       </geometry>
     </visual>
@@ -90,5 +91,5 @@
       <origin xyz='-0.245 0 0.201' rpy='0 0 -1.5708'/>
       <geometry>
-        <mesh filename='meshes/darpa_jetson_back.stl' scale='0.001 0.001 0.001'/>
+        <mesh filename='package://${robot_description_package}/meshes/darpa_jetson_back.stl' scale='0.001 0.001 0.001'/>
       </geometry>
     </visual>
@@ -96,5 +97,5 @@
       <origin xyz='0.3482 0 0.161624' rpy='0 -0 0'/>
       <geometry>
-        <mesh filename='meshes/darpa_head_1.stl' scale='0.001 0.001 0.001'/>
+        <mesh filename='package://${robot_description_package}/meshes/darpa_head_1.stl' scale='0.001 0.001 0.001'/>
       </geometry>
     </visual>
@@ -102,5 +103,5 @@
       <origin xyz='0.388757 -0.000224 0.057675' rpy='-0.009501 0.382227 0'/>
       <geometry>
-        <mesh filename='meshes/realsense_d435.dae' scale='0.001 0.001 0.001'/>
+        <mesh filename='package://${robot_description_package}/meshes/realsense_d435.dae' scale='0.001 0.001 0.001'/>
       </geometry>
     </visual>
@@ -108,5 +109,5 @@
       <origin xyz='0.27 0 0.2299' rpy='0 -0 0'/>
       <geometry>
-        <mesh filename='meshes/VLP16_base_1.dae' scale='1 1 1'/>
+        <mesh filename='package://${robot_description_package}/meshes/VLP16_base_1.dae' scale='1 1 1'/>
       </geometry>
     </visual>
@@ -114,5 +115,5 @@
       <origin xyz='0.27 0 0.2299' rpy='0 -0 0'/>
       <geometry>
-        <mesh filename='meshes/VLP16_base_2.dae' scale='1 1 1'/>
+        <mesh filename='package://${robot_description_package}/meshes/VLP16_base_2.dae' scale='1 1 1'/>
       </geometry>
     </visual>
@@ -120,5 +121,5 @@
       <origin xyz='0.27 0 0.2299' rpy='0 -0 0'/>
       <geometry>
-        <mesh filename='meshes/VLP16_scan.dae' scale='1 1 1'/>
+        <mesh filename='package://${robot_description_package}/meshes/VLP16_scan.dae' scale='1 1 1'/>
       </geometry>
     </visual>
@@ -205,5 +206,5 @@
       <origin xyz='0 0 0' rpy='0 -0 0'/>
       <geometry>
-        <mesh filename='meshes/anymal_hip_l.dae' scale='0.001 0.001 0.001'/>
+        <mesh filename='package://${robot_description_package}/meshes/anymal_hip_l.dae' scale='0.001 0.001 0.001'/>
       </geometry>
     </visual>
@@ -236,5 +237,5 @@
       <origin xyz='0 0 0' rpy='0 -0 0'/>
       <geometry>
-        <mesh filename='meshes/anymal_thigh_l.dae' scale='0.001 0.001 0.001'/>
+        <mesh filename='package://${robot_description_package}/meshes/anymal_thigh_l.dae' scale='0.001 0.001 0.001'/>
       </geometry>
     </visual>
@@ -267,5 +268,5 @@
       <origin xyz='0 0 0' rpy='0 -0 0'/>
       <geometry>
-        <mesh filename='meshes/anymal_shank_l.dae' scale='0.001 0.001 0.001'/>
+        <mesh filename='package://${robot_description_package}/meshes/anymal_shank_l.dae' scale='0.001 0.001 0.001'/>
       </geometry>
     </visual>
@@ -273,5 +274,5 @@
       <origin xyz='0.1 -0.02 0.032' rpy='0 -0 0'/>
       <geometry>
-        <mesh filename='meshes/anymal_foot.dae' scale='0.001 0.001 0.001'/>
+        <mesh filename='package://${robot_description_package}/meshes/anymal_foot.dae' scale='0.001 0.001 0.001'/>
       </geometry>
     </visual>
@@ -298,5 +299,5 @@
       <origin xyz='0 0 0' rpy='0 -0 3.14159'/>
       <geometry>
-        <mesh filename='meshes/anymal_hip_r.dae' scale='0.001 0.001 0.001'/>
+        <mesh filename='package://${robot_description_package}/meshes/anymal_hip_r.dae' scale='0.001 0.001 0.001'/>
       </geometry>
     </visual>
@@ -329,5 +330,5 @@
       <origin xyz='0 0 0' rpy='0 -0 3.14159'/>
       <geometry>
-        <mesh filename='meshes/anymal_thigh_r.dae' scale='0.001 0.001 0.001'/>
+        <mesh filename='package://${robot_description_package}/meshes/anymal_thigh_r.dae' scale='0.001 0.001 0.001'/>
       </geometry>
     </visual>
@@ -360,5 +361,5 @@
       <origin xyz='0 0 0' rpy='0 -0 3.14159'/>
       <geometry>
-        <mesh filename='meshes/anymal_shank_r.dae' scale='0.001 0.001 0.001'/>
+        <mesh filename='package://${robot_description_package}/meshes/anymal_shank_r.dae' scale='0.001 0.001 0.001'/>
       </geometry>
     </visual>
@@ -366,5 +367,5 @@
       <origin xyz='-0.1 -0.02 0.032' rpy='0 -0 3.14159'/>
       <geometry>
-        <mesh filename='meshes/anymal_foot.dae' scale='0.001 0.001 0.001'/>
+        <mesh filename='package://${robot_description_package}/meshes/anymal_foot.dae' scale='0.001 0.001 0.001'/>
       </geometry>
     </visual>
@@ -391,5 +392,5 @@
       <origin xyz='0 0 0' rpy='0 -0 0'/>
       <geometry>
-        <mesh filename='meshes/anymal_hip_r.dae' scale='0.001 0.001 0.001'/>
+        <mesh filename='package://${robot_description_package}/meshes/anymal_hip_r.dae' scale='0.001 0.001 0.001'/>
       </geometry>
     </visual>
@@ -422,5 +423,5 @@
       <origin xyz='0 0 0' rpy='0 -0 0'/>
       <geometry>
-        <mesh filename='meshes/anymal_thigh_r.dae' scale='0.001 0.001 0.001'/>
+        <mesh filename='package://${robot_description_package}/meshes/anymal_thigh_r.dae' scale='0.001 0.001 0.001'/>
       </geometry>
     </visual>
@@ -453,5 +454,5 @@
       <origin xyz='0 0 0' rpy='0 -0 0'/>
       <geometry>
-        <mesh filename='meshes/anymal_shank_r.dae' scale='0.001 0.001 0.001'/>
+        <mesh filename='package://${robot_description_package}/meshes/anymal_shank_r.dae' scale='0.001 0.001 0.001'/>
       </geometry>
     </visual>
@@ -459,5 +460,5 @@
       <origin xyz='0.1 0.02 0.032' rpy='0 -0 0'/>
       <geometry>
-        <mesh filename='meshes/anymal_foot.dae' scale='0.001 0.001 0.001'/>
+        <mesh filename='package://${robot_description_package}/meshes/anymal_foot.dae' scale='0.001 0.001 0.001'/>
       </geometry>
     </visual>
@@ -484,5 +485,5 @@
       <origin xyz='0 0 0' rpy='0 -0 3.14159'/>
       <geometry>
-        <mesh filename='meshes/anymal_hip_l.dae' scale='0.001 0.001 0.001'/>
+        <mesh filename='package://${robot_description_package}/meshes/anymal_hip_l.dae' scale='0.001 0.001 0.001'/>
       </geometry>
     </visual>
@@ -515,5 +516,5 @@
       <origin xyz='0 0 0' rpy='0 -0 3.14159'/>
       <geometry>
-        <mesh filename='meshes/anymal_thigh_l.dae' scale='0.001 0.001 0.001'/>
+        <mesh filename='package://${robot_description_package}/meshes/anymal_thigh_l.dae' scale='0.001 0.001 0.001'/>
       </geometry>
     </visual>
@@ -546,5 +547,5 @@
       <origin xyz='0 0 0' rpy='0 -0 3.14159'/>
       <geometry>
-        <mesh filename='meshes/anymal_shank_l.dae' scale='0.001 0.001 0.001'/>
+        <mesh filename='package://${robot_description_package}/meshes/anymal_shank_l.dae' scale='0.001 0.001 0.001'/>
       </geometry>
     </visual>
@@ -552,5 +553,5 @@
       <origin xyz='-0.1 0.02 0.032' rpy='0 -0 3.14159'/>
       <geometry>
-        <mesh filename='meshes/anymal_foot.dae' scale='0.001 0.001 0.001'/>
+        <mesh filename='package://${robot_description_package}/meshes/anymal_foot.dae' scale='0.001 0.001 0.001'/>
       </geometry>
     </visual>
