Commit message: Robotika Freyja - fix mount parts of the wheel

File: submitted_models/robotika_freyja_sensor_config_1/urdf/model.urdf (robot description, URDF)
Before this commit: robot ROBOTIKA_FREYJA, 5 links, 4 joints
Links:
- link base_link: geometry collision box size=0.08 0.1 0.115; collision box size=0.08 0.1 0.115
- link front_left_wheel: geometry collision cylinder length=0.082 radius=0.1275; visual cylinder length=0.025 radius=0.04
- link front_right_wheel: geometry collision cylinder length=0.082 radius=0.1275; visual cylinder length=0.025 radius=0.04
- link rear_left_wheel: geometry collision cylinder length=0.082 radius=0.1275; visual cylinder length=0.025 radius=0.04
- link rear_right_wheel: geometry collision cylinder length=0.082 radius=0.1275; visual cylinder length=0.025 radius=0.04

File: submitted_models/robotika_freyja_sensor_config_1/urdf/model.xacro (robot description, xacro)
@@ -1,5 +1,5 @@
 <?xml version="1.0" encoding="utf-8"?>
 <!-- =================================================================================== -->
-<!-- |    This document was autogenerated by xacro from /model.sdf                     | -->
+<!-- |    This document was autogenerated by xacro from src/subt/submitted_models/robotika_freyja_sensor_config_1/model.sdf | -->
 <!-- |    EDITING THIS FILE BY HAND IS NOT RECOMMENDED                                 | -->
 <!-- =================================================================================== -->
@@ -27,5 +27,5 @@
       </inertial>
       <!-- This bounding box covers also wheel mounts at the bottom and
-           lidars on the top. -->
+                 lidars on the top. -->
       <collision name="chassis_collision">
         <pose>0 0 0.105 0 0 0</pose>
@@ -44,6 +44,6 @@
         </geometry>
         <material>
-          <ambient>222 184 135 1</ambient>
-          <diffuse>222 184 135 1</diffuse>
+          <ambient>0.8706 0.7216 0.5294 1.0</ambient>
+          <diffuse>0.8706 0.7216 0.5294 1.0</diffuse>
         </material>
       </visual>
@@ -56,6 +56,6 @@
         </geometry>
         <material>
-          <ambient>222 184 135 1</ambient>
-          <diffuse>222 184 135 1</diffuse>
+          <ambient>0.8706 0.7216 0.5294 1.0</ambient>
+          <diffuse>0.8706 0.7216 0.5294 1.0</diffuse>
         </material>
       </visual>
@@ -68,6 +68,6 @@
         </geometry>
         <material>
-          <ambient>222 184 135 1</ambient>
-          <diffuse>222 184 135 1</diffuse>
+          <ambient>0.8706 0.7216 0.5294 1.0</ambient>
+          <diffuse>0.8706 0.7216 0.5294 1.0</diffuse>
         </material>
       </visual>
@@ -80,6 +80,6 @@
         </geometry>
         <material>
-          <ambient>0 180 0 1</ambient>
-          <diffuse>0 180 0 1</diffuse>
+          <ambient>0.0 0.7059 0.0 1.0</ambient>
+          <diffuse>0.0 0.7059 0.0 1.0</diffuse>
         </material>
       </visual>
@@ -92,6 +92,6 @@
         </geometry>
         <material>
-          <ambient>222 184 135 1</ambient>
-          <diffuse>222 184 135 1</diffuse>
+          <ambient>0.8706 0.7216 0.5294 1.0</ambient>
+          <diffuse>0.8706 0.7216 0.5294 1.0</diffuse>
         </material>
       </visual>
@@ -104,6 +104,6 @@
         </geometry>
         <material>
-          <ambient>222 184 135 1</ambient>
-          <diffuse>222 184 135 1</diffuse>
+          <ambient>0.8706 0.7216 0.5294 1.0</ambient>
+          <diffuse>0.8706 0.7216 0.5294 1.0</diffuse>
         </material>
       </visual>
@@ -116,6 +116,6 @@
         </geometry>
         <material>
-          <ambient>222 184 135 1</ambient>
-          <diffuse>222 184 135 1</diffuse>
+          <ambient>0.8706 0.7216 0.5294 1.0</ambient>
+          <diffuse>0.8706 0.7216 0.5294 1.0</diffuse>
         </material>
       </visual>
@@ -128,6 +128,6 @@
         </geometry>
         <material>
-          <ambient>222 184 135 1</ambient>
-          <diffuse>222 184 135 1</diffuse>
+          <ambient>0.8706 0.7216 0.5294 1.0</ambient>
+          <diffuse>0.8706 0.7216 0.5294 1.0</diffuse>
         </material>
       </visual>
@@ -140,6 +140,6 @@
         </geometry>
         <material>
-          <ambient>180 0 0 1</ambient>
-          <diffuse>180 0 0 1</diffuse>
+          <ambient>0.7059 0.0 0.0 1.0</ambient>
+          <diffuse>0.7059 0.0 0.0 1.0</diffuse>
         </material>
       </visual>
@@ -152,6 +152,6 @@
         </geometry>
         <material>
-          <ambient>222 184 135 1</ambient>
-          <diffuse>222 184 135 1</diffuse>
+          <ambient>0.8706 0.7216 0.5294 1.0</ambient>
+          <diffuse>0.8706 0.7216 0.5294 1.0</diffuse>
         </material>
       </visual>
@@ -164,6 +164,6 @@
         </geometry>
         <material>
-          <ambient>222 184 135 1</ambient>
-          <diffuse>222 184 135 1</diffuse>
+          <ambient>0.8706 0.7216 0.5294 1.0</ambient>
+          <diffuse>0.8706 0.7216 0.5294 1.0</diffuse>
         </material>
       </visual>
@@ -176,6 +176,6 @@
         </geometry>
         <material>
-          <ambient>222 184 135 1</ambient>
-          <diffuse>222 184 135 1</diffuse>
+          <ambient>0.8706 0.7216 0.5294 1.0</ambient>
+          <diffuse>0.8706 0.7216 0.5294 1.0</diffuse>
         </material>
       </visual>
@@ -188,6 +188,6 @@
         </geometry>
         <material>
-          <ambient>222 184 135 1</ambient>
-          <diffuse>222 184 135 1</diffuse>
+          <ambient>0.8706 0.7216 0.5294 1.0</ambient>
+          <diffuse>0.8706 0.7216 0.5294 1.0</diffuse>
         </material>
       </visual>
@@ -200,6 +200,6 @@
         </geometry>
         <material>
-          <ambient>222 184 135 1</ambient>
-          <diffuse>222 184 135 1</diffuse>
+          <ambient>0.8706 0.7216 0.5294 1.0</ambient>
+          <diffuse>0.8706 0.7216 0.5294 1.0</diffuse>
         </material>
       </visual>
@@ -212,6 +212,6 @@
         </geometry>
         <material>
-          <ambient>222 184 135 1</ambient>
-          <diffuse>222 184 135 1</diffuse>
+          <ambient>0.8706 0.7216 0.5294 1.0</ambient>
+          <diffuse>0.8706 0.7216 0.5294 1.0</diffuse>
         </material>
       </visual>
@@ -232,6 +232,6 @@
         </geometry>
         <material>
-          <ambient>222 184 135 1</ambient>
-          <diffuse>222 184 135 1</diffuse>
+          <ambient>0.8706 0.7216 0.5294 1.0</ambient>
+          <diffuse>0.8706 0.7216 0.5294 1.0</diffuse>
         </material>
       </visual>
@@ -244,6 +244,6 @@
         </geometry>
         <material>
-          <ambient>0 0 180 1</ambient>
-          <diffuse>0 0 180 1</diffuse>
+          <ambient>0.0 0.0 0.7059 1.0</ambient>
+          <diffuse>0.0 0.0 0.7059 1.0</diffuse>
         </material>
       </visual>
@@ -264,6 +264,6 @@
         </geometry>
         <material>
-          <ambient>222 184 135 1</ambient>
-          <diffuse>222 184 135 1</diffuse>
+          <ambient>0.8706 0.7216 0.5294 1.0</ambient>
+          <diffuse>0.8706 0.7216 0.5294 1.0</diffuse>
         </material>
       </visual>
@@ -276,6 +276,6 @@
         </geometry>
         <material>
-          <ambient>220 220 0 1</ambient>
-          <diffuse>220 220 0 1</diffuse>
+          <ambient>0.8627 0.8627 0.0 1.0</ambient>
+          <diffuse>0.8627 0.8627 0.0 1.0</diffuse>
         </material>
       </visual>
@@ -289,6 +289,6 @@
         </geometry>
         <material>
-          <ambient>180 180 180</ambient>
-          <diffuse>180 180 180</diffuse>
+          <ambient>0.7059 0.7059 0.7059 1.0</ambient>
+          <diffuse>0.7059 0.7059 0.7059 1.0</diffuse>
         </material>
       </visual>
@@ -302,6 +302,6 @@
         </geometry>
         <material>
-          <ambient>255 0 0</ambient>
-          <diffuse>255 0 0</diffuse>
+          <ambient>1.0 0.0 0.0 1.0</ambient>
+          <diffuse>1.0 0.0 0.0 1.0</diffuse>
         </material>
       </visual>
@@ -315,6 +315,6 @@
         </geometry>
         <material>
-          <ambient>0 0 0</ambient>
-          <diffuse>0 0 0</diffuse>
+          <ambient>0.0 0.0 0.0 1.0</ambient>
+          <diffuse>0.0 0.0 0.0 1.0</diffuse>
         </material>
       </visual>
@@ -328,6 +328,6 @@
         </geometry>
         <material>
-          <ambient>180 180 180</ambient>
-          <diffuse>180 180 180</diffuse>
+          <ambient>0.7059 0.7059 0.7059 1.0</ambient>
+          <diffuse>0.7059 0.7059 0.7059 1.0</diffuse>
         </material>
       </visual>
@@ -340,6 +340,106 @@
         </geometry>
         <material>
-          <ambient>0 0 0</ambient>
-          <diffuse>0 0 0</diffuse>
+          <ambient>0.0 0.0 0.0 1.0</ambient>
+          <diffuse>0.0 0.0 0.0 1.0</diffuse>
+        </material>
+      </visual>
+      <visual name="wheel_mount_front_left_axis_visual">
+        <pose>0.19 0.11 0 1.5707963267948966 0 0</pose>
+        <geometry>
+          <cylinder>
+            <length>0.05</length>
+            <radius>0.008</radius>
+          </cylinder>
+        </geometry>
+        <material>
+          <ambient>0.0 0.0 0.0 1.0</ambient>
+          <diffuse>0.0 0.0 0.0 1.0</diffuse>
+        </material>
+      </visual>
+      <visual name="wheel_mount_front_left_visual">
+        <pose>0.19 0.08 0 0 0 0</pose>
+        <geometry>
+          <box>
+            <size>0.05 0.07 0.025</size>
+          </box>
+        </geometry>
+        <material>
+          <ambient>0.502 0.502 0.502 1.0</ambient>
+          <diffuse>0.502 0.502 0.502 1.0</diffuse>
+        </material>
+      </visual>
+      <visual name="wheel_mount_front_right_axis_visual">
+        <pose>0.19 -0.11 0 1.5707963267948966 0 0</pose>
+        <geometry>
+          <cylinder>
+            <length>0.05</length>
+            <radius>0.008</radius>
+          </cylinder>
+        </geometry>
+        <material>
+          <ambient>0.0 0.0 0.0 1.0</ambient>
+          <diffuse>0.0 0.0 0.0 1.0</diffuse>
+        </material>
+      </visual>
+      <visual name="wheel_mount_front_right_visual">
+        <pose>0.19 -0.08 0 0 0 0</pose>
+        <geometry>
+          <box>
+            <size>0.05 0.07 0.025</size>
+          </box>
+        </geometry>
+        <material>
+          <ambient>0.502 0.502 0.502 1.0</ambient>
+          <diffuse>0.502 0.502 0.502 1.0</diffuse>
+        </material>
+      </visual>
+      <visual name="wheel_mount_rear_left_axis_visual">
+        <pose>-0.19 0.11 0 1.5707963267948966 0 0</pose>
+        <geometry>
+          <cylinder>
+            <length>0.05</length>
+            <radius>0.008</radius>
+          </cylinder>
+        </geometry>
+        <material>
+          <ambient>0.0 0.0 0.0 1.0</ambient>
+          <diffuse>0.0 0.0 0.0 1.0</diffuse>
+        </material>
+      </visual>
+      <visual name="wheel_mount_rear_left_visual">
+        <pose>-0.19 0.08 0 0 0 0</pose>
+        <geometry>
+          <box>
+            <size>0.05 0.07 0.025</size>
+          </box>
+        </geometry>
+        <material>
+          <ambient>0.502 0.502 0.502 1.0</ambient>
+          <diffuse>0.502 0.502 0.502 1.0</diffuse>
+        </material>
+      </visual>
+      <visual name="wheel_mount_rear_right_axis_visual">
+        <pose>-0.19 -0.11 0 1.5707963267948966 0 0</pose>
+        <geometry>
+          <cylinder>
+            <length>0.05</length>
+            <radius>0.008</radius>
+          </cylinder>
+        </geometry>
+        <material>
+          <ambient>0.0 0.0 0.0 1.0</ambient>
+          <diffuse>0.0 0.0 0.0 1.0</diffuse>
+        </material>
+      </visual>
+      <visual name="wheel_mount_rear_right_visual">
+        <pose>-0.19 -0.08 0 0 0 0</pose>
+        <geometry>
+          <box>
+            <size>0.05 0.07 0.025</size>
+          </box>
+        </geometry>
+        <material>
+          <ambient>0.502 0.502 0.502 1.0</ambient>
+          <diffuse>0.502 0.502 0.502 1.0</diffuse>
         </material>
       </visual>
@@ -466,6 +566,6 @@
         </geometry>
         <material>
-          <ambient>200 180 180 1</ambient>
-          <diffuse>200 180 180 1</diffuse>
+          <ambient>0.7843 0.7059 0.7059 1.0</ambient>
+          <diffuse>0.7843 0.7059 0.7059 1.0</diffuse>
         </material>
       </visual>
@@ -479,6 +579,6 @@
         </geometry>
         <material>
-          <ambient>0 0 0 1</ambient>
-          <diffuse>0 0 0 1</diffuse>
+          <ambient>0.0 0.0 0.0 1.0</ambient>
+          <diffuse>0.0 0.0 0.0 1.0</diffuse>
         </material>
       </visual>
@@ -492,6 +592,6 @@
         </geometry>
         <material>
-          <ambient>120 255 120 1</ambient>
-          <diffuse>120 255 120 1</diffuse>
+          <ambient>0.4706 1.0 0.4706 1.0</ambient>
+          <diffuse>0.4706 1.0 0.4706 1.0</diffuse>
         </material>
       </visual>
@@ -505,6 +605,6 @@
         </geometry>
         <material>
-          <ambient>10 10 10 1</ambient>
-          <diffuse>10 10 10 1</diffuse>
+          <ambient>0.03922 0.03922 0.03922 1.0</ambient>
+          <diffuse>0.03922 0.03922 0.03922 1.0</diffuse>
         </material>
       </visual>
@@ -541,6 +641,6 @@
         </geometry>
         <material>
-          <ambient>200 180 180 1</ambient>
-          <diffuse>200 180 180 1</diffuse>
+          <ambient>0.7843 0.7059 0.7059 1.0</ambient>
+          <diffuse>0.7843 0.7059 0.7059 1.0</diffuse>
         </material>
       </visual>
@@ -554,6 +654,6 @@
         </geometry>
         <material>
-          <ambient>0 0 0 1</ambient>
-          <diffuse>0 0 0 1</diffuse>
+          <ambient>0.0 0.0 0.0 1.0</ambient>
+          <diffuse>0.0 0.0 0.0 1.0</diffuse>
         </material>
       </visual>
@@ -567,6 +667,6 @@
         </geometry>
         <material>
-          <ambient>120 255 120 1</ambient>
-          <diffuse>120 255 120 1</diffuse>
+          <ambient>0.4706 1.0 0.4706 1.0</ambient>
+          <diffuse>0.4706 1.0 0.4706 1.0</diffuse>
         </material>
       </visual>
@@ -580,6 +680,6 @@
         </geometry>
         <material>
-          <ambient>10 10 10 1</ambient>
-          <diffuse>10 10 10 1</diffuse>
+          <ambient>0.03922 0.03922 0.03922 1.0</ambient>
+          <diffuse>0.03922 0.03922 0.03922 1.0</diffuse>
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