Commit message: update model to use tf2 static pose messages, and added a better xacro file
Signed-off-by: Nate Koenig <nate@openrobotics.org>

File: submitted_models/robotika_freyja_sensor_config_1/urdf/model.urdf (robot description, URDF)
Before this commit: robot ROBOTIKA_FREYJA, 5 links, 4 joints
Links:
- added link base_footprint
Joints:
- added joint base_footprint_joint: type fixed, parent base_link, child base_footprint, origin xyz=0 0 -0.1275 rpy=0 0 0

File: submitted_models/robotika_freyja_sensor_config_1/urdf/model.xacro (robot description, xacro)
@@ -1,1468 +1,520 @@
 <?xml version="1.0" encoding="utf-8"?>
-<!-- =================================================================================== -->
-<!-- |    This document was autogenerated by xacro from robotika_freyja_sensor_config_1/model.sdf | -->
-<!-- |    EDITING THIS FILE BY HAND IS NOT RECOMMENDED                                 | -->
-<!-- =================================================================================== -->
-<sdf version="1.6">
-  <model name="ROBOTIKA_FREYJA">
-    <pose>0 0 0.1275 0 0 0</pose>
-    <enable_wind>1</enable_wind>
-    <link name="base_link">
-      <!-- Mass modelled as solid 0.3 x 0.24 x 0.08 cuboid at central
-                 bottom part of the robot, where battery and onboard computer
-                 are located, surrounded by ventilation space and lightweight
-                 chassis.
-                 Note: Most of the mass of the robot is *not* in the main body,
-                       but in wheels, which contain hub motors.
-                 https://en.wikipedia.org/wiki/List_of_moments_of_inertia
-            -->
-      <inertial>
-        <pose>0 0 0.0725 0 0 0</pose>
-        <mass>9.6</mass>
-        <inertia>
-          <ixx>0.0512</ixx>
-          <iyy>0.07712</iyy>
-          <izz>0.11808</izz>
-        </inertia>
-      </inertial>
-      <!-- This bounding box covers also wheel mounts at the bottom and
-                 lidars on the top. -->
-      <collision name="chassis_collision">
-        <pose>0 0 0.105 0 0 0</pose>
-        <geometry>
-          <box>
-            <size>0.50 0.24 0.235</size>
-          </box>
-        </geometry>
-      </collision>
-      <visual name="chassis_main_visual">
-        <pose>0 0 0.0725 0 0 0</pose>
-        <geometry>
-          <box>
-            <size>0.46 0.24 0.12</size>
-          </box>
-        </geometry>
-        <material>
-          <ambient>0.8706 0.7216 0.5294 1.0</ambient>
-          <diffuse>0.8706 0.7216 0.5294 1.0</diffuse>
-        </material>
-      </visual>
-      <visual name="chassis_front_face_bottom">
-        <pose>0.24 0 0.0175 0 0 0</pose>
-        <geometry>
-          <box>
-            <size>0.02001 0.24 0.01</size>
-          </box>
-        </geometry>
-        <material>
-          <ambient>0.8706 0.7216 0.5294 1.0</ambient>
-          <diffuse>0.8706 0.7216 0.5294 1.0</diffuse>
-        </material>
-      </visual>
-      <visual name="chassis_front_face_top">
-        <pose>0.24 0 0.1275 0 0 0</pose>
-        <geometry>
-          <box>
-            <size>0.02001 0.24 0.01</size>
-          </box>
-        </geometry>
-        <material>
-          <ambient>0.8706 0.7216 0.5294 1.0</ambient>
-          <diffuse>0.8706 0.7216 0.5294 1.0</diffuse>
-        </material>
-      </visual>
-      <visual name="chassis_front_face_top_marker">
-        <pose>0.245 0 0.1325 0 0 0</pose>
-        <geometry>
-          <box>
-            <size>0.01 0.12 0.0001</size>
-          </box>
-        </geometry>
-        <material>
-          <ambient>0.0 0.7059 0.0 1.0</ambient>
-          <diffuse>0.0 0.7059 0.0 1.0</diffuse>
-        </material>
-      </visual>
-      <visual name="chassis_front_face_left">
-        <pose>0.24 0.115 0.0725 0 0 0</pose>
-        <geometry>
-          <box>
-            <size>0.02001 0.01 0.12</size>
-          </box>
-        </geometry>
-        <material>
-          <ambient>0.8706 0.7216 0.5294 1.0</ambient>
-          <diffuse>0.8706 0.7216 0.5294 1.0</diffuse>
-        </material>
-      </visual>
-      <visual name="chassis_front_face_right">
-        <pose>0.24 -0.115 0.0725 0 0 0</pose>
-        <geometry>
-          <box>
-            <size>0.02001 0.01 0.12</size>
-          </box>
-        </geometry>
-        <material>
-          <ambient>0.8706 0.7216 0.5294 1.0</ambient>
-          <diffuse>0.8706 0.7216 0.5294 1.0</diffuse>
-        </material>
-      </visual>
-      <visual name="chassis_rear_face_bottom">
-        <pose>-0.24 0 0.0175 0 0 0</pose>
-        <geometry>
-          <box>
-            <size>0.02001 0.24 0.01</size>
-          </box>
-        </geometry>
-        <material>
-          <ambient>0.8706 0.7216 0.5294 1.0</ambient>
-          <diffuse>0.8706 0.7216 0.5294 1.0</diffuse>
-        </material>
-      </visual>
-      <visual name="chassis_rear_face_top">
-        <pose>-0.24 0 0.1275 0 0 0</pose>
-        <geometry>
-          <box>
-            <size>0.02001 0.24 0.01</size>
-          </box>
-        </geometry>
-        <material>
-          <ambient>0.8706 0.7216 0.5294 1.0</ambient>
-          <diffuse>0.8706 0.7216 0.5294 1.0</diffuse>
-        </material>
-      </visual>
-      <visual name="chassis_rear_face_top_marker">
-        <pose>-0.245 0 0.1325 0 0 0</pose>
-        <geometry>
-          <box>
-            <size>0.01 0.12 0.0001</size>
-          </box>
-        </geometry>
-        <material>
-          <ambient>0.7059 0.0 0.0 1.0</ambient>
-          <diffuse>0.7059 0.0 0.0 1.0</diffuse>
-        </material>
-      </visual>
-      <visual name="chassis_rear_face_left">
-        <pose>-0.24 0.115 0.0725 0 0 0</pose>
-        <geometry>
-          <box>
-            <size>0.02001 0.01 0.12</size>
-          </box>
-        </geometry>
-        <material>
-          <ambient>0.8706 0.7216 0.5294 1.0</ambient>
-          <diffuse>0.8706 0.7216 0.5294 1.0</diffuse>
-        </material>
-      </visual>
-      <visual name="chassis_rear_face_right">
-        <pose>-0.24 -0.115 0.0725 0 0 0</pose>
-        <geometry>
-          <box>
-            <size>0.02001 0.01 0.12</size>
-          </box>
-        </geometry>
-        <material>
-          <ambient>0.8706 0.7216 0.5294 1.0</ambient>
-          <diffuse>0.8706 0.7216 0.5294 1.0</diffuse>
-        </material>
-      </visual>
-      <visual name="lidar_base_visual">
-        <pose>0 0 0.135 0 0 0</pose>
-        <geometry>
-          <box>
-            <size>0.3001 0.21 0.005</size>
-          </box>
-        </geometry>
-        <material>
-          <ambient>0.8706 0.7216 0.5294 1.0</ambient>
-          <diffuse>0.8706 0.7216 0.5294 1.0</diffuse>
-        </material>
-      </visual>
-      <visual name="cable_cover_left_visual">
-        <pose>0 0.095 0.1475 0 0 0</pose>
-        <geometry>
-          <box>
-            <size>0.07 0.02 0.02001</size>
-          </box>
-        </geometry>
-        <material>
-          <ambient>0.8706 0.7216 0.5294 1.0</ambient>
-          <diffuse>0.8706 0.7216 0.5294 1.0</diffuse>
-        </material>
-      </visual>
-      <visual name="cable_cover_right_visual">
-        <pose>0 -0.095 0.1475 0 0 0</pose>
-        <geometry>
-          <box>
-            <size>0.07 0.02 0.02001</size>
-          </box>
-        </geometry>
-        <material>
-          <ambient>0.8706 0.7216 0.5294 1.0</ambient>
-          <diffuse>0.8706 0.7216 0.5294 1.0</diffuse>
-        </material>
-      </visual>
-      <visual name="cable_cover_top_visual">
-        <pose>0 0.0 0.16 0 0 0</pose>
-        <geometry>
-          <box>
-            <size>0.07 0.21 0.005</size>
-          </box>
-        </geometry>
-        <material>
-          <ambient>0.8706 0.7216 0.5294 1.0</ambient>
-          <diffuse>0.8706 0.7216 0.5294 1.0</diffuse>
-        </material>
-      </visual>
-      <collision name="left_mount_collision">
-        <pose>0.0 0.17 0.085 0 0 0</pose>
-        <geometry>
-          <box>
-            <size>0.08 0.1 0.115</size>
-          </box>
-        </geometry>
-      </collision>
-      <visual name="left_mount_visual">
-        <pose>0.0 0.17 0.0725 0 0 0</pose>
-        <geometry>
-          <box>
-            <size>0.08 0.1 0.09</size>
-          </box>
-        </geometry>
-        <material>
-          <ambient>0.8706 0.7216 0.5294 1.0</ambient>
-          <diffuse>0.8706 0.7216 0.5294 1.0</diffuse>
-        </material>
-      </visual>
-      <visual name="left_mount_top_marker_visual">
-        <pose>0.0 0.215 0.1175 0 0 0</pose>
-        <geometry>
-          <box>
-            <size>0.08 0.01 0.0001</size>
-          </box>
-        </geometry>
-        <material>
-          <ambient>0.0 0.0 0.7059 1.0</ambient>
-          <diffuse>0.0 0.0 0.7059 1.0</diffuse>
-        </material>
-      </visual>
-      <collision name="right_mount_collision">
-        <pose>0.0 -0.17 0.085 0 0 0</pose>
-        <geometry>
-          <box>
-            <size>0.08 0.1 0.115</size>
-          </box>
-        </geometry>
-      </collision>
-      <visual name="right_mount_visual">
-        <pose>0.0 -0.17 0.0725 0 0 0</pose>
-        <geometry>
-          <box>
-            <size>0.08 0.1 0.09</size>
-          </box>
-        </geometry>
-        <material>
-          <ambient>0.8706 0.7216 0.5294 1.0</ambient>
-          <diffuse>0.8706 0.7216 0.5294 1.0</diffuse>
-        </material>
-      </visual>
-      <visual name="right_mount_top_marker_visual">
-        <pose>0.0 -0.215 0.1175 0 0 0</pose>
-        <geometry>
-          <box>
-            <size>0.08 0.01 0.0001</size>
-          </box>
-        </geometry>
-        <material>
-          <ambient>0.8627 0.8627 0.0 1.0</ambient>
-          <diffuse>0.8627 0.8627 0.0 1.0</diffuse>
-        </material>
-      </visual>
-      <visual name="emergency_stop_bottom_visual">
-        <pose>0.0 -0.155 0.125 0 0 0</pose>
-        <geometry>
-          <cylinder>
-            <length>0.015</length>
-            <radius>0.015</radius>
-          </cylinder>
-        </geometry>
-        <material>
-          <ambient>0.7059 0.7059 0.7059 1.0</ambient>
-          <diffuse>0.7059 0.7059 0.7059 1.0</diffuse>
-        </material>
-      </visual>
-      <visual name="emergency_stop_top_visual">
-        <pose>0.0 -0.155 0.135 0 0 0</pose>
-        <geometry>
-          <cylinder>
-            <length>0.005</length>
-            <radius>0.02</radius>
-          </cylinder>
-        </geometry>
-        <material>
-          <ambient>1.0 0.0 0.0 1.0</ambient>
-          <diffuse>1.0 0.0 0.0 1.0</diffuse>
-        </material>
-      </visual>
-      <visual name="power_switch_bottom_visual">
-        <pose>0.0 0.155 0.1225 0 0 0</pose>
-        <geometry>
-          <cylinder>
-            <length>0.005</length>
-            <radius>0.015</radius>
-          </cylinder>
-        </geometry>
-        <material>
-          <ambient>0.0 0.0 0.0 1.0</ambient>
-          <diffuse>0.0 0.0 0.0 1.0</diffuse>
-        </material>
-      </visual>
-      <visual name="power_switch_middle_visual">
-        <pose>0.0 0.155 0.1275 0 0 0</pose>
-        <geometry>
-          <cylinder>
-            <length>0.005</length>
-            <radius>0.015</radius>
-          </cylinder>
-        </geometry>
-        <material>
-          <ambient>0.7059 0.7059 0.7059 1.0</ambient>
-          <diffuse>0.7059 0.7059 0.7059 1.0</diffuse>
-        </material>
-      </visual>
-      <visual name="power_switch_top_visual">
-        <pose>0.0 0.155 0.1375 0 0 0.35</pose>
-        <geometry>
-          <box>
-            <size>0.025 0.005 0.01</size>
-          </box>
-        </geometry>
-        <material>
-          <ambient>0.0 0.0 0.0 1.0</ambient>
-          <diffuse>0.0 0.0 0.0 1.0</diffuse>
-        </material>
-      </visual>
-      <visual name="wheel_mount_front_left_axis_visual">
-        <pose>0.19 0.11 0 1.5707963267948966 0 0</pose>
-        <geometry>
-          <cylinder>
-            <length>0.05</length>
-            <radius>0.008</radius>
-          </cylinder>
-        </geometry>
-        <material>
-          <ambient>0.0 0.0 0.0 1.0</ambient>
-          <diffuse>0.0 0.0 0.0 1.0</diffuse>
-        </material>
-      </visual>
-      <visual name="wheel_mount_front_left_visual">
-        <pose>0.19 0.08 0 0 0 0</pose>
-        <geometry>
-          <box>
-            <size>0.05 0.07 0.025</size>
-          </box>
-        </geometry>
-        <material>
-          <ambient>0.502 0.502 0.502 1.0</ambient>
-          <diffuse>0.502 0.502 0.502 1.0</diffuse>
-        </material>
-      </visual>
-      <visual name="wheel_mount_front_right_axis_visual">
-        <pose>0.19 -0.11 0 1.5707963267948966 0 0</pose>
-        <geometry>
-          <cylinder>
-            <length>0.05</length>
-            <radius>0.008</radius>
-          </cylinder>
-        </geometry>
-        <material>
-          <ambient>0.0 0.0 0.0 1.0</ambient>
-          <diffuse>0.0 0.0 0.0 1.0</diffuse>
-        </material>
-      </visual>
-      <visual name="wheel_mount_front_right_visual">
-        <pose>0.19 -0.08 0 0 0 0</pose>
-        <geometry>
-          <box>
-            <size>0.05 0.07 0.025</size>
-          </box>
-        </geometry>
-        <material>
-          <ambient>0.502 0.502 0.502 1.0</ambient>
-          <diffuse>0.502 0.502 0.502 1.0</diffuse>
-        </material>
-      </visual>
-      <visual name="wheel_mount_rear_left_axis_visual">
-        <pose>-0.19 0.11 0 1.5707963267948966 0 0</pose>
-        <geometry>
-          <cylinder>
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