Commit message: Corrected path for Freyja model.xacro file wheel.dae reference.

File: submitted_models/robotika_freyja_sensor_config_1/urdf/model.xacro (robot description, xacro)
@@ -405,5 +405,5 @@
       <origin xyz='0 0 0' rpy='1.5708 -0 0'/>
       <geometry>
-        <mesh filename='meshes/wheel_left.dae' scale='1.30102 1.30102 2.05'/>
+        <mesh filename='package://robotika_freyja_sensor_config_1/meshes/wheel_left.dae' scale='1.30102 1.30102 2.05'/>
       </geometry>
     </visual>
@@ -430,5 +430,5 @@
       <origin xyz='0 0 0' rpy='1.5708 -0 0'/>
       <geometry>
-        <mesh filename='meshes/wheel_right.dae' scale='1.30102 1.30102 2.05'/>
+        <mesh filename='package://robotika_freyja_sensor_config_1/meshes/wheel_right.dae' scale='1.30102 1.30102 2.05'/>
       </geometry>
     </visual>
@@ -455,5 +455,5 @@
       <origin xyz='0 0 0' rpy='1.5708 -0 0'/>
       <geometry>
-        <mesh filename='meshes/wheel_left.dae' scale='1.30102 1.30102 2.05'/>
+        <mesh filename='package://robotika_freyja_sensor_config_1/meshes/wheel_left.dae' scale='1.30102 1.30102 2.05'/>
       </geometry>
     </visual>
@@ -480,5 +480,5 @@
       <origin xyz='0 0 0' rpy='1.5708 -0 0'/>
       <geometry>
-        <mesh filename='meshes/wheel_right.dae' scale='1.30102 1.30102 2.05'/>
+        <mesh filename='package://robotika_freyja_sensor_config_1/meshes/wheel_right.dae' scale='1.30102 1.30102 2.05'/>
       </geometry>
     </visual>
