Commit message: Robotika Kloubak URDF ver1

File: submitted_models/robotika_kloubak_sensor_config_1/urdf/model.xacro (robot description, xacro)
@@ -5,5 +5,5 @@
 <!-- =================================================================================== -->
 <sdf version="1.6">
-  <model name="Robotika_K2">
+  <model name="ROBOTIKA_KLOUBAK">
     <static>false</static>
     <enable_wind>1</enable_wind>
@@ -20,5 +20,5 @@
       </inertial>
       <!-- Box and axle -->
-      <collision name="collision_fron_box">
+      <collision name="collision_front_box">
         <pose>0 0 0.08 0 0 0</pose>
         <geometry>
@@ -75,5 +75,5 @@
         </geometry>
       </visual>
-      <!-- LORD IMU and magnetometer?? -->
+      <!-- LORD IMU and magnetometer -->
       <sensor name="imu_sensor_front" type="imu">
         <always_on>1</always_on>
@@ -170,5 +170,5 @@
         </magnetometer>
       </sensor>
-      <!-- Infineon DPS310 TODO ???
+      <!-- Infineon DPS310
             https://www.infineon.com/cms/en/product/sensor/pressure-sensors/absolute-pressure-sensors-map-bap/dps310/
         -->
@@ -183,5 +183,5 @@
         </air_pressure>
       </sensor>
-      <!--LED lihgt -->
+      <!--LED light -->
       <collision name="collision_light_lidar_camera">
         <pose>0.05 0 0.2325 0 0 0</pose>
@@ -277,8 +277,8 @@
               <fx>17.8229</fx>
               <fy>17.8229</fy>
-              <!-- cx = ( width + 1 ) / 2 -->
-              <cx>512.5</cx>
-              <!-- cy = ( height + 1 ) / 2 -->
-              <cy>384.5</cy>
+              <!-- cx = ( width - 1 ) / 2 -->
+              <cx>511.5</cx>
+              <!-- cy = ( height - 1 ) / 2 -->
+              <cy>383.5</cy>
               <s>0</s>
             </intrinsics>
@@ -341,14 +341,14 @@
         <camera name="depth_camera_front">
           <pose frame="">0 0 0 0 -1.5707 1.5707</pose>
-          <horizontal_fov>1.2113</horizontal_fov>
+          <horizontal_fov>1.5184</horizontal_fov>
           <lens>
             <intrinsics>
               <!-- fx = fy = width / ( 2 * tan (hfov / 2 ) ) -->
-              <fx>462.1</fx>
-              <fy>462.1</fy>
-              <!-- cx = ( width + 1 ) / 2 -->
-              <cx>320.5</cx>
-              <!-- cy = ( height + 1 ) / 2 -->
-              <cy>180.5</cy>
+              <fx>337.22</fx>
+              <fy>337.22</fy>
+              <!-- cx = ( width - 1 ) / 2 -->
+              <cx>319.5</cx>
+              <!-- cy = ( height - 1 ) / 2 -->
+              <cy>179.5</cy>
               <s>0</s>
             </intrinsics>
@@ -419,5 +419,5 @@
         </geometry>
       </visual>
-      <!-- LORD IMU and magnetometer??? -->
+      <!-- LORD IMU and magnetometer -->
       <sensor name="imu_sensor_back" type="imu">
         <always_on>1</always_on>
@@ -514,5 +514,5 @@
         </magnetometer>
       </sensor>
-      <!--LED lihgt -->
+      <!--LED light -->
       <collision name="collision_light_lidar_camera">
         <pose>-0.07 0 0.2925 0 0 0</pose>
@@ -608,8 +608,8 @@
               <fx>17.8229</fx>
               <fy>17.8229</fy>
-              <!-- cx = ( width + 1 ) / 2 -->
-              <cx>512.5</cx>
-              <!-- cy = ( height + 1 ) / 2 -->
-              <cy>384.5</cy>
+              <!-- cx = ( width - 1 ) / 2 -->
+              <cx>511.5</cx>
+              <!-- cy = ( height - 1 ) / 2 -->
+              <cy>383.5</cy>
               <s>0</s>
             </intrinsics>
@@ -672,14 +672,14 @@
         <camera name="depth_camera_back">
           <pose frame="">0 0 0 0 -1.5707 1.5707</pose>
-          <horizontal_fov>1.2113</horizontal_fov>
+          <horizontal_fov>1.5184</horizontal_fov>
           <lens>
             <intrinsics>
               <!-- fx = fy = width / ( 2 * tan (hfov / 2 ) ) -->
-              <fx>462.1</fx>
-              <fy>462.1</fy>
-              <!-- cx = ( width + 1 ) / 2 -->
-              <cx>320.5</cx>
-              <!-- cy = ( height + 1 ) / 2 -->
-              <cy>180.5</cy>
+              <fx>337.22</fx>
+              <fy>337.22</fy>
+              <!-- cx = ( width - 1 ) / 2 -->
+              <cx>319.5</cx>
+              <!-- cy = ( height - 1 ) / 2 -->
+              <cy>179.5</cy>
               <s>0</s>
             </intrinsics>
@@ -741,6 +741,6 @@
         </geometry>
         <material>
-          <ambient>204 204 204 </ambient>
-          <diffuse>204 204 204 </diffuse>
+          <ambient>204 204 204 1</ambient>
+          <diffuse>204 204 204 1</diffuse>
         </material>
       </visual>

Commit message: Updating tf
Signed-off-by: Nate Koenig <nate@openrobotics.org>

File: submitted_models/robotika_kloubak_sensor_config_1/urdf/model.xacro (robot description, xacro)
@@ -1,1050 +1,381 @@
 <?xml version="1.0" encoding="utf-8"?>
-<!-- =================================================================================== -->
-<!-- |    This document was autogenerated by xacro from /tmp/model.sdf                 | -->
-<!-- |    EDITING THIS FILE BY HAND IS NOT RECOMMENDED                                 | -->
-<!-- =================================================================================== -->
-<sdf version="1.6">
-  <model name="ROBOTIKA_KLOUBAK">
-    <static>false</static>
-    <enable_wind>1</enable_wind>
-    <link name="chassis_front">
-      <pose>0 0 0.2 0 0 0</pose>
-      <inertial>
-        <pose>-0.05 0 0.08 0 0 0</pose>
-        <mass>8</mass>
-        <inertia>
-          <ixx>0.1119</ixx>
-          <iyy>0.1286</iyy>
-          <izz>0.2159</izz>
-        </inertia>
-      </inertial>
-      <!-- Box and axle -->
-      <collision name="collision_front_box">
-        <pose>0 0 0.08 0 0 0</pose>
-        <geometry>
-          <box>
-            <size>0.3 0.4 0.16</size>
-          </box>
-        </geometry>
-      </collision>
-      <collision name="collision_bar">
-        <pose>-0.17 0 0.02 0 0 0</pose>
-        <geometry>
-          <box>
-            <size>0.3 0.04 0.04</size>
-          </box>
-        </geometry>
-      </collision>
-      <collision name="collision_joint_upper">
-        <pose>-0.335 0 0.05 0 0 0</pose>
-        <geometry>
-          <box>
-            <size>0.07 0.06 0.02</size>
-          </box>
-        </geometry>
-      </collision>
-      <collision name="collision_joint_bottom">
-        <pose>-0.335 0 -0.01 0 0 0</pose>
-        <geometry>
-          <box>
-            <size>0.07 0.06 0.02</size>
-          </box>
-        </geometry>
-      </collision>
-      <collision name="collision_wheel_hinge_left">
-        <pose>0 0.18 -0.02 0 0 0</pose>
-        <geometry>
-          <box>
-            <size>0.04 0.06 0.04</size>
-          </box>
-        </geometry>
-      </collision>
-      <collision name="collision_wheel_hinge_right">
-        <pose>0 -0.18 -0.02 0 0 0</pose>
-        <geometry>
-          <box>
-            <size>0.04 0.06 0.04</size>
-          </box>
-        </geometry>
-      </collision>
-      <visual name="visual_chassis">
-        <geometry>
-          <mesh>
-            <uri>meshes/chassis_front.dae</uri>
-          </mesh>
-        </geometry>
-      </visual>
-      <!-- LORD IMU and magnetometer -->
-      <sensor name="imu_sensor_front" type="imu">
-        <always_on>1</always_on>
-        <update_rate>50</update_rate>
-        <imu>
-          <angular_velocity>
-            <x>
-              <noise type="gaussian">
-                <mean>0</mean>
-                <stddev>2e-4</stddev>
-                <bias_mean>0.0000075</bias_mean>
-                <bias_stddev>0.0000008</bias_stddev>
-                <dynamic_bias_stddev>0.0000004</dynamic_bias_stddev>
-                <dynamic_bias_correlation_time>1000.0</dynamic_bias_correlation_time>
-              </noise>
-            </x>
-            <y>
-              <noise type="gaussian">
-                <mean>0</mean>
-                <stddev>2e-4</stddev>
-                <bias_mean>0.0000075</bias_mean>
-                <bias_stddev>0.0000008</bias_stddev>
-                <dynamic_bias_stddev>0.0000004</dynamic_bias_stddev>
-                <dynamic_bias_correlation_time>1000.0</dynamic_bias_correlation_time>
-              </noise>
-            </y>
-            <z>
-              <noise type="gaussian">
-                <mean>0</mean>
-                <stddev>2e-4</stddev>
-                <bias_mean>0.0000075</bias_mean>
-                <bias_stddev>0.0000008</bias_stddev>
-                <dynamic_bias_stddev>0.0000004</dynamic_bias_stddev>
-                <dynamic_bias_correlation_time>1000.0</dynamic_bias_correlation_time>
-              </noise>
-            </z>
-          </angular_velocity>
-          <linear_acceleration>
-            <x>
-              <noise type="gaussian">
-                <mean>0</mean>
-                <stddev>1e-2</stddev>
-                <bias_mean>0.1</bias_mean>
-                <bias_stddev>0.001</bias_stddev>
-                <dynamic_bias_stddev>0.002</dynamic_bias_stddev>
-                <dynamic_bias_correlation_time>300.0</dynamic_bias_correlation_time>
-              </noise>
-            </x>
-            <y>
-              <noise type="gaussian">
-                <mean>0</mean>
-                <stddev>1e-2</stddev>
-                <bias_mean>0.1</bias_mean>
-                <bias_stddev>0.001</bias_stddev>
-                <dynamic_bias_stddev>0.002</dynamic_bias_stddev>
-                <dynamic_bias_correlation_time>300.0</dynamic_bias_correlation_time>
-              </noise>
-            </y>
-            <z>
-              <noise type="gaussian">
-                <mean>0</mean>
-                <stddev>1e-2</stddev>
-                <bias_mean>0.1</bias_mean>
-                <bias_stddev>0.001</bias_stddev>
-                <dynamic_bias_stddev>0.002</dynamic_bias_stddev>
-                <dynamic_bias_correlation_time>300.0</dynamic_bias_correlation_time>
-              </noise>
-            </z>
-          </linear_acceleration>
-        </imu>
-      </sensor>
-      <sensor name="magnetometer_front" type="magnetometer">
-        <always_on>1</always_on>
-        <update_rate>50</update_rate>
-        <magnetometer>
-          <x>
-            <noise type="gaussian">
-              <mean>0.000000080</mean>
-              <bias_mean>0.000000400</bias_mean>
-            </noise>
-          </x>
-          <y>
-            <noise type="gaussian">
-              <mean>0.000000080</mean>
-              <bias_mean>0.000000400</bias_mean>
-            </noise>
-          </y>
-          <z>
-            <noise type="gaussian">
-              <mean>0.000000080</mean>
-              <bias_mean>0.000000400</bias_mean>
-            </noise>
-          </z>
-        </magnetometer>
-      </sensor>
-      <!-- Infineon DPS310
-            https://www.infineon.com/cms/en/product/sensor/pressure-sensors/absolute-pressure-sensors-map-bap/dps310/
-        -->
-      <sensor name="air_pressure" type="air_pressure">
-        <always_on>1</always_on>
-        <update_rate>20</update_rate>
-        <air_pressure>
-          <reference_altitude>0</reference_altitude>
-          <noise type="gaussian">
-            <mean>0.00000008</mean>
-          </noise>
-        </air_pressure>
-      </sensor>
-      <!--LED light -->
-      <collision name="collision_light_lidar_camera">
-        <pose>0.05 0 0.2325 0 0 0</pose>
-        <geometry>
-          <box>
-            <size>0.2 0.15 0.145</size>
-          </box>
-        </geometry>
-      </collision>
-      <visual name="visual_light">
-        <pose>0.09 0 0.16 0 0 0</pose>
-        <geometry>
-          <mesh>
-            <uri>meshes/light.dae</uri>
-          </mesh>
-        </geometry>
-      </visual>
-      <light name="light_front" type="spot">
-        <pose>0.15 0 0.29 0 0 0</pose>
-        <attenuation>
-          <range>25</range>
-          <linear>0</linear>
-          <constant>0.1</constant>
-          <quadratic>0.005</quadratic>
-        </attenuation>
-        <diffuse>0.8 0.8 0.5 1.0</diffuse>
-        <specular>0.8 0.8 0.5 1</specular>
-        <spot>
-          <inner_angle>1.571</inner_angle>
-          <outer_angle>2.1</outer_angle>
-          <falloff>1</falloff>
-        </spot>
-        <direction>1 0 0</direction>
-        <cast_shadows>1</cast_shadows>
-      </light>
-      <!--SICK TIM881P lidar, a prototype without a good public URL. It is derived from
-            the TIM58x family:
-            https://www.sick.com/ch/en/detection-and-ranging-solutions/2d-lidar-sensors/tim5xx/tim581-2050101/p/p619344
-        -->
-      <visual name="visual_lidar_front">
-        <pose>0.015 0 0.18 0 0 0</pose>
-        <geometry>
-          <mesh>
-            <uri>meshes/lidar.dae</uri>
-          </mesh>
-        </geometry>
-      </visual>
-      <sensor name="lidar_front" type="gpu_lidar">
-        <pose>0.04 0 0.235 0 0 0</pose>
-        <update_rate>15</update_rate>
-        <lidar>
-          <scan>
-            <horizontal>
-              <samples>811</samples>
-              <resolution>1</resolution>
-              <min_angle>-2.3562</min_angle>
-              <max_angle>2.3562</max_angle>
-            </horizontal>
-          </scan>
-          <range>
-            <min>0.04</min>
-            <max>25</max>
-            <resolution>0.01</resolution>
-          </range>
-          <noise>
-            <type>gaussian</type>
-            <mean>0</mean>
-            <stddev>0.01</stddev>
-          </noise>
-        </lidar>
-      </sensor>
-      <!--Camera Arecont AV3216DN and lens MPL1.55
-            https://sales.arecontvision.com/product/MegaVideo%20G5%20Series/AV3216DN
-            https://sales.arecontvision.com/product/Lenses/MPL1.55
-        -->
-      <visual name="visual_camera_front">
-        <pose>0.114 0 0.16 0 0 0</pose>
-        <geometry>
-          <mesh>
-            <uri>meshes/camera.dae</uri>
-          </mesh>
-        </geometry>
-      </visual>
-      <sensor name="camera_front" type="camera">
-        <pose>0.15 0 0.192 0 0 0</pose>
-        <always_on>1</always_on>
-        <update_rate>10</update_rate>
-        <camera name="camera_front">
-          <horizontal_fov>3.072</horizontal_fov>
-          <lens>
-            <intrinsics>
-              <!-- fx = fy = width / ( 2 * tan (hfov / 2 ) ) -->
-              <fx>17.8229</fx>
-              <fy>17.8229</fy>
-              <!-- cx = ( width - 1 ) / 2 -->
-              <cx>511.5</cx>
-              <!-- cy = ( height - 1 ) / 2 -->
-              <cy>383.5</cy>
-              <s>0</s>
-            </intrinsics>
-          </lens>
-          <distortion>
-            <k1>0.0</k1>
-            <k2>0.0</k2>
-            <k3>0.0</k3>
-            <p1>0.0</p1>
-            <p2>0.0</p2>
-            <center>0.5 0.5</center>
-          </distortion>
-          <image>
-            <width>1024</width>
-            <height>768</height>
-            <format>R8G8B8</format>
-          </image>
-          <clip>
-            <near>0.01</near>
-            <far>300</far>
-          </clip>
-          <noise>
-            <type>gaussian</type>
-            <mean>0</mean>
-            <stddev>0.007</stddev>
-          </noise>
-        </camera>
-      </sensor>
-      <!-- RealSense depth camera D435i
-            https://www.intelrealsense.com/depth-camera-d435i/
-        -->
-      <collision name="collision_depth_camera_front">
-        <pose>0.165 0 0.11 0 0 0</pose>
-        <geometry>
-          <box>
-            <size>0.03 0.2 0.06</size>
-          </box>
-        </geometry>
-      </collision>
-      <visual name="visual_depth_camera_shield_front">
-        <pose>0.15 0 0.11 0 0 0</pose>
-        <geometry>
-          <mesh>
-            <uri>meshes/depth_camera_shield.dae</uri>
-          </mesh>
-        </geometry>
-      </visual>
-      <visual name="visual_depth_camera_front">
-        <pose>0.15 0 0.113 0 0 0</pose>
-        <geometry>
-          <mesh>
-            <uri>meshes/depth_camera.dae</uri>
-          </mesh>
-        </geometry>
-      </visual>
-      <sensor name="depth_camera_front" type="rgbd_camera">
-        <pose>0.18 0 0.113 0 0 0</pose>
-        <always_on>1</always_on>
-        <update_rate>20</update_rate>
-        <camera name="depth_camera_front">
-          <pose frame="">0 0 0 0 -1.5707 1.5707</pose>
-          <horizontal_fov>1.5184</horizontal_fov>
-          <lens>
-            <intrinsics>
-              <!-- fx = fy = width / ( 2 * tan (hfov / 2 ) ) -->
-              <fx>337.22</fx>
-              <fy>337.22</fy>
-              <!-- cx = ( width - 1 ) / 2 -->
-              <cx>319.5</cx>
-              <!-- cy = ( height - 1 ) / 2 -->
-              <cy>179.5</cy>
-              <s>0</s>
-            </intrinsics>
-          </lens>
-          <distortion>
-            <k1>0.0</k1>
-            <k2>0.0</k2>
-            <k3>0.0</k3>
-            <p1>0.0</p1>
-            <p2>0.0</p2>
-            <center>0.5 0.5</center>
-          </distortion>
-          <image>
-            <width>640</width>
-            <height>360</height>
-            <format>R8G8B8</format>
-          </image>
-          <clip>
-            <near>0.01</near>
-            <far>300</far>
-          </clip>
-          <depth_camera>
-            <clip>
-              <near>0.1</near>
-              <far>10</far>
-            </clip>
-          </depth_camera>
-          <noise>
-            <type>gaussian</type>
-            <mean>0</mean>
-            <stddev>0.007</stddev>
-          </noise>
-        </camera>
-      </sensor>
-    </link>
-    <link name="chassis_back">
-      <pose>-0.7 0 0.2 0 0 0</pose>
-      <inertial>
-        <pose>0.025 0 0.116 0 0 0</pose>
-        <mass>7.2</mass>
-        <inertia>
-          <ixx>0.0468</ixx>
-          <iyy>0.1117</iyy>
-          <izz>0.1228</izz>
-        </inertia>
-      </inertial>
-      <collision name="collision_back_box">
-        <pose>0 0 0.13 0 0 0</pose>
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
Commit message: Fix spawning
Signed-off-by: Nate Koenig <nate@openrobotics.org>

File: submitted_models/robotika_kloubak_sensor_config_1/urdf/model.xacro (robot description, xacro)
@@ -3,5 +3,4 @@
   <xacro:arg name="name" default="robotika_kloubak_sensor_config_1"/>
   <xacro:property name="robot_namespace" value="$(arg name)"/>
-  <link name='${robot_namespace}/base_link'/>
   <link name='${robot_namespace}/chassis_front'>
     <inertial>
