Commit message: Updates based on review

File: teambase_description/urdf/teambase.xacro (robot description, xacro)
@@ -2,5 +2,5 @@
 <robot name="TeamBase" xmlns:xacro="http://ros.org/wiki/xacro">
   <xacro:property name="robot_namespace" value="TeamBase"/>
-  <link name='${robot_namespace}/base_link'>
+  <link name='${robot_namespace}/link'>
    <visual name='visual'>
       <origin xyz='0 0 0.05' rpy='0 0 0'/>

Commit message: Allow a custom name to be used for the teambase, and handle different capitalization for teambase config
Signed-off-by: Nate Koenig <nate@openrobotics.org>

File: teambase_description/urdf/teambase.xacro (robot description, xacro)
@@ -1,5 +1,6 @@
 <?xml version='1.0' encoding='utf-8'?>
 <robot name="TeamBase" xmlns:xacro="http://ros.org/wiki/xacro">
-  <xacro:property name="robot_namespace" value="TeamBase"/>
+  <xacro:arg name="name" default="TeamBase"/>
+  <xacro:property name="robot_namespace" value="$(arg name)"/>
   <link name='${robot_namespace}/link'>
    <visual name='visual'>
