Commit message: Submitted models/explorer ds1 sensor config1 (#492)
* add spinning rotors and propoller. change weight and specifications. add light mesh

* add spinning rotors and propoller. change weight and specifications. add light mesh

Co-authored-by: Hong <hongbiaz@andrew.cmu.edu>

File: submitted_models/explorer_ds1_sensor_config_1/urdf/model.orig.xacro (robot description, xacro)
@@ -3,7 +3,5 @@
   <xacro:arg name="name" default="ds1"/>
   <xacro:property name="name" value="$(arg name)"/>
-  <xacro:property name="name" value="$(arg name)"/>
-  <xacro:property name="robot_namespace" value="$(arg name)"/>
-  <link name='${robot_namespace}/base_link'>
+  <link name='${name}/base_link'>
     <inertial>
       <origin xyz='0 0 0' rpy='0 -0 0'/>
@@ -14,8 +12,5 @@
       <origin xyz='0 0 0' rpy='0 -0 0'/>
       <geometry>
-        <!-- <mesh filename='package://explorer_ds1_sensor_config_1/meshes/DS1_COLLISION.STL' scale='1 1 1'/> -->
-        <box>
-            <size>0.47 0.47 0.11</size>
-        </box>
+        <mesh filename='package://explorer_ds1_sensor_config_1/meshes/DS1_COLLISION.STL' scale='1 1 1'/>
       </geometry>
     </collision>
@@ -23,10 +18,10 @@
       <origin xyz='0 0 0' rpy='0 -0 0'/>
       <geometry>
-        <mesh filename='package://explorer_ds1_sensor_config_1/meshes/DS1.STL' scale='1 1 1'/>
+        <mesh filename='package://explorer_ds1_sensor_config_1/meshes/DS1.dae' scale='1 1 1'/>
       </geometry>
     </visual>
     <!-- camera_visual -->
     <visual name='rs_up_visual'>
-      <origin xyz='0.305 0 0.11' rpy='0 -1.57079632679 0'/>
+      <origin xyz='0.305 0 0.11' rpy='-1.57079632679 0 1.57079632679'/>
       <geometry>
         <mesh filename='package://explorer_ds1_sensor_config_1/meshes/realsense.dae' scale='1 1 1'/>
@@ -34,5 +29,5 @@
     </visual>
     <visual name='rs_down_visual'>
-      <origin xyz='0.305 0 0.03' rpy='0 1.57079632679 0'/>
+      <origin xyz='0.305 0 0.03' rpy='1.57079632679 0 1.57079632679'/>
       <geometry>
         <mesh filename='package://explorer_ds1_sensor_config_1/meshes/realsense.dae' scale='1 1 1'/>
@@ -40,5 +35,5 @@
     </visual>
     <visual name='rs_front_visual'>
-      <origin xyz='0.325 0 0.07' rpy='0 -0 0'/>
+      <origin xyz='0.325 0 0.07' rpy='0 -0 1.57079632679'/>
       <geometry>
         <mesh filename='package://explorer_ds1_sensor_config_1/meshes/realsense.dae' scale='1 1 1'/>
@@ -59,5 +54,5 @@
     </visual>
     <visual name='laser_visual_scan'>
-      <origin xyz='0.18 0 0.1523' rpy='0 -0 0'/>
+      <origin xyz='0.18 0 0.19' rpy='0 -0 0'/>
       <geometry>
         <mesh filename="package://explorer_ds1_sensor_config_1/meshes/VLP16_scan.dae" />
@@ -102,5 +97,5 @@
     <origin xyz='0.18 0 0.284' rpy='0 -0 0'/>
   </sensor>
-  <link name='${robot_namespace}/rotor_0'>
+  <link name='${name}/rotor_0'>
     <inertial>
       <origin xyz='0 0 0' rpy='0 -0 0'/>
@@ -108,18 +103,12 @@
       <inertia ixx='9.75e-07' ixy='0' ixz='0' iyy='4.17041e-05' iyz='0' izz='4.26041e-05'/>
     </inertial>
-    <collision name='rotor_0_collision'>
-      <origin xyz='0 0 0' rpy='0 -0 0'/>
-      <geometry>
-        <cylinder radius='0.1' length='0.005'/>
-      </geometry>
-    </collision>
     <visual name='rotor_0_visual'>
       <origin xyz='0 0 0' rpy='0 -0 0'/>
       <geometry>
-        <mesh filename='package://explorer_ds1_sensor_config_1/meshes/propeller_ccw.dae' scale='0.1 0.1 0.1'/>
+        <mesh filename='package://explorer_ds1_sensor_config_1/meshes/propeller_ccw.dae' scale='0.12 0.12 0.12'/>
       </geometry>
     </visual>
   </link>
-  <link name='${robot_namespace}/rotor_1'>
+  <link name='${name}/rotor_1'>
     <inertial>
       <origin xyz='0 0 0' rpy='0 -0 0'/>
@@ -127,18 +116,12 @@
       <inertia ixx='9.75e-07' ixy='0' ixz='0' iyy='4.17041e-05' iyz='0' izz='4.26041e-05'/>
     </inertial>
-    <collision name='rotor_1_collision'>
-      <origin xyz='0 0 0' rpy='0 -0 0'/>
-      <geometry>
-        <cylinder radius='0.1' length='0.005'/>
-      </geometry>
-    </collision>
     <visual name='rotor_1_visual'>
       <origin xyz='0 0 0' rpy='0 -0 0'/>
       <geometry>
-        <mesh filename='package://explorer_ds1_sensor_config_1/meshes/propeller_ccw.dae' scale='0.1 0.1 0.1'/>
+        <mesh filename='package://explorer_ds1_sensor_config_1/meshes/propeller_ccw.dae' scale='0.12 0.12 0.12'/>
       </geometry>
     </visual>
   </link>
-  <link name='${robot_namespace}/rotor_2'>
+  <link name='${name}/rotor_2'>
     <inertial>
       <origin xyz='0 0 0' rpy='0 -0 0'/>
@@ -146,18 +129,12 @@
       <inertia ixx='9.75e-07' ixy='0' ixz='0' iyy='4.17041e-05' iyz='0' izz='4.26041e-05'/>
     </inertial>
-    <collision name='rotor_2_collision'>
-      <origin xyz='0 0 0' rpy='0 -0 0'/>
-      <geometry>
-        <cylinder radius='0.1' length='0.005'/>
-      </geometry>
-    </collision>
     <visual name='rotor_2_visual'>
       <origin xyz='0 0 0' rpy='0 -0 0'/>
       <geometry>
-        <mesh filename='package://explorer_ds1_sensor_config_1/meshes/propeller_cw.dae' scale='0.1 0.1 0.1'/>
+        <mesh filename='package://explorer_ds1_sensor_config_1/meshes/propeller_cw.dae' scale='0.12 0.12 0.12'/>
       </geometry>
     </visual>
   </link>
-  <link name='${robot_namespace}/rotor_3'>
+  <link name='${name}/rotor_3'>
     <inertial>
       <origin xyz='0 0 0' rpy='0 -0 0'/>
@@ -165,21 +142,15 @@
       <inertia ixx='9.75e-07' ixy='0' ixz='0' iyy='4.17041e-05' iyz='0' izz='4.26041e-05'/>
     </inertial>
-    <collision name='rotor_3_collision'>
-      <origin xyz='0 0 0' rpy='0 -0 0'/>
-      <geometry>
-        <cylinder radius='0.1' length='0.005'/>
-      </geometry>
-    </collision>
     <visual name='rotor_3_visual'>
       <origin xyz='0 0 0' rpy='0 -0 0'/>
       <geometry>
-        <mesh filename='package://explorer_ds1_sensor_config_1/meshes/propeller_cw.dae' scale='0.1 0.1 0.1'/>
+        <mesh filename='package://explorer_ds1_sensor_config_1/meshes/propeller_cw.dae' scale='0.12 0.12 0.12'/>
       </geometry>
     </visual>
   </link>
   <joint name='rotor_0_joint' type='revolute'>
-    <origin xyz='0.13 -0.22 0.023' rpy='0 -0 0'/>
-    <parent link='${robot_namespace}/base_link'/>
-    <child link='${robot_namespace}/rotor_0'/>
+    <origin xyz='0.1644 -0.166 0.023' rpy='0 -0 0'/>
+    <parent link='${name}/base_link'/>
+    <child link='${name}/rotor_0'/>
     <dynamics damping='0' friction='0' />
     <axis xyz='0 0 1'/>
@@ -187,7 +158,7 @@
   </joint>
   <joint name='rotor_1_joint' type='revolute'>
-    <origin xyz='-0.13 0.2 0.023' rpy='0 -0 0'/>
-    <parent link='${robot_namespace}/base_link'/>
-    <child link='${robot_namespace}/rotor_1'/>
+    <origin xyz='-0.16443 0.1661 0.023' rpy='0 -0 0'/>
+    <parent link='${name}/base_link'/>
+    <child link='${name}/rotor_1'/>
     <dynamics damping='0' friction='0' />
     <axis xyz='0 0 1'/>
@@ -195,7 +166,7 @@
   </joint>
   <joint name='rotor_2_joint' type='revolute'>
-    <origin xyz='0.13 0.22 0.023' rpy='0 -0 0'/>
-    <parent link='${robot_namespace}/base_link'/>
-    <child link='${robot_namespace}/rotor_2'/>
+    <origin xyz='0.16443 0.1661 0.023' rpy='0 -0 0'/>
+    <parent link='${name}/base_link'/>
+    <child link='${name}/rotor_2'/>
     <dynamics damping='0' friction='0' />
     <axis xyz='0 0 1'/>
@@ -203,7 +174,7 @@
   </joint>
   <joint name='rotor_3_joint' type='revolute'>
-    <origin xyz='-0.13 -0.2 0.023' rpy='0 -0 0'/>
-    <parent link='${robot_namespace}/base_link'/>
-    <child link='${robot_namespace}/rotor_3'/>
+    <origin xyz='-0.16443 -0.1661 0.023' rpy='0 -0 0'/>
+    <parent link='${name}/base_link'/>
+    <child link='${name}/rotor_3'/>
     <dynamics damping='0' friction='0' />
     <axis xyz='0 0 1'/>
