Commit message: Fixed realsense, omnicam, lights and mass properties.

File: submitted_models/ctu_cras_norlab_absolem_sensor_config_1/urdf/_d435.xacro (robot description, xacro)
@@ -44,13 +44,16 @@
         </joint>
         <link name="$(arg prefix)${name}_link">
-            <visual>
-                <origin xyz="${d435_cam_mount_from_center_offset} ${-d435_cam_depth_py} 0" rpy="${M_PI/2} 0 ${M_PI/2}"/>
-                <geometry>
-                    <!-- <box size="${d435_cam_width} ${d435_cam_height} ${d435_cam_depth}"/> -->
-                    <mesh filename="package://ctu_cras_norlab_absolem_sensor_config_1/meshes/realsense_d435.dae" />
-                    <!--<mesh filename="package://realsense2_description/meshes/d435/d435.dae" />-->
-                </geometry>
-                <material name="${name}_aluminum"/>
-            </visual>
+            <!-- For some reason, Gazebo sees the camera itself, which is bad... -->
+            <xacro:if value="${'$(arg rendering_target)' == 'urdf'}">
+                <visual>
+                    <origin xyz="${d435_cam_mount_from_center_offset} ${-d435_cam_depth_py} 0" rpy="${M_PI/2} 0 ${M_PI/2}"/>
+                    <geometry>
+                        <!-- <box size="${d435_cam_width} ${d435_cam_height} ${d435_cam_depth}"/> -->
+                        <mesh filename="package://ctu_cras_norlab_absolem_sensor_config_1/meshes/realsense_d435.dae" />
+                        <!--<mesh filename="package://realsense2_description/meshes/d435/d435.dae" />-->
+                    </geometry>
+                    <material name="${name}_aluminum"/>
+                </visual>
+            </xacro:if>
             <collision>
                 <origin xyz="0 ${-d435_cam_depth_py} 0" rpy="0 0 0"/>

File: submitted_models/ctu_cras_norlab_absolem_sensor_config_1/urdf/nifti_robot.xacro (robot description, xacro)
@@ -270,7 +270,7 @@
 	<!-- MEASURED CONSTANTS -->
 	<xacro:property name="body_scale" value="1.0" />
-	<xacro:property name="body_mass" value="6.746" />
+	<xacro:property name="body_mass" value="16.0" />
 	<xacro:property name="battery_scale" value="1.0" />
-	<xacro:property name="battery_mass" value="3.18" />
+	<xacro:property name="battery_mass" value="2.7" />
 	<xacro:property name="top_box_scale" value="1.0" />
 	<xacro:property name="top_box_mass" value="0.24" />
@@ -986,4 +986,6 @@
 			<xacro:calibrated_fixed_joint name="camera_5_j" parent="omnicam" child="camera_5" />
 			<xacro:if value="$(arg has_omnicam_sensor_mount)">
+				<!-- For some reason, the mount is visible in simulated cameras, so we hide it in Gazebo. -->
+				<xacro:if value="${'$(arg rendering_target)' == 'urdf'}">
 					<link name="$(arg prefix)omnicam_sensor_mount">
 							<visual>
@@ -1014,4 +1016,8 @@
 							</collision>
 					</link>
+				</xacro:if>
+				<xacro:unless value="${'$(arg rendering_target)' == 'urdf'}">
+					<xacro:empty_link name="$(arg prefix)omnicam_sensor_mount" />
+				</xacro:unless>
 					<joint name="omnicam_sensor_mount_j" type="fixed">
 							<child link="$(arg prefix)omnicam_sensor_mount"/>
@@ -1199,5 +1205,11 @@
     <xacro:macro name="omnicam_camera" params="num name">
 				<xacro:empty_link name="$(arg prefix)${name}_sim" />
-				<xacro:fixed_joint name="${name}_sim_j" parent="${name}" child="${name}_sim" rpy="1.5707963267948966 0 0" />
+				<xacro:if value="${num != 5}">
+					<xacro:property name="rpy" value="${pi/2} 0 0" />
+				</xacro:if>
+				<xacro:if value="${num == 5}">
+					<xacro:property name="rpy" value="0 ${-pi/2} 0" />
+				</xacro:if>
+				<xacro:fixed_joint name="${name}_sim_j" parent="${name}" child="${name}_sim" rpy="${rpy}" />
 				<gazebo reference="$(arg prefix)${name}_sim">
 					<sensor name="omnicam_sensor${num}" type="camera">
@@ -1317,5 +1329,39 @@
 		<gazebo reference="$(arg prefix)base_link">
 			<light name="light_left" type="spot">
-				<pose>0 0.13 0.1 0 0 0</pose>
+				<pose>0 0.13 0.2 ${pi/2} ${pi/2} 0</pose>
+				<attenuation>
+					<range>50</range>
+					<linear>0</linear>
+					<constant>0.1</constant>
+					<quadratic>0.0025</quadratic>
+				</attenuation>
+				<diffuse>0.8 0.8 0.5 1</diffuse>
+				<specular>0.8 0.8 0.5 1</specular>
+				<spot>
+					<inner_angle>2.8</inner_angle>
+					<outer_angle>2.9</outer_angle>
+					<falloff>1</falloff>
+				</spot>
+				<direction>1 0 0</direction>
+			</light>
+			<light name="light_right" type="spot">
+				<pose>0 -0.13 0.2 ${3*pi/2} ${pi/2} 0</pose>
+				<attenuation>
+					<range>50</range>
+					<linear>0</linear>
+					<constant>0.1</constant>
+					<quadratic>0.0025</quadratic>
+				</attenuation>
+				<diffuse>0.8 0.8 0.5 1</diffuse>
+				<specular>0.8 0.8 0.5 1</specular>
+				<spot>
+					<inner_angle>2.8</inner_angle>
+					<outer_angle>2.9</outer_angle>
+					<falloff>1</falloff>
+				</spot>
+				<direction>1 0 0</direction>
+			</light>
+			<light name="light_front_left" type="spot">
+				<pose>0.3 0.13 0.2 ${7*pi/8} ${pi/2} 0</pose>
 				<attenuation>
 					<range>30</range>
@@ -1327,12 +1373,12 @@
 				<specular>0.8 0.8 0.5 1</specular>
 				<spot>
-					<inner_angle>2.8</inner_angle>
-					<outer_angle>2.9</outer_angle>
+					<inner_angle>1.5</inner_angle>
+					<outer_angle>1.6</outer_angle>
 					<falloff>1</falloff>
 				</spot>
-				<direction>0 1 0</direction>
+				<direction>1 0 0</direction>
 			</light>
-			<light name="light_right" type="spot">
-				<pose>0 -0.13 0.1 0 0 0</pose>
+			<light name="light_front_right" type="spot">
+				<pose>0.3 -0.13 0.2 ${9*pi/8} ${pi/2} 0</pose>
 				<attenuation>
 					<range>30</range>
@@ -1344,12 +1390,12 @@
 				<specular>0.8 0.8 0.5 1</specular>
 				<spot>
-					<inner_angle>2.8</inner_angle>
-					<outer_angle>2.9</outer_angle>
+					<inner_angle>1.5</inner_angle>
+					<outer_angle>1.6</outer_angle>
 					<falloff>1</falloff>
 				</spot>
-				<direction>0 -1 0</direction>
+				<direction>1 0 0</direction>
 			</light>
-			<light name="light_front_left" type="spot">
-				<pose>0.3 0.13 0.1 0 0 0</pose>
+			<light name="light_rear" type="spot">
+				<pose>-0.4 0 0.2 0 ${pi/2} 0</pose>
 				<attenuation>
 					<range>30</range>
@@ -1361,43 +1407,9 @@
 				<specular>0.8 0.8 0.5 1</specular>
 				<spot>
-					<inner_angle>2.8</inner_angle>
-					<outer_angle>2.9</outer_angle>
+					<inner_angle>1.5</inner_angle>
+					<outer_angle>1.8</outer_angle>
 					<falloff>1</falloff>
 				</spot>
-				<direction>1 1 0</direction>
-			</light>
-			<light name="light_front_right" type="spot">
-				<pose>0.3 -0.13 0.1 0 0 0</pose>
-				<attenuation>
-					<range>30</range>
-					<linear>0</linear>
-					<constant>0.2</constant>
-					<quadratic>0.0025</quadratic>
-				</attenuation>
-				<diffuse>0.8 0.8 0.5 1</diffuse>
-				<specular>0.8 0.8 0.5 1</specular>
-				<spot>
-					<inner_angle>2.8</inner_angle>
-					<outer_angle>2.9</outer_angle>
-					<falloff>1</falloff>
-				</spot>
-				<direction>1 -1 0</direction>
-			</light>
-			<light name="light_rear" type="spot">
-				<pose>-0.2 0 0.1 0 0 0</pose>
-				<attenuation>
-					<range>30</range>
-					<linear>0</linear>
-					<constant>0.2</constant>
-					<quadratic>0.0025</quadratic>
-				</attenuation>
-				<diffuse>0.8 0.8 0.5 1</diffuse>
-				<specular>0.8 0.8 0.5 1</specular>
-				<spot>
-					<inner_angle>2.8</inner_angle>
-					<outer_angle>2.9</outer_angle>
-					<falloff>1</falloff>
-				</spot>
-				<direction>-1 0 0</direction>
+				<direction>1 0 0</direction>
 			</light>
 		</gazebo>

Commit message: Absolem: Fixed track properties and realsense visuals and pose.

File: submitted_models/ctu_cras_norlab_absolem_sensor_config_1/urdf/_d435.xacro (robot description, xacro)
@@ -45,15 +45,13 @@
         <link name="$(arg prefix)${name}_link">
             <!-- For some reason, Gazebo sees the camera itself, which is bad... -->
-            <xacro:if value="${'$(arg rendering_target)' == 'urdf'}">
-                <visual>
-                    <origin xyz="${d435_cam_mount_from_center_offset} ${-d435_cam_depth_py} 0" rpy="${M_PI/2} 0 ${M_PI/2}"/>
-                    <geometry>
-                        <!-- <box size="${d435_cam_width} ${d435_cam_height} ${d435_cam_depth}"/> -->
-                        <mesh filename="package://ctu_cras_norlab_absolem_sensor_config_1/meshes/realsense_d435.dae" />
-                        <!--<mesh filename="package://realsense2_description/meshes/d435/d435.dae" />-->
-                    </geometry>
-                    <material name="${name}_aluminum"/>
-                </visual>
-            </xacro:if>
+            <visual>
+                <origin xyz="${d435_cam_mount_from_center_offset} ${-d435_cam_depth_py} 0" rpy="${M_PI/2} 0 ${M_PI/2}"/>
+                <geometry>
+                    <!-- <box size="${d435_cam_width} ${d435_cam_height} ${d435_cam_depth}"/> -->
+                    <mesh filename="package://ctu_cras_norlab_absolem_sensor_config_1/meshes/realsense_d435.dae" />
+                    <!--<mesh filename="package://realsense2_description/meshes/d435/d435.dae" />-->
+                </geometry>
+                <material name="${name}_aluminum"/>
+            </visual>
             <collision>
                 <origin xyz="0 ${-d435_cam_depth_py} 0" rpy="0 0 0"/>

File: submitted_models/ctu_cras_norlab_absolem_sensor_config_1/urdf/nifti_robot.xacro (robot description, xacro)
@@ -804,5 +804,5 @@
 	<xacro:macro name="flipper_fake_wheel" params="prefix1 prefix2 reflect_y do_inward_enlargement num_wheels wheel_num">
 			<link name="$(arg prefix)${prefix1}_${prefix2}_flipper_wheel${wheel_num}">
-					<collision name="${prefix1}_${prefix2}_flipper_collision_wheel${wheel_num}">
+					<collision name="${prefix1}_${prefix2}_flipper_wheel${wheel_num}_collision">
 							<origin rpy="${pi/2} 0 0" xyz="0 0 0"/>
 							<geometry>
@@ -1070,18 +1070,23 @@
         <kinematic>false</kinematic>
     </xacro:macro>
-    <xacro:macro name="gazebo_flipper_tags">
-        <selfCollide>true</selfCollide>
-    </xacro:macro>
     <xacro:macro name="track_base_surface">
         <surface>
-            <friction>
-                <ode>
-                    <mu>$(arg track_mu)</mu>
-                    <mu2>$(arg track_mu2)</mu2>
-                    <fdir1>0 1 0</fdir1> <!-- is overridden by the plugin -->
-                </ode>
-            </friction>
+			<contact>
+				<ode>
+					<kp>1e+07</kp>
+					<kd>1</kd>
+				</ode>
+			</contact>
+			<friction>
+				<ode>
+					<mu>$(arg track_mu)</mu>
+					<mu2>$(arg track_mu2)</mu2>
+					<slip1>0.035</slip1>
+					<slip2>0</slip2>
+					<fdir1>0 0 1</fdir1>
+				</ode>
+			</friction>
         </surface>
-        <max_contacts>20</max_contacts>
+<!--        <max_contacts>20</max_contacts>-->
     </xacro:macro>
     <xacro:macro name="flipper_surface">
@@ -1089,51 +1094,62 @@
     <xacro:macro name="track_surface">
     </xacro:macro>
-    <gazebo reference="$(arg prefix)left_track">
+	<xacro:macro name="gazebo_track_tags">
 		<xacro:gazebo_default_tags />
-        <collision>
-            <xacro:track_base_surface />
-            <xacro:track_surface />
-        </collision>
-	</gazebo>
-    <gazebo reference="$(arg prefix)right_track">
+		<collision>
+			<xacro:track_base_surface />
+			<xacro:track_surface />
+		</collision>
+	</xacro:macro>
+	<xacro:macro name="gazebo_flipper_tags">
 		<xacro:gazebo_default_tags />
-        <collision>
-            <xacro:track_base_surface />
-            <xacro:track_surface />
-        </collision>
-    </gazebo>
+		<selfCollide>true</selfCollide>
+		<collision>
+			<xacro:track_base_surface />
+			<xacro:flipper_surface />
+		</collision>
+	</xacro:macro>
+    <gazebo reference="$(arg prefix)left_track"><xacro:gazebo_track_tags /></gazebo>
+    <gazebo reference="$(arg prefix)right_track"><xacro:gazebo_track_tags /></gazebo>
+    <gazebo reference="$(arg prefix)left_track_wheel1"><xacro:gazebo_track_tags /></gazebo>
+    <gazebo reference="$(arg prefix)right_track_wheel1"><xacro:gazebo_track_tags /></gazebo>
+    <gazebo reference="$(arg prefix)left_track_wheel2"><xacro:gazebo_track_tags /></gazebo>
+    <gazebo reference="$(arg prefix)right_track_wheel2"><xacro:gazebo_track_tags /></gazebo>
+    <gazebo reference="$(arg prefix)left_track_wheel3"><xacro:gazebo_track_tags /></gazebo>
+    <gazebo reference="$(arg prefix)right_track_wheel3"><xacro:gazebo_track_tags /></gazebo>
+    <gazebo reference="$(arg prefix)left_track_wheel4"><xacro:gazebo_track_tags /></gazebo>
+    <gazebo reference="$(arg prefix)right_track_wheel4"><xacro:gazebo_track_tags /></gazebo>
+    <gazebo reference="$(arg prefix)left_track_wheel5"><xacro:gazebo_track_tags /></gazebo>
+    <gazebo reference="$(arg prefix)right_track_wheel5"><xacro:gazebo_track_tags /></gazebo>
+    <gazebo reference="$(arg prefix)left_track_wheel6"><xacro:gazebo_track_tags /></gazebo>
+    <gazebo reference="$(arg prefix)right_track_wheel6"><xacro:gazebo_track_tags /></gazebo>
+    <gazebo reference="$(arg prefix)left_track_wheel7"><xacro:gazebo_track_tags /></gazebo>
+    <gazebo reference="$(arg prefix)right_track_wheel7"><xacro:gazebo_track_tags /></gazebo>
+    <gazebo reference="$(arg prefix)left_track_wheel8"><xacro:gazebo_track_tags /></gazebo>
+    <gazebo reference="$(arg prefix)right_track_wheel8"><xacro:gazebo_track_tags /></gazebo>
     <xacro:if value="$(arg has_flippers)">
-        <gazebo reference="$(arg prefix)front_left_flipper">
-            <xacro:gazebo_default_tags />
-            <xacro:gazebo_flipper_tags />
-            <collision>
-                <xacro:track_base_surface />
-                <xacro:flipper_surface />
-            </collision>
-        </gazebo>
-        <gazebo reference="$(arg prefix)front_right_flipper">
-            <xacro:gazebo_default_tags />
-            <xacro:gazebo_flipper_tags />
-            <collision>
-                <xacro:track_base_surface />
-                <xacro:flipper_surface />
-            </collision>
-        </gazebo>
-        <gazebo reference="$(arg prefix)rear_left_flipper">
-            <xacro:gazebo_default_tags />
-            <xacro:gazebo_flipper_tags />
-            <collision>
-                <xacro:track_base_surface />
-                <xacro:flipper_surface />
-            </collision>
-        </gazebo>
-        <gazebo reference="$(arg prefix)rear_right_flipper">
-            <xacro:gazebo_default_tags />
-            <xacro:gazebo_flipper_tags />
-            <collision>
-                <xacro:track_base_surface />
-                <xacro:flipper_surface />
-            </collision>
-        </gazebo>
+        <gazebo reference="$(arg prefix)front_left_flipper"><xacro:gazebo_flipper_tags /></gazebo>
+        <gazebo reference="$(arg prefix)front_right_flipper"><xacro:gazebo_flipper_tags /></gazebo>
+        <gazebo reference="$(arg prefix)rear_left_flipper"><xacro:gazebo_flipper_tags /></gazebo>
+        <gazebo reference="$(arg prefix)rear_right_flipper"><xacro:gazebo_flipper_tags /></gazebo>
+        <gazebo reference="$(arg prefix)front_left_flipper_wheel1"><xacro:gazebo_flipper_tags /></gazebo>
+        <gazebo reference="$(arg prefix)front_right_flipper_wheel1"><xacro:gazebo_flipper_tags /></gazebo>
+        <gazebo reference="$(arg prefix)rear_left_flipper_wheel1"><xacro:gazebo_flipper_tags /></gazebo>
+        <gazebo reference="$(arg prefix)rear_right_flipper_wheel1"><xacro:gazebo_flipper_tags /></gazebo>
+        <gazebo reference="$(arg prefix)front_left_flipper_wheel2"><xacro:gazebo_flipper_tags /></gazebo>
+        <gazebo reference="$(arg prefix)front_right_flipper_wheel2"><xacro:gazebo_flipper_tags /></gazebo>
+        <gazebo reference="$(arg prefix)rear_left_flipper_wheel2"><xacro:gazebo_flipper_tags /></gazebo>
+        <gazebo reference="$(arg prefix)rear_right_flipper_wheel2"><xacro:gazebo_flipper_tags /></gazebo>
+        <gazebo reference="$(arg prefix)front_left_flipper_wheel3"><xacro:gazebo_flipper_tags /></gazebo>
+        <gazebo reference="$(arg prefix)front_right_flipper_wheel3"><xacro:gazebo_flipper_tags /></gazebo>
+        <gazebo reference="$(arg prefix)rear_left_flipper_wheel3"><xacro:gazebo_flipper_tags /></gazebo>
+        <gazebo reference="$(arg prefix)rear_right_flipper_wheel3"><xacro:gazebo_flipper_tags /></gazebo>
+        <gazebo reference="$(arg prefix)front_left_flipper_wheel4"><xacro:gazebo_flipper_tags /></gazebo>
+        <gazebo reference="$(arg prefix)front_right_flipper_wheel4"><xacro:gazebo_flipper_tags /></gazebo>
+        <gazebo reference="$(arg prefix)rear_left_flipper_wheel4"><xacro:gazebo_flipper_tags /></gazebo>
+        <gazebo reference="$(arg prefix)rear_right_flipper_wheel4"><xacro:gazebo_flipper_tags /></gazebo>
+        <gazebo reference="$(arg prefix)front_left_flipper_wheel5"><xacro:gazebo_flipper_tags /></gazebo>
+        <gazebo reference="$(arg prefix)front_right_flipper_wheel5"><xacro:gazebo_flipper_tags /></gazebo>
+        <gazebo reference="$(arg prefix)rear_left_flipper_wheel5"><xacro:gazebo_flipper_tags /></gazebo>
+        <gazebo reference="$(arg prefix)rear_right_flipper_wheel5"><xacro:gazebo_flipper_tags /></gazebo>
     </xacro:if>
     <xacro:if value="$(arg has_sick_lidar)">
@@ -1168,5 +1184,4 @@
 <!--                <time_increment>2.77777780866e-05</time_increment>-->
 <!--                <scan_time>0.019999999553</scan_time>-->
-<!--                <angle_increment>0.00872664619237</angle_increment>-->
                 </sensor>
             </xacro:if>

File: submitted_models/ctu_cras_norlab_absolem_sensor_config_1/urdf/realsense.gazebo.xacro (robot description, xacro)
@@ -37,10 +37,10 @@
             </image>
             <clip>
-              <near>0.01</near>
+              <near>0.1</near> <!-- not less, the image would be obstructed-->
               <far>100</far>
             </clip>
             <depth_camera>
               <clip>
-                <near>0.1</near>
+                <near>0.1</near> <!-- not less, the image would be obstructed-->
                 <far>10</far>
               </clip>
@@ -57,3 +57,19 @@
         </sensor>
     </gazebo>
+    <gazebo reference="$(arg prefix)realsense_holder_part2">
+      <visual>
+        <material>
+          <diffuse>.5 0.5 0.5 1</diffuse>
+          <ambient>.1 0.1 0.1 1</ambient>
+        </material>
+      </visual>
+    </gazebo>
+    <gazebo reference="$(arg prefix)$(arg realsense_name)_link">
+      <visual>
+        <material>
+          <diffuse>.5 0.5 0.5 1</diffuse>
+          <ambient>.1 0.1 0.1 1</ambient>
+        </material>
+      </visual>
+    </gazebo>
 </robot>

File: submitted_models/ctu_cras_norlab_absolem_sensor_config_1/urdf/realsense_d435_with_holder.xacro (robot description, xacro)
@@ -153,5 +153,5 @@
         <link name="$(arg prefix)realsense_holder_part2">
             <visual>
-                <origin rpy="-0.504467 0 1.5758" xyz="-0.002 -0.055 -0.051"/>
+                <origin rpy="-0.504467 0 1.5758" xyz="-0.002 -0.055 -0.0595"/>
                 <geometry>
                     <mesh scale="0.001 0.001 0.001"
