Commit message: Absolem: Synchronize Xacro and SDF files.

File: submitted_models/ctu_cras_norlab_absolem_sensor_config_1/urdf/_d435.xacro (robot description, xacro)
@@ -44,16 +44,18 @@
         </joint>
         <link name="$(arg prefix)${name}_link">
-            <!-- For some reason, Gazebo sees the camera itself, which is bad... -->
-            <xacro:if value="${'$(arg rendering_target)' == 'urdf'}">
-                <visual>
+            <visual>
+                <xacro:if value="${'$(arg rendering_target)' == 'sdf'}">
+                    <origin xyz="${d435_cam_mount_from_center_offset-0.001} ${-d435_cam_depth_py} -0.008" rpy="${M_PI/2} 0 ${M_PI/2}"/>
+                </xacro:if>
+                <xacro:unless value="${'$(arg rendering_target)' == 'sdf'}">
                     <origin xyz="${d435_cam_mount_from_center_offset} ${-d435_cam_depth_py} 0" rpy="${M_PI/2} 0 ${M_PI/2}"/>
-                    <geometry>
-                        <!-- <box size="${d435_cam_width} ${d435_cam_height} ${d435_cam_depth}"/> -->
-                        <mesh filename="package://ctu_cras_norlab_absolem_sensor_config_1/meshes/realsense_d435.dae" />
-                        <!--<mesh filename="package://realsense2_description/meshes/d435/d435.dae" />-->
-                    </geometry>
-                    <material name="${name}_aluminum"/>
-                </visual>
-            </xacro:if>
+                </xacro:unless>
+                <geometry>
+                    <!-- <box size="${d435_cam_width} ${d435_cam_height} ${d435_cam_depth}"/> -->
+                    <mesh filename="package://ctu_cras_norlab_absolem_sensor_config_1/meshes/realsense_d435.dae" />
+                    <!--<mesh filename="package://realsense2_description/meshes/d435/d435.dae" />-->
+                </geometry>
+                <material name="${name}_aluminum"/>
+            </visual>
             <collision>
                 <origin xyz="0 ${-d435_cam_depth_py} 0" rpy="0 0 0"/>

File: submitted_models/ctu_cras_norlab_absolem_sensor_config_1/urdf/nifti_robot.xacro (robot description, xacro)
@@ -804,5 +804,5 @@
 	<xacro:macro name="flipper_fake_wheel" params="prefix1 prefix2 reflect_y do_inward_enlargement num_wheels wheel_num">
 			<link name="$(arg prefix)${prefix1}_${prefix2}_flipper_wheel${wheel_num}">
-					<collision name="${prefix1}_${prefix2}_flipper_collision_wheel${wheel_num}">
+					<collision name="${prefix1}_${prefix2}_flipper_wheel${wheel_num}_collision">
 							<origin rpy="${pi/2} 0 0" xyz="0 0 0"/>
 							<geometry>
@@ -834,5 +834,5 @@
 			</xacro:if>
 			<xacro:unless value="${flipper_fixed}">
-					<joint name="${prefix1}_${prefix2}_flipper_j" type="continuous">
+					<joint name="${prefix1}_${prefix2}_flipper_j" type="revolute">
 							<xacro:flipper_joint_inner flipper_fixed="${flipper_fixed}" flipper_angle="${flipper_angle}" />
 					</joint>
@@ -848,5 +848,5 @@
 			</xacro:if>
 			<xacro:unless value="${flipper_fixed}">
-					<limit effort="50" velocity="${pi/4}" />
+					<limit lower="-1e+16" upper="1e+16" effort="20" velocity="${pi/4}" />
 			</xacro:unless>
 	</xacro:macro>
@@ -1031,37 +1031,17 @@
 						<plugin filename="libflipper_control_plugin.so" name="cras::FlipperControlPlugin">
 							<joint_name>front_left_flipper_j</joint_name>
+							<max_velocity>0.8</max_velocity>
 						</plugin>
-						<plugin filename="libignition-gazebo-joint-controller-system.so" name="ignition::gazebo::systems::JointController">
+						<plugin filename="libflipper_control_plugin.so" name="cras::FlipperControlPlugin">
 							<joint_name>front_right_flipper_j</joint_name>
-							<use_force_commands>true</use_force_commands>
-							<p_gain>30.0</p_gain>
-							<i_gain>0.1</i_gain>
-							<d_gain>0.01</d_gain>
-							<i_max>10</i_max>
-							<i_min>-10</i_min>
-							<cmd_max>100</cmd_max>
-							<cmd_min>-100</cmd_min>
+							<max_velocity>0.8</max_velocity>
 						</plugin>
-						<plugin filename="libignition-gazebo-joint-controller-system.so" name="ignition::gazebo::systems::JointController">
+						<plugin filename="libflipper_control_plugin.so" name="cras::FlipperControlPlugin">
 							<joint_name>rear_left_flipper_j</joint_name>
-							<use_force_commands>true</use_force_commands>
-							<p_gain>30.0</p_gain>
-							<i_gain>0.1</i_gain>
-							<d_gain>0.01</d_gain>
-							<i_max>10</i_max>
-							<i_min>-10</i_min>
-							<cmd_max>100</cmd_max>
-							<cmd_min>-100</cmd_min>
+							<max_velocity>0.8</max_velocity>
 						</plugin>
-						<plugin filename="libignition-gazebo-joint-controller-system.so" name="ignition::gazebo::systems::JointController">
+						<plugin filename="libflipper_control_plugin.so" name="cras::FlipperControlPlugin">
 							<joint_name>rear_right_flipper_j</joint_name>
-							<use_force_commands>true</use_force_commands>
-							<p_gain>30.0</p_gain>
-							<i_gain>0.1</i_gain>
-							<d_gain>0.01</d_gain>
-							<i_max>10</i_max>
-							<i_min>-10</i_min>
-							<cmd_max>100</cmd_max>
-							<cmd_min>-100</cmd_min>
+							<max_velocity>0.8</max_velocity>
 						</plugin>
         </xacro:if>
@@ -1074,6 +1054,6 @@
         </xacro:if>
 				<plugin filename="libignition-gazebo-joint-state-publisher-system.so" name="ignition::gazebo::systems::JointStatePublisher">
-					<joint_name>left_track_j</joint_name>
-					<joint_name>right_track_j</joint_name>
+					<!--joint_name>left_track_j</joint_name>
+					<joint_name>right_track_j</joint_name-->
 					<xacro:if value="$(arg has_flippers)">
 						<joint_name>front_left_flipper_j</joint_name>
@@ -1094,18 +1074,52 @@
         <kinematic>false</kinematic>
     </xacro:macro>
-    <xacro:macro name="gazebo_flipper_tags">
-        <selfCollide>true</selfCollide>
-    </xacro:macro>
     <xacro:macro name="track_base_surface">
         <surface>
-            <friction>
-                <ode>
-                    <mu>$(arg track_mu)</mu>
-                    <mu2>$(arg track_mu2)</mu2>
-                    <fdir1>0 1 0</fdir1> <!-- is overridden by the plugin -->
-                </ode>
-            </friction>
+			<friction>
+				<ode>
+					<mu>$(arg track_mu)</mu>
+					<mu2>$(arg track_mu2)</mu2>
+					<fdir1>0 0 1</fdir1>
+				</ode>
+			</friction>
         </surface>
-        <max_contacts>20</max_contacts>
+    </xacro:macro>
+    <xacro:macro name="track_wheel_surface">
+        <surface>
+			<contact>
+				<ode>
+					<kp>1e+07</kp>
+					<kd>1</kd>
+				</ode>
+			</contact>
+			<friction>
+				<ode>
+					<mu>1</mu>
+					<mu2>1</mu2>
+					<slip1>0.035</slip1>
+					<slip2>0</slip2>
+					<fdir1>0 0 1</fdir1>
+				</ode>
+			</friction>
+        </surface>
+    </xacro:macro>
+    <xacro:macro name="flipper_wheel_surface">
+        <surface>
+			<contact>
+				<ode>
+					<kp>1e+07</kp>
+					<kd>1</kd>
+				</ode>
+			</contact>
+			<friction>
+				<ode>
+					<mu>1</mu>
+					<mu2>1</mu2>
+					<slip1>0.035</slip1>
+					<slip2>0</slip2>
+					<fdir1>0 0 1</fdir1>
+				</ode>
+			</friction>
+        </surface>
     </xacro:macro>
     <xacro:macro name="flipper_surface">
@@ -1113,51 +1127,77 @@
     <xacro:macro name="track_surface">
     </xacro:macro>
-    <gazebo reference="$(arg prefix)left_track">
+	<xacro:macro name="gazebo_track_tags">
 		<xacro:gazebo_default_tags />
-        <collision>
-            <xacro:track_base_surface />
-            <xacro:track_surface />
-        </collision>
-	</gazebo>
-    <gazebo reference="$(arg prefix)right_track">
+		<collision>
+			<xacro:track_base_surface />
+			<xacro:track_surface />
+		</collision>
+	</xacro:macro>
+	<xacro:macro name="gazebo_track_wheel_tags">
 		<xacro:gazebo_default_tags />
-        <collision>
-            <xacro:track_base_surface />
-            <xacro:track_surface />
-        </collision>
-    </gazebo>
+		<collision>
+			<xacro:track_wheel_surface />
+			<xacro:track_surface />
+		</collision>
+	</xacro:macro>
+	<xacro:macro name="gazebo_flipper_tags">
+		<xacro:gazebo_default_tags />
+		<!--<selfCollide>true</selfCollide>-->
+		<collision>
+			<xacro:track_base_surface />
+			<xacro:flipper_surface />
+		</collision>
+	</xacro:macro>
+	<xacro:macro name="gazebo_flipper_wheel_tags">
+		<xacro:gazebo_default_tags />
+		<!--<selfCollide>true</selfCollide>-->
+		<collision>
+			<xacro:flipper_wheel_surface />
+			<xacro:flipper_surface />
+		</collision>
+	</xacro:macro>
+	<gazebo reference="$(arg prefix)left_track"><xacro:gazebo_track_tags /></gazebo>
+	<gazebo reference="$(arg prefix)right_track"><xacro:gazebo_track_tags /></gazebo>
+	<gazebo reference="$(arg prefix)left_track_wheel1"><xacro:gazebo_track_wheel_tags /></gazebo>
+	<gazebo reference="$(arg prefix)right_track_wheel1"><xacro:gazebo_track_wheel_tags /></gazebo>
+	<gazebo reference="$(arg prefix)left_track_wheel2"><xacro:gazebo_track_wheel_tags /></gazebo>
+	<gazebo reference="$(arg prefix)right_track_wheel2"><xacro:gazebo_track_wheel_tags /></gazebo>
+	<gazebo reference="$(arg prefix)left_track_wheel3"><xacro:gazebo_track_wheel_tags /></gazebo>
+	<gazebo reference="$(arg prefix)right_track_wheel3"><xacro:gazebo_track_wheel_tags /></gazebo>
+	<gazebo reference="$(arg prefix)left_track_wheel4"><xacro:gazebo_track_wheel_tags /></gazebo>
+	<gazebo reference="$(arg prefix)right_track_wheel4"><xacro:gazebo_track_wheel_tags /></gazebo>
+	<gazebo reference="$(arg prefix)left_track_wheel5"><xacro:gazebo_track_wheel_tags /></gazebo>
+	<gazebo reference="$(arg prefix)right_track_wheel5"><xacro:gazebo_track_wheel_tags /></gazebo>
+	<gazebo reference="$(arg prefix)left_track_wheel6"><xacro:gazebo_track_wheel_tags /></gazebo>
+	<gazebo reference="$(arg prefix)right_track_wheel6"><xacro:gazebo_track_wheel_tags /></gazebo>
+	<gazebo reference="$(arg prefix)left_track_wheel7"><xacro:gazebo_track_wheel_tags /></gazebo>
+	<gazebo reference="$(arg prefix)right_track_wheel7"><xacro:gazebo_track_wheel_tags /></gazebo>
+	<gazebo reference="$(arg prefix)left_track_wheel8"><xacro:gazebo_track_wheel_tags /></gazebo>
+	<gazebo reference="$(arg prefix)right_track_wheel8"><xacro:gazebo_track_wheel_tags /></gazebo>
     <xacro:if value="$(arg has_flippers)">
-        <gazebo reference="$(arg prefix)front_left_flipper">
-            <xacro:gazebo_default_tags />
-            <xacro:gazebo_flipper_tags />
-            <collision>
-                <xacro:track_base_surface />
-                <xacro:flipper_surface />
-            </collision>
-        </gazebo>
-        <gazebo reference="$(arg prefix)front_right_flipper">
-            <xacro:gazebo_default_tags />
-            <xacro:gazebo_flipper_tags />
-            <collision>
-                <xacro:track_base_surface />
-                <xacro:flipper_surface />
-            </collision>
-        </gazebo>
-        <gazebo reference="$(arg prefix)rear_left_flipper">
-            <xacro:gazebo_default_tags />
-            <xacro:gazebo_flipper_tags />
-            <collision>
-                <xacro:track_base_surface />
-                <xacro:flipper_surface />
-            </collision>
-        </gazebo>
-        <gazebo reference="$(arg prefix)rear_right_flipper">
-            <xacro:gazebo_default_tags />
-            <xacro:gazebo_flipper_tags />
-            <collision>
-                <xacro:track_base_surface />
-                <xacro:flipper_surface />
-            </collision>
-        </gazebo>
+		<gazebo reference="$(arg prefix)front_left_flipper"><xacro:gazebo_flipper_tags /></gazebo>
+		<gazebo reference="$(arg prefix)front_right_flipper"><xacro:gazebo_flipper_tags /></gazebo>
+		<gazebo reference="$(arg prefix)rear_left_flipper"><xacro:gazebo_flipper_tags /></gazebo>
+		<gazebo reference="$(arg prefix)rear_right_flipper"><xacro:gazebo_flipper_tags /></gazebo>
+		<gazebo reference="$(arg prefix)front_left_flipper_wheel1"><xacro:gazebo_flipper_wheel_tags /></gazebo>
+		<gazebo reference="$(arg prefix)front_right_flipper_wheel1"><xacro:gazebo_flipper_wheel_tags /></gazebo>
+		<gazebo reference="$(arg prefix)rear_left_flipper_wheel1"><xacro:gazebo_flipper_wheel_tags /></gazebo>
+		<gazebo reference="$(arg prefix)rear_right_flipper_wheel1"><xacro:gazebo_flipper_wheel_tags /></gazebo>
+		<gazebo reference="$(arg prefix)front_left_flipper_wheel2"><xacro:gazebo_flipper_wheel_tags /></gazebo>
+		<gazebo reference="$(arg prefix)front_right_flipper_wheel2"><xacro:gazebo_flipper_wheel_tags /></gazebo>
+		<gazebo reference="$(arg prefix)rear_left_flipper_wheel2"><xacro:gazebo_flipper_wheel_tags /></gazebo>
+		<gazebo reference="$(arg prefix)rear_right_flipper_wheel2"><xacro:gazebo_flipper_wheel_tags /></gazebo>
+		<gazebo reference="$(arg prefix)front_left_flipper_wheel3"><xacro:gazebo_flipper_wheel_tags /></gazebo>
+		<gazebo reference="$(arg prefix)front_right_flipper_wheel3"><xacro:gazebo_flipper_wheel_tags /></gazebo>
+		<gazebo reference="$(arg prefix)rear_left_flipper_wheel3"><xacro:gazebo_flipper_wheel_tags /></gazebo>
+		<gazebo reference="$(arg prefix)rear_right_flipper_wheel3"><xacro:gazebo_flipper_wheel_tags /></gazebo>
+		<gazebo reference="$(arg prefix)front_left_flipper_wheel4"><xacro:gazebo_flipper_wheel_tags /></gazebo>
+		<gazebo reference="$(arg prefix)front_right_flipper_wheel4"><xacro:gazebo_flipper_wheel_tags /></gazebo>
+		<gazebo reference="$(arg prefix)rear_left_flipper_wheel4"><xacro:gazebo_flipper_wheel_tags /></gazebo>
+		<gazebo reference="$(arg prefix)rear_right_flipper_wheel4"><xacro:gazebo_flipper_wheel_tags /></gazebo>
+		<gazebo reference="$(arg prefix)front_left_flipper_wheel5"><xacro:gazebo_flipper_wheel_tags /></gazebo>
+		<gazebo reference="$(arg prefix)front_right_flipper_wheel5"><xacro:gazebo_flipper_wheel_tags /></gazebo>
+		<gazebo reference="$(arg prefix)rear_left_flipper_wheel5"><xacro:gazebo_flipper_wheel_tags /></gazebo>
+		<gazebo reference="$(arg prefix)rear_right_flipper_wheel5"><xacro:gazebo_flipper_wheel_tags /></gazebo>
     </xacro:if>
     <xacro:if value="$(arg has_sick_lidar)">
@@ -1192,5 +1232,4 @@
 <!--                <time_increment>2.77777780866e-05</time_increment>-->
 <!--                <scan_time>0.019999999553</scan_time>-->
-<!--                <angle_increment>0.00872664619237</angle_increment>-->
                 </sensor>
             </xacro:if>

File: submitted_models/ctu_cras_norlab_absolem_sensor_config_1/urdf/realsense.gazebo.xacro (robot description, xacro)
@@ -10,8 +10,13 @@
     <xacro:arg name="realsense_visualize" default="[]" />
     <xacro:property name="deg_to_rad" value="${pi/180}" />
-    <gazebo reference="$(arg prefix)$(arg realsense_name)_link">
+    <link name="$(arg prefix)$(arg realsense_name)_link_sim" />
+    <xacro:fixed_joint name="$(arg realsense_name)_link_sim_j"
+                       parent="$(arg prefix)$(arg realsense_name)_link"
+                       child="$(arg prefix)$(arg realsense_name)_link_sim"
+                       xyz="0.017 -0.023 -0.009" />
+    <gazebo reference="$(arg prefix)$(arg realsense_name)_link_sim">
         <sensor name="$(arg realsense_name)" type="rgbd_camera">
           <camera name="$(arg realsense_name)_camera">
-            <horizontal_fov>${69.4*deg_to_rad}</horizontal_fov>
+            <horizontal_fov>1.5184</horizontal_fov>
             <lens>
               <intrinsics>
@@ -57,3 +62,19 @@
         </sensor>
     </gazebo>
+    <gazebo reference="$(arg prefix)realsense_holder_part2">
+        <visual>
+            <material>
+                <diffuse>.5 0.5 0.5 1</diffuse>
+                <ambient>.1 0.1 0.1 1</ambient>
+            </material>
+        </visual>
+    </gazebo>
+    <gazebo reference="$(arg prefix)$(arg realsense_name)_link">
+        <visual>
+            <material>
+                <diffuse>.5 0.5 0.5 1</diffuse>
+                <ambient>.1 0.1 0.1 1</ambient>
+            </material>
+        </visual>
+    </gazebo>
 </robot>

File: submitted_models/ctu_cras_norlab_absolem_sensor_config_1/urdf/realsense_d435_with_holder.xacro (robot description, xacro)
@@ -153,5 +153,10 @@
         <link name="$(arg prefix)realsense_holder_part2">
             <visual>
-                <origin rpy="-0.504467 0 1.5758" xyz="-0.002 -0.055 -0.051"/>
+                <xacro:if value="${'$(arg rendering_target)' == 'sdf'}">
+                    <origin rpy="-0.504467 0 1.5758" xyz="0.001 -0.055 -0.058"/>
+                </xacro:if>
+                <xacro:unless value="${'$(arg rendering_target)' == 'sdf'}">
+                    <origin rpy="-0.504467 0 1.5758" xyz="-0.002 -0.055 -0.051"/>
+                </xacro:unless>
                 <geometry>
                     <mesh scale="0.001 0.001 0.001"
