Commit message: Absolem: Added Basler cameras intrinsics.

File: submitted_models/ctu_cras_norlab_absolem_sensor_config_1/urdf/basler_cameras.xacro (robot description, xacro)
@@ -84,4 +84,16 @@
                             </lens>
                         </xacro:if>
+                        <xacro:unless value="${fisheye and '$(arg rendering_target)' == 'gz'}">
+                            <lens>
+                                <intrinsics>
+                                    <xacro:property name="f" value="${resolution_x / (2 * tan(radians(hfov_deg)/2))}" />
+                                    <fx>${f}</fx>
+                                    <fy>${f}</fy>
+                                    <cx>${(resolution_x - 1) / 2}</cx>
+                                    <cy>${(resolution_y - 1) / 2}</cy>
+                                    <s>0</s>
+                                </intrinsics>
+                            </lens>
+                        </xacro:unless>
                     </camera>
                 </sensor>
