Commit message: Model submission for Absolem sensor configurations 6,7,8 by CTU-CRAS-Norlab (#860)
* Absolem: Added sensor configs 6, 7 and 8.

* remove ros from the x500 plugin (#891)

Signed-off-by: Nate Koenig <nate@openrobotics.org>

Co-authored-by: Nate Koenig <nate@openrobotics.org>

* Model Submission for Emesent Hovermap (#892)

* Model submission for Hovermap sensor config 1 from Emesent

Signed-off-by: Rowan Ramamurthy <rowan.ramamurthy@emesent.io>

* updated specifications for the Emesent Hovermap

Signed-off-by: Rowan Ramamurthy <rowan.ramamurthy@emesent.io>

* Updated gimbal controller - fixed issue with battery usage

Signed-off-by: Rowan Ramamurthy <rowan.ramamurthy@emesent.io>

* Specifications updated for emesent hovermap sensor config 1

Signed-off-by: Rowan Ramamurthy <rowan.ramamurthy@emesent.io>

* Update specifications.md

Signed-off-by: Rowan Ramamurthy <rowan.ramamurthy@emesent.io>

* Update submitted_models/emesent_hovermap_sensor_config_1/CMakeLists.txt

Co-authored-by: Nate Koenig <nkoenig@users.noreply.github.com>

* Added details in the model.config

* Updated the min and max angle for the gpu lidar for the hovermap

* Updating min range and resolution for lidar

* Removing visualisation for lidar

* Added the number of horizontal samples for the gpu to 900

* Updated camera resolution, and also updated the weight in the specifications file to match the sdf values

* Updated noise parameters for the gimbal stabilising imu

* Added /sensor prefix to magnetometer output

* Added sensor prefixes for other sensor outputs

* Updated the imu with the new noise model

* Adding imu topic and specifications as per validation data

* Update submitted_models/emesent_hovermap_sensor_config_1/launch/spawner.rb

Co-authored-by: Nate Koenig <nkoenig@users.noreply.github.com>

* Renamed node with repeated name

* Updating the battery plugin to support a 21.6min flight time

* Updated specifications.md to align with provided validation data and spawner.rb accelerations.

* Adjusted limits on gimbals to align with observed behavior in validation data.

Co-authored-by: Rowan Ramamurthy <rowan.ramamurthy@emesent.io>
Co-authored-by: Peter <PeterQFR@users.noreply.github.com>
Co-authored-by: Nate Koenig <nkoenig@users.noreply.github.com>
Co-authored-by: Peter Milani <peter@emesent.io>

* Model Submission for CTU-CRAS-NORLAB MARV (#886)

* Added CTU_CRAS_NORLAB_MARV_SENSOR_CONFIG_1 (and other sensor configs).

* MARV: prefix links in URDF with robot name.

* MARV: Update RViz config.

* Removed debug prints

* MARV: Added mapping server relay.

* MARV: Downgraded model.sdf to SDF 1.6.

* MARV: Fixed IMU topic.

* MARV: Fixed cliff sensors ROS bridge.

* MARV: Fixed odom rate.

* MARV: Fixed flickering of lights.

* MARV: Update IMU parameters.

* MARV: Added camera intrinsics.

* MARV: Fixed lower bound of temperature for Boson camera.

* MARV: Changed Ouster precision and stddev to 0.01 to follow other SubT sensors.

* Added experimental validation of camera FoV to the specifications.

* Reduced battery life to 60 minutes until validation is complete.  The current maximum velocity and acceleration are set to the default limits for models without validation data.

* Added endurance adjustment to the specifications.md file.

Co-authored-by: Martin Pecka <peckama2@fel.cvut.cz>

* Model submission for BOSDYN_SPOT and two sensor configs of CTU-CRAS-Norlab (#841)

* Spot: First version, has actuators, but no control.

* Spot walking.

* Spot: improved modularity and made CCN_SPOT_SC1 compatible with BOSDYN_SPOT again.

The interface between BOSDYN_SPOT and sensor configs can be considered more or less stable now.

* Spot: Added cameras.

* Spot: Fixed a bug in handling leg collisions.

* Spot: specifications.md

* Spot: Fixed xacro utils to be compatible with MARV.

* Spot: Mono camera now also relays set_rate requests.

* Spot: Fixed IMU bridge.

* Spot: Added payload to CCN_SPOT_SC1.

* CCN_SPOT_SC1: Removed the total_mass_* helper link from URDF to avoid RViz displaying an error.

* Spot: Added CTU_CRAS_NORLAB_SPOT_SENSOR_CONFIG_2.

* CCN_SPOT_SC1: Added specifications.md.

* Spot: Added thumbnails.

* CCN_SPOT_SC1: Added thumbnails.

* Spot: Added mapping server bridge.

* Spot: Downgraded model.sdf to SDF 1.6.

* Spot: update IMU params.

* Spot: Add camera intrinsics.

Body depth camera is still just estimated.

* Spot: Fixed specifications.md part about contact system.

* Spot: Fixed mass by adding battery and tuned the PIDs a bit.

* Spot: Battery life set to 60 minutes.

* CCN_SPOT: Changed Ouster resolution and stddev to 0.01.

* Spot: removed unintentional change.

Signed-off-by: Martin Pecka <peckama2@fel.cvut.cz>

* Spot: Improvements of specifications.md.

* Spot: Adjusted battery life to 60 minutes.

* Spot: Resolved relative references to Fuel parts.

* added feedforward to bridge, controller msgs are now printed only once (#895)

* Set the state properly when recording is complete (#894)

Signed-off-by: Nate Koenig <nate@openrobotics.org>

Co-authored-by: Nate Koenig <nate@openrobotics.org>

* Absolem: Remove debug visuals [SDF 1.6] (#878)

* Absolem: Sync Xacro: Change IMU and friction parameters in Xacro to correspond to the desired values in SDF.

* Absolem: Sync Xacro: Re-generate model.sdf using libsdformat 8.9.1 .

This commit makes no real change to the geometry of the model, it just represents some numbers and rotations differently.

* Absolem: Removed empty link visuals as they obstructed the omnicam and were not good for anything else.

* Add missing robot platform types (#890)

* Add missing robot platform types

Signed-off-by: Nate Koenig <nate@openrobotics.org>

* Added hovermap and marv

Signed-off-by: Nate Koenig <nate@openrobotics.org>

* Added spot and fix dependency

Signed-off-by: Nate Koenig <nate@openrobotics.org>

Co-authored-by: Nate Koenig <nate@openrobotics.org>

* Fix CMakeLists (#897)

* Model Submission for CTU-CRAS-NORLAB Lily hexapod robot, sensor configs 1 and 2 (#867)

* added ctu_cras_norlab_lily ign simulation models

* changed thumbnails

* Fixed links in specifications.md .

* Downgraded model.sdf to SDF 1.6.

* Lily: Corrected mass.

* Lily: Added camera intrinsics.

* Lily: Changed ouster resolution and stddev to 0.01.

* Lily: Changed battery endurance to 60 minutes.

* Lily: Added robot_state_publisher to fill in missing static TFs.

* Lily: Edited Basler cam FOV to match in all places and correspond to intrinsics.

Co-authored-by: petr <petr.cizek@fel.cvut.cz>
Co-authored-by: Martin Pecka <peckama2@fel.cvut.cz>

* Spot: Disable nodelets because of spurious broken bonds. (#898)

* Model Submission for Coordinated Robotics' Crystal UAV Sensor Config 1 (#866)

* Coordinated Robotics Crystal UAV Sensor Config 1

* Updates based on reviews of other robots

* Camera precedent update, change colors to floats

* Adjust lighting to match camera change

* Update xacro

* Correct down lidar position, set top_scan to zero

Co-authored-by: Kevin <ak619@lafn.org>

* Model Submission for Coordinated Robotics Rocky Sensor Configs 1, 2 and 3 (#862)

* Coordinated Robotics Rocky

* Updates based on reviews of other robots

* Remove wheel slip plugin from Ackermann type steering vehicle

* Fixed camera name, changed color to floats

* Update cameras to match precedent

Co-authored-by: Kevin <ak619@lafn.org>

* Model Submission Coordinated Robotics Mike (#845)

* Add Coordinated Robotics Mike

* Updates based on reviews of other robots

* Add thermal camera to sensor list, fix wheel plugin wheel diameter, change to floating point colors, increase wheel joint speed

Co-authored-by: Kevin <ak619@lafn.org>

* Move battery plugin to the end of plugin list (#901)

Signed-off-by: Michael Carroll <michael@openrobotics.org>

* fixed pose of rs_up, rs_down rgbd cameras (#903)

* Update robot classes and marsupial pairs (#900)

* Adding lily to include

Signed-off-by: Nate Koenig <nate@openrobotics.org>

* Added CRYSTAL, MIKE, and ROCKY

Signed-off-by: Nate Koenig <nate@openrobotics.org>

* Added crystal as marsupial child

Signed-off-by: Nate Koenig <nate@openrobotics.org>

* Added new Coordinated marsupial pairs, adjusted Karen's collisions, and tweaked a few spawner z-offsets

Signed-off-by: Nate Koenig <nate@openrobotics.org>

* Remove debug statement

Signed-off-by: Nate Koenig <nate@openrobotics.org>

Co-authored-by: Nate Koenig <nate@openrobotics.org>

* Update to use the lattest fog emitter code (#896)

* Update to use the lastest fog emitter code

Signed-off-by: Nate Koenig <nate@openrobotics.org>

* Merged with master

Signed-off-by: Nate Koenig <nate@openrobotics.org>

* Adjust pose based on latest emitter model

Signed-off-by: Nate Koenig <nate@openrobotics.org>

Co-authored-by: Nate Koenig <nate@openrobotics.org>

* fixed fx, fy focal length of front camera to be consistent with hfov (#907)

* add set_rate service to X500 UAV (#906)

* added feedforward to bridge, controller msgs are now printed only once

* added set_rate services to laser, rgb, rgbd sensors

* dot_generator tweaks for tunnels (#884)

* Unified comms parameters across circuits.

Signed-off-by: Carlos Agüero <caguero@openrobotics.org>

* Absolem: Changed lidar and thermocam parameters, fixed RViz model.

* Absolem: Added Basler cameras intrinsics.

Co-authored-by: Nate Koenig <nkoenig@users.noreply.github.com>
Co-authored-by: Nate Koenig <nate@openrobotics.org>
Co-authored-by: acschang <61025344+acschang@users.noreply.github.com>
Co-authored-by: Rowan Ramamurthy <rowan.ramamurthy@emesent.io>
Co-authored-by: Peter <PeterQFR@users.noreply.github.com>
Co-authored-by: Peter Milani <peter@emesent.io>
Co-authored-by: Matej Petrlik <petrlmat@fel.cvut.cz>
Co-authored-by: Petr Cizek <cizekpet@gmail.com>
Co-authored-by: petr <petr.cizek@fel.cvut.cz>
Co-authored-by: knoedler <knoedler@dslextreme.com>
Co-authored-by: Kevin <ak619@lafn.org>
Co-authored-by: Michael Carroll <michael@openrobotics.org>
Co-authored-by: Carlos Agüero <caguero@osrfoundation.org>

File: submitted_models/ctu_cras_norlab_absolem_sensor_config_1/urdf/boson_thermocam.xacro (robot description, xacro)
@@ -27,9 +27,22 @@
                     <visualize>${visualize}</visualize>
                     <camera name="thermal_camera">
-                        <horizontal_fov>${92 * pi/180}</horizontal_fov>
+                        <xacro:property name="hfov" value="${radians(92)}" />
+                        <xacro:property name="width" value="320" />
+                        <xacro:property name="height" value="256" />
+                        <horizontal_fov>${hfov}</horizontal_fov>
+                        <lens>
+                            <intrinsics>
+                                <xacro:property name="focal_length" value="${320 / (2 * tan(radians(92) / 2))}" />
+                                <fx>${focal_length}</fx>
+                                <fy>${focal_length}</fy>
+                                <cx>${(width + 1) / 2.0}</cx>
+                                <cy>${(height + 1) / 2.0}</cy>
+                                <s>0</s>
+                            </intrinsics>
+                        </lens>
                         <image>
-                            <width>320</width>
-                            <height>256</height>
-                            <format>L16</format>
+                            <width>${width}</width>
+                            <height>${height}</height>
+                            <format>L8</format>
                         </image>
                         <clip>
@@ -39,7 +52,7 @@
                     </camera>
                     <plugin filename="ignition-gazebo-thermal-sensor-system" name="ignition::gazebo::systems::ThermalSensor">
-                        <min_temp>233.15</min_temp>
-                        <max_temp>453.15</max_temp>
-                        <resolution>0.06</resolution>
+                        <min_temp>253.15</min_temp>
+                        <max_temp>673.15</max_temp>
+                        <resolution>1.6</resolution>
                     </plugin>
                 </sensor>

File: submitted_models/ctu_cras_norlab_absolem_sensor_config_1/urdf/nifti_robot.xacro (robot description, xacro)
@@ -395,4 +395,7 @@
 		<xacro:include filename="$(find ctu_cras_norlab_absolem_sensor_config_1)/urdf/boson_thermocam.xacro" />
 	</xacro:if>
+	<xacro:if value="$(arg has_omnicam_vras)">
+		<xacro:include filename="$(find ctu_cras_norlab_absolem_sensor_config_1)/urdf/basler_cameras.xacro" />
+	</xacro:if>
 	<!-- NIFTI ROBOT LINKS AND JOINTS SPECIFICATION -->
 	<xacro:property name="body_color" value="$(arg body_color)" />
@@ -668,4 +671,12 @@
 							</geometry>
 					</visual>
+					<xacro:if value="${'$(arg revision)' == '2021' and $(arg has_omnicam_vras)}">
+						<visual>
+							<origin rpy="0 ${3*pi/2} 0" xyz="-0.075 0.0 0.12" />
+							<geometry>
+								<mesh filename="package://ctu_cras_norlab_absolem_sensor_config_1/meshes/reflector.dae" />
+							</geometry>
+						</visual>
+					</xacro:if>
 					<xacro:if value="${$(arg simplified_collision)==0}">
 							<collision>
@@ -742,5 +753,35 @@
 				<xacro:fixed_joint name="top_box_j" parent="$(arg prefix)rear_right_box" child="$(arg prefix)top_box" xyz="${top_box_j_x-0.0635} ${$(arg rover_robotWidthBody)/2} 0.0" rpy="0 0 0"/>
 				<xacro:if value="$(arg has_omnicam_vras)">
-					<!-- -->
+					<link name="$(arg prefix)top_box_step">
+						<xacro:property name="top_box_step_width" value="0.12" />
+						<xacro:property name="top_box_step_height" value="0.1" />
+						<visual>
+							<origin rpy="0 0 0" xyz="0 0 ${top_box_step_height/2}"/>
+							<geometry>
+								<box size="0.1270 ${top_box_step_width} ${top_box_step_height}" />
+							</geometry>
+							<material name="body_color">
+								<color rgba="0 ${94/255.0} ${184/255.0} 1.0"/>
+							</material>
+						</visual>
+						<visual>
+							<origin rpy="0 $(arg ouster_rpy_p) 0" xyz="${$(arg ouster_pos_x) - 0.01} 0 ${$(arg ouster_pos_z) - 0.075}"/>
+							<geometry>
+								<cylinder radius="0.025" length="0.05" />
+							</geometry>
+							<material name="body_color">
+								<color rgba="0 ${94/255.0} ${184/255.0} 1.0"/>
+							</material>
+						</visual>
+						<collision>
+							<origin rpy="0 0 0" xyz="0 0 ${top_box_step_height/2}"/>
+							<geometry>
+								<box size="0.1270 ${top_box_step_width} ${top_box_step_height}" />
+							</geometry>
+						</collision>
+						<xacro:box_inertial mass="1.0" width="${top_box_step_width}" height="${top_box_step_height}" depth="0.1270" xyz="0 0 ${top_box_step_height/2}" />
+					</link>
+					<xacro:fixed_joint name="top_box_step_j" parent="$(arg prefix)top_box" child="$(arg prefix)top_box_step" xyz="0 0 0.06252" />
+					<xacro:solid_color_link_material link="$(arg prefix)top_box_step" r="0" g="${94/255.0}" b="${184/255.0}" />
 				</xacro:if>
 			</xacro:if>
@@ -801,5 +842,10 @@
 	</link>
 	<xacro:if value="${'$(arg revision)' == '2021'}">
-		<xacro:fixed_joint name="antenna_j" parent="$(arg prefix)base_link" child="$(arg prefix)antenna" xyz="${-$(arg rover_robotLengthBody)/2 + 0.12} 0.0789 0.1551" rpy="0 0 0" />
+		<xacro:if value="$(arg has_omnicam)">
+			<xacro:fixed_joint name="antenna_j" parent="$(arg prefix)base_link" child="$(arg prefix)antenna" xyz="${-$(arg rover_robotLengthBody)/2 + 0.12} 0.0789 0.1551" rpy="0 0 0" />
+		</xacro:if>
+		<xacro:if value="$(arg has_omnicam_vras)">
+			<xacro:fixed_joint name="antenna_j" parent="$(arg prefix)base_link" child="$(arg prefix)antenna" xyz="${-$(arg rover_robotLengthBody)/2 + 0.12} 0.1 0.1551" rpy="0 0 0" />
+		</xacro:if>
 	</xacro:if>
 	<xacro:unless value="${'$(arg revision)' == '2021'}">
@@ -1207,20 +1253,42 @@
 			</xacro:if>
 	</xacro:if>
+	<!-- Omnicamera -->
+	<xacro:if value="$(arg has_omnicam_vras)">
+		<xacro:basler_ace_omnicam name="camera_0" simulate="$(arg simulate_omnicam_vras)" visualize="$(arg visualize_sensors)" />
+		<xacro:fixed_joint name="camera_0_j" parent="$(arg prefix)rear_right_box" child="$(arg prefix)camera_0"
+						   xyz="${$(arg rover_robotLengthBody) - 0.11} ${$(arg rover_robotWidthBody)/2} 0.01" lump="0" />
+		<link name="$(arg prefix)front_camera_holder"><visual><geometry><box size="0.04 0.025 0.01" /></geometry></visual></link>
+		<xacro:fixed_joint name="front_camera_holder_j" parent="$(arg prefix)camera_0" child="$(arg prefix)front_camera_holder" xyz="0.02 0 -0.005" />
+		<xacro:basler_ace_omnicam name="camera_1" simulate="$(arg simulate_omnicam_vras)" visualize="$(arg visualize_sensors)" />
+		<xacro:fixed_joint name="camera_1_j" parent="$(arg prefix)rear_right_box" child="$(arg prefix)camera_1"
+						   xyz="${$(arg rover_robotLengthBody)/2-0.02} 0.083 0" rpy="0 0 ${-pi/2}" lump="0" />
+		<xacro:basler_ace_omnicam name="camera_2" simulate="$(arg simulate_omnicam_vras)" visualize="$(arg visualize_sensors)" />
+		<xacro:fixed_joint name="camera_2_j" parent="$(arg prefix)rear_right_box" child="$(arg prefix)camera_2"
+						   xyz="0.05 ${$(arg rover_robotWidthBody)/2} 0" rpy="0 0 ${-pi}" lump="0" />
+		<xacro:basler_ace_omnicam name="camera_3" simulate="$(arg simulate_omnicam_vras)" visualize="$(arg visualize_sensors)" />
+		<xacro:fixed_joint name="camera_3_j" parent="$(arg prefix)rear_right_box" child="$(arg prefix)camera_3"
+						   xyz="${$(arg rover_robotLengthBody)/2-0.02} ${$(arg rover_robotWidthBody) - 0.083} 0" rpy="0 0 ${-3*pi/2}" lump="0" />
+		<xacro:basler_ace_omnicam name="camera_4" simulate="$(arg simulate_omnicam_vras)" visualize="$(arg visualize_sensors)" />
+		<xacro:fixed_joint name="camera_4_j" parent="$(arg prefix)top_box" child="$(arg prefix)camera_4"
+						   xyz="-0.048 -0.0145 ${0.06252 + top_box_step_height - 0.08}" rpy="${pi} ${-pi/2} ${pi/2}" lump="0" />
+	</xacro:if>
 	<!-- 3D lidar -->
 	<xacro:if value="$(arg has_ouster_lidar)">
 		<xacro:ouster_os0_128 name="laser" simulate="$(arg simulate_ouster_lidar)" visualize="$(arg visualize_sensors)" />
 		<xacro:calibrated_fixed_joint name="laser_j" parent="top_box" child="laser" prefix="ouster" lump="0"/>
-		<link name="$(arg prefix)ouster_holder">
-			<visual>
-				<origin xyz="0 0 0" />
-				<geometry>
-					<mesh filename="package://ctu_cras_norlab_absolem_sensor_config_1/meshes/ouster_holder_ladybug.dae" />
-				</geometry>
-			</visual>
-			<xacro:cylinder_inertial mass="0.2" radius="0.07" length="0.02"
-								xyz="0 0 -0.01" />
-		</link>
-		<xacro:fixed_joint name="ouster_holder_j" parent="$(arg prefix)omnicam_top" child="$(arg prefix)ouster_holder"
-			xyz="0 0 0.005" rpy="0 0 ${radians(36)}" />
+		<xacro:if value="$(arg has_omnicam)">
+			<link name="$(arg prefix)ouster_holder">
+				<visual>
+					<origin xyz="0 0 0" />
+					<geometry>
+						<mesh filename="package://ctu_cras_norlab_absolem_sensor_config_1/meshes/ouster_holder_ladybug.dae" />
+					</geometry>
+				</visual>
+				<xacro:cylinder_inertial mass="0.2" radius="0.07" length="0.02"
+									xyz="0 0 -0.01" />
+			</link>
+			<xacro:fixed_joint name="ouster_holder_j" parent="$(arg prefix)omnicam_top" child="$(arg prefix)ouster_holder"
+				xyz="0 0 0.005" rpy="0 0 ${radians(36)}" />
+		</xacro:if>
 	</xacro:if>
 	<!-- Thermal camera -->
@@ -1530,6 +1598,12 @@
     <xacro:if value="$(arg has_mote_deployer)">
         <!-- The link is included automatically in the payload xacro -->
-        <xacro:fixed_joint name="mote_deployer_j" parent="$(arg prefix)rear_right_box" child="$(arg prefix)mote_deployer"
-            xyz="0.09 0.16 -0.01" rpy="0 0 ${pi}" />
+		<xacro:if value="$(arg has_omnicam)">
+			<xacro:fixed_joint name="mote_deployer_j" parent="$(arg prefix)rear_right_box" child="$(arg prefix)mote_deployer"
+				xyz="0.09 0.16 -0.01" rpy="0 0 ${pi}" />
+		</xacro:if>
+		<xacro:if value="$(arg has_omnicam_vras)">
+			<xacro:fixed_joint name="mote_deployer_j" parent="$(arg prefix)rear_right_box" child="$(arg prefix)mote_deployer"
+				xyz="0.09 0.18 -0.01" rpy="0 0 ${pi}" />
+		</xacro:if>
     </xacro:if>
     <xacro:macro name="stiff_joint_tags">

File: submitted_models/ctu_cras_norlab_absolem_sensor_config_1/urdf/ouster_lidar.xacro (robot description, xacro)
@@ -42,10 +42,10 @@
                             <min>0.1</min>
                             <max>50</max>
-                            <resolution>0.003</resolution>
+                            <resolution>0.01</resolution>
                         </range>
                         <noise>
                             <type>gaussian</type>
                             <mean>0</mean>
-                            <stddev>0.03</stddev>
+                            <stddev>0.01</stddev>
                         </noise>
                     </lidar>
