Commit message: Absolem: configurable length of big collision box.

File: submitted_models/ctu_cras_norlab_absolem_sensor_config_1/urdf/nifti_robot.xacro (robot description, xacro)
@@ -281,4 +281,5 @@
 	<xacro:arg name="big_collision_box_height" default="0.25" />
 	<xacro:arg name="big_collision_box_width" default="0.31" />
+	<xacro:arg name="big_collision_box_length" default="0.65" />
 	<xacro:arg name="big_collision_box_x" default="-0.21" />
 	<xacro:arg name="flipper_inflation_ratio" default="1.0" />
@@ -555,5 +556,5 @@
 							<origin rpy="0 0 0" xyz="$(arg big_collision_box_x) 0 ${0.08 + $(arg big_collision_box_height)/2}"/>
 							<geometry>
-									<box size="0.65 $(arg big_collision_box_width) $(arg big_collision_box_height)" />
+									<box size="$(arg big_collision_box_length) $(arg big_collision_box_width) $(arg big_collision_box_height)" />
 							</geometry>
 					</collision>

Commit message: Absolem: Added ceiling light.

File: submitted_models/ctu_cras_norlab_absolem_sensor_config_1/urdf/nifti_robot.xacro (robot description, xacro)
@@ -389,4 +389,7 @@
 		<xacro:include filename="$(find ctu_cras_norlab_absolem_sensor_config_1)/urdf/mote_deployer.xacro" />
 	</xacro:if>
+	<xacro:if value="${'$(arg revision)' == '2021'}">
+		<xacro:include filename="$(find ctu_cras_norlab_absolem_sensor_config_1)/urdf/lights.xacro" />
+	</xacro:if>
 	<xacro:if value="$(arg has_boson_thermocam)">
 		<xacro:include filename="$(find ctu_cras_norlab_absolem_sensor_config_1)/urdf/boson_thermocam.xacro" />
@@ -450,4 +453,12 @@
 					</xacro:unless>
 			</xacro:if>
+			<xacro:if value="${'$(arg revision)' == '2021' and $(arg has_omnicam)}">
+				<visual>
+					<origin rpy="0 ${3*pi/2} ${pi/2}" xyz="-0.18 0 0.185" />
+					<geometry>
+						<mesh filename="package://ctu_cras_norlab_absolem_sensor_config_1/meshes/reflector.dae" />
+					</geometry>
+				</visual>
+			</xacro:if>
 			<xacro:if value="${$(arg simplified_collision)==0}">
 					<collision>
@@ -644,10 +655,5 @@
 	<xacro:if value="$(arg has_top_box)">
 		<xacro:if value="${'$(arg revision)' == '2021'}">
-			<xacro:if value="$(arg has_omnicam)">
-				<xacro:property name="top_box_mesh_name" value="top_box_2021_ladybug.dae" />
-			</xacro:if>
-			<xacro:if value="$(arg has_omnicam_vras)">
-				<xacro:property name="top_box_mesh_name" value="top_box_2021_omnicam_vras.dae" />
-			</xacro:if>
+			<xacro:property name="top_box_mesh_name" value="top_box_2021_ladybug.dae" />
 		</xacro:if>
 		<xacro:unless value="${'$(arg revision)' == '2021'}">
@@ -684,13 +690,8 @@
 							<collision>
 								<xacro:if value="${'$(arg revision)' == '2021'}">
-									<xacro:if value="$(arg has_omnicam)">
-										<origin rpy="0 0 0" xyz="0 0 0.0315"/>
-										<geometry>
-											<box size="0.1270 0.231 0.06252" />
-										</geometry>
-									</xacro:if>
-									<xacro:if value="$(arg has_omnicam_vras)">
-										<!-- TODO -->
-									</xacro:if>
+									<origin rpy="0 0 0" xyz="0 0 0.0315"/>
+									<geometry>
+										<box size="0.1270 0.231 0.06252" />
+									</geometry>
 								</xacro:if>
 								<xacro:unless value="${'$(arg revision)' == '2021'}">
@@ -704,10 +705,5 @@
 							<collision>
 									<xacro:if value="${'$(arg revision)' == '2021'}">
-										<xacro:if value="$(arg has_omnicam)">
-											<origin rpy="0 0 0" xyz="-0.04 0.09 0.0690"/>
-										</xacro:if>
-										<xacro:if value="$(arg has_omnicam_vras)">
-											<origin rpy="0 0 0" xyz="fail"/>
-										</xacro:if>
+										<origin rpy="0 0 0" xyz="-0.04 0.09 0.0690"/>
 									</xacro:if>
 									<xacro:unless value="${'$(arg revision)' == '2021'}">
@@ -721,10 +717,5 @@
 							<collision>
 									<xacro:if value="${'$(arg revision)' == '2021'}">
-										<xacro:if value="$(arg has_omnicam)">
-											<origin rpy="0 0 0" xyz="0.01474 -0.08352 0.07996"/>
-										</xacro:if>
-										<xacro:if value="$(arg has_omnicam_vras)">
-											<origin rpy="0 0 0" xyz="fail"/>
-										</xacro:if>
+										<origin rpy="0 0 0" xyz="0.01474 -0.08352 0.07996"/>
 									</xacro:if>
 									<xacro:unless value="${'$(arg revision)' == '2021'}">
@@ -748,8 +739,6 @@
 			<xacro:property name="top_box_j_x" value="$(arg top_box_j_x)" />
 			<xacro:if value="${'$(arg revision)' == '2021'}">
-				<xacro:if value="$(arg has_omnicam)">
-					<!-- Origin of top box is 0.0635 m from the front side. And top_box_j_x is distance from robot's back to top box' front. -->
-					<xacro:fixed_joint name="top_box_j" parent="$(arg prefix)rear_right_box" child="$(arg prefix)top_box" xyz="${top_box_j_x-0.0635} ${$(arg rover_robotWidthBody)/2} 0.0" rpy="0 0 0"/>
-				</xacro:if>
+				<!-- Origin of top box is 0.0635 m from the front side. And top_box_j_x is distance from robot's back to top box' front. -->
+				<xacro:fixed_joint name="top_box_j" parent="$(arg prefix)rear_right_box" child="$(arg prefix)top_box" xyz="${top_box_j_x-0.0635} ${$(arg rover_robotWidthBody)/2} 0.0" rpy="0 0 0"/>
 				<xacro:if value="$(arg has_omnicam_vras)">
 					<!-- -->
@@ -1710,4 +1699,16 @@
 			</xacro:if>
 		</gazebo>
+	<xacro:if value="${'$(arg revision)' == '2021'}">
+		<xacro:if value="$(arg has_omnicam)">
+			<gazebo reference="$(arg prefix)base_link">
+				<xacro:spot_light_up name="light_up" pose="-0.18 0 0.185 0 ${-pi} 0" />
+			</gazebo>
+		</xacro:if>
+		<xacro:if value="$(arg has_omnicam_vras)">
+			<gazebo reference="$(arg prefix)top_box">
+				<xacro:spot_light_up name="light_up" pose="-0.075 0.0 0.12 0 ${-pi} 0" />
+			</gazebo>
+		</xacro:if>
+	</xacro:if>
     <gazebo reference="$(arg prefix)imu">
 		<xacro:gazebo_invisible_tags />
