Commit message: Absolem: Added sensor config 3 (facelifted version with 3D lidar).

File: submitted_models/ctu_cras_norlab_absolem_sensor_config_1/urdf/nifti_robot.xacro (robot description, xacro)
@@ -178,4 +178,30 @@
 	<xacro:arg default="0.000000" name="d435_pos_y"/>
 	<xacro:arg default="0.000000" name="d435_pos_x"/>
+	<xacro:arg default="1.000000" name="ouster_quat_w"/>
+	<xacro:arg default="0.000000" name="ouster_quat_z"/>
+	<xacro:arg default="0.000000" name="ouster_quat_y"/>
+	<xacro:arg default="0.000000" name="ouster_quat_x"/>
+	<xacro:arg default="0.000000" name="ouster_gzrpy_y"/>
+	<xacro:arg default="0.000000" name="ouster_gzrpy_p"/>
+	<xacro:arg default="0.000000" name="ouster_gzrpy_r"/>
+	<xacro:arg default="0.000000" name="ouster_rpy_y"/>
+	<xacro:arg default="0.000000" name="ouster_rpy_p"/>
+	<xacro:arg default="0.000000" name="ouster_rpy_r"/>
+	<xacro:arg default="0.200000" name="ouster_pos_z"/>
+	<xacro:arg default="0.000000" name="ouster_pos_y"/>
+	<xacro:arg default="0.070000" name="ouster_pos_x"/>
+	<xacro:arg default="0.042087" name="camera_0_pos_x"/>
+	<xacro:arg default="0.000000" name="cliff_sensor_0_x"/>
+	<xacro:arg default="0.000000" name="cliff_sensor_0_y"/>
+	<xacro:arg default="0.000000" name="cliff_sensor_0_yaw"/>
+	<xacro:arg default="0.000000" name="cliff_sensor_1_x"/>
+	<xacro:arg default="0.000000" name="cliff_sensor_1_y"/>
+	<xacro:arg default="0.000000" name="cliff_sensor_1_yaw"/>
+	<xacro:arg default="0.000000" name="cliff_sensor_2_x"/>
+	<xacro:arg default="0.000000" name="cliff_sensor_2_y"/>
+	<xacro:arg default="0.000000" name="cliff_sensor_2_yaw"/>
+	<xacro:arg default="0.000000" name="cliff_sensor_3_x"/>
+	<xacro:arg default="0.000000" name="cliff_sensor_3_y"/>
+	<xacro:arg default="0.000000" name="cliff_sensor_3_yaw"/>
 	<xacro:arg default="0.070500" name="rover_referentialZ"/>
 	<xacro:arg default="0.600000" name="rover_vMaxRun"/>
@@ -193,4 +219,7 @@
 	<xacro:arg default="0.300000" name="rover_vMaxTravel"/>
 	<xacro:arg default="0.240930" name="rover_robotWidthBody"/>
+	<xacro:arg default="0.500170" name="rover_robotLengthBody"/>
+	<xacro:arg default="-0.12200" name="rover_robotBodyShift"/>
+	<xacro:arg default="0.022000" name="rover_bodyEdgeCurvature"/> <!-- curvature of the front and rear bottom edges -->
 	<xacro:arg default="0.397000" name="rover_trackDistance"/>
 	<xacro:arg default="0.330000" name="rover_flipperLength"/>
@@ -209,15 +238,25 @@
 			 Example of value: '0 1 0 1' (don't forget to set alpha to 1!). -->
 	<xacro:arg name="body_color" default="" />
+	<!-- Body shape revision. Possible values are 2010, 2014 and 2021 -->
+	<xacro:arg name="revision" default="2014" />
 	<xacro:arg name="has_top_box" default="1" />
 	<!-- Distance from robot's back to top box' front panel. Default is the front-most position. -->
 	<xacro:arg name="top_box_j_x" default="0.4977" />
 	<xacro:arg name="has_sick_lidar" default="1" />
+	<xacro:arg name="has_ouster_lidar" default="0" />
 	<xacro:arg name="has_omnicam" default="1" />
+	<xacro:arg name="has_omnicam_vras" default="0" />
 	<xacro:arg name="has_omnicam_sensor_mount" default="1" />
 	<xacro:arg name="has_flippers" default="1" />
 	<xacro:arg name="has_differential" default="1" />
+	<xacro:arg name="has_new_realsense" default="0" />
+	<xacro:arg name="has_realsense_d435" default="0" />
+	<xacro:arg name="has_realsense_t265" default="0" />
+	<xacro:arg name="has_jetson" default="0" />
+	<xacro:arg name="num_cliff_sensors" default="0" />
 	<xacro:arg name="has_rear_sensor_item" default="1" />
 	<xacro:arg name="rear_sensor_item_x" default="0.084" />
 	<xacro:arg name="rear_sensor_item_y" default="0.02" />
+	<xacro:arg name="rear_sensor_item_height" default="0.35" />
 	<xacro:arg name="laser_pitch" default="0.0" />
 	<!-- render_xacro.py allows use of arguments like $(arg rover_trackLength) etc. which are not defined here -->
@@ -263,7 +302,11 @@
     <xacro:arg name="perfect_odometry" default="False" /> <!-- If True, ground truth position will be published as odom frame. -->
     <xacro:arg name="simulate_sick_lidar" default="True" />
+    <xacro:arg name="simulate_ouster_lidar" default="True" />
     <xacro:arg name="simulate_omnicam" default="True" />
+    <xacro:arg name="simulate_omnicam_vras" default="True" />
     <xacro:arg name="simulate_realsense_d435" default="True" />
     <xacro:arg name="simulate_imu" default="True" />
+    <xacro:arg name="simulate_cliff_sensors" default="True" />
+    <xacro:arg name="visualize_sensors" default="False" />
     <xacro:arg name="differential_locked" default="true" />
     <xacro:arg name="laser_update_rate" default="1000.0" />
@@ -287,5 +330,5 @@
 	<!-- MACRO SPECIFICATIONS -->
 	<xacro:include filename="$(find ctu_cras_norlab_absolem_sensor_config_1)/urdf/utils.xacro" />
-	<xacro:macro name="calibrated_fixed_joint" params="name parent child prefix:=''">
+	<xacro:macro name="calibrated_fixed_joint" params="name parent child prefix:='' lump:='1'">
 			<!-- These arguments are filled by render_xacro.py from calibration data. -->
 			<xacro:if value="${prefix == ''}">
@@ -297,10 +340,17 @@
 			<xacro:fixed_joint name="${name}" parent="$(arg prefix)${parent}" child="$(arg prefix)${child}"
 												 xyz="$(arg ${pref}_pos_x) $(arg ${pref}_pos_y) $(arg ${pref}_pos_z)"
-												 rpy="$(arg ${pref}_rpy_r) $(arg ${pref}_rpy_p) $(arg ${pref}_rpy_y)" />
+												 rpy="$(arg ${pref}_rpy_r) $(arg ${pref}_rpy_p) $(arg ${pref}_rpy_y)"
+												 lump="${lump}"/>
 	</xacro:macro>
 	<!-- SPECIAL LINKS -->
 	<!-- This is a virtual link that specifies the origin to which parts attachable to the top of the robot should be related. -->
 	<link name="$(arg prefix)rear_right_box" />
-	<xacro:fixed_joint name="rear_right_box_j" parent="$(arg prefix)base_link" child="$(arg prefix)rear_right_box" rpy="0 0 0" xyz="-0.379 -0.1265 0.185"/>
+	<xacro:if value="${'$(arg revision)' == '2021'}">
+		<xacro:fixed_joint name="rear_right_box_j" parent="$(arg prefix)base_link" child="$(arg prefix)rear_right_box" rpy="0 0 0"
+						   xyz="${-$(arg rover_robotLengthBody)/2} ${-$(arg rover_robotWidthBody)/2} 0.185"/>
+	</xacro:if>
+	<xacro:unless value="${'$(arg revision)' == '2021'}">
+		<xacro:fixed_joint name="rear_right_box_j" parent="$(arg prefix)base_link" child="$(arg prefix)rear_right_box" rpy="0 0 0" xyz="-0.379 -0.1265 0.185"/>
+	</xacro:unless>
 	<!-- INCLUDES -->
 	<xacro:if value="$(arg has_jetson)">
@@ -316,7 +366,16 @@
 		<xacro:include filename="$(find ctu_cras_norlab_absolem_sensor_config_1)/urdf/t265_attach_to_robot.xacro" />
 	</xacro:if>
+	<xacro:if value="$(arg has_ouster_lidar)">
+		<xacro:include filename="$(find ctu_cras_norlab_absolem_sensor_config_1)/urdf/ouster_lidar.xacro" />
+	</xacro:if>
 	<!-- NIFTI ROBOT LINKS AND JOINTS SPECIFICATION -->
 	<xacro:property name="body_color" value="$(arg body_color)" />
 	<link name="$(arg prefix)base_link">
+			<xacro:if value="${'$(arg revision)' == '2021'}">
+				<xacro:property name="body_mesh_name" value="body_2021.dae" />
+			</xacro:if>
+			<xacro:unless value="${'$(arg revision)' == '2021'}">
+				<xacro:property name="body_mesh_name" value="body.dae" />
+			</xacro:unless>
 			<xacro:if value="${len(body_color) == 0}">
 					<visual>
@@ -324,5 +383,5 @@
 							<geometry>
 									<mesh scale="${body_scale} ${body_scale} ${body_scale}"
-												filename="package://ctu_cras_norlab_absolem_sensor_config_1/meshes/body.dae"/>
+												filename="package://ctu_cras_norlab_absolem_sensor_config_1/meshes/${body_mesh_name}"/>
 							</geometry>
 					</visual>
@@ -330,7 +389,7 @@
 			<xacro:if value="${len(body_color) > 0}">
 					<visual>
-							<origin rpy="0 0 0" xyz="-0.1220 0 0.118"/>
-							<geometry>
-									<box size="0.50017 $(arg rover_robotWidthBody) 0.1390" />
+							<origin rpy="0 0 0" xyz="$(arg rover_robotBodyShift) 0 0.118"/>
+							<geometry>
+									<box size="$(arg rover_robotLengthBody) $(arg rover_robotWidthBody) 0.1390" />
 							</geometry>
 							<material name="body_color">
@@ -338,31 +397,33 @@
 							</material>
 					</visual>
-					<visual>
-							<origin rpy="0 0 0" xyz="0.157 0 0.118"/>
-							<geometry>
-									<box size="0.056 0.12093 0.1390" />
-							</geometry>
-							<material name="body_color">
-									<color rgba="$(arg body_color)"/>
-							</material>
-					</visual>
-					<visual>
-							<origin rpy="0 0 0.785398" xyz="0.144 -0.076 0.118"/>
-							<geometry>
-									<box size="0.083 0.040 0.1390" />
-							</geometry>
-							<material name="body_color">
-									<color rgba="$(arg body_color)"/>
-							</material>
-					</visual>
-					<visual>
-							<origin rpy="0 0 -0.785398" xyz="0.144 0.076 0.118"/>
-							<geometry>
-									<box size="0.083 0.040 0.1390" />
-							</geometry>
-							<material name="body_color">
-									<color rgba="$(arg body_color)"/>
-							</material>
-					</visual>
+					<xacro:unless value="${'$(arg revision)' == '2021'}">
+						<visual>
+								<origin rpy="0 0 0" xyz="0.157 0 0.118"/>
+								<geometry>
+										<box size="0.056 0.12093 0.1390" />
+								</geometry>
+								<material name="body_color">
+										<color rgba="$(arg body_color)"/>
+								</material>
+						</visual>
+						<visual>
+								<origin rpy="0 0 0.785398" xyz="0.144 -0.076 0.118"/>
+								<geometry>
+										<box size="0.083 0.040 0.1390" />
+								</geometry>
+								<material name="body_color">
+										<color rgba="$(arg body_color)"/>
+								</material>
+						</visual>
+						<visual>
+								<origin rpy="0 0 -0.785398" xyz="0.144 0.076 0.118"/>
+								<geometry>
+										<box size="0.083 0.040 0.1390" />
+								</geometry>
+								<material name="body_color">
+										<color rgba="$(arg body_color)"/>
+								</material>
+						</visual>
+					</xacro:unless>
 			</xacro:if>
 			<xacro:if value="${$(arg simplified_collision)==0}">
@@ -371,5 +432,5 @@
 							<geometry>
 									<mesh scale="${body_scale} ${body_scale} ${body_scale}"
-												filename="package://ctu_cras_norlab_absolem_sensor_config_1/meshes/body.dae"/>
+												filename="package://ctu_cras_norlab_absolem_sensor_config_1/meshes/${body_mesh_name}"/>
 							</geometry>
 					</collision>
@@ -380,5 +441,5 @@
 							<geometry>
 									<mesh scale="${body_scale} ${body_scale} ${body_scale}"
-												filename="package://ctu_cras_norlab_absolem_sensor_config_1/meshes/collide/body.dae"/>
+												filename="package://ctu_cras_norlab_absolem_sensor_config_1/meshes/collide/${body_mesh_name}"/>
 							</geometry>
 					</collision>
@@ -386,27 +447,37 @@
 			<xacro:if value="${$(arg simplified_collision)==2}">
 					<collision>
-							<origin rpy="0 0 0" xyz="-0.1220 0 0.118"/>
-							<geometry>
-									<box size="0.50017 $(arg rover_robotWidthBody) 0.1390" />
-							</geometry>
-					</collision>
-					<collision>
-							<origin rpy="0 0 0" xyz="0.157 0 0.118"/>
-							<geometry>
-									<box size="0.056 0.12093 0.1390" />
-							</geometry>
-					</collision>
-					<collision>
-							<origin rpy="0 0 0.785398" xyz="0.144 -0.076 0.118"/>
-							<geometry>
-									<box size="0.083 0.040 0.1390" />
-							</geometry>
-					</collision>
-					<collision>
-							<origin rpy="0 0 -0.785398" xyz="0.144 0.076 0.118"/>
-							<geometry>
-									<box size="0.083 0.040 0.1390" />
-							</geometry>
-					</collision>
+							<xacro:if value="${'$(arg revision)' == '2021'}">
+								<xacro:property name="bodyCollHeight" value="${0.1390 - $(arg rover_bodyEdgeCurvature)}" />
+								<xacro:property name="bodyCollZshift" value="${0.118 + $(arg rover_bodyEdgeCurvature)/2}" />
+							</xacro:if>
+							<xacro:unless value="${'$(arg revision)' == '2021'}">
+								<xacro:property name="bodyCollHeight" value="0.1390" />
+								<xacro:property name="bodyCollZshift" value="0.118" />
+							</xacro:unless>
+							<origin rpy="0 0 0" xyz="$(arg rover_robotBodyShift) 0 ${bodyCollZshift}"/>
+							<geometry>
+									<box size="$(arg rover_robotLengthBody) $(arg rover_robotWidthBody) ${bodyCollHeight}" />
+							</geometry>
+					</collision>
+				    <xacro:unless value="${'$(arg revision)' == '2021'}">
+						<collision>
+								<origin rpy="0 0 0" xyz="0.157 0 0.118"/>
+								<geometry>
+										<box size="0.056 0.12093 0.1390" />
+								</geometry>
+						</collision>
+						<collision>
+								<origin rpy="0 0 0.785398" xyz="0.144 -0.076 0.118"/>
+								<geometry>
+										<box size="0.083 0.040 0.1390" />
+								</geometry>
+						</collision>
+						<collision>
+								<origin rpy="0 0 -0.785398" xyz="0.144 0.076 0.118"/>
+								<geometry>
+										<box size="0.083 0.040 0.1390" />
+								</geometry>
+						</collision>
+					</xacro:unless>
 					<collision>
 							<origin rpy="0 0 0" xyz="0 0.135 0.09"/>
@@ -433,4 +504,28 @@
 							</geometry>
 					</collision>
+					<xacro:if value="${'$(arg revision)' == '2021'}">
+						<collision>
+							<origin rpy="0 0 0" xyz="0 0 ${0.048 + $(arg rover_bodyEdgeCurvature)/2}"/>
+							<geometry>
+								<box size="${$(arg rover_robotLengthBody) - 2*$(arg rover_bodyEdgeCurvature)} $(arg rover_robotWidthBody) $(arg rover_bodyEdgeCurvature)" />
+							</geometry>
+						</collision>
+						<collision>
+							<!-- We enlarge the radius a tiny bit to avoid wrong contact forces on the interface between the bottom plate and the cylinder -->
+							<origin xyz="${$(arg rover_robotLengthBody)/2-$(arg rover_bodyEdgeCurvature)} 0 ${0.048 + $(arg rover_bodyEdgeCurvature)}"
+									rpy="${pi/2} 0 0"/>
+							<geometry>
+								<cylinder length="$(arg rover_robotWidthBody)" radius="${$(arg rover_bodyEdgeCurvature)*1.001}" />
+							</geometry>
+						</collision>
+						<collision>
+							<!-- We enlarge the radius a tiny bit to avoid wrong contact forces on the interface between the bottom plate and the cylinder -->
+							<origin xyz="${-$(arg rover_robotLengthBody)/2+$(arg rover_bodyEdgeCurvature)} 0 ${0.048 + $(arg rover_bodyEdgeCurvature)}"
+									rpy="${pi/2} 0 0"/>
+							<geometry>
+								<cylinder length="$(arg rover_robotWidthBody)" radius="${$(arg rover_bodyEdgeCurvature)*1.001}" />
+							</geometry>
+						</collision>
+					</xacro:if>
 			</xacro:if>
 			<xacro:if value="$(arg big_collision_box_on_top)">
@@ -456,7 +551,7 @@
 			<link name="$(arg prefix)rear_sensor_item">
 					<visual>
-							<origin xyz="0 0 ${0.35/2}" rpy="0 0 0" />
-							<geometry>
-									<box size="0.02 0.02 0.35"/>
+							<origin xyz="0 0 ${$(arg rear_sensor_item_height)/2}" rpy="0 0 0" />
+							<geometry>
+									<box size="0.02 0.02 $(arg rear_sensor_item_height)"/>
 							</geometry>
 							<material name="aluminium">
@@ -465,7 +560,7 @@
 					</visual>
 					<collision>
-							<origin xyz="0 0 ${0.35/2}" rpy="0 0 0" />
-							<geometry>
-									<box size="0.02 0.02 0.35" />
+							<origin xyz="0 0 ${$(arg rear_sensor_item_height)/2}" rpy="0 0 0" />
+							<geometry>
+									<box size="0.02 0.02 $(arg rear_sensor_item_height)" />
 							</geometry>
 					</collision>
@@ -518,6 +613,22 @@
 			</inertial>
 	</link>
-	<xacro:fixed_joint name="battery_j" parent="$(arg prefix)base_link" child="$(arg prefix)battery" xyz="-0.2836 -0.0221 0.0722" rpy="0 0 0" />
+	<xacro:unless value="${'$(arg revision)' == '2021'}">
+		<xacro:fixed_joint name="battery_j" parent="$(arg prefix)base_link" child="$(arg prefix)battery" xyz="-0.2836 -0.0221 0.0722" rpy="0 0 0" />
+	</xacro:unless>
+	<xacro:if value="${'$(arg revision)' == '2021'}">
+		<xacro:fixed_joint name="battery_j" parent="$(arg prefix)base_link" child="$(arg prefix)battery" xyz="-0.12 0 0.12" rpy="0 ${pi/2} 0" />
+	</xacro:if>
 	<xacro:if value="$(arg has_top_box)">
+		<xacro:if value="${'$(arg revision)' == '2021'}">
+			<xacro:if value="$(arg has_omnicam)">
+				<xacro:property name="top_box_mesh_name" value="top_box_2021_ladybug.dae" />
+			</xacro:if>
+			<xacro:if value="$(arg has_omnicam_vras)">
+				<xacro:property name="top_box_mesh_name" value="top_box_2021_omnicam_vras.dae" />
+			</xacro:if>
+		</xacro:if>
+		<xacro:unless value="${'$(arg revision)' == '2021'}">
+			<xacro:property name="top_box_mesh_name" value="top_box.dae" />
+		</xacro:unless>
 			<link name="$(arg prefix)top_box">
 					<visual>
@@ -525,5 +636,5 @@
 							<geometry>
 									<mesh scale="${top_box_scale} ${top_box_scale} ${top_box_scale}"
-												filename="package://ctu_cras_norlab_absolem_sensor_config_1/meshes/top_box.dae"/>
+												filename="package://ctu_cras_norlab_absolem_sensor_config_1/meshes/${top_box_mesh_name}"/>
 							</geometry>
 					</visual>
@@ -533,5 +644,5 @@
 									<geometry>
 											<mesh scale="${top_box_scale} ${top_box_scale} ${top_box_scale}"
-														filename="package://ctu_cras_norlab_absolem_sensor_config_1/meshes/top_box.dae"/>
+														filename="package://ctu_cras_norlab_absolem_sensor_config_1/meshes/${top_box_mesh_name}"/>
 									</geometry>
 							</collision>
@@ -542,23 +653,59 @@
 									<geometry>
 											<mesh scale="${top_box_scale} ${top_box_scale} ${top_box_scale}"
-														filename="package://ctu_cras_norlab_absolem_sensor_config_1/meshes/collide/top_box.dae"/>
+														filename="package://ctu_cras_norlab_absolem_sensor_config_1/meshes/collide/${top_box_mesh_name}"/>
 									</geometry>
 							</collision>
 					</xacro:if>
 					<xacro:if value="${$(arg simplified_collision)==2}">
+							<!-- the box -->
 							<collision>
+								<xacro:if value="${'$(arg revision)' == '2021'}">
+									<xacro:if value="$(arg has_omnicam)">
+										<origin rpy="0 0 0" xyz="0 0 0.0315"/>
+										<geometry>
+											<box size="0.1270 0.231 0.06252" />
+										</geometry>
+									</xacro:if>
+									<xacro:if value="$(arg has_omnicam_vras)">
+										<!-- TODO -->
+									</xacro:if>
+								</xacro:if>
+								<xacro:unless value="${'$(arg revision)' == '2021'}">
 									<origin rpy="0 0 0" xyz="-0.0290 0 0.0315"/>
 									<geometry>
 											<box size="0.2000 0.1330 0.06252" />
 									</geometry>
+								</xacro:unless>
 							</collision>
+							<!-- GPS antenna -->
 							<collision>
-									<origin rpy="0 0 0" xyz="-0.09824 0.04127 0.0690"/>
+									<xacro:if value="${'$(arg revision)' == '2021'}">
+										<xacro:if value="$(arg has_omnicam)">
+											<origin rpy="0 0 0" xyz="-0.04 0.09 0.0690"/>
+										</xacro:if>
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