Commit message: Model submission for Absolem sensor configurations 3,4,5 by CTU-CRAS-Norlab (#859)
* Absolem: Sync Xacro: Change IMU and friction parameters in Xacro to correspond to the desired values in SDF.

* Absolem: Sync Xacro: Re-generate model.sdf using libsdformat 8.9.1 .

This commit makes no real change to the geometry of the model, it just represents some numbers and rotations differently.

* Absolem: Removed empty link visuals as they obstructed the omnicam and were not good for anything else.

* Absolem: Modernized tooling for reuse by other sensor configs.

model.sdf remains unchanged (up to a comment at the very top)

spawner.rb and vehicle_topics.launch changed a lot, but I tested them thoroughly and they keep behaving exactly the same as before.

* Absolem: Added sensor config 3 (facelifted version with 3D lidar).

* Absolem: Added Sensor Config 4.

* Absolem: Added sensor config 5.

* Absolem: Added <depend> tags to sensor configs that pull resources from sensor config 1.

* Absolem: configurable length of big collision box.

* Absolem: Added ceiling light.

* Absolem SC5: Fixed ceiling light position.

* Absolem: update.

* Absolem: Changed lidar and thermocam parameters, fixed RViz model.

File: submitted_models/ctu_cras_norlab_absolem_sensor_config_1/urdf/nifti_robot.xacro (robot description, xacro)
@@ -178,4 +178,43 @@
 	<xacro:arg default="0.000000" name="d435_pos_y"/>
 	<xacro:arg default="0.000000" name="d435_pos_x"/>
+	<xacro:arg default="1.000000" name="ouster_quat_w"/>
+	<xacro:arg default="0.000000" name="ouster_quat_z"/>
+	<xacro:arg default="0.000000" name="ouster_quat_y"/>
+	<xacro:arg default="0.000000" name="ouster_quat_x"/>
+	<xacro:arg default="0.000000" name="ouster_gzrpy_y"/>
+	<xacro:arg default="0.000000" name="ouster_gzrpy_p"/>
+	<xacro:arg default="0.000000" name="ouster_gzrpy_r"/>
+	<xacro:arg default="0.000000" name="ouster_rpy_y"/>
+	<xacro:arg default="0.000000" name="ouster_rpy_p"/>
+	<xacro:arg default="0.000000" name="ouster_rpy_r"/>
+	<xacro:arg default="0.200000" name="ouster_pos_z"/>
+	<xacro:arg default="0.000000" name="ouster_pos_y"/>
+	<xacro:arg default="0.070000" name="ouster_pos_x"/>
+	<xacro:arg default="1.000000" name="boson_quat_w"/>
+	<xacro:arg default="0.000000" name="boson_quat_z"/>
+	<xacro:arg default="0.000000" name="boson_quat_y"/>
+	<xacro:arg default="0.000000" name="boson_quat_x"/>
+	<xacro:arg default="0.000000" name="boson_gzrpy_y"/>
+	<xacro:arg default="0.000000" name="boson_gzrpy_p"/>
+	<xacro:arg default="0.000000" name="boson_gzrpy_r"/>
+	<xacro:arg default="0.000000" name="boson_rpy_y"/>
+	<xacro:arg default="0.000000" name="boson_rpy_p"/>
+	<xacro:arg default="0.000000" name="boson_rpy_r"/>
+	<xacro:arg default="0.000000" name="boson_pos_z"/>
+	<xacro:arg default="0.000000" name="boson_pos_y"/>
+	<xacro:arg default="0.000000" name="boson_pos_x"/>
+	<xacro:arg default="0.042087" name="camera_0_pos_x"/>
+	<xacro:arg default="0.000000" name="cliff_sensor_0_x"/>
+	<xacro:arg default="0.000000" name="cliff_sensor_0_y"/>
+	<xacro:arg default="0.000000" name="cliff_sensor_0_yaw"/>
+	<xacro:arg default="0.000000" name="cliff_sensor_1_x"/>
+	<xacro:arg default="0.000000" name="cliff_sensor_1_y"/>
+	<xacro:arg default="0.000000" name="cliff_sensor_1_yaw"/>
+	<xacro:arg default="0.000000" name="cliff_sensor_2_x"/>
+	<xacro:arg default="0.000000" name="cliff_sensor_2_y"/>
+	<xacro:arg default="0.000000" name="cliff_sensor_2_yaw"/>
+	<xacro:arg default="0.000000" name="cliff_sensor_3_x"/>
+	<xacro:arg default="0.000000" name="cliff_sensor_3_y"/>
+	<xacro:arg default="0.000000" name="cliff_sensor_3_yaw"/>
 	<xacro:arg default="0.070500" name="rover_referentialZ"/>
 	<xacro:arg default="0.600000" name="rover_vMaxRun"/>
@@ -193,4 +232,7 @@
 	<xacro:arg default="0.300000" name="rover_vMaxTravel"/>
 	<xacro:arg default="0.240930" name="rover_robotWidthBody"/>
+	<xacro:arg default="0.500170" name="rover_robotLengthBody"/>
+	<xacro:arg default="-0.12200" name="rover_robotBodyShift"/>
+	<xacro:arg default="0.022000" name="rover_bodyEdgeCurvature"/> <!-- curvature of the front and rear bottom edges -->
 	<xacro:arg default="0.397000" name="rover_trackDistance"/>
 	<xacro:arg default="0.330000" name="rover_flipperLength"/>
@@ -209,15 +251,27 @@
 			 Example of value: '0 1 0 1' (don't forget to set alpha to 1!). -->
 	<xacro:arg name="body_color" default="" />
+	<!-- Body shape revision. Possible values are 2010, 2014 and 2021 -->
+	<xacro:arg name="revision" default="2014" />
 	<xacro:arg name="has_top_box" default="1" />
 	<!-- Distance from robot's back to top box' front panel. Default is the front-most position. -->
 	<xacro:arg name="top_box_j_x" default="0.4977" />
 	<xacro:arg name="has_sick_lidar" default="1" />
+	<xacro:arg name="has_ouster_lidar" default="0" />
 	<xacro:arg name="has_omnicam" default="1" />
+	<xacro:arg name="has_omnicam_vras" default="0" />
 	<xacro:arg name="has_omnicam_sensor_mount" default="1" />
 	<xacro:arg name="has_flippers" default="1" />
 	<xacro:arg name="has_differential" default="1" />
+	<xacro:arg name="has_new_realsense" default="0" />
+	<xacro:arg name="has_realsense_d435" default="0" />
+	<xacro:arg name="has_realsense_t265" default="0" />
+	<xacro:arg name="has_jetson" default="0" />
+	<xacro:arg name="has_mote_deployer" default="0" />
+	<xacro:arg name="has_boson_thermocam" default="0" />
+	<xacro:arg name="num_cliff_sensors" default="0" />
 	<xacro:arg name="has_rear_sensor_item" default="1" />
 	<xacro:arg name="rear_sensor_item_x" default="0.084" />
 	<xacro:arg name="rear_sensor_item_y" default="0.02" />
+	<xacro:arg name="rear_sensor_item_height" default="0.35" />
 	<xacro:arg name="laser_pitch" default="0.0" />
 	<!-- render_xacro.py allows use of arguments like $(arg rover_trackLength) etc. which are not defined here -->
@@ -227,4 +281,5 @@
 	<xacro:arg name="big_collision_box_height" default="0.25" />
 	<xacro:arg name="big_collision_box_width" default="0.31" />
+	<xacro:arg name="big_collision_box_length" default="0.65" />
 	<xacro:arg name="big_collision_box_x" default="-0.21" />
 	<xacro:arg name="flipper_inflation_ratio" default="1.0" />
@@ -263,7 +318,12 @@
     <xacro:arg name="perfect_odometry" default="False" /> <!-- If True, ground truth position will be published as odom frame. -->
     <xacro:arg name="simulate_sick_lidar" default="True" />
+    <xacro:arg name="simulate_ouster_lidar" default="True" />
     <xacro:arg name="simulate_omnicam" default="True" />
+    <xacro:arg name="simulate_omnicam_vras" default="True" />
     <xacro:arg name="simulate_realsense_d435" default="True" />
     <xacro:arg name="simulate_imu" default="True" />
+    <xacro:arg name="simulate_cliff_sensors" default="True" />
+    <xacro:arg name="simulate_thermocam" default="True" />
+    <xacro:arg name="visualize_sensors" default="False" />
     <xacro:arg name="differential_locked" default="true" />
     <xacro:arg name="laser_update_rate" default="1000.0" />
@@ -287,5 +347,5 @@
 	<!-- MACRO SPECIFICATIONS -->
 	<xacro:include filename="$(find ctu_cras_norlab_absolem_sensor_config_1)/urdf/utils.xacro" />
-	<xacro:macro name="calibrated_fixed_joint" params="name parent child prefix:=''">
+	<xacro:macro name="calibrated_fixed_joint" params="name parent child prefix:='' lump:='1'">
 			<!-- These arguments are filled by render_xacro.py from calibration data. -->
 			<xacro:if value="${prefix == ''}">
@@ -297,10 +357,17 @@
 			<xacro:fixed_joint name="${name}" parent="$(arg prefix)${parent}" child="$(arg prefix)${child}"
 												 xyz="$(arg ${pref}_pos_x) $(arg ${pref}_pos_y) $(arg ${pref}_pos_z)"
-												 rpy="$(arg ${pref}_rpy_r) $(arg ${pref}_rpy_p) $(arg ${pref}_rpy_y)" />
+												 rpy="$(arg ${pref}_rpy_r) $(arg ${pref}_rpy_p) $(arg ${pref}_rpy_y)"
+												 lump="${lump}"/>
 	</xacro:macro>
 	<!-- SPECIAL LINKS -->
 	<!-- This is a virtual link that specifies the origin to which parts attachable to the top of the robot should be related. -->
 	<link name="$(arg prefix)rear_right_box" />
-	<xacro:fixed_joint name="rear_right_box_j" parent="$(arg prefix)base_link" child="$(arg prefix)rear_right_box" rpy="0 0 0" xyz="-0.379 -0.1265 0.185"/>
+	<xacro:if value="${'$(arg revision)' == '2021'}">
+		<xacro:fixed_joint name="rear_right_box_j" parent="$(arg prefix)base_link" child="$(arg prefix)rear_right_box" rpy="0 0 0"
+						   xyz="${-$(arg rover_robotLengthBody)/2} ${-$(arg rover_robotWidthBody)/2} 0.185"/>
+	</xacro:if>
+	<xacro:unless value="${'$(arg revision)' == '2021'}">
+		<xacro:fixed_joint name="rear_right_box_j" parent="$(arg prefix)base_link" child="$(arg prefix)rear_right_box" rpy="0 0 0" xyz="-0.379 -0.1265 0.185"/>
+	</xacro:unless>
 	<!-- INCLUDES -->
 	<xacro:if value="$(arg has_jetson)">
@@ -316,7 +383,25 @@
 		<xacro:include filename="$(find ctu_cras_norlab_absolem_sensor_config_1)/urdf/t265_attach_to_robot.xacro" />
 	</xacro:if>
+	<xacro:if value="$(arg has_ouster_lidar)">
+		<xacro:include filename="$(find ctu_cras_norlab_absolem_sensor_config_1)/urdf/ouster_lidar.xacro" />
+	</xacro:if>
+	<xacro:if value="$(arg has_mote_deployer)">
+		<xacro:include filename="$(find ctu_cras_norlab_absolem_sensor_config_1)/urdf/mote_deployer.xacro" />
+	</xacro:if>
+	<xacro:if value="${'$(arg revision)' == '2021'}">
+		<xacro:include filename="$(find ctu_cras_norlab_absolem_sensor_config_1)/urdf/lights.xacro" />
+	</xacro:if>
+	<xacro:if value="$(arg has_boson_thermocam)">
+		<xacro:include filename="$(find ctu_cras_norlab_absolem_sensor_config_1)/urdf/boson_thermocam.xacro" />
+	</xacro:if>
 	<!-- NIFTI ROBOT LINKS AND JOINTS SPECIFICATION -->
 	<xacro:property name="body_color" value="$(arg body_color)" />
 	<link name="$(arg prefix)base_link">
+			<xacro:if value="${'$(arg revision)' == '2021'}">
+				<xacro:property name="body_mesh_name" value="body_2021.dae" />
+			</xacro:if>
+			<xacro:unless value="${'$(arg revision)' == '2021'}">
+				<xacro:property name="body_mesh_name" value="body.dae" />
+			</xacro:unless>
 			<xacro:if value="${len(body_color) == 0}">
 					<visual>
@@ -324,5 +409,5 @@
 							<geometry>
 									<mesh scale="${body_scale} ${body_scale} ${body_scale}"
-												filename="package://ctu_cras_norlab_absolem_sensor_config_1/meshes/body.dae"/>
+												filename="package://ctu_cras_norlab_absolem_sensor_config_1/meshes/${body_mesh_name}"/>
 							</geometry>
 					</visual>
@@ -330,7 +415,7 @@
 			<xacro:if value="${len(body_color) > 0}">
 					<visual>
-							<origin rpy="0 0 0" xyz="-0.1220 0 0.118"/>
-							<geometry>
-									<box size="0.50017 $(arg rover_robotWidthBody) 0.1390" />
+							<origin rpy="0 0 0" xyz="$(arg rover_robotBodyShift) 0 0.118"/>
+							<geometry>
+									<box size="$(arg rover_robotLengthBody) $(arg rover_robotWidthBody) 0.1390" />
 							</geometry>
 							<material name="body_color">
@@ -338,31 +423,41 @@
 							</material>
 					</visual>
-					<visual>
-							<origin rpy="0 0 0" xyz="0.157 0 0.118"/>
-							<geometry>
-									<box size="0.056 0.12093 0.1390" />
-							</geometry>
-							<material name="body_color">
-									<color rgba="$(arg body_color)"/>
-							</material>
-					</visual>
-					<visual>
-							<origin rpy="0 0 0.785398" xyz="0.144 -0.076 0.118"/>
-							<geometry>
-									<box size="0.083 0.040 0.1390" />
-							</geometry>
-							<material name="body_color">
-									<color rgba="$(arg body_color)"/>
-							</material>
-					</visual>
-					<visual>
-							<origin rpy="0 0 -0.785398" xyz="0.144 0.076 0.118"/>
-							<geometry>
-									<box size="0.083 0.040 0.1390" />
-							</geometry>
-							<material name="body_color">
-									<color rgba="$(arg body_color)"/>
-							</material>
-					</visual>
+					<xacro:unless value="${'$(arg revision)' == '2021'}">
+						<visual>
+								<origin rpy="0 0 0" xyz="0.157 0 0.118"/>
+								<geometry>
+										<box size="0.056 0.12093 0.1390" />
+								</geometry>
+								<material name="body_color">
+										<color rgba="$(arg body_color)"/>
+								</material>
+						</visual>
+						<visual>
+								<origin rpy="0 0 0.785398" xyz="0.144 -0.076 0.118"/>
+								<geometry>
+										<box size="0.083 0.040 0.1390" />
+								</geometry>
+								<material name="body_color">
+										<color rgba="$(arg body_color)"/>
+								</material>
+						</visual>
+						<visual>
+								<origin rpy="0 0 -0.785398" xyz="0.144 0.076 0.118"/>
+								<geometry>
+										<box size="0.083 0.040 0.1390" />
+								</geometry>
+								<material name="body_color">
+										<color rgba="$(arg body_color)"/>
+								</material>
+						</visual>
+					</xacro:unless>
+			</xacro:if>
+			<xacro:if value="${'$(arg revision)' == '2021' and $(arg has_omnicam)}">
+				<visual>
+					<origin rpy="0 ${3*pi/2} ${pi/2}" xyz="-0.18 0 0.185" />
+					<geometry>
+						<mesh filename="package://ctu_cras_norlab_absolem_sensor_config_1/meshes/reflector.dae" />
+					</geometry>
+				</visual>
 			</xacro:if>
 			<xacro:if value="${$(arg simplified_collision)==0}">
@@ -371,5 +466,5 @@
 							<geometry>
 									<mesh scale="${body_scale} ${body_scale} ${body_scale}"
-												filename="package://ctu_cras_norlab_absolem_sensor_config_1/meshes/body.dae"/>
+												filename="package://ctu_cras_norlab_absolem_sensor_config_1/meshes/${body_mesh_name}"/>
 							</geometry>
 					</collision>
@@ -380,5 +475,5 @@
 							<geometry>
 									<mesh scale="${body_scale} ${body_scale} ${body_scale}"
-												filename="package://ctu_cras_norlab_absolem_sensor_config_1/meshes/collide/body.dae"/>
+												filename="package://ctu_cras_norlab_absolem_sensor_config_1/meshes/collide/${body_mesh_name}"/>
 							</geometry>
 					</collision>
@@ -386,27 +481,37 @@
 			<xacro:if value="${$(arg simplified_collision)==2}">
 					<collision>
-							<origin rpy="0 0 0" xyz="-0.1220 0 0.118"/>
-							<geometry>
-									<box size="0.50017 $(arg rover_robotWidthBody) 0.1390" />
-							</geometry>
-					</collision>
-					<collision>
-							<origin rpy="0 0 0" xyz="0.157 0 0.118"/>
-							<geometry>
-									<box size="0.056 0.12093 0.1390" />
-							</geometry>
-					</collision>
-					<collision>
-							<origin rpy="0 0 0.785398" xyz="0.144 -0.076 0.118"/>
-							<geometry>
-									<box size="0.083 0.040 0.1390" />
-							</geometry>
-					</collision>
-					<collision>
-							<origin rpy="0 0 -0.785398" xyz="0.144 0.076 0.118"/>
-							<geometry>
-									<box size="0.083 0.040 0.1390" />
-							</geometry>
-					</collision>
+							<xacro:if value="${'$(arg revision)' == '2021'}">
+								<xacro:property name="bodyCollHeight" value="${0.1390 - $(arg rover_bodyEdgeCurvature)}" />
+								<xacro:property name="bodyCollZshift" value="${0.118 + $(arg rover_bodyEdgeCurvature)/2}" />
+							</xacro:if>
+							<xacro:unless value="${'$(arg revision)' == '2021'}">
+								<xacro:property name="bodyCollHeight" value="0.1390" />
+								<xacro:property name="bodyCollZshift" value="0.118" />
+							</xacro:unless>
+							<origin rpy="0 0 0" xyz="$(arg rover_robotBodyShift) 0 ${bodyCollZshift}"/>
+							<geometry>
+									<box size="$(arg rover_robotLengthBody) $(arg rover_robotWidthBody) ${bodyCollHeight}" />
+							</geometry>
+					</collision>
+				    <xacro:unless value="${'$(arg revision)' == '2021'}">
+						<collision>
+								<origin rpy="0 0 0" xyz="0.157 0 0.118"/>
+								<geometry>
+										<box size="0.056 0.12093 0.1390" />
+								</geometry>
+						</collision>
+						<collision>
+								<origin rpy="0 0 0.785398" xyz="0.144 -0.076 0.118"/>
+								<geometry>
+										<box size="0.083 0.040 0.1390" />
+								</geometry>
+						</collision>
+						<collision>
+								<origin rpy="0 0 -0.785398" xyz="0.144 0.076 0.118"/>
+								<geometry>
+										<box size="0.083 0.040 0.1390" />
+								</geometry>
+						</collision>
+					</xacro:unless>
 					<collision>
 							<origin rpy="0 0 0" xyz="0 0.135 0.09"/>
@@ -433,4 +538,28 @@
 							</geometry>
 					</collision>
+					<xacro:if value="${'$(arg revision)' == '2021'}">
+						<collision>
+							<origin rpy="0 0 0" xyz="0 0 ${0.048 + $(arg rover_bodyEdgeCurvature)/2}"/>
+							<geometry>
+								<box size="${$(arg rover_robotLengthBody) - 2*$(arg rover_bodyEdgeCurvature)} $(arg rover_robotWidthBody) $(arg rover_bodyEdgeCurvature)" />
+							</geometry>
+						</collision>
+						<collision>
+							<!-- We enlarge the radius a tiny bit to avoid wrong contact forces on the interface between the bottom plate and the cylinder -->
+							<origin xyz="${$(arg rover_robotLengthBody)/2-$(arg rover_bodyEdgeCurvature)} 0 ${0.048 + $(arg rover_bodyEdgeCurvature)}"
+									rpy="${pi/2} 0 0"/>
+							<geometry>
+								<cylinder length="$(arg rover_robotWidthBody)" radius="${$(arg rover_bodyEdgeCurvature)*1.001}" />
+							</geometry>
+						</collision>
+						<collision>
+							<!-- We enlarge the radius a tiny bit to avoid wrong contact forces on the interface between the bottom plate and the cylinder -->
+							<origin xyz="${-$(arg rover_robotLengthBody)/2+$(arg rover_bodyEdgeCurvature)} 0 ${0.048 + $(arg rover_bodyEdgeCurvature)}"
+									rpy="${pi/2} 0 0"/>
+							<geometry>
+								<cylinder length="$(arg rover_robotWidthBody)" radius="${$(arg rover_bodyEdgeCurvature)*1.001}" />
+							</geometry>
+						</collision>
+					</xacro:if>
 			</xacro:if>
 			<xacro:if value="$(arg big_collision_box_on_top)">
@@ -438,5 +567,5 @@
 							<origin rpy="0 0 0" xyz="$(arg big_collision_box_x) 0 ${0.08 + $(arg big_collision_box_height)/2}"/>
 							<geometry>
-									<box size="0.65 $(arg big_collision_box_width) $(arg big_collision_box_height)" />
+									<box size="$(arg big_collision_box_length) $(arg big_collision_box_width) $(arg big_collision_box_height)" />
 							</geometry>
 					</collision>
@@ -456,7 +585,7 @@
 			<link name="$(arg prefix)rear_sensor_item">
 					<visual>
-							<origin xyz="0 0 ${0.35/2}" rpy="0 0 0" />
-							<geometry>
-									<box size="0.02 0.02 0.35"/>
+							<origin xyz="0 0 ${$(arg rear_sensor_item_height)/2}" rpy="0 0 0" />
+							<geometry>
+									<box size="0.02 0.02 $(arg rear_sensor_item_height)"/>
 							</geometry>
 							<material name="aluminium">
@@ -465,7 +594,7 @@
 					</visual>
 					<collision>
-							<origin xyz="0 0 ${0.35/2}" rpy="0 0 0" />
-							<geometry>
-									<box size="0.02 0.02 0.35" />
+							<origin xyz="0 0 ${$(arg rear_sensor_item_height)/2}" rpy="0 0 0" />
+							<geometry>
+									<box size="0.02 0.02 $(arg rear_sensor_item_height)" />
 							</geometry>
 					</collision>
@@ -518,6 +647,17 @@
 			</inertial>
 	</link>
-	<xacro:fixed_joint name="battery_j" parent="$(arg prefix)base_link" child="$(arg prefix)battery" xyz="-0.2836 -0.0221 0.0722" rpy="0 0 0" />
+	<xacro:unless value="${'$(arg revision)' == '2021'}">
+		<xacro:fixed_joint name="battery_j" parent="$(arg prefix)base_link" child="$(arg prefix)battery" xyz="-0.2836 -0.0221 0.0722" rpy="0 0 0" />
+	</xacro:unless>
+	<xacro:if value="${'$(arg revision)' == '2021'}">
+		<xacro:fixed_joint name="battery_j" parent="$(arg prefix)base_link" child="$(arg prefix)battery" xyz="-0.12 0 0.12" rpy="0 ${pi/2} 0" />
+	</xacro:if>
 	<xacro:if value="$(arg has_top_box)">
+		<xacro:if value="${'$(arg revision)' == '2021'}">
+			<xacro:property name="top_box_mesh_name" value="top_box_2021_ladybug.dae" />
+		</xacro:if>
+		<xacro:unless value="${'$(arg revision)' == '2021'}">
+			<xacro:property name="top_box_mesh_name" value="top_box.dae" />
+		</xacro:unless>
 			<link name="$(arg prefix)top_box">
 					<visual>
@@ -525,5 +665,5 @@
 							<geometry>
 									<mesh scale="${top_box_scale} ${top_box_scale} ${top_box_scale}"
-												filename="package://ctu_cras_norlab_absolem_sensor_config_1/meshes/top_box.dae"/>
+												filename="package://ctu_cras_norlab_absolem_sensor_config_1/meshes/${top_box_mesh_name}"/>
 							</geometry>
 					</visual>
@@ -533,5 +673,5 @@
 									<geometry>
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
File: submitted_models/ctu_cras_norlab_absolem_sensor_config_1/urdf/utils.xacro (robot description, xacro)
@@ -7,8 +7,8 @@
                 izz="${izz*scale*scale}"/>
     </xacro:macro>
-    <xacro:macro name="sphere_inertial" params="radius mass *origin">
+    <xacro:macro name="sphere_inertial" params="radius mass xyz:='0 0 0'">
         <inertial>
             <mass value="${mass}" />
-            <xacro:insert_block name="origin" />
+            <origin xyz="${xyz}" rpy="0 0 0"/>
             <inertia ixx="${2.0/5 * mass * radius * radius}" ixy="0.0" ixz="0.0"
                      iyy="${2.0/5 * mass * radius * radius}" iyz="0.0"
@@ -16,17 +16,17 @@
         </inertial>
     </xacro:macro>
-    <xacro:macro name="box_inertial" params="width height depth mass *origin">
+    <xacro:macro name="box_inertial" params="width height depth mass xyz:='0 0 0' rpy:='0 0 0'">
         <inertial>
             <mass value="${mass}" />
-            <xacro:insert_block name="origin" />
-            <inertia ixx="${1.0/12 * mass * (height * height + depth * depth)}" ixy="0.0" ixz="0.0"
-                     iyy="${1.0/12 * mass * (width * width + depth * depth)}" iyz="0.0"
-                     izz="${1.0/12 * mass * (width * width + height * height)}" />
+            <origin xyz="${xyz}" rpy="${rpy}"/>
+            <inertia ixx="${1.0/12 * mass * (width * width + height * height)}" ixy="0.0" ixz="0.0"
+                     iyy="${1.0/12 * mass * (height * height + depth * depth)}" iyz="0.0"
+                     izz="${1.0/12 * mass * (width * width + depth * depth)}" />
         </inertial>
     </xacro:macro>
-    <xacro:macro name="cylinder_inertial" params="radius length mass *origin">
+    <xacro:macro name="cylinder_inertial" params="radius length mass xyz:='0 0 0' rpy:='0 0 0'">
         <inertial>
             <mass value="${mass}" />
-            <xacro:insert_block name="origin" />
+            <origin xyz="${xyz}" rpy="${rpy}"/>
             <inertia ixx="${1.0/12 * mass * (3 * radius * radius + length * length)}" ixy="0.0" ixz="0.0"
                      iyy="${1.0/12 * mass * (3 * radius * radius + length * length)}" iyz="0.0"
@@ -48,5 +48,5 @@
         </link>
     </xacro:macro>
-    <xacro:macro name="fixed_joint" params="name parent child xyz='0 0 0' rpy='0 0 0'">
+    <xacro:macro name="fixed_joint" params="name parent child xyz:='0 0 0' rpy:='0 0 0' lump:=1">
         <joint name="${name}" type="fixed">
             <parent link="${parent}"/>
@@ -54,4 +54,10 @@
             <origin xyz="${xyz}" rpy="${rpy}"/>
         </joint>
+        <xacro:if value="${lump == 0}">
+            <!-- workaround for https://github.com/osrf/sdformat/issues/378 -->
+            <gazebo reference="${name}">
+                <preserveFixedJoint>true</preserveFixedJoint>
+            </gazebo>
+        </xacro:if>
     </xacro:macro>
 </root>
