Commit message: Implement proper tracked motion model (#958)
* Absolem: fix bad merge.

* Implement more plausible model of tracks.

* Merge upstream thermal cam settings for MARV SC3

* Update with latest changes.

* Removed empty wheel slip plugin.

* Use power_draining_topic to start battery drain for tracked vehicles.

File: submitted_models/ctu_cras_norlab_absolem_sensor_config_1/urdf/nifti_robot.xacro (robot description, xacro)
@@ -302,4 +302,5 @@
 	<xacro:arg name="base_link_cog_offset" default="0.0" />
 	<xacro:arg name="rendering_target" default="urdf" /> <!-- Pass either "urdf" or "sdf" to tell the parser what is the desired target format. -->
+	<xacro:arg name="wheels_instead_of_tracks" default="true" />
     <!-- 17.0 for real max torque, 3.0; 40.0 for real 6.0 -->
     <xacro:arg name="max_flipper_torque" default="17.0" />
@@ -893,11 +894,43 @@
 							</visual>
 					</xacro:if>
-					<collision>
-							<origin rpy="0 0 0" xyz="0 0 0"/>
-							<geometry>
-									<box size="0.01 0.01 0.01"/>
-							</geometry>
-					</collision>
-					<xacro:default_inertial />
+					<xacro:if value="${$(arg wheels_instead_of_tracks)}">
+						<collision>
+								<origin rpy="0 0 0" xyz="0 0 0"/>
+								<geometry>
+										<box size="0.01 0.01 0.01"/>
+								</geometry>
+						</collision>
+						<xacro:default_inertial />
+					</xacro:if>
+					<xacro:unless value="${$(arg wheels_instead_of_tracks)}">
+						<collision>
+							<origin xyz="0 0 0.01855" rpy="${pi/2} 0 ${pi/2}" />
+							<geometry>
+								<box size="$(arg rover_trackWidth) ${2*$(arg rover_trackWheelRadius)} $(arg rover_trackLength)"/>
+							</geometry>
+						</collision>
+						<collision>
+							<origin rpy="${pi/2} 0 0" xyz="${$(arg rover_trackLength)/2} ${-reflect*$(arg track_inward_enlargement)} 0.01855"/>
+							<geometry>
+								<!-- enlarged because of laser filtering problems -->
+								<cylinder radius="$(arg rover_trackWheelRadius)" length="${$(arg rover_trackWidth)+$(arg track_inward_enlargement)}"/>
+							</geometry>
+						</collision>
+						<collision>
+							<origin rpy="${pi/2} 0 0" xyz="${-$(arg rover_trackLength)/2} 0 0.01855"/>
+							<geometry>
+								<cylinder radius="$(arg rover_trackWheelRadius)" length="$(arg rover_trackWidth)"/>
+							</geometry>
+						</collision>
+						<inertial>
+							<origin xyz="0 0 0.0141" rpy="0 0 0"/>
+							<mass value="${track_mass}"/>
+							<xacro:inertia_meshlab
+									ixx="0.002731" ixy="0" ixz="0"
+									iyy="0.032554" iyz="0.000015"
+									izz="0.031391"
+									scale="${track_scale}" mass="${track_mass}" />
+						</inertial>
+					</xacro:unless>
 			</link>
 			<joint name="${prefix}_track_j" type="revolute">
@@ -912,12 +945,14 @@
 					</xacro:if>
 			</joint>
-			<xacro:fake_wheel prefix="${prefix}" reflect="${reflect}" num_wheels="8" wheel_num="1" />
-			<xacro:fake_wheel prefix="${prefix}" reflect="${reflect}" num_wheels="8" wheel_num="2" />
-			<xacro:fake_wheel prefix="${prefix}" reflect="${reflect}" num_wheels="8" wheel_num="3" />
-			<xacro:fake_wheel prefix="${prefix}" reflect="${reflect}" num_wheels="8" wheel_num="4" />
-			<xacro:fake_wheel prefix="${prefix}" reflect="${reflect}" num_wheels="8" wheel_num="5" />
-			<xacro:fake_wheel prefix="${prefix}" reflect="${reflect}" num_wheels="8" wheel_num="6" />
-			<xacro:fake_wheel prefix="${prefix}" reflect="${reflect}" num_wheels="8" wheel_num="7" />
-			<xacro:fake_wheel prefix="${prefix}" reflect="${reflect}" num_wheels="8" wheel_num="8" />
+			<xacro:if value="${$(arg wheels_instead_of_tracks)}">
+				<xacro:fake_wheel prefix="${prefix}" reflect="${reflect}" num_wheels="8" wheel_num="1" />
+				<xacro:fake_wheel prefix="${prefix}" reflect="${reflect}" num_wheels="8" wheel_num="2" />
+				<xacro:fake_wheel prefix="${prefix}" reflect="${reflect}" num_wheels="8" wheel_num="3" />
+				<xacro:fake_wheel prefix="${prefix}" reflect="${reflect}" num_wheels="8" wheel_num="4" />
+				<xacro:fake_wheel prefix="${prefix}" reflect="${reflect}" num_wheels="8" wheel_num="5" />
+				<xacro:fake_wheel prefix="${prefix}" reflect="${reflect}" num_wheels="8" wheel_num="6" />
+				<xacro:fake_wheel prefix="${prefix}" reflect="${reflect}" num_wheels="8" wheel_num="7" />
+				<xacro:fake_wheel prefix="${prefix}" reflect="${reflect}" num_wheels="8" wheel_num="8" />
+			</xacro:if>
 	</xacro:macro>
 	<xacro:macro name="fake_wheel" params="prefix reflect num_wheels wheel_num">
@@ -982,11 +1017,54 @@
 							</geometry>
 					</visual>
-					<collision>
-							<origin rpy="0 0 0" xyz="0 0 0"/>
-							<geometry>
-									<box size="0.01 0.01 0.01"/>
-							</geometry>
-					</collision>
-					<xacro:default_inertial />
+					<xacro:if value="${$(arg wheels_instead_of_tracks)}">
+						<collision>
+								<origin rpy="0 0 0" xyz="0 0 0"/>
+								<geometry>
+										<box size="0.01 0.01 0.01"/>
+								</geometry>
+						</collision>
+						<xacro:default_inertial />
+					</xacro:if>
+					<xacro:unless value="${$(arg wheels_instead_of_tracks)}">
+						<collision name="${prefix1}_${prefix2}_flipper_collision_large_wheel">
+							<origin rpy="${pi/2} 0 0" xyz="0 ${-reflect_y*$(arg flipper_inward_enlargement)*do_inward_enlargement/2.0} 0"/>
+							<geometry>
+								<cylinder length="${$(arg rover_flipperWidth)+$(arg flipper_inward_enlargement)*do_inward_enlargement}" radius="$(arg rover_trackWheelRadius)" />
+							</geometry>
+						</collision>
+						<collision name="${prefix1}_${prefix2}_flipper_collision_small_wheel">
+							<origin rpy="${pi/2} 0 0" xyz="${reflect_y*$(arg rover_flipperLength)} ${-reflect_y*$(arg flipper_inward_enlargement)*do_inward_enlargement/2.0} 0.0"/>
+							<geometry>
+								<cylinder length="${$(arg rover_flipperWidth)+$(arg flipper_inward_enlargement)*do_inward_enlargement}" radius="${0.029 + 0.029*($(arg flipper_inflation_ratio)-1)*do_inward_enlargement}" />
+							</geometry>
+						</collision>
+						<collision name="${prefix1}_${prefix2}_flipper_collision_top_bar">
+							<origin rpy="0 0.184162095 ${(1-reflect_y)*pi/2}" xyz="${reflect_y*$(arg rover_flipperLength)/2.0} ${-reflect_y*$(arg flipper_inward_enlargement)*do_inward_enlargement/2.0} 0.0325"/>
+							<geometry>
+								<box size="$(arg rover_flipperLength) ${$(arg rover_flipperWidth)+$(arg flipper_inward_enlargement)*do_inward_enlargement} ${0.055 + 0.055*($(arg flipper_inflation_ratio)-1)*do_inward_enlargement}" />
+							</geometry>
+						</collision>
+						<collision name="${prefix1}_${prefix2}_flipper_collision_bottom_bar">
+							<origin rpy="0 -0.184162095 ${(1-reflect_y)*pi/2}" xyz="${reflect_y*$(arg rover_flipperLength)/2} ${-reflect_y*$(arg flipper_inward_enlargement)*do_inward_enlargement/2.0} -0.0325"/>
+							<geometry>
+								<box size="$(arg rover_flipperLength) ${$(arg rover_flipperWidth)+$(arg flipper_inward_enlargement)*do_inward_enlargement} ${0.055 + 0.055*($(arg flipper_inflation_ratio)-1)*do_inward_enlargement}" />
+							</geometry>
+						</collision>
+						<collision name="${prefix1}_${prefix2}_flipper_collision_middle_bar">
+							<origin rpy="0 -0.02 ${(1-reflect_y)*pi/2}" xyz="${reflect_y*($(arg rover_flipperLength)/2.0 + 0.001)} ${-reflect_y*$(arg flipper_inward_enlargement)*do_inward_enlargement/2.0} 0.004"/>
+							<geometry>
+								<box size="0.20 ${$(arg rover_flipperWidth)+$(arg flipper_inward_enlargement)*do_inward_enlargement} 0.07" />
+							</geometry>
+						</collision>
+						<inertial>
+							<origin xyz="${reflect_y*0.08} 0 0.0" rpy="0 0 0"/>
+							<mass value="${flipper_mass}"/>
+							<xacro:inertia_meshlab
+									ixx="1.7491e-003" ixy="2.8512e-007" ixz="1.8277e-003"
+									iyy="1.2277e-002" iyz="-3.6288e-007"
+									izz="1.0941e-002"
+									scale="${flipper_scale}" mass="${flipper_mass}" />
+						</inertial>
+					</xacro:unless>
 <!--					<sensor name="${prefix1}_${prefix2}_flipper_contact" type="contact">-->
 <!--							<contact>-->
@@ -1011,9 +1089,11 @@
 					<xacro:flipper_joint flipper_fixed="$(arg robot_fixed)" flipper_angle="$(arg rear_right_flipper_angle)" />
 			</xacro:if>
-			<xacro:flipper_fake_wheel prefix1="${prefix1}" prefix2="${prefix2}" reflect_y="${reflect_y}" do_inward_enlargement="${do_inward_enlargement}" num_wheels="5" wheel_num="1" />
-			<xacro:flipper_fake_wheel prefix1="${prefix1}" prefix2="${prefix2}" reflect_y="${reflect_y}" do_inward_enlargement="${do_inward_enlargement}" num_wheels="5" wheel_num="2" />
-			<xacro:flipper_fake_wheel prefix1="${prefix1}" prefix2="${prefix2}" reflect_y="${reflect_y}" do_inward_enlargement="${do_inward_enlargement}" num_wheels="5" wheel_num="3" />
-			<xacro:flipper_fake_wheel prefix1="${prefix1}" prefix2="${prefix2}" reflect_y="${reflect_y}" do_inward_enlargement="${do_inward_enlargement}" num_wheels="5" wheel_num="4" />
-			<xacro:flipper_fake_wheel prefix1="${prefix1}" prefix2="${prefix2}" reflect_y="${reflect_y}" do_inward_enlargement="${do_inward_enlargement}" num_wheels="5" wheel_num="5" />
+			<xacro:if value="${$(arg wheels_instead_of_tracks)}">
+				<xacro:flipper_fake_wheel prefix1="${prefix1}" prefix2="${prefix2}" reflect_y="${reflect_y}" do_inward_enlargement="${do_inward_enlargement}" num_wheels="5" wheel_num="1" />
+				<xacro:flipper_fake_wheel prefix1="${prefix1}" prefix2="${prefix2}" reflect_y="${reflect_y}" do_inward_enlargement="${do_inward_enlargement}" num_wheels="5" wheel_num="2" />
+				<xacro:flipper_fake_wheel prefix1="${prefix1}" prefix2="${prefix2}" reflect_y="${reflect_y}" do_inward_enlargement="${do_inward_enlargement}" num_wheels="5" wheel_num="3" />
+				<xacro:flipper_fake_wheel prefix1="${prefix1}" prefix2="${prefix2}" reflect_y="${reflect_y}" do_inward_enlargement="${do_inward_enlargement}" num_wheels="5" wheel_num="4" />
+				<xacro:flipper_fake_wheel prefix1="${prefix1}" prefix2="${prefix2}" reflect_y="${reflect_y}" do_inward_enlargement="${do_inward_enlargement}" num_wheels="5" wheel_num="5" />
+			</xacro:if>
 			<link name="$(arg prefix)${prefix1}_${prefix2}_flipper_end_point"/>
 			<joint name="${prefix1}_${prefix2}_flipper_end_point_j" type="fixed">
@@ -1429,20 +1509,22 @@
 	<gazebo reference="$(arg prefix)left_track"><xacro:gazebo_track_tags /></gazebo>
 	<gazebo reference="$(arg prefix)right_track"><xacro:gazebo_track_tags /></gazebo>
-	<gazebo reference="$(arg prefix)left_track_wheel1"><xacro:gazebo_track_wheel_tags /></gazebo>
-	<gazebo reference="$(arg prefix)right_track_wheel1"><xacro:gazebo_track_wheel_tags /></gazebo>
-	<gazebo reference="$(arg prefix)left_track_wheel2"><xacro:gazebo_track_wheel_tags /></gazebo>
-	<gazebo reference="$(arg prefix)right_track_wheel2"><xacro:gazebo_track_wheel_tags /></gazebo>
-	<gazebo reference="$(arg prefix)left_track_wheel3"><xacro:gazebo_track_wheel_tags /></gazebo>
-	<gazebo reference="$(arg prefix)right_track_wheel3"><xacro:gazebo_track_wheel_tags /></gazebo>
-	<gazebo reference="$(arg prefix)left_track_wheel4"><xacro:gazebo_track_wheel_tags /></gazebo>
-	<gazebo reference="$(arg prefix)right_track_wheel4"><xacro:gazebo_track_wheel_tags /></gazebo>
-	<gazebo reference="$(arg prefix)left_track_wheel5"><xacro:gazebo_track_wheel_tags /></gazebo>
-	<gazebo reference="$(arg prefix)right_track_wheel5"><xacro:gazebo_track_wheel_tags /></gazebo>
-	<gazebo reference="$(arg prefix)left_track_wheel6"><xacro:gazebo_track_wheel_tags /></gazebo>
-	<gazebo reference="$(arg prefix)right_track_wheel6"><xacro:gazebo_track_wheel_tags /></gazebo>
-	<gazebo reference="$(arg prefix)left_track_wheel7"><xacro:gazebo_track_wheel_tags /></gazebo>
-	<gazebo reference="$(arg prefix)right_track_wheel7"><xacro:gazebo_track_wheel_tags /></gazebo>
-	<gazebo reference="$(arg prefix)left_track_wheel8"><xacro:gazebo_track_wheel_tags /></gazebo>
-	<gazebo reference="$(arg prefix)right_track_wheel8"><xacro:gazebo_track_wheel_tags /></gazebo>
+	<xacro:if value="${$(arg wheels_instead_of_tracks)}">
+		<gazebo reference="$(arg prefix)left_track_wheel1"><xacro:gazebo_track_wheel_tags /></gazebo>
+		<gazebo reference="$(arg prefix)right_track_wheel1"><xacro:gazebo_track_wheel_tags /></gazebo>
+		<gazebo reference="$(arg prefix)left_track_wheel2"><xacro:gazebo_track_wheel_tags /></gazebo>
+		<gazebo reference="$(arg prefix)right_track_wheel2"><xacro:gazebo_track_wheel_tags /></gazebo>
+		<gazebo reference="$(arg prefix)left_track_wheel3"><xacro:gazebo_track_wheel_tags /></gazebo>
+		<gazebo reference="$(arg prefix)right_track_wheel3"><xacro:gazebo_track_wheel_tags /></gazebo>
+		<gazebo reference="$(arg prefix)left_track_wheel4"><xacro:gazebo_track_wheel_tags /></gazebo>
+		<gazebo reference="$(arg prefix)right_track_wheel4"><xacro:gazebo_track_wheel_tags /></gazebo>
+		<gazebo reference="$(arg prefix)left_track_wheel5"><xacro:gazebo_track_wheel_tags /></gazebo>
+		<gazebo reference="$(arg prefix)right_track_wheel5"><xacro:gazebo_track_wheel_tags /></gazebo>
+		<gazebo reference="$(arg prefix)left_track_wheel6"><xacro:gazebo_track_wheel_tags /></gazebo>
+		<gazebo reference="$(arg prefix)right_track_wheel6"><xacro:gazebo_track_wheel_tags /></gazebo>
+		<gazebo reference="$(arg prefix)left_track_wheel7"><xacro:gazebo_track_wheel_tags /></gazebo>
+		<gazebo reference="$(arg prefix)right_track_wheel7"><xacro:gazebo_track_wheel_tags /></gazebo>
+		<gazebo reference="$(arg prefix)left_track_wheel8"><xacro:gazebo_track_wheel_tags /></gazebo>
+		<gazebo reference="$(arg prefix)right_track_wheel8"><xacro:gazebo_track_wheel_tags /></gazebo>
+	</xacro:if>
     <xacro:if value="$(arg has_flippers)">
 		<gazebo reference="$(arg prefix)front_left_flipper"><xacro:gazebo_flipper_tags /></gazebo>
@@ -1450,24 +1532,26 @@
 		<gazebo reference="$(arg prefix)rear_left_flipper"><xacro:gazebo_flipper_tags /></gazebo>
 		<gazebo reference="$(arg prefix)rear_right_flipper"><xacro:gazebo_flipper_tags /></gazebo>
-		<gazebo reference="$(arg prefix)front_left_flipper_wheel1"><xacro:gazebo_flipper_wheel_tags /></gazebo>
-		<gazebo reference="$(arg prefix)front_right_flipper_wheel1"><xacro:gazebo_flipper_wheel_tags /></gazebo>
-		<gazebo reference="$(arg prefix)rear_left_flipper_wheel1"><xacro:gazebo_flipper_wheel_tags /></gazebo>
-		<gazebo reference="$(arg prefix)rear_right_flipper_wheel1"><xacro:gazebo_flipper_wheel_tags /></gazebo>
-		<gazebo reference="$(arg prefix)front_left_flipper_wheel2"><xacro:gazebo_flipper_wheel_tags /></gazebo>
-		<gazebo reference="$(arg prefix)front_right_flipper_wheel2"><xacro:gazebo_flipper_wheel_tags /></gazebo>
-		<gazebo reference="$(arg prefix)rear_left_flipper_wheel2"><xacro:gazebo_flipper_wheel_tags /></gazebo>
-		<gazebo reference="$(arg prefix)rear_right_flipper_wheel2"><xacro:gazebo_flipper_wheel_tags /></gazebo>
-		<gazebo reference="$(arg prefix)front_left_flipper_wheel3"><xacro:gazebo_flipper_wheel_tags /></gazebo>
-		<gazebo reference="$(arg prefix)front_right_flipper_wheel3"><xacro:gazebo_flipper_wheel_tags /></gazebo>
-		<gazebo reference="$(arg prefix)rear_left_flipper_wheel3"><xacro:gazebo_flipper_wheel_tags /></gazebo>
-		<gazebo reference="$(arg prefix)rear_right_flipper_wheel3"><xacro:gazebo_flipper_wheel_tags /></gazebo>
-		<gazebo reference="$(arg prefix)front_left_flipper_wheel4"><xacro:gazebo_flipper_wheel_tags /></gazebo>
-		<gazebo reference="$(arg prefix)front_right_flipper_wheel4"><xacro:gazebo_flipper_wheel_tags /></gazebo>
-		<gazebo reference="$(arg prefix)rear_left_flipper_wheel4"><xacro:gazebo_flipper_wheel_tags /></gazebo>
-		<gazebo reference="$(arg prefix)rear_right_flipper_wheel4"><xacro:gazebo_flipper_wheel_tags /></gazebo>
-		<gazebo reference="$(arg prefix)front_left_flipper_wheel5"><xacro:gazebo_flipper_wheel_tags /></gazebo>
-		<gazebo reference="$(arg prefix)front_right_flipper_wheel5"><xacro:gazebo_flipper_wheel_tags /></gazebo>
-		<gazebo reference="$(arg prefix)rear_left_flipper_wheel5"><xacro:gazebo_flipper_wheel_tags /></gazebo>
-		<gazebo reference="$(arg prefix)rear_right_flipper_wheel5"><xacro:gazebo_flipper_wheel_tags /></gazebo>
+		<xacro:if value="${$(arg wheels_instead_of_tracks)}">
+			<gazebo reference="$(arg prefix)front_left_flipper_wheel1"><xacro:gazebo_flipper_wheel_tags /></gazebo>
+			<gazebo reference="$(arg prefix)front_right_flipper_wheel1"><xacro:gazebo_flipper_wheel_tags /></gazebo>
+			<gazebo reference="$(arg prefix)rear_left_flipper_wheel1"><xacro:gazebo_flipper_wheel_tags /></gazebo>
+			<gazebo reference="$(arg prefix)rear_right_flipper_wheel1"><xacro:gazebo_flipper_wheel_tags /></gazebo>
+			<gazebo reference="$(arg prefix)front_left_flipper_wheel2"><xacro:gazebo_flipper_wheel_tags /></gazebo>
+			<gazebo reference="$(arg prefix)front_right_flipper_wheel2"><xacro:gazebo_flipper_wheel_tags /></gazebo>
+			<gazebo reference="$(arg prefix)rear_left_flipper_wheel2"><xacro:gazebo_flipper_wheel_tags /></gazebo>
+			<gazebo reference="$(arg prefix)rear_right_flipper_wheel2"><xacro:gazebo_flipper_wheel_tags /></gazebo>
+			<gazebo reference="$(arg prefix)front_left_flipper_wheel3"><xacro:gazebo_flipper_wheel_tags /></gazebo>
+			<gazebo reference="$(arg prefix)front_right_flipper_wheel3"><xacro:gazebo_flipper_wheel_tags /></gazebo>
+			<gazebo reference="$(arg prefix)rear_left_flipper_wheel3"><xacro:gazebo_flipper_wheel_tags /></gazebo>
+			<gazebo reference="$(arg prefix)rear_right_flipper_wheel3"><xacro:gazebo_flipper_wheel_tags /></gazebo>
+			<gazebo reference="$(arg prefix)front_left_flipper_wheel4"><xacro:gazebo_flipper_wheel_tags /></gazebo>
+			<gazebo reference="$(arg prefix)front_right_flipper_wheel4"><xacro:gazebo_flipper_wheel_tags /></gazebo>
+			<gazebo reference="$(arg prefix)rear_left_flipper_wheel4"><xacro:gazebo_flipper_wheel_tags /></gazebo>
+			<gazebo reference="$(arg prefix)rear_right_flipper_wheel4"><xacro:gazebo_flipper_wheel_tags /></gazebo>
+			<gazebo reference="$(arg prefix)front_left_flipper_wheel5"><xacro:gazebo_flipper_wheel_tags /></gazebo>
+			<gazebo reference="$(arg prefix)front_right_flipper_wheel5"><xacro:gazebo_flipper_wheel_tags /></gazebo>
+			<gazebo reference="$(arg prefix)rear_left_flipper_wheel5"><xacro:gazebo_flipper_wheel_tags /></gazebo>
+			<gazebo reference="$(arg prefix)rear_right_flipper_wheel5"><xacro:gazebo_flipper_wheel_tags /></gazebo>
+		</xacro:if>
     </xacro:if>
     <xacro:if value="$(arg has_sick_lidar)">
@@ -1793,4 +1877,5 @@
 				<update_rate>50</update_rate>
 				<imu>
+					<enable_orientation>0</enable_orientation>
 					<angular_velocity>
 						<xacro:macro name="angular_imu_noise">

File: submitted_models/ctu_cras_norlab_marv_sensor_config_1/urdf/marv.xacro (robot description, xacro)
@@ -398,5 +398,5 @@
                 </geometry>
             </visual>
-            <xacro:if value="${'$(arg rendering_target)' == 'urdf'}">
+            <xacro:if value="${'$(arg rendering_target)' == 'urdf' or $(arg num_wheels) == 0}">
                 <xacro:property name="inflated_big_wheel" value="${$(arg flipper_inflation_ratio) * $(arg rover_flipperBigRadius)}" />
                 <xacro:property name="inflated_small_wheel" value="${$(arg flipper_inflation_ratio) * $(arg rover_flipperSmallRadius)}" />
@@ -435,5 +435,18 @@
                 </collision>
             </xacro:if>
-            <xacro:default_inertial />
+            <xacro:if value="${$(arg num_wheels) > 0}">
+                <xacro:default_inertial />
+            </xacro:if>
+            <xacro:if value="${$(arg num_wheels) == 0}">
+                <inertial>
+                    <origin xyz="${reflect_y*0.08} 0 0.0" rpy="0 0 0"/>
+                    <mass value="${flipper_arm_mass + flipper_big_wheel_mass + 2*flipper_small_wheel_mass + belt_mass}"/>
+                    <xacro:inertia_meshlab
+                            ixx="1.7491e-003" ixy="2.8512e-007" ixz="1.8277e-003"
+                            iyy="1.2277e-002" iyz="-3.6288e-007"
+                            izz="1.0941e-002" scale="1.0"
+                            mass="${flipper_arm_mass + flipper_big_wheel_mass + 2*flipper_small_wheel_mass + belt_mass}" />
+                </inertial>
+            </xacro:if>
         </link>
         <joint name="${prefix1}_${prefix2}_flipper_j" type="revolute">
@@ -670,5 +683,5 @@
         </xacro:macro>
         <xacro:flipper_wheel_tags wheel_num="${$(arg num_wheels)}" />
-        <xacro:if value="${'$(arg rendering_target)' == 'ign'}">
+        <xacro:if value="${'$(arg rendering_target)' == 'ign' and $(arg num_wheels) > 0}">
             <gazebo>
                 <xacro:property name="inflation_coef" value="$(arg flipper_inflation_ratio)" />
@@ -751,4 +764,5 @@
                 <update_rate>50</update_rate>
                 <imu>
+                    <enable_orientation>0</enable_orientation>
                     <angular_velocity>
                         <xacro:macro name="angular_imu_noise">
