Commit message: Fixed urdf/xacro

File: submitted_models/marble_hd2_sensor_config_3/urdf/robot_from_sdf.xacro (robot description, xacro)
@@ -1,10 +1,10 @@
 <?xml version='1.0' encoding='utf-8'?>
-<robot name='marble_hd2_sensor_config_1' xmlns:xacro='http://ros.org/wiki/xacro'>
-  <xacro:arg name="name" default="marble_hd2_sensor_config_1"/>
+<robot name='marble_hd2_sensor_config_3' xmlns:xacro='http://ros.org/wiki/xacro'>
+  <xacro:arg name="name" default="marble_hd2_sensor_config_3"/>
   <xacro:property name="robot_namespace" value="$(arg name)"/>
   <link name='${robot_namespace}/base_link'>
     <inertial>
       <origin xyz='-0.000649 -0.084945 0.062329' rpy='0 -0 0'/>
-      <mass value='34.02'/>
+      <mass value='21.8194'/>
       <inertia ixx='0.615397' ixy='-0.0240585' ixz='-0.120749' iyy='1.75388' iyz='-0.0028322' izz='2.03641'/>
     </inertial>
@@ -34,5 +34,5 @@
     </collision>
     <collision name='base_link_fixed_joint_lump__camera/camera_link_collision_2'>
-      <origin xyz='0.478 0 0.285' rpy='0 -0 0'/>
+      <origin xyz='0.485 0 0.31' rpy='0 -0 0'/>
       <geometry>
         <box size='0.0078 0.13 0.0192'/>
@@ -46,5 +46,5 @@
     </collision>
     <collision name='base_link_fixed_joint_lump__velodyne_base_link_collision_6'>
-      <origin xyz='0.424 0 0.327' rpy='0 -0 0'/>
+      <origin xyz='0.403 0 0.36' rpy='0 -0 0'/>
       <geometry>
         <cylinder radius='0.0516' length='0.0717'/>
@@ -52,5 +52,5 @@
     </collision>
     <collision name='base_link_fixed_joint_lump__velodyne_gimbal_plate_base_link_collision_7'>
-      <origin xyz='0.424 0 0.4' rpy='0 -0 0'/>
+      <origin xyz='0.403 0 0.41' rpy='0 -0 0'/>
       <geometry>
         <box size='0.1 0.1 0.01'/>
@@ -69,113 +69,113 @@
       </geometry>
     </collision>
-    <visual name='base_link_visual'>
-      <origin xyz='0 0 0' rpy='1.57 -0 1.57'/>
-      <geometry>
-        <mesh filename='package://marble_hd2_sensor_config_1/meshes/hd2_chassis.stl' scale='1 1 1'/>
-      </geometry>
-    </visual>
-    <visual name='track_left_visual'>
-      <origin xyz='0 0.2625 0' rpy='1.57 -0 1.57'/>
-      <geometry>
-        <mesh filename='package://marble_hd2_sensor_config_1/meshes/track.stl' scale='1 1 1'/>
-      </geometry>
-    </visual>
-    <visual name='track_right_visual'>
-      <origin xyz='0 -0.2625 0' rpy='1.57 -0 1.57'/>
-      <geometry>
-        <mesh filename='package://marble_hd2_sensor_config_1/meshes/track.stl' scale='1 1 1'/>
-      </geometry>
-    </visual>
-    <visual name='base_link_fixed_joint_lump__camera/camera_link_visual_1'>
-      <origin xyz='0.44 0 0.26' rpy='0 0.5236 0'/>
-      <geometry>
-        <mesh filename='package://marble_hd2_sensor_config_1/meshes/realsense.dae' scale='1 1 1'/>
-      </geometry>
-    </visual>
-    <visual name='base_link_fixed_joint_lump__camera/camera_link_visual_2'>
-      <origin xyz='0.44 0 0.295' rpy='0 -0 0'/>
-      <geometry>
-        <mesh filename='package://marble_hd2_sensor_config_1/meshes/realsense.dae' scale='1 1 1'/>
+    <visual name='Body_visual'>
+      <origin xyz='0 0 -0.135' rpy='0 -0 1.57'/>
+      <geometry>
+        <mesh filename='package://marble_hd2_sensor_config_3/meshes/hd2.dae' scale='1 1 1'/>
+      </geometry>
+    </visual>
+  </link>
+  <sensor name='camera_down' update_rate='30'>
+    <parent link='${robot_namespace}/base_link'/>
+    <origin xyz='0.473 0 0.26' rpy='0 0.5236 0'/>
+    <camera>
+      <image width='320' height='240' format='R8G8B8' hfov='1.5184' near='0.01' far='300' />
+    </camera>
+  </sensor>
+  <sensor name='planar_laser' update_rate='10'>
+    <parent link='${robot_namespace}/base_link'/>
+    <origin xyz='0.403 0 0.127' rpy='0 -0 0'/>
+  </sensor>
+  <sensor name='imu_sensor' update_rate='50'>
+    <parent link='${robot_namespace}/base_link'/>
+    <origin xyz='0 0 0' rpy='0 -0 0'/>
+  </sensor>
+  <link name='${robot_namespace}/sensor_head_link'>
+    <inertial>
+      <origin xyz='0 0 0' rpy='0 -0 0'/>
+      <mass value='0.1'/>
+      <inertia ixx='0.01' ixy='0' ixz='0' iyy='0.01' iyz='0' izz='0.01'/>
+    </inertial>
+    <visual name='sensor_head_visual'>
+      <origin xyz='0 0 0' rpy='0 -0 0'/>
+      <geometry>
+        <box size='0.1 0.1 0.1'/>
       </geometry>
     </visual>
     <visual name='base_link_fixed_joint_lump__velodyne_base_link_visual_10'>
-      <origin xyz='0.354 0 0.327' rpy='0 -0 0'/>
-      <geometry>
-        <mesh filename='package://marble_hd2_sensor_config_1/meshes/VLP16_base_1.dae' scale='1 1 1'/>
+      <origin xyz='0 0 0.086' rpy='0 -0 0'/>
+      <geometry>
+        <mesh filename='package://marble_hd2_sensor_config_3/meshes/VLP16_base_1.dae' scale='1 1 1'/>
       </geometry>
     </visual>
     <visual name='base_link_fixed_joint_lump__velodyne_base_link_visual_11'>
-      <origin xyz='0.354 0 0.327' rpy='0 -0 0'/>
-      <geometry>
-        <mesh filename='package://marble_hd2_sensor_config_1/meshes/VLP16_base_2.dae' scale='1 1 1'/>
+      <origin xyz='0 0 0.086' rpy='0 -0 0'/>
+      <geometry>
+        <mesh filename='package://marble_hd2_sensor_config_3/meshes/VLP16_base_2.dae' scale='1 1 1'/>
       </geometry>
     </visual>
     <visual name='base_link_fixed_joint_lump__velodyne_visual_12'>
-      <origin xyz='0.354 0 0.327' rpy='0 -0 0'/>
-      <geometry>
-        <mesh filename='package://marble_hd2_sensor_config_1/meshes/VLP16_scan.dae' scale='1 1 1'/>
-      </geometry>
-    </visual>
-    <visual name='base_link_fixed_joint_lump__planar_lidar_link_visual_14'>
-      <origin xyz='0.354 0 0.127' rpy='0 -0 0'/>
-      <geometry>
-        <cylinder radius='0.045' length='0.05'/>
-      </geometry>
-    </visual>
-    <visual name='base_link_fixed_joint_lump__velodyne_gimbal_plate_15'>
-      <origin xyz='0.354 0 0.4' rpy='0 -0 0'/>
-      <geometry>
-        <box size='0.06 0.06 0.01'/>
-      </geometry>
-    </visual>
-    <visual name='base_link_fixed_joint_lump__sensor_tower_16'>
-      <origin xyz='0.354 0 0.19' rpy='0 -0 0'/>
-      <geometry>
-        <box size='0.18 0.25 0.275'/>
-      </geometry>
-    </visual>
-    <visual name='base_link_fixed_joint_lump__computer_block_17'>
-      <origin xyz='0.05 0 0.135' rpy='0 -0 0'/>
-      <geometry>
-        <box size='0.3 0.355 0.175'/>
-      </geometry>
-    </visual>
-    <visual name='base_link_fixed_joint_lid_18'>
-      <origin xyz='0 0 0.05' rpy='0 -0 0'/>
-      <geometry>
-        <box size='0.7 0.35 0.02'/>
-      </geometry>
-    </visual>
-  </link>
-  <sensor name='camera_front' update_rate='30'>
-    <parent link='${robot_namespace}/base_link'/>
-    <origin xyz='0.44 0 0.36' rpy='0 -0 0'/>
+      <origin xyz='0 0 0.086' rpy='0 -0 0'/>
+      <geometry>
+        <mesh filename='package://marble_hd2_sensor_config_3/meshes/VLP16_scan.dae' scale='1 1 1'/>
+      </geometry>
+    </visual>
+    <visual name='base_link_fixed_joint_lump__velodyne_base_link_visual_13'>
+      <origin xyz='-0.158 0 -0.086' rpy='3.14159 1.57079 3.14159'/>
+      <geometry>
+        <mesh filename='package://marble_hd2_sensor_config_3/meshes/VLP16_base_1.dae' scale='1 1 1'/>
+      </geometry>
+    </visual>
+    <visual name='base_link_fixed_joint_lump__velodyne_base_link_visual_14'>
+      <origin xyz='-0.158 0 -0.086' rpy='3.14159 1.57079 3.14159'/>
+      <geometry>
+        <mesh filename='package://marble_hd2_sensor_config_3/meshes/VLP16_base_2.dae' scale='1 1 1'/>
+      </geometry>
+    </visual>
+    <visual name='base_link_fixed_joint_lump__velodyne_visual_15'>
+      <origin xyz='-0.158 0 -0.086' rpy='3.14159 1.57079 3.14159'/>
+      <geometry>
+        <mesh filename='package://marble_hd2_sensor_config_3/meshes/VLP16_scan.dae' scale='1 1 1'/>
+      </geometry>
+    </visual>
+    <visual name='camera_front_visual'>
+      <origin xyz='0.1 0 0.013' rpy='0 -0 0'/>
+      <geometry>
+        <box size='0.02 0.02 0.02'/>
+      </geometry>
+    </visual>
+    <visual name='camera_back_visual'>
+      <origin xyz='-0.1 0 0.013' rpy='0 -0 0'/>
+      <geometry>
+        <box size='0.02 0.02 0.02'/>
+      </geometry>
+    </visual>
+  </link>
+  <sensor name='horiz_laser' update_rate='20'>
+    <parent link='${robot_namespace}/sensor_head_link'/>
+    <origin xyz='0 0 0.086' rpy='0 -0 0'/>
+  </sensor>
+  <sensor name='vert_laser' update_rate='20'>
+    <parent link='${robot_namespace}/sensor_head_link'/>
+    <origin xyz='-0.158 0 -0.086' rpy='3.14159 1.57079 3.14159'/>
+  </sensor>
+  <sensor name='camera_front' update_rate='15'>
+    <parent link='${robot_namespace}/sensor_head_link'/>
+    <origin xyz='0.12 0 0.013' rpy='0 -0 0'/>
     <camera>
-      <image width='1280' height='720' format='R8G8B8' hfov='1.5184' near='0.01' far='300' />
+      <image width='1280' height='960' format='R8G8B8' hfov='1.0472' near='0.01' far='300' />
     </camera>
   </sensor>
-  <sensor name='camera_down' update_rate='30'>
-    <parent link='${robot_namespace}/base_link'/>
-    <origin xyz='0.44 0 0.335' rpy='0 0.5236 0'/>
+  <sensor name='camera_back' update_rate='15'>
+    <parent link='${robot_namespace}/sensor_head_link'/>
+    <origin xyz='-0.12 0 0.013' rpy='0 -0 3.14159'/>
     <camera>
-      <image width='1280' height='720' format='R8G8B8' hfov='1.5184' near='0.01' far='300' />
+      <image width='1280' height='960' format='R8G8B8' hfov='1.0472' near='0.01' far='300' />
     </camera>
   </sensor>
-  <sensor name='planar_laser' update_rate='10'>
-    <parent link='${robot_namespace}/base_link'/>
-    <origin xyz='0.354 0 0.127' rpy='0 -0 0'/>
-  </sensor>
-  <sensor name='front_laser' update_rate='20'>
-    <parent link='${robot_namespace}/base_link'/>
-    <origin xyz='0.354 0 0.387' rpy='0 -0 0'/>
-  </sensor>
-  <sensor name='imu_sensor' update_rate='250'>
-    <parent link='${robot_namespace}/base_link'/>
-    <origin xyz='0 0 0' rpy='0 -0 0'/>
-  </sensor>
   <link name='${robot_namespace}/front_left_wheel_link'>
     <inertial>
       <origin xyz='0 0 0' rpy='0 -0 0'/>
-      <mass value='2.637'/>
+      <mass value='1.5'/>
       <inertia ixx='0.02467' ixy='0' ixz='0' iyy='0.04411' iyz='0' izz='0.02467'/>
     </inertial>
@@ -186,15 +186,9 @@
       </geometry>
     </collision>
-    <visual name='front_left_wheel_link_visual'>
-      <origin xyz='0 0 0' rpy='1.5708 -0 0'/>
-      <geometry>
-        <cylinder radius='0.129' length='0.1'/>
-      </geometry>
-    </visual>
   </link>
   <link name='${robot_namespace}/front_middle_left_wheel_link'>
     <inertial>
       <origin xyz='0 0 0' rpy='0 -0 0'/>
-      <mass value='2.637'/>
+      <mass value='1.5'/>
       <inertia ixx='0.02467' ixy='0' ixz='0' iyy='0.04411' iyz='0' izz='0.02467'/>
     </inertial>
@@ -205,15 +199,9 @@
       </geometry>
     </collision>
-    <visual name='front_middle_left_wheel_link_visual'>
-      <origin xyz='0 0 0' rpy='1.5708 -0 0'/>
-      <geometry>
-        <cylinder radius='0.129' length='0.1'/>
-      </geometry>
-    </visual>
   </link>
   <link name='${robot_namespace}/rear_middle_left_wheel_link'>
     <inertial>
       <origin xyz='0 0 0' rpy='0 -0 0'/>
-      <mass value='2.637'/>
+      <mass value='1.5'/>
       <inertia ixx='0.02467' ixy='0' ixz='0' iyy='0.04411' iyz='0' izz='0.02467'/>
     </inertial>
@@ -224,15 +212,9 @@
       </geometry>
     </collision>
-    <visual name='rear_middle_left_wheel_link_visual'>
-      <origin xyz='0 0 0' rpy='1.5708 -0 0'/>
-      <geometry>
-        <cylinder radius='0.129' length='0.1'/>
-      </geometry>
-    </visual>
   </link>
   <link name='${robot_namespace}/rear_left_wheel_link'>
     <inertial>
       <origin xyz='0 0 0' rpy='0 -0 0'/>
-      <mass value='2.637'/>
+      <mass value='1.5'/>
       <inertia ixx='0.02467' ixy='0' ixz='0' iyy='0.04411' iyz='0' izz='0.02467'/>
     </inertial>
@@ -243,15 +225,9 @@
       </geometry>
     </collision>
-    <visual name='rear_left_wheel_link_visual'>
-      <origin xyz='0 0 0' rpy='1.5708 -0 0'/>
-      <geometry>
-        <cylinder radius='0.129' length='0.1'/>
-      </geometry>
-    </visual>
   </link>
   <link name='${robot_namespace}/front_right_wheel_link'>
     <inertial>
       <origin xyz='0 0 0' rpy='0 -0 0'/>
-      <mass value='2.637'/>
+      <mass value='1.5'/>
       <inertia ixx='0.02467' ixy='0' ixz='0' iyy='0.04411' iyz='0' izz='0.02467'/>
     </inertial>
@@ -262,15 +238,9 @@
       </geometry>
     </collision>
-    <visual name='front_right_wheel_link_visual'>
-      <origin xyz='0 0 0' rpy='1.5708 -0 0'/>
-      <geometry>
-        <cylinder radius='0.129' length='0.1'/>
-      </geometry>
-    </visual>
   </link>
   <link name='${robot_namespace}/front_middle_right_wheel_link'>
     <inertial>
       <origin xyz='0 0 0' rpy='0 -0 0'/>
-      <mass value='2.637'/>
+      <mass value='1.5'/>
       <inertia ixx='0.02467' ixy='0' ixz='0' iyy='0.04411' iyz='0' izz='0.02467'/>
     </inertial>
@@ -281,15 +251,9 @@
       </geometry>
     </collision>
-    <visual name='front_middle_right_wheel_link_visual'>
-      <origin xyz='0 0 0' rpy='1.5708 -0 0'/>
-      <geometry>
-        <cylinder radius='0.129' length='0.1'/>
-      </geometry>
-    </visual>
   </link>
   <link name='${robot_namespace}/rear_middle_right_wheel_link'>
     <inertial>
       <origin xyz='0 0 0' rpy='0 -0 0'/>
-      <mass value='2.637'/>
+      <mass value='1.5'/>
       <inertia ixx='0.02467' ixy='0' ixz='0' iyy='0.04411' iyz='0' izz='0.02467'/>
     </inertial>
@@ -300,15 +264,9 @@
       </geometry>
     </collision>
-    <visual name='rear_middle_right_wheel_link_visual'>
-      <origin xyz='0 0 0' rpy='1.5708 -0 0'/>
-      <geometry>
-        <cylinder radius='0.129' length='0.1'/>
-      </geometry>
-    </visual>
   </link>
   <link name='${robot_namespace}/rear_right_wheel_link'>
     <inertial>
       <origin xyz='0 0 0' rpy='0 -0 0'/>
-      <mass value='2.637'/>
+      <mass value='1.5'/>
       <inertia ixx='0.02467' ixy='0' ixz='0' iyy='0.04411' iyz='0' izz='0.02467'/>
     </inertial>
@@ -319,80 +277,12 @@
       </geometry>
     </collision>
-    <visual name='rear_right_wheel_link_visual'>
-      <origin xyz='0 0 0' rpy='1.5708 -0 0'/>
-      <geometry>
-        <cylinder radius='0.129' length='0.1'/>
-      </geometry>
-    </visual>
-  </link>
-  <link name='${robot_namespace}/pan_gimbal_link'>
-    <inertial>
-      <origin xyz='0 0 0' rpy='0 -0 0'/>
-      <mass value='0.1'/>
-      <inertia ixx='1' ixy='0' ixz='0' iyy='1' iyz='0' izz='1'/>
-    </inertial>
-    <collision name='pan_gimbal_link_collision'>
-      <origin xyz='0 0 0' rpy='0 -0 0'/>
-      <geometry>
-        <cylinder radius='0.014' length='0.045'/>
-      </geometry>
-    </collision>
-    <visual name='pan_gimbal_link_visual'>
-      <origin xyz='0 0 0' rpy='0 -0 0'/>
-      <geometry>
-        <cylinder radius='0.014' length='0.045'/>
-      </geometry>
-    </visual>
-  </link>
-  <link name='${robot_namespace}/tilt_gimbal_link'>
-    <inertial>
-      <origin xyz='0 0 0' rpy='1.5708 -0 0'/>
-      <mass value='0.1'/>
-      <inertia ixx='1' ixy='0' ixz='0' iyy='1' iyz='0' izz='1'/>
-    </inertial>
-    <collision name='tilt_gimbal_link_collision'>
-      <origin xyz='0 0 0' rpy='1.5708 -0 0'/>
-      <geometry>
-        <cylinder radius='0.014' length='0.045'/>
-      </geometry>
-    </collision>
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
Commit message: addressed issues in PR, still need to connect floating sensors, add docs for the camera, and figure out steering issue

File: submitted_models/marble_hd2_sensor_config_3/urdf/robot_from_sdf.xacro (robot description, xacro)
@@ -145,5 +145,5 @@
       </geometry>
     </visual>
-    <visual name='camera_back_visual'>
+    <visual name='camera_rear_visual'>
       <origin xyz='-0.1 0 0.013' rpy='0 -0 0'/>
       <geometry>
@@ -167,5 +167,5 @@
     </camera>
   </sensor>
-  <sensor name='camera_back' update_rate='15'>
+  <sensor name='camera_rear' update_rate='15'>
     <parent link='${robot_namespace}/sensor_head_link'/>
     <origin xyz='-0.12 0 0.013' rpy='0 -0 3.14159'/>
