Commit message: add more data

File: submitted_models/cerberus_anymal_c_sensor_config_1/urdf/robot_from_sdf.xacro (robot description, xacro)
@@ -7,5 +7,5 @@
     <inertial>
       <origin xyz='-0.02203 -0.000162 0.009216' rpy='0 -0 0'/>
-      <mass value='26.9398'/>
+      <mass value='29.23832'/>
       <inertia ixx='0.236867' ixy='0.00846724' ixz='0.0854364' iyy='2.06849' iyz='-0.000253399' izz='2.09006'/>
     </inertial>
