Commit message: Spot: improved modularity and made CCN_SPOT_SC1 compatible with BOSDYN_SPOT again.
The interface between BOSDYN_SPOT and sensor configs can be considered more or less stable now.

File: submitted_models/bosdyn_spot/urdf/spot_leg.urdf.xacro (robot description, xacro)
@@ -1,4 +1,15 @@
 <?xml version="1.0"?>
 <robot xmlns:xacro="http://ros.org/wiki/xacro">
+    <xacro:arg name="leg_kp" default="1e+07" />
+    <xacro:arg name="leg_kd" default="100.0" />
+    <xacro:arg name="leg_mu1" default="0.8" />
+    <xacro:arg name="leg_mu2" default="0.8" />
+    <xacro:arg name="leg_fdir1" default="" />
+    <xacro:arg name="max_knee_effort" default="80" />
+    <xacro:arg name="max_knee_velocity" default="15" />
+    <xacro:arg name="max_hip_x_effort" default="80" />
+    <xacro:arg name="max_hip_x_velocity" default="15" />
+    <xacro:arg name="max_hip_y_effort" default="80" />
+    <xacro:arg name="max_hip_y_velocity" default="15" />
     <xacro:macro name="spot_leg" params="leg_name prefix" >
         <xacro:if value="${leg_name == 'front_left'}">
@@ -41,5 +52,5 @@
             <parent link="${prefix}base_link" />
             <child link="${prefix}${leg_name}_hip" />
-            <limit effort="80" velocity="15" lower="-0.78539816339744827899" upper="0.78539816339744827899" />
+            <limit effort="$(arg max_hip_x_effort)" velocity="$(arg max_hip_x_velocity)" lower="-0.78539816339744827899" upper="0.78539816339744827899" />
         </joint>
         <link name="${prefix}${leg_name}_upper_leg">
@@ -67,5 +78,5 @@
             <parent link="${prefix}${leg_name}_hip" />
             <child link="${prefix}${leg_name}_upper_leg" />
-            <limit effort="80" velocity="15" lower="-0.89884456477707963539" upper="2.2951079663725435509" />
+            <limit effort="$(arg max_hip_y_effort)" velocity="$(arg max_hip_y_velocity)" lower="-0.89884456477707963539" upper="2.2951079663725435509" />
         </joint>
         <link name="${prefix}${leg_name}_lower_leg">
@@ -95,8 +106,11 @@
         </link>
          <gazebo reference="${prefix}${leg_name}_lower_leg">
-            <kp>1e+7</kp>
-            <kd>100.0</kd>
-            <mu1>0.8</mu1>
-            <mu2>0.8</mu2>
+            <kp>$(arg leg_kp)</kp>
+            <kd>$(arg leg_kd)</kd>
+            <mu1>$(arg leg_mu1)</mu1>
+            <mu2>$(arg leg_mu2)</mu2>
+             <xacro:if value="${'$(arg leg_fdir1)' != ''}">
+                 <fdir1>$(arg leg_fdir1)</fdir1>
+             </xacro:if>
              <sensor name="contact" type="contact">
                 <contact>
@@ -110,5 +124,5 @@
             <parent link="${prefix}${leg_name}_upper_leg" />
             <child link="${prefix}${leg_name}_lower_leg" />
-            <limit effort="80" velocity="15" lower="-2.7929" upper="-0.254801" />
+            <limit effort="$(arg max_knee_effort)" velocity="$(arg max_knee_velocity)" lower="-2.7929" upper="-0.254801" />
         </joint>
         <xacro:empty_link name="${prefix}${leg_name}_ee" />

Commit message: Spot: Fixed a bug in handling leg collisions.

File: submitted_models/bosdyn_spot/urdf/spot_leg.urdf.xacro (robot description, xacro)
@@ -116,4 +116,5 @@
                 <contact>
                     <collision>${leg_name}_lower_leg_collision</collision>
+                    <collision>${leg_name}_lower_leg_collision_1</collision>
                 </contact>
              </sensor>
