Commit message: Spot: Fixed xacro utils to be compatible with MARV.

File: submitted_models/bosdyn_spot/urdf/utils.xacro (robot description, xacro)
@@ -7,8 +7,8 @@
                 izz="${izz*scale*scale}"/>
     </xacro:macro>
-    <xacro:macro name="sphere_inertial" params="radius mass *origin">
+    <xacro:macro name="sphere_inertial" params="radius mass xyz:='0 0 0'">
         <inertial>
             <mass value="${mass}" />
-            <xacro:insert_block name="origin" />
+            <origin xyz="${xyz}" rpy="0 0 0"/>
             <inertia ixx="${2.0/5 * mass * radius * radius}" ixy="0.0" ixz="0.0"
                      iyy="${2.0/5 * mass * radius * radius}" iyz="0.0"
@@ -16,17 +16,17 @@
         </inertial>
     </xacro:macro>
-    <xacro:macro name="box_inertial" params="width height depth mass *origin">
+    <xacro:macro name="box_inertial" params="width height depth mass xyz:='0 0 0' rpy:='0 0 0'">
         <inertial>
             <mass value="${mass}" />
-            <xacro:insert_block name="origin" />
-            <inertia ixx="${1.0/12 * mass * (height * height + depth * depth)}" ixy="0.0" ixz="0.0"
-                     iyy="${1.0/12 * mass * (width * width + depth * depth)}" iyz="0.0"
-                     izz="${1.0/12 * mass * (width * width + height * height)}" />
+            <origin xyz="${xyz}" rpy="${rpy}"/>
+            <inertia ixx="${1.0/12 * mass * (width * width + height * height)}" ixy="0.0" ixz="0.0"
+                     iyy="${1.0/12 * mass * (height * height + depth * depth)}" iyz="0.0"
+                     izz="${1.0/12 * mass * (width * width + depth * depth)}" />
         </inertial>
     </xacro:macro>
-    <xacro:macro name="cylinder_inertial" params="radius length mass *origin">
+    <xacro:macro name="cylinder_inertial" params="radius length mass xyz:='0 0 0' rpy:='0 0 0'">
         <inertial>
             <mass value="${mass}" />
-            <xacro:insert_block name="origin" />
+            <origin xyz="${xyz}" rpy="${rpy}"/>
             <inertia ixx="${1.0/12 * mass * (3 * radius * radius + length * length)}" ixy="0.0" ixz="0.0"
                      iyy="${1.0/12 * mass * (3 * radius * radius + length * length)}" iyz="0.0"
