Commit message: Spot: Add camera intrinsics.
Body depth camera is still just estimated.

File: submitted_models/bosdyn_spot/urdf/camera.xacro (robot description, xacro)
@@ -21,5 +21,5 @@
                     <visualize>${visualize}</visualize>
                     <camera>
-                        <horizontal_fov>${radians(95)}</horizontal_fov>
+                        <horizontal_fov>${radians(102.35)}</horizontal_fov> <!-- computed from real fx -->
                         <image>
                             <width>640</width>
@@ -36,4 +36,13 @@
                             <stddev>0.007</stddev>
                         </noise>
+                        <lens>
+                            <intrinsics>
+                                <fx>257.4866</fx> <!-- from real Spot of CoSTAR -->
+                                <fy>257.4866</fy> <!-- =fx; real Spot has 256.9733 -->
+                                <cx>319.5</cx> <!-- ideal value -->
+                                <cy>239.5</cy> <!-- ideal value -->
+                                <s>0</s>
+                            </intrinsics>
+                        </lens>
                     </camera>
                     <plugin filename="mono-camera-system" name="subt::MonoCameraSystem" />
@@ -44,5 +53,5 @@
                     <visualize>${visualize}</visualize>
                     <camera>
-                        <horizontal_fov>${radians(92)}</horizontal_fov>
+                        <horizontal_fov>${radians(102.35)}</horizontal_fov> <!-- put here equal to mono cam -->
                         <image>
                             <width>424</width>
@@ -59,4 +68,13 @@
                             <stddev>0.007</stddev>
                         </noise>
+                        <lens>
+                            <intrinsics>
+                                <fx>170.6</fx> <!-- computed from FOV -->
+                                <fy>170.6</fy> <!-- computed from FOV -->
+                                <cx>211.5</cx> <!-- ideal value -->
+                                <cy>119.5</cy> <!-- ideal value -->
+                                <s>0</s>
+                            </intrinsics>
+                        </lens>
                     </camera>
                 </sensor>

File: submitted_models/ctu_cras_norlab_spot_sensor_config_1/urdf/basler_cameras.xacro (robot description, xacro)
@@ -77,12 +77,20 @@
                             <stddev>0.007</stddev>
                         </noise>
-                        <xacro:if value="${fisheye and '$(arg rendering_target)' == 'gz'}">
-                            <lens>
+                        <lens>
+                            <intrinsics>
+                                <xacro:property name="f" value="${resolution_x / (2 * tan(radians(hfov_deg)/2))}" />
+                                <fx>${f}</fx>
+                                <fy>${f}</fy>
+                                <cx>${(resolution_x - 1) / 2}</cx>
+                                <cy>${(resolution_y - 1) / 2}</cy>
+                                <s>0</s>
+                            </intrinsics>
+                            <xacro:if value="${fisheye and '$(arg rendering_target)' == 'gz'}">
                                 <type>stereographic</type>
                                 <scale_to_hfov>true</scale_to_hfov>
                                 <cutoff_angle>${pi}</cutoff_angle>
                                 <env_texture_size>1024</env_texture_size>
-                            </lens>
-                        </xacro:if>
+                            </xacro:if>
+                        </lens>
                     </camera>
                 </sensor>
