Commit message: Spot walking.

File: submitted_models/bosdyn_spot/urdf/spot.urdf.xacro (robot description, xacro)
@@ -8,5 +8,5 @@
         <xacro:arg name="prefix" default="$(arg name)/"/>
     </xacro:unless>
-    <!-- Pass either "urdf" or "sdf" to tell the parser what is the desired target format. -->
+    <!-- Pass either "urdf" or "ign" to tell the parser what is the desired target format. -->
     <xacro:arg name="rendering_target" default="urdf"/>
     <xacro:arg name="simulate_cameras" default="True"/>
@@ -33,16 +33,10 @@
         </inertial>
     </link>
-    <link name="$(arg prefix)front_rail"/>
-    <joint name="front_rail_joint" type="fixed">
-        <origin xyz="0.223 0 0.0805" rpy="0 0 0" />
-        <parent link="$(arg prefix)base_link" />
-        <child link="$(arg prefix)front_rail" />
-    </joint>
-    <link name="$(arg prefix)rear_rail"/>
-    <joint name="rear_rail_joint" type="fixed">
-        <origin xyz="-0.223 0 0.0805" rpy="0 0 0" />
-        <parent link="$(arg prefix)base_link" />
-        <child link="$(arg prefix)rear_rail" />
-    </joint>
+    <xacro:empty_link name="$(arg prefix)body"/>
+    <xacro:fixed_joint name="base_link_joint" parent="$(arg prefix)base_link" child="$(arg prefix)body" />
+    <xacro:empty_link name="$(arg prefix)front_rail"/>
+    <xacro:fixed_joint name="front_rail_joint" parent="$(arg prefix)body" child="$(arg prefix)front_rail" xyz="0.223 0 0.0805" />
+    <xacro:empty_link name="$(arg prefix)rear_rail"/>
+    <xacro:fixed_joint name="rear_rail_joint" parent="$(arg prefix)body" child="$(arg prefix)rear_rail" xyz="-0.223 0 0.0805" />
     <xacro:spot_leg leg_name="front_left" prefix="$(arg prefix)" />
     <xacro:spot_leg leg_name="front_right" prefix="$(arg prefix)" />
@@ -51,7 +45,5 @@
     <!-- virtual link to specify IMU position -->
     <xacro:empty_link name="$(arg prefix)imu"/>
-    <xacro:fixed_joint name="imu_j"
-      parent="$(arg prefix)base_link" child="$(arg prefix)imu"
-      xyz="0 0 0" rpy="0 0 0"/>
+    <xacro:fixed_joint name="imu_j" parent="$(arg prefix)base_link" child="$(arg prefix)imu" />
     <gazebo reference="$(arg prefix)imu">
         <xacro:if value="$(arg simulate_imu)">
@@ -61,5 +53,5 @@
                 <imu>
                     <angular_velocity>
-                        <x>
+                        <xacro:macro name="angular_imu_noise">
                             <noise type="gaussian">
                                 <mean>0</mean>
@@ -67,34 +59,16 @@
                                 <bias_mean>0.0000075</bias_mean>
                                 <bias_stddev>0.0000008</bias_stddev>
-                                <dynamic_bias_stddev>0.0000004</dynamic_bias_stddev>
-                                <dynamic_bias_correlation_time>1000.0
-                                </dynamic_bias_correlation_time>
+                                <xacro:if value="${'$(arg rendering_target)' == 'ign'}">
+                                    <dynamic_bias_stddev>0.0000004</dynamic_bias_stddev>
+                                    <dynamic_bias_correlation_time>1000.0</dynamic_bias_correlation_time>
+                                </xacro:if>
                             </noise>
-                        </x>
-                        <y>
-                            <noise type="gaussian">
-                                <mean>0</mean>
-                                <stddev>2e-4</stddev>
-                                <bias_mean>0.0000075</bias_mean>
-                                <bias_stddev>0.0000008</bias_stddev>
-                                <dynamic_bias_stddev>0.0000004</dynamic_bias_stddev>
-                                <dynamic_bias_correlation_time>1000.0
-                                </dynamic_bias_correlation_time>
-                            </noise>
-                        </y>
-                        <z>
-                            <noise type="gaussian">
-                                <mean>0</mean>
-                                <stddev>2e-4</stddev>
-                                <bias_mean>0.0000075</bias_mean>
-                                <bias_stddev>0.0000008</bias_stddev>
-                                <dynamic_bias_stddev>0.0000004</dynamic_bias_stddev>
-                                <dynamic_bias_correlation_time>1000.0
-                                </dynamic_bias_correlation_time>
-                            </noise>
-                        </z>
+                        </xacro:macro>
+                        <x><xacro:angular_imu_noise/></x>
+                        <y><xacro:angular_imu_noise/></y>
+                        <z><xacro:angular_imu_noise/></z>
                     </angular_velocity>
                     <linear_acceleration>
-                        <x>
+                        <xacro:macro name="linear_imu_noise">
                             <noise type="gaussian">
                                 <mean>0</mean>
@@ -102,28 +76,13 @@
                                 <bias_mean>0.1</bias_mean>
                                 <bias_stddev>0.001</bias_stddev>
-                                <dynamic_bias_stddev>0.002</dynamic_bias_stddev>
-                                <dynamic_bias_correlation_time>300.0</dynamic_bias_correlation_time>
+                                <xacro:if value="${'$(arg rendering_target)' == 'ign'}">
+                                    <dynamic_bias_stddev>0.002</dynamic_bias_stddev>
+                                    <dynamic_bias_correlation_time>300.0</dynamic_bias_correlation_time>
+                                </xacro:if>
                             </noise>
-                        </x>
-                        <y>
-                            <noise type="gaussian">
-                                <mean>0</mean>
-                                <stddev>1e-2</stddev>
-                                <bias_mean>0.1</bias_mean>
-                                <bias_stddev>0.001</bias_stddev>
-                                <dynamic_bias_stddev>0.002</dynamic_bias_stddev>
-                                <dynamic_bias_correlation_time>300.0</dynamic_bias_correlation_time>
-                            </noise>
-                        </y>
-                        <z>
-                            <noise type="gaussian">
-                                <mean>0</mean>
-                                <stddev>1e-2</stddev>
-                                <bias_mean>0.1</bias_mean>
-                                <bias_stddev>0.001</bias_stddev>
-                                <dynamic_bias_stddev>0.002</dynamic_bias_stddev>
-                                <dynamic_bias_correlation_time>300.0</dynamic_bias_correlation_time>
-                            </noise>
-                        </z>
+                        </xacro:macro>
+                        <x><xacro:linear_imu_noise /></x>
+                        <y><xacro:linear_imu_noise /></y>
+                        <z><xacro:linear_imu_noise /></z>
                     </linear_acceleration>
                 </imu>

File: submitted_models/bosdyn_spot/urdf/spot_leg.urdf.xacro (robot description, xacro)
@@ -41,5 +41,5 @@
             <parent link="${prefix}base_link" />
             <child link="${prefix}${leg_name}_hip" />
-            <limit effort="100" velocity="1.0" lower="-0.78539816339744827899" upper="0.78539816339744827899" />
+            <limit effort="80" velocity="15" lower="-0.78539816339744827899" upper="0.78539816339744827899" />
         </joint>
         <link name="${prefix}${leg_name}_upper_leg">
@@ -67,5 +67,5 @@
             <parent link="${prefix}${leg_name}_hip" />
             <child link="${prefix}${leg_name}_upper_leg" />
-            <limit effort="100" velocity="1.0" lower="-0.89884456477707963539" upper="2.2951079663725435509" />
+            <limit effort="80" velocity="15" lower="-0.89884456477707963539" upper="2.2951079663725435509" />
         </joint>
         <link name="${prefix}${leg_name}_lower_leg">
@@ -80,4 +80,10 @@
                 </geometry>
             </collision>
+            <collision>
+                <origin xyz="0 0 -${lower_leg_to_foot_z - 0.04 + 0.003}" />
+                <geometry>
+                    <sphere radius="0.04" />
+                </geometry>
+            </collision>
             <inertial>
                 <origin xyz="0 0 -0.16" rpy="0 0 0" />
@@ -89,10 +95,13 @@
         </link>
          <gazebo reference="${prefix}${leg_name}_lower_leg">
-            <kp>100000.0</kp>
-            <kd>1.0</kd>
+            <kp>1e+7</kp>
+            <kd>100.0</kd>
             <mu1>0.8</mu1>
             <mu2>0.8</mu2>
-            <maxVel>0.0</maxVel>
-            <minDepth>0.001</minDepth>
+             <sensor name="contact" type="contact">
+                <contact>
+                    <collision>${leg_name}_lower_leg_collision</collision>
+                </contact>
+             </sensor>
         </gazebo>
         <joint name="${leg_name}_knee" type="revolute">
@@ -101,12 +110,39 @@
             <parent link="${prefix}${leg_name}_upper_leg" />
             <child link="${prefix}${leg_name}_lower_leg" />
-            <limit effort="100" velocity="1.0" lower="-2.7929" upper="-0.254801" />
+            <limit effort="80" velocity="15" lower="-2.7929" upper="-0.254801" />
         </joint>
-        <link name="${prefix}${leg_name}_ee" />
-        <joint name="${leg_name}_foot" type="fixed">
-            <parent link="${prefix}${leg_name}_lower_leg" />
-            <child link="${prefix}${leg_name}_ee" />
-            <origin xyz="0 0 -${lower_leg_to_foot_z}" rpy="0 0 0" />
-        </joint>
+        <xacro:empty_link name="${prefix}${leg_name}_ee" />
+        <xacro:fixed_joint name="${leg_name}_foot" parent="${prefix}${leg_name}_lower_leg" child="${prefix}${leg_name}_ee" xyz="0 0 -${lower_leg_to_foot_z}" />
+        <!-- Not actually used now, but doesn't hurt to have it here ready for future use with ros_ign_control. -->
+        <transmission name="${leg_name}_hip_x_trans">
+            <type>transmission_interface/SimpleTransmission</type>
+            <joint name="${leg_name}_hip_x">
+                <hardwareInterface>hardware_interface/EffortJointInterface</hardwareInterface>
+            </joint>
+            <actuator name="${leg_name}_hip_x_actuator">
+                <hardwareInterface>hardware_interface/EffortJointInterface</hardwareInterface>
+                <mechanicalReduction>1</mechanicalReduction>
+            </actuator>
+        </transmission>
+        <transmission name="${leg_name}_hip_y_trans">
+            <type>transmission_interface/SimpleTransmission</type>
+            <joint name="${leg_name}_hip_y">
+                <hardwareInterface>hardware_interface/EffortJointInterface</hardwareInterface>
+            </joint>
+            <actuator name="${leg_name}_hip_y_actuator">
+                <hardwareInterface>hardware_interface/EffortJointInterface</hardwareInterface>
+                <mechanicalReduction>1</mechanicalReduction>
+            </actuator>
+        </transmission>
+        <transmission name="${leg_name}_knee_trans">
+            <type>transmission_interface/SimpleTransmission</type>
+            <joint name="${leg_name}_knee">
+                <hardwareInterface>hardware_interface/EffortJointInterface</hardwareInterface>
+            </joint>
+            <actuator name="${leg_name}_knee_actuator">
+                <hardwareInterface>hardware_interface/EffortJointInterface</hardwareInterface>
+                <mechanicalReduction>1</mechanicalReduction>
+            </actuator>
+        </transmission>
     </xacro:macro>
 </robot>

File: submitted_models/bosdyn_spot/urdf/utils.xacro (robot description, xacro)
@@ -45,17 +45,9 @@
     <xacro:macro name="empty_link" params="name">
         <link name="${name}">
-            <visual>
-                <origin xyz="0 0 0" rpy="0 0 0" />
-                <geometry>
-                    <box size="0.005 0.005 0.005"/>
-                </geometry>
-                <material name="invisible_color">
-                    <color rgba="1 0 0 0.5"/>
-                </material>
-            </visual>
             <xacro:default_inertial />
+            <selfCollide>false</selfCollide>
         </link>
     </xacro:macro>
-    <xacro:macro name="fixed_joint" params="name parent child xyz='0 0 0' rpy='0 0 0'">
+    <xacro:macro name="fixed_joint" params="name parent child xyz:='0 0 0' rpy:='0 0 0' lump:=0">
         <joint name="${name}" type="fixed">
             <parent link="${parent}"/>
@@ -63,4 +55,10 @@
             <origin xyz="${xyz}" rpy="${rpy}"/>
         </joint>
+        <xacro:if value="${lump == 0}">
+            <!-- workaround for https://github.com/osrf/sdformat/issues/378 -->
+            <gazebo reference="${name}">
+                <preserveFixedJoint>true</preserveFixedJoint>
+            </gazebo>
+        </xacro:if>
     </xacro:macro>
 </root>

Commit message: Spot: Fixed mass by adding battery and tuned the PIDs a bit.

File: submitted_models/bosdyn_spot/urdf/spot.urdf.xacro (robot description, xacro)
@@ -12,4 +12,7 @@
     <xacro:arg name="simulate_cameras" default="True"/>
     <xacro:arg name="simulate_imu" default="True"/>
+    <xacro:arg name="body_color_r" default="${str(234/255.0)}" />
+    <xacro:arg name="body_color_g" default="${str(167/255.0)}" />
+    <xacro:arg name="body_color_b" default="0" />
     <xacro:include filename="utils.xacro"/>
     <xacro:include filename="constants.urdf.xacro" />
@@ -34,4 +37,22 @@
         </inertial>
     </link>
+    <link name="$(arg prefix)battery">
+        <visual>
+            <geometry>
+                <box size="0.324 0.168 0.093" />
+            </geometry>
+            <material name="spot_color">
+                <color rgba="$(arg body_color_r) $(arg body_color_g) $(arg body_color_b) 1.0"/>
+            </material>
+        </visual>
+        <collision>
+            <geometry>
+                <box size="0.324 0.168 0.093" />
+            </geometry>
+        </collision>
+        <xacro:box_inertial mass="4.0" depth="0.324" width="0.168" height="0.093" />
+    </link>
+    <xacro:solid_color_link_material link="$(arg prefix)battery" r="$(arg body_color_r)" g="$(arg body_color_g)" b="$(arg body_color_b)" />
+    <xacro:fixed_joint name="battery_joint" parent="$(arg prefix)base_link" child="$(arg prefix)battery" xyz="0 0 -0.03" />
     <xacro:empty_link name="$(arg prefix)body"/>
     <xacro:fixed_joint name="base_link_joint" parent="$(arg prefix)base_link" child="$(arg prefix)body" />

File: submitted_models/bosdyn_spot/urdf/utils.xacro (robot description, xacro)
@@ -62,3 +62,17 @@
         </xacro:if>
     </xacro:macro>
+    <xacro:macro name="solid_color_link_material" params="link r g b">
+        <xacro:unless value="${'$(arg rendering_target)' == 'urdf'}">
+            <gazebo reference="${link}">
+                <visual>
+                    <material>
+                        <ambient>${r} ${g} ${b} 1</ambient>
+                        <diffuse>${r} ${g} ${b} 1</diffuse>
+                        <specular>${r} ${g} ${b} 1</specular>
+                        <emissive>0 0 0 0</emissive>
+                    </material>
+                </visual>
+            </gazebo>
+        </xacro:unless>
+    </xacro:macro>
 </root>
