Commit message: Addressed review comments regarding executable name and T265 sensor visual.

File: submitted_models/coro_pam_sensor_config_1/urdf/model.xacro (robot description, xacro)
@@ -259,10 +259,4 @@
       <geometry>
         <box size='0.001 0.02 0.06'/>
-      </geometry>
-    </visual>
-    <visual name='t265_visual'>
-      <origin xyz='0.09 0 -0.143' rpy='0 0.75 0'/>
-      <geometry>
-        <box size='0.013 0.108 0.025'/>
       </geometry>
     </visual>
