Commit message: added missing meshes

File: submitted_models/ctu_cras_norlab_x500_sensor_config_2/urdf/model.xacro (robot description, xacro)
@@ -1,5 +1,5 @@
 <?xml version='1.0' encoding='utf-8'?>
 <robot name='ctu_cras_norlab_x500_sensor_config_2' xmlns:xacro='http://ros.org/wiki/xacro'>
-  <xacro:arg name="name" default="ctu_cras_norlab_x500_sensor_config_1"/>
+  <xacro:arg name="name" default="ctu_cras_norlab_x500_sensor_config_2"/>
   <xacro:property name="robot_namespace" value="$(arg name)"/>
   <link name='${robot_namespace}/base_link'>
@@ -72,5 +72,5 @@
       <origin xyz='0 0 -0.022' rpy='1.5708 0 -1.5708'/>
       <geometry>
-        <mesh filename='package://ctu_cras_norlab_x500_sensor_config_1/meshes/holders/holder_rs_down_bfox.dae' scale='1 1 1'/>
+        <mesh filename='package://ctu_cras_norlab_x500_sensor_config_2/meshes/holders/holder_rs_down_bfox.dae' scale='1 1 1'/>
       </geometry>
     </collision>
@@ -78,5 +78,5 @@
       <origin xyz='0.107 0 0' rpy='0 -0 0'/>
       <geometry>
-        <mesh filename='package://ctu_cras_norlab_x500_sensor_config_1/meshes/sensors/bluefox.dae' scale='1 1 1'/>
+        <mesh filename='package://ctu_cras_norlab_x500_sensor_config_2/meshes/sensors/bluefox.dae' scale='1 1 1'/>
       </geometry>
     </visual>
@@ -84,5 +84,5 @@
       <origin xyz='-0.064 0 0.03' rpy='0 -0 1.5708'/>
       <geometry>
-        <mesh filename='package://ctu_cras_norlab_x500_sensor_config_1/meshes/holders/side_mrs.dae' scale='1 1 1'/>
+        <mesh filename='package://ctu_cras_norlab_x500_sensor_config_2/meshes/holders/side_mrs.dae' scale='1 1 1'/>
       </geometry>
     </visual>
@@ -90,5 +90,5 @@
       <origin xyz='0 0 0' rpy='0 -0 2.35619'/>
       <geometry>
-        <mesh filename='package://ctu_cras_norlab_x500_sensor_config_1/meshes/holybro/holybro_x500_arm.dae' scale='1 1 1'/>
+        <mesh filename='package://ctu_cras_norlab_x500_sensor_config_2/meshes/holybro/holybro_x500_arm.dae' scale='1 1 1'/>
       </geometry>
     </visual>
@@ -96,5 +96,5 @@
       <origin xyz='-0.177484 0.177484 0.021' rpy='0 -0 0'/>
       <geometry>
-        <mesh filename='package://ctu_cras_norlab_x500_sensor_config_1/meshes/holybro/holybro_x500_motor.dae' scale='1 1 1'/>
+        <mesh filename='package://ctu_cras_norlab_x500_sensor_config_2/meshes/holybro/holybro_x500_motor.dae' scale='1 1 1'/>
       </geometry>
     </visual>
@@ -102,5 +102,5 @@
       <origin xyz='0 0 0' rpy='0 0 -2.35619'/>
       <geometry>
-        <mesh filename='package://ctu_cras_norlab_x500_sensor_config_1/meshes/holybro/holybro_x500_arm.dae' scale='1 1 1'/>
+        <mesh filename='package://ctu_cras_norlab_x500_sensor_config_2/meshes/holybro/holybro_x500_arm.dae' scale='1 1 1'/>
       </geometry>
     </visual>
@@ -108,5 +108,5 @@
       <origin xyz='-0.177484 -0.177484 0.021' rpy='0 -0 0'/>
       <geometry>
-        <mesh filename='package://ctu_cras_norlab_x500_sensor_config_1/meshes/holybro/holybro_x500_motor.dae' scale='1 1 1'/>
+        <mesh filename='package://ctu_cras_norlab_x500_sensor_config_2/meshes/holybro/holybro_x500_motor.dae' scale='1 1 1'/>
       </geometry>
     </visual>
@@ -114,5 +114,5 @@
       <origin xyz='-0.02 0.03 0' rpy='0 -0 0'/>
       <geometry>
-        <mesh filename='package://ctu_cras_norlab_x500_sensor_config_1/meshes/holybro/holybro_x500_battery.dae' scale='1 1 1'/>
+        <mesh filename='package://ctu_cras_norlab_x500_sensor_config_2/meshes/holybro/holybro_x500_battery.dae' scale='1 1 1'/>
       </geometry>
     </visual>
@@ -120,5 +120,5 @@
       <origin xyz='-0.02 -0.03 0' rpy='0 -0 0'/>
       <geometry>
-        <mesh filename='package://ctu_cras_norlab_x500_sensor_config_1/meshes/holybro/holybro_x500_battery.dae' scale='1 1 1'/>
+        <mesh filename='package://ctu_cras_norlab_x500_sensor_config_2/meshes/holybro/holybro_x500_battery.dae' scale='1 1 1'/>
       </geometry>
     </visual>
@@ -126,5 +126,5 @@
       <origin xyz='0 0 0' rpy='0 -0 0'/>
       <geometry>
-        <mesh filename='package://ctu_cras_norlab_x500_sensor_config_1/meshes/holybro/holybro_x500_bottom_board.dae' scale='1 1 1'/>
+        <mesh filename='package://ctu_cras_norlab_x500_sensor_config_2/meshes/holybro/holybro_x500_bottom_board.dae' scale='1 1 1'/>
       </geometry>
     </visual>
@@ -150,5 +150,5 @@
       <origin xyz='0 0 0' rpy='0 -0 0.785398'/>
       <geometry>
-        <mesh filename='package://ctu_cras_norlab_x500_sensor_config_1/meshes/holybro/holybro_x500_arm.dae' scale='1 1 1'/>
+        <mesh filename='package://ctu_cras_norlab_x500_sensor_config_2/meshes/holybro/holybro_x500_arm.dae' scale='1 1 1'/>
       </geometry>
     </visual>
@@ -156,5 +156,5 @@
       <origin xyz='0.162635 0.162635 -0.157' rpy='0 -0 0.785398'/>
       <geometry>
-        <mesh filename='package://ctu_cras_norlab_x500_sensor_config_1/meshes/holybro/holybro_x500_leg.dae' scale='1 1 1'/>
+        <mesh filename='package://ctu_cras_norlab_x500_sensor_config_2/meshes/holybro/holybro_x500_leg.dae' scale='1 1 1'/>
       </geometry>
     </visual>
@@ -168,5 +168,5 @@
       <origin xyz='0.177484 0.177484 0.021' rpy='0 -0 0'/>
       <geometry>
-        <mesh filename='package://ctu_cras_norlab_x500_sensor_config_1/meshes/holybro/holybro_x500_motor.dae' scale='1 1 1'/>
+        <mesh filename='package://ctu_cras_norlab_x500_sensor_config_2/meshes/holybro/holybro_x500_motor.dae' scale='1 1 1'/>
       </geometry>
     </visual>
@@ -174,5 +174,5 @@
       <origin xyz='0 0 0' rpy='0 0 -0.785398'/>
       <geometry>
-        <mesh filename='package://ctu_cras_norlab_x500_sensor_config_1/meshes/holybro/holybro_x500_arm.dae' scale='1 1 1'/>
+        <mesh filename='package://ctu_cras_norlab_x500_sensor_config_2/meshes/holybro/holybro_x500_arm.dae' scale='1 1 1'/>
       </geometry>
     </visual>
@@ -180,5 +180,5 @@
       <origin xyz='0.162635 -0.162635 -0.157' rpy='0 0 -0.785398'/>
       <geometry>
-        <mesh filename='package://ctu_cras_norlab_x500_sensor_config_1/meshes/holybro/holybro_x500_leg.dae' scale='1 1 1'/>
+        <mesh filename='package://ctu_cras_norlab_x500_sensor_config_2/meshes/holybro/holybro_x500_leg.dae' scale='1 1 1'/>
       </geometry>
     </visual>
@@ -192,5 +192,5 @@
       <origin xyz='0.177484 -0.177484 0.021' rpy='0 -0 0'/>
       <geometry>
-        <mesh filename='package://ctu_cras_norlab_x500_sensor_config_1/meshes/holybro/holybro_x500_motor.dae' scale='1 1 1'/>
+        <mesh filename='package://ctu_cras_norlab_x500_sensor_config_2/meshes/holybro/holybro_x500_motor.dae' scale='1 1 1'/>
       </geometry>
     </visual>
@@ -198,5 +198,5 @@
       <origin xyz='0 0.064 0.03' rpy='0 0 -3.14159'/>
       <geometry>
-        <mesh filename='package://ctu_cras_norlab_x500_sensor_config_1/meshes/holders/side_ctu.dae' scale='1 1 1'/>
+        <mesh filename='package://ctu_cras_norlab_x500_sensor_config_2/meshes/holders/side_ctu.dae' scale='1 1 1'/>
       </geometry>
     </visual>
@@ -204,5 +204,5 @@
       <origin xyz='0 0 0.06' rpy='0 -0 1.5708'/>
       <geometry>
-        <mesh filename='package://ctu_cras_norlab_x500_sensor_config_1/meshes/sensors/os1_64.dae' scale='1 1 1'/>
+        <mesh filename='package://ctu_cras_norlab_x500_sensor_config_2/meshes/sensors/os1_64.dae' scale='1 1 1'/>
       </geometry>
     </visual>
@@ -216,5 +216,5 @@
       <origin xyz='0 0 0' rpy='0 -0 0'/>
       <geometry>
-        <mesh filename='package://ctu_cras_norlab_x500_sensor_config_1/meshes/holybro/holybro_x500_pc_mount.dae' scale='1 1 1'/>
+        <mesh filename='package://ctu_cras_norlab_x500_sensor_config_2/meshes/holybro/holybro_x500_pc_mount.dae' scale='1 1 1'/>
       </geometry>
     </visual>
@@ -222,5 +222,5 @@
       <origin xyz='0 0 0.036' rpy='0 -0 0'/>
       <geometry>
-        <mesh filename='package://ctu_cras_norlab_x500_sensor_config_1/meshes/sensors/pixhawk.dae' scale='1 1 1'/>
+        <mesh filename='package://ctu_cras_norlab_x500_sensor_config_2/meshes/sensors/pixhawk.dae' scale='1 1 1'/>
       </geometry>
     </visual>
@@ -228,5 +228,5 @@
       <origin xyz='-0.162635 0.162635 -0.157' rpy='0 -0 2.35619'/>
       <geometry>
-        <mesh filename='package://ctu_cras_norlab_x500_sensor_config_1/meshes/holybro/holybro_x500_leg.dae' scale='1 1 1'/>
+        <mesh filename='package://ctu_cras_norlab_x500_sensor_config_2/meshes/holybro/holybro_x500_leg.dae' scale='1 1 1'/>
       </geometry>
     </visual>
@@ -234,5 +234,5 @@
       <origin xyz='-0.162635 -0.162635 -0.157' rpy='0 0 -2.35619'/>
       <geometry>
-        <mesh filename='package://ctu_cras_norlab_x500_sensor_config_1/meshes/holybro/holybro_x500_leg.dae' scale='1 1 1'/>
+        <mesh filename='package://ctu_cras_norlab_x500_sensor_config_2/meshes/holybro/holybro_x500_leg.dae' scale='1 1 1'/>
       </geometry>
     </visual>
@@ -240,5 +240,5 @@
       <origin xyz='0 -0.064 0.03' rpy='0 -0 0'/>
       <geometry>
-        <mesh filename='package://ctu_cras_norlab_x500_sensor_config_1/meshes/holders/side_ctu.dae' scale='1 1 1'/>
+        <mesh filename='package://ctu_cras_norlab_x500_sensor_config_2/meshes/holders/side_ctu.dae' scale='1 1 1'/>
       </geometry>
     </visual>
@@ -246,5 +246,5 @@
       <origin xyz='0 0 -0.022' rpy='1.5708 0 -1.5708'/>
       <geometry>
-        <mesh filename='package://ctu_cras_norlab_x500_sensor_config_1/meshes/holders/holder_rs_down_bfox.dae' scale='1 1 1'/>
+        <mesh filename='package://ctu_cras_norlab_x500_sensor_config_2/meshes/holders/holder_rs_down_bfox.dae' scale='1 1 1'/>
       </geometry>
     </visual>
@@ -287,5 +287,5 @@
       <origin xyz='-0.177484 0.177484 -0.057' rpy='0 -0 0'/>
       <geometry>
-        <mesh filename='package://ctu_cras_norlab_x500_sensor_config_1/meshes/holybro/holybro_x500_prop.dae' scale='1 1 1'/>
+        <mesh filename='package://ctu_cras_norlab_x500_sensor_config_2/meshes/holybro/holybro_x500_prop.dae' scale='1 1 1'/>
       </geometry>
     </visual>
@@ -306,5 +306,5 @@
       <origin xyz='0.177484 -0.177484 -0.057' rpy='0 -0 0'/>
       <geometry>
-        <mesh filename='package://ctu_cras_norlab_x500_sensor_config_1/meshes/holybro/holybro_x500_prop.dae' scale='1 1 1'/>
+        <mesh filename='package://ctu_cras_norlab_x500_sensor_config_2/meshes/holybro/holybro_x500_prop.dae' scale='1 1 1'/>
       </geometry>
     </visual>
@@ -325,5 +325,5 @@
       <origin xyz='-0.177484 -0.177484 -0.057' rpy='0 -0 0'/>
       <geometry>
-        <mesh filename='package://ctu_cras_norlab_x500_sensor_config_1/meshes/holybro/holybro_x500_prop.dae' scale='-1 1 1'/>
+        <mesh filename='package://ctu_cras_norlab_x500_sensor_config_2/meshes/holybro/holybro_x500_prop.dae' scale='-1 1 1'/>
       </geometry>
     </visual>
@@ -344,5 +344,5 @@
       <origin xyz='0.177484 0.177484 -0.057' rpy='0 -0 0'/>
       <geometry>
-        <mesh filename='package://ctu_cras_norlab_x500_sensor_config_1/meshes/holybro/holybro_x500_prop.dae' scale='-1 1 1'/>
+        <mesh filename='package://ctu_cras_norlab_x500_sensor_config_2/meshes/holybro/holybro_x500_prop.dae' scale='-1 1 1'/>
       </geometry>
     </visual>
