Commit message: MARV: Added camera intrinsics.

File: submitted_models/ctu_cras_norlab_marv_sensor_config_1/urdf/basler_cameras.xacro (robot description, xacro)
@@ -75,12 +75,20 @@
                             <stddev>0.007</stddev>
                         </noise>
-                        <xacro:if value="${fisheye and '$(arg rendering_target)' == 'gz'}">
-                            <lens>
+                        <lens>
+                            <intrinsics>
+                                <xacro:property name="f" value="${resolution_x / (2 * tan(radians(hfov_deg)/2))}" />
+                                <fx>${f}</fx>
+                                <fy>${f}</fy>
+                                <cx>${(resolution_x - 1) / 2}</cx>
+                                <cy>${(resolution_y - 1) / 2}</cy>
+                                <s>0</s>
+                            </intrinsics>
+                            <xacro:if value="${fisheye and '$(arg rendering_target)' == 'gz'}">
                                 <type>stereographic</type>
                                 <scale_to_hfov>true</scale_to_hfov>
                                 <cutoff_angle>${pi}</cutoff_angle>
                                 <env_texture_size>1024</env_texture_size>
-                            </lens>
-                        </xacro:if>
+                            </xacro:if>
+                        </lens>
                     </camera>
                 </sensor>
