Commit message: Lily: Corrected mass.

File: submitted_models/ctu_cras_norlab_lily_sensor_config_1/urdf/link.xacro (robot description, xacro)
@@ -177,4 +177,20 @@
           </contact>
         </sensor>
+        <collision>
+          <surface>
+            <contact>
+              <ode>
+                <kp>1e+10</kp>
+                <kd>1</kd>
+              </ode>
+            </contact>
+            <friction>
+              <ode>
+                <mu>10.0</mu>
+                <!--<mu2>10.0</mu2>-->
+              </ode>
+            </friction>
+          </surface>
+        </collision>
       </gazebo>
     </xacro:if>

File: submitted_models/ctu_cras_norlab_lily_sensor_config_1/urdf/payload.xacro (robot description, xacro)
@@ -28,7 +28,8 @@
       <!-- simplified inertia -->
       <!-- mass including chasis, onboard computer, breadcrumbs (???) etc.-->
-      <xacro:box_inertial x_size="0.4" y_size="0.2" z_size="0.1" mass="1.5"
+      <xacro:box_inertial x_size="0.4" y_size="0.2" z_size="0.1" mass="7"
                           xyz="0 0 0.05" rpy="0 0 0"/>
-      <!-- upper box -->
+    </link>
+    <link name="$(arg prefix)upper_box">
       <!--
       <visual>
@@ -47,6 +48,9 @@
       <!-- simplified inertia -->
       <!-- mass including chasis, cameras, wifi, etc.-->
-      <xacro:box_inertial x_size="0.25" y_size="0.2" z_size="0.1" mass="1"
+      <xacro:box_inertial x_size="0.25" y_size="0.2" z_size="0.1" mass="5"
                           xyz="-0.05 0 0.15" rpy="0 0 0"/>
+    </link>
+    <xacro:fixed_joint name="upper_box_j" parent="$(arg prefix)base_link" child="$(arg prefix)upper_box" />
+    <link name="$(arg prefix)battery_right">
       <!-- battery-right -->
       <visual>
@@ -67,4 +71,7 @@
       </inertial>
       <!-- AUTOGENERATE END -->
+    </link>
+    <xacro:fixed_joint name="battery_right_j" parent="$(arg prefix)base_link" child="$(arg prefix)battery_right" />
+    <link name="$(arg prefix)battery_left">
       <!-- battery-left -->
       <visual>
@@ -86,6 +93,16 @@
       <!-- AUTOGENERATE END -->
     </link>
+    <xacro:fixed_joint name="battery_left_j" parent="$(arg prefix)base_link" child="$(arg prefix)battery_left" />
     <!-- material -->
-    <gazebo reference="base_link">
+    <gazebo reference="$(arg prefix)base_link">
+      <xacro:gazebo_black_material/>
+    </gazebo>
+    <gazebo reference="$(arg prefix)upper_box">
+      <xacro:gazebo_black_material/>
+    </gazebo>
+    <gazebo reference="$(arg prefix)battery_right">
+      <xacro:gazebo_black_material/>
+    </gazebo>
+    <gazebo reference="$(arg prefix)battery_left">
       <xacro:gazebo_black_material/>
     </gazebo>
