Commit message: Updates to both sensor configurations based upon PR feedback.

File: submitted_models/marble_spot_sensor_config_1/urdf/basler_cameras.xacro (robot description, xacro)
@@ -94,5 +94,5 @@
             fisheye="${fisheye}" simulate="${simulate}" visualize="${visualize}"
             camera_length="0.0555" origin_to_camera_front_dist="0.0524" camera_mass="${basler_ace2_pro_mass}"
-            camera_mesh="package://ctu_cras_norlab_spot_sensor_config_1/meshes/basler_ace2_pro.dae"
+            camera_mesh="package://marble_spot_sensor_config_1/meshes/basler_ace2_pro.dae"
             lens_length="${lens_length}" lens_back_focal_distance="${lens_back_focal_distance}"
             lens_entrance_pupil_position="${lens_entrance_pupil_position}" lens_mass="${lens_mass}" lens_mesh="${lens_mesh}"
@@ -103,5 +103,5 @@
         <xacro:basler_ace2_pro_link name="${name}" hfov_deg="86.5" simulate="${simulate}" visualize="${visualize}"
             lens_back_focal_distance="0.00809" lens_entrance_pupil_position="0.01066" lens_length="0.03974" lens_mass="${omnicam_lens_mass}"
-            lens_mesh="package://ctu_cras_norlab_spot_sensor_config_1/meshes/evetar_lens.dae" />
+            lens_mesh="package://marble_spot_sensor_config_1/meshes/evetar_lens.dae" />
     </xacro:macro>
 </root>

File: submitted_models/marble_spot_sensor_config_1/urdf/flir_cameras.xacro (robot description, xacro)
@@ -90,5 +90,5 @@
             fisheye="${fisheye}" simulate="${simulate}" visualize="${visualize}"
             camera_length="0.0555" origin_to_camera_front_dist="0.0524" camera_mass="${flir_backly_mass}"
-            camera_mesh="package://ctu_cras_norlab_spot_sensor_config_1/meshes/basler_ace2_pro.dae"
+            camera_mesh="package://marble_spot_sensor_config_1/meshes/basler_ace2_pro.dae"
             lens_length="${lens_length}" lens_back_focal_distance="${lens_back_focal_distance}"
             lens_entrance_pupil_position="${lens_entrance_pupil_position}" lens_mass="${lens_mass}" lens_mesh="${lens_mesh}"
@@ -99,5 +99,5 @@
         <xacro:flir_backly_link name="${name}" hfov_deg="80" simulate="${simulate}" visualize="${visualize}"
             lens_back_focal_distance="0.00809" lens_entrance_pupil_position="0.01066" lens_length="0.03974" lens_mass="${lens_mass}"
-            lens_mesh="package://ctu_cras_norlab_spot_sensor_config_1/meshes/evetar_lens.dae" />
+            lens_mesh="package://marble_spot_sensor_config_1/meshes/evetar_lens.dae" />
     </xacro:macro>
 </root>

File: submitted_models/marble_spot_sensor_config_1/urdf/imu.xacro (robot description, xacro)
@@ -25,10 +25,11 @@
                                 <noise type="gaussian">
                                     <mean>0</mean>
-                                    <stddev>2e-4</stddev>
-                                    <bias_mean>0.0000075</bias_mean>
-                                    <bias_stddev>0.0000008</bias_stddev>
+                                    <stddev>0.009</stddev>
+                                    <bias_mean>0.00075</bias_mean>
+                                    <bias_stddev>0.005</bias_stddev>
                                     <xacro:if value="${'$(arg rendering_target)' == 'ign'}">
-                                        <dynamic_bias_stddev>0.0000004</dynamic_bias_stddev>
-                                        <dynamic_bias_correlation_time>1000.0</dynamic_bias_correlation_time>
+                                        <dynamic_bias_stddev>0.00002</dynamic_bias_stddev>
+                                        <dynamic_bias_correlation_time>400.0</dynamic_bias_correlation_time>
+                                        <precision>0.00025</precision>
                                     </xacro:if>
                                 </noise>
@@ -42,10 +43,11 @@
                                 <noise type="gaussian">
                                     <mean>0</mean>
-                                    <stddev>1e-2</stddev>
-                                    <bias_mean>0.1</bias_mean>
-                                    <bias_stddev>0.001</bias_stddev>
+                                    <stddev>0.021</stddev>
+                                    <bias_mean>0.05</bias_mean>
+                                    <bias_stddev>0.0075</bias_stddev>
                                     <xacro:if value="${'$(arg rendering_target)' == 'ign'}">
-                                        <dynamic_bias_stddev>0.002</dynamic_bias_stddev>
-                                        <dynamic_bias_correlation_time>300.0</dynamic_bias_correlation_time>
+                                        <dynamic_bias_stddev>0.000375</dynamic_bias_stddev>
+                                        <dynamic_bias_correlation_time>175.0</dynamic_bias_correlation_time>
+                                        <precision>0.005</precision>
                                     </xacro:if>
                                 </noise>

File: submitted_models/marble_spot_sensor_config_1/urdf/mote_deployer.xacro (robot description, xacro)
@@ -9,5 +9,5 @@
             <visual>
                 <geometry>
-                    <mesh filename="package://ctu_cras_norlab_spot_sensor_config_1/meshes/mote_deployer.dae" />
+                    <mesh filename="package://marble_spot_sensor_config_1/meshes/mote_deployer.dae" />
                 </geometry>
             </visual>

File: submitted_models/marble_spot_sensor_config_1/urdf/ouster_lidar.xacro (robot description, xacro)
@@ -7,5 +7,5 @@
             <visual>
                 <geometry>
-                    <mesh filename="package://ctu_cras_norlab_spot_sensor_config_1/meshes/ouster-os0.dae"/>
+                    <mesh filename="package://marble_spot_sensor_config_1/meshes/ouster-os0.dae"/>
                 </geometry>
             </visual>
@@ -43,10 +43,10 @@
                             <min>0.1</min>
                             <max>50</max>
-                            <resolution>0.003</resolution>
+                            <resolution>0.01</resolution>
                         </range>
                         <noise>
                             <type>gaussian</type>
                             <mean>0</mean>
-                            <stddev>0.03</stddev>
+                            <stddev>0.01</stddev>
                         </noise>
                     </lidar>

File: submitted_models/marble_spot_sensor_config_1/urdf/ouster_lidar_alt.xacro (robot description, xacro)
@@ -7,5 +7,5 @@
             <visual>
                 <geometry>
-                    <mesh filename="package://ctu_cras_norlab_spot_sensor_config_1/meshes/ouster-os0.dae"/>
+                    <mesh filename="package://marble_spot_sensor_config_1/meshes/ouster-os0.dae"/>
                 </geometry>
             </visual>
@@ -42,11 +42,11 @@
                         <range>
                             <min>0.1</min>
-                            <max>50</max>
-                            <resolution>0.003</resolution>
+                            <max>120</max>
+                            <resolution>0.01</resolution>
                         </range>
                         <noise>
                             <type>gaussian</type>
                             <mean>0</mean>
-                            <stddev>0.03</stddev>
+                            <stddev>0.01</stddev>
                         </noise>
                     </lidar>

File: submitted_models/marble_spot_sensor_config_1/urdf/spot.urdf.xacro (robot description, xacro)
@@ -1,4 +1,4 @@
 <?xml version="1.0" ?>
-<robot name="ctu_cras_norlab_spot_sensor_config_1" xmlns:xacro="http://www.ros.org/wiki/xacro">
+<robot name="marble_spot_sensor_config_1" xmlns:xacro="http://www.ros.org/wiki/xacro">
     <xacro:arg name="has_flir_cameras" default="1" />
     <xacro:arg name="has_ouster_lidar" default="0" />
@@ -10,5 +10,5 @@
     <xacro:arg name="simulate_omnicam_vras" default="True" />
     <xacro:arg name="simulate_flircams" default="True" />
-    <xacro:arg name="simulate_imu" default="False" />
+    <xacro:arg name="simulate_imu" default="True" />
     <xacro:arg name="visualize_sensors" default="0" />
     <xacro:property name="payload_z_top" value="0.105" />
@@ -18,8 +18,8 @@
     <!-- Colon-separated list of payload Xacro files to include. Whitespace around is ignored. -->
     <xacro:arg name="payload_xacros" default="
-      $(find ctu_cras_norlab_spot_sensor_config_1)/urdf/basler_cameras.xacro :
-      $(find ctu_cras_norlab_spot_sensor_config_1)/urdf/imu.xacro :
-      $(find ctu_cras_norlab_spot_sensor_config_1)/urdf/mote_deployer.xacro :
-      $(find ctu_cras_norlab_spot_sensor_config_1)/urdf/ouster_lidar.xacro :
+      $(find marble_spot_sensor_config_1)/urdf/basler_cameras.xacro :
+      $(find marble_spot_sensor_config_1)/urdf/imu.xacro :
+      $(find marble_spot_sensor_config_1)/urdf/mote_deployer.xacro :
+      $(find marble_spot_sensor_config_1)/urdf/ouster_lidar.xacro :
       $(find marble_spot_sensor_config_1)/urdf/ouster_lidar_alt.xacro :
       $(find marble_spot_sensor_config_1)/urdf/flir_cameras.xacro :
@@ -46,5 +46,5 @@
             <origin rpy="1.5708 0 1.5708" xyz="0.325 0 0.005"/>
             <geometry>
-                <mesh filename="package://ctu_cras_norlab_spot_sensor_config_1/meshes/spot_sensor_rig_assembly.dae" />
+                <mesh filename="package://marble_spot_sensor_config_1/meshes/spot_sensor_rig_assembly.dae" />
             </geometry>
         </visual>
@@ -135,5 +135,5 @@
     </xacro:if>
     <!-- LIGHTS -->
-    <xacro:include filename="$(find ctu_cras_norlab_spot_sensor_config_1)/urdf/lights.xacro" />
+    <xacro:include filename="$(find marble_spot_sensor_config_1)/urdf/lights.xacro" />
     <gazebo reference="$(arg prefix)payload">
         <xacro:led_stripe name="light_left" range="20" linear="0.2" constant="0.1" quadratic="0.0025"

File: submitted_models/marble_spot_sensor_config_2/urdf/basler_cameras.xacro (robot description, xacro)
@@ -94,5 +94,5 @@
             fisheye="${fisheye}" simulate="${simulate}" visualize="${visualize}"
             camera_length="0.0555" origin_to_camera_front_dist="0.0524" camera_mass="${basler_ace2_pro_mass}"
-            camera_mesh="package://ctu_cras_norlab_spot_sensor_config_1/meshes/basler_ace2_pro.dae"
+            camera_mesh="package://marble_spot_sensor_config_2/meshes/basler_ace2_pro.dae"
             lens_length="${lens_length}" lens_back_focal_distance="${lens_back_focal_distance}"
             lens_entrance_pupil_position="${lens_entrance_pupil_position}" lens_mass="${lens_mass}" lens_mesh="${lens_mesh}"
@@ -103,5 +103,5 @@
         <xacro:basler_ace2_pro_link name="${name}" hfov_deg="86.5" simulate="${simulate}" visualize="${visualize}"
             lens_back_focal_distance="0.00809" lens_entrance_pupil_position="0.01066" lens_length="0.03974" lens_mass="${omnicam_lens_mass}"
-            lens_mesh="package://ctu_cras_norlab_spot_sensor_config_1/meshes/evetar_lens.dae" />
+            lens_mesh="package://marble_spot_sensor_config_2/meshes/evetar_lens.dae" />
     </xacro:macro>
 </root>

File: submitted_models/marble_spot_sensor_config_2/urdf/flir_cameras.xacro (robot description, xacro)
@@ -90,5 +90,5 @@
             fisheye="${fisheye}" simulate="${simulate}" visualize="${visualize}"
             camera_length="0.0555" origin_to_camera_front_dist="0.0524" camera_mass="${flir_backly_mass}"
-            camera_mesh="package://ctu_cras_norlab_spot_sensor_config_1/meshes/basler_ace2_pro.dae"
+            camera_mesh="package://marble_spot_sensor_config_2/meshes/basler_ace2_pro.dae"
             lens_length="${lens_length}" lens_back_focal_distance="${lens_back_focal_distance}"
             lens_entrance_pupil_position="${lens_entrance_pupil_position}" lens_mass="${lens_mass}" lens_mesh="${lens_mesh}"
@@ -99,5 +99,5 @@
         <xacro:flir_backly_link name="${name}" hfov_deg="80" simulate="${simulate}" visualize="${visualize}"
             lens_back_focal_distance="0.00809" lens_entrance_pupil_position="0.01066" lens_length="0.03974" lens_mass="${lens_mass}"
-            lens_mesh="package://ctu_cras_norlab_spot_sensor_config_1/meshes/evetar_lens.dae" />
+            lens_mesh="package://marble_spot_sensor_config_2/meshes/evetar_lens.dae" />
     </xacro:macro>
 </root>

File: submitted_models/marble_spot_sensor_config_2/urdf/mote_deployer.xacro (robot description, xacro)
@@ -9,5 +9,5 @@
             <visual>
                 <geometry>
-                    <mesh filename="package://ctu_cras_norlab_spot_sensor_config_1/meshes/mote_deployer.dae" />
+                    <mesh filename="package://marble_spot_sensor_config_2/meshes/mote_deployer.dae" />
                 </geometry>
             </visual>

File: submitted_models/marble_spot_sensor_config_2/urdf/ouster_lidar.xacro (robot description, xacro)
@@ -7,5 +7,5 @@
             <visual>
                 <geometry>
-                    <mesh filename="package://ctu_cras_norlab_spot_sensor_config_1/meshes/ouster-os0.dae"/>
+                    <mesh filename="package://marble_spot_sensor_config_2/meshes/ouster-os0.dae"/>
                 </geometry>
             </visual>
@@ -43,10 +43,10 @@
                             <min>0.1</min>
                             <max>50</max>
-                            <resolution>0.003</resolution>
+                            <resolution>0.01</resolution>
                         </range>
                         <noise>
                             <type>gaussian</type>
                             <mean>0</mean>
-                            <stddev>0.03</stddev>
+                            <stddev>0.01</stddev>
                         </noise>
                     </lidar>

File: submitted_models/marble_spot_sensor_config_2/urdf/ouster_lidar_alt.xacro (robot description, xacro)
@@ -7,5 +7,5 @@
             <visual>
                 <geometry>
-                    <mesh filename="package://ctu_cras_norlab_spot_sensor_config_1/meshes/ouster-os0.dae"/>
+                    <mesh filename="package://marble_spot_sensor_config_2/meshes/ouster-os0.dae"/>
                 </geometry>
             </visual>
@@ -42,11 +42,11 @@
                         <range>
                             <min>0.1</min>
-                            <max>50</max>
-                            <resolution>0.003</resolution>
+                            <max>120</max>
+                            <resolution>0.01</resolution>
                         </range>
                         <noise>
                             <type>gaussian</type>
                             <mean>0</mean>
-                            <stddev>0.03</stddev>
+                            <stddev>0.01</stddev>
                         </noise>
                     </lidar>

File: submitted_models/marble_spot_sensor_config_2/urdf/spot.urdf.xacro (robot description, xacro)
@@ -1,4 +1,4 @@
 <?xml version="1.0" ?>
-<robot name="ctu_cras_norlab_spot_sensor_config_1" xmlns:xacro="http://www.ros.org/wiki/xacro">
+<robot name="marble_spot_sensor_config_2" xmlns:xacro="http://www.ros.org/wiki/xacro">
     <xacro:arg name="has_flir_cameras" default="1" />
     <xacro:arg name="has_ouster_lidar" default="0" />
@@ -10,5 +10,5 @@
     <xacro:arg name="simulate_omnicam_vras" default="True" />
     <xacro:arg name="simulate_flircams" default="True" />
-    <xacro:arg name="simulate_imu" default="False" />
+    <xacro:arg name="simulate_imu" default="True" />
     <xacro:arg name="visualize_sensors" default="0" />
     <xacro:property name="payload_z_top" value="0.105" />
@@ -18,8 +18,8 @@
     <!-- Colon-separated list of payload Xacro files to include. Whitespace around is ignored. -->
     <xacro:arg name="payload_xacros" default="
-      $(find ctu_cras_norlab_spot_sensor_config_1)/urdf/basler_cameras.xacro :
-      $(find ctu_cras_norlab_spot_sensor_config_1)/urdf/imu.xacro :
-      $(find ctu_cras_norlab_spot_sensor_config_1)/urdf/mote_deployer.xacro :
-      $(find ctu_cras_norlab_spot_sensor_config_1)/urdf/ouster_lidar.xacro :
+      $(find marble_spot_sensor_config_2)/urdf/basler_cameras.xacro :
+      $(find marble_spot_sensor_config_2)/urdf/imu.xacro :
+      $(find marble_spot_sensor_config_2)/urdf/mote_deployer.xacro :
+      $(find marble_spot_sensor_config_2)/urdf/ouster_lidar.xacro :
       $(find marble_spot_sensor_config_2)/urdf/ouster_lidar_alt.xacro :
       $(find marble_spot_sensor_config_2)/urdf/flir_cameras.xacro :
@@ -46,5 +46,5 @@
             <origin rpy="1.5708 0 1.5708" xyz="0.325 0 0.005"/>
             <geometry>
-                <mesh filename="package://ctu_cras_norlab_spot_sensor_config_1/meshes/spot_sensor_rig_assembly.dae" />
+                <mesh filename="package://marble_spot_sensor_config_2/meshes/spot_sensor_rig_assembly.dae" />
             </geometry>
         </visual>
@@ -135,5 +135,5 @@
     </xacro:if>
     <!-- LIGHTS -->
-    <xacro:include filename="$(find ctu_cras_norlab_spot_sensor_config_1)/urdf/lights.xacro" />
+    <xacro:include filename="$(find marble_spot_sensor_config_2)/urdf/lights.xacro" />
     <gazebo reference="$(arg prefix)payload">
         <xacro:led_stripe name="light_left" range="20" linear="0.2" constant="0.1" quadratic="0.0025"
