Commit message: Addressed review comments

File: submitted_models/coro_jeanine_sensor_config_1/urdf/model.xacro (robot description, xacro)
@@ -217,5 +217,5 @@
     </camera>
   </sensor>
-  <sensor name='camera_front' update_rate='30'>
+  <sensor name='camera_front' update_rate='25'>
     <parent link='${robot_namespace}/base_link'/>
     <origin xyz='0.11 0.06 0.42' rpy='0 -0 0'/>
@@ -224,5 +224,5 @@
     </camera>
   </sensor>
-  <sensor name='camera_rear' update_rate='30'>
+  <sensor name='camera_rear' update_rate='25'>
     <parent link='${robot_namespace}/base_link'/>
     <origin xyz='-0.11 0 0.42' rpy='0 -0 3.14159'/>
@@ -231,5 +231,5 @@
     </camera>
   </sensor>
-  <sensor name='camera_left' update_rate='30'>
+  <sensor name='camera_left' update_rate='25'>
     <parent link='${robot_namespace}/base_link'/>
     <origin xyz='0 0.11 0.42' rpy='0 -0 1.5708'/>
@@ -238,5 +238,5 @@
     </camera>
   </sensor>
-  <sensor name='camera_right' update_rate='30'>
+  <sensor name='camera_right' update_rate='25'>
     <parent link='${robot_namespace}/base_link'/>
     <origin xyz='0 -0.11 0.42' rpy='0 0 -1.5708'/>
@@ -264,5 +264,5 @@
       <origin xyz='0 0 0' rpy='1.5708 -0 0'/>
       <geometry>
-        <mesh filename='package://coro_jeanine_sensor_config_1/meshes/wheel_left.dae' scale='1.41 1.41 1.71'/>
+        <mesh filename='package://coro_jeanine_sensor_config_1/meshes/wheel_left.dae' scale='1.22 1.22 1.71'/>
       </geometry>
     </visual>
@@ -283,5 +283,5 @@
       <origin xyz='0 0 0' rpy='1.5708 -0 0'/>
       <geometry>
-        <cylinder radius='0.145' length='0.075'/>
+        <cylinder radius='0.1275' length='0.075'/>
       </geometry>
     </collision>
@@ -289,5 +289,5 @@
       <origin xyz='0 0 0' rpy='1.5708 -0 0'/>
       <geometry>
-        <mesh filename='package://coro_jeanine_sensor_config_1/meshes/wheel_right.dae' scale='1.41 1.41 1.71'/>
+        <mesh filename='package://coro_jeanine_sensor_config_1/meshes/wheel_right.dae' scale='1.22 1.22 1.71'/>
       </geometry>
     </visual>
@@ -308,5 +308,5 @@
       <origin xyz='0 0 0' rpy='-1.5708 0 0'/>
       <geometry>
-        <cylinder radius='0.145' length='0.075'/>
+        <cylinder radius='0.1275' length='0.075'/>
       </geometry>
     </collision>
@@ -314,5 +314,5 @@
       <origin xyz='0 0 0' rpy='1.5708 -0 0'/>
       <geometry>
-        <mesh filename='package://coro_jeanine_sensor_config_1/meshes/wheel_left.dae' scale='1.41 1.41 1.71'/>
+        <mesh filename='package://coro_jeanine_sensor_config_1/meshes/wheel_left.dae' scale='1.22 1.22 1.71'/>
       </geometry>
     </visual>
@@ -333,5 +333,5 @@
       <origin xyz='0 0 0' rpy='1.5708 -0 0'/>
       <geometry>
-        <cylinder radius='0.145' length='0.075'/>
+        <cylinder radius='0.1275' length='0.075'/>
       </geometry>
     </collision>
@@ -339,5 +339,5 @@
       <origin xyz='0 0 0' rpy='1.5708 -0 0'/>
       <geometry>
-        <mesh filename='package://coro_jeanine_sensor_config_1/meshes/wheel_right.dae' scale='1.41 1.41 1.71'/>
+        <mesh filename='package://coro_jeanine_sensor_config_1/meshes/wheel_right.dae' scale='1.22 1.22 1.71'/>
       </geometry>
     </visual>
