Commit message: updated lights

File: submitted_models/marble_husky_sensor_config_6/urdf/robot_from_sdf.xacro (robot description, xacro)
@@ -27,10 +27,4 @@
       </geometry>
     </collision>
-    <collision name='base_link_fixed_joint_lump__camera/camera_link_collision_1'>
-      <origin xyz='0 0 0.05' rpy='0 -0 0'/>
-      <geometry>
-        <box size='0.0078 0.13 0.0192'/>
-      </geometry>
-    </collision>
     <collision name='base_link_fixed_joint_lump__camera/camera_link_collision_2'>
       <origin xyz='0.478 0 0.285' rpy='0 -0 0'/>
@@ -51,10 +45,4 @@
       </geometry>
     </collision>
-    <collision name='base_link_fixed_joint_lump__velodyne_gimbal_plate_base_link_collision_7'>
-      <origin xyz='0.424 0 0.4' rpy='0 -0 0'/>
-      <geometry>
-        <box size='0.1 0.1 0.01'/>
-      </geometry>
-    </collision>
     <collision name='base_link_fixed_joint_lump__sensor_tower_8'>
       <origin xyz='0.374 0 0.215' rpy='0 -0 0'/>
@@ -69,20 +57,68 @@
       </geometry>
     </collision>
+    <collision name='tof_left_camera_mount_collision'>
+      <origin xyz='0.5105 0.01 0.439' rpy='-1.34452 0.47634 0.465309'/>
+      <geometry>
+        <box size='0.04 0.135 0.0385'/>
+      </geometry>
+    </collision>
+    <collision name='tof_right_camera_mount_collision'>
+      <origin xyz='0.5105 -0.01 0.439' rpy='-1.79707 0.47634 -0.465309'/>
+      <geometry>
+        <box size='0.04 0.135 0.0385'/>
+      </geometry>
+    </collision>
+    <collision name='sensor_head_collision'>
+      <origin xyz='0.4379 0 0.54818' rpy='0 -0 0'/>
+      <geometry>
+        <box size='0.1 0.1 0.125'/>
+      </geometry>
+    </collision>
+    <collision name='sensor_tower_support_collision'>
+      <origin xyz='0.4379 0 0.39918' rpy='0 -0 0'/>
+      <geometry>
+        <box size='0.04 0.04 0.25'/>
+      </geometry>
+    </collision>
+    <collision name='vertical_lidar_support_collision'>
+      <origin xyz='0.4029 0 0.44418' rpy='0 -0 0'/>
+      <geometry>
+        <box size='0.2 0.04 0.04'/>
+      </geometry>
+    </collision>
+    <collision name='diagonal_lidar_support_collision'>
+      <origin xyz='0.3779 0 0.36418' rpy='0 0.8854 0'/>
+      <geometry>
+        <box size='0.18 0.04 0.04'/>
+      </geometry>
+    </collision>
+    <collision name='camera_front_collision'>
+      <origin xyz='0.5179 0 0.53718' rpy='3.14159 1.57069 3.14159'/>
+      <geometry>
+        <cylinder radius='0.03' length='0.065'/>
+      </geometry>
+    </collision>
+    <collision name='camera_back_collision'>
+      <origin xyz='0.3579 0 0.53718' rpy='3.14159 1.57069 3.14159'/>
+      <geometry>
+        <cylinder radius='0.03' length='0.065'/>
+      </geometry>
+    </collision>
+    <collision name='camera_left_collision'>
+      <origin xyz='0.4379 0.08 0.53718' rpy='1.5709 -0 0'/>
+      <geometry>
+        <cylinder radius='0.03' length='0.065'/>
+      </geometry>
+    </collision>
+    <collision name='camera_right_collision'>
+      <origin xyz='0.4379 -0.08 0.53718' rpy='1.5709 -0 0'/>
+      <geometry>
+        <cylinder radius='0.03' length='0.065'/>
+      </geometry>
+    </collision>
     <visual name='base_link_visual'>
       <origin xyz='0 0 0' rpy='0 -0 0'/>
       <geometry>
-        <mesh filename='package://marble_husky_sensor_config_6/meshes/base_link.dae' scale='1 1 1'/>
-      </geometry>
-    </visual>
-    <visual name='base_link_fixed_joint_lump__camera/camera_link_visual_1'>
-      <origin xyz='0.478 0 0.26' rpy='0 0.5236 0'/>
-      <geometry>
-        <mesh filename='package://marble_husky_sensor_config_6/meshes/realsense.dae' scale='1 1 1'/>
-      </geometry>
-    </visual>
-    <visual name='base_link_fixed_joint_lump__camera/camera_link_visual_2'>
-      <origin xyz='0.478 0 0.285' rpy='0 -0 0'/>
-      <geometry>
-        <mesh filename='package://marble_husky_sensor_config_6/meshes/realsense.dae' scale='1 1 1'/>
+        <mesh filename='meshes/base_link.dae' scale='1 1 1'/>
       </geometry>
     </visual>
@@ -90,5 +126,5 @@
       <origin xyz='0.48 0 0.091' rpy='0 -0 0'/>
       <geometry>
-        <mesh filename='package://marble_husky_sensor_config_6/meshes/bumper.dae' scale='1 1 1'/>
+        <mesh filename='meshes/bumper.dae' scale='1 1 1'/>
       </geometry>
     </visual>
@@ -96,5 +132,5 @@
       <origin xyz='-0.48 0 0.091' rpy='0 -0 3.14159'/>
       <geometry>
-        <mesh filename='package://marble_husky_sensor_config_6/meshes/bumper.dae' scale='1 1 1'/>
+        <mesh filename='meshes/bumper.dae' scale='1 1 1'/>
       </geometry>
     </visual>
@@ -102,23 +138,5 @@
       <origin xyz='0 0 0' rpy='0 -0 0'/>
       <geometry>
-        <mesh filename='package://marble_husky_sensor_config_6/meshes/top_chassis.dae' scale='1 1 1'/>
-      </geometry>
-    </visual>
-    <visual name='base_link_fixed_joint_lump__velodyne_base_link_visual_10'>
-      <origin xyz='0.424 0 0.327' rpy='0 -0 0'/>
-      <geometry>
-        <mesh filename='package://marble_husky_sensor_config_6/meshes/VLP16_base_1.dae' scale='1 1 1'/>
-      </geometry>
-    </visual>
-    <visual name='base_link_fixed_joint_lump__velodyne_base_link_visual_11'>
-      <origin xyz='0.424 0 0.327' rpy='0 -0 0'/>
-      <geometry>
-        <mesh filename='package://marble_husky_sensor_config_6/meshes/VLP16_base_2.dae' scale='1 1 1'/>
-      </geometry>
-    </visual>
-    <visual name='base_link_fixed_joint_lump__velodyne_visual_12'>
-      <origin xyz='0.424 0 0.327' rpy='0 -0 0'/>
-      <geometry>
-        <mesh filename='package://marble_husky_sensor_config_6/meshes/VLP16_scan.dae' scale='1 1 1'/>
+        <mesh filename='meshes/top_chassis.dae' scale='1 1 1'/>
       </geometry>
     </visual>
@@ -126,5 +144,5 @@
       <origin xyz='0.272 0 0.245' rpy='0 -0 0'/>
       <geometry>
-        <mesh filename='package://marble_husky_sensor_config_6/meshes/user_rail.dae' scale='1 1 1'/>
+        <mesh filename='meshes/user_rail.dae' scale='1 1 1'/>
       </geometry>
     </visual>
@@ -135,10 +153,4 @@
       </geometry>
     </visual>
-    <visual name='base_link_fixed_joint_lump__velodyne_gimbal_plate_15'>
-      <origin xyz='0.424 0 0.4' rpy='0 -0 0'/>
-      <geometry>
-        <box size='0.06 0.06 0.01'/>
-      </geometry>
-    </visual>
     <visual name='base_link_fixed_joint_lump__sensor_tower_16'>
       <origin xyz='0.374 0 0.215' rpy='0 -0 0'/>
@@ -153,30 +165,170 @@
       </geometry>
     </visual>
+    <visual name='tof_left_camera_visual'>
+      <origin xyz='0.527 0.015 0.429' rpy='-1.34452 0.47634 0.465309'/>
+      <geometry>
+        <mesh filename='meshes/realsense.dae' scale='1 1 1'/>
+      </geometry>
+    </visual>
+    <visual name='tof_left_camera_mount_visual'>
+      <origin xyz='0.5105 0.01 0.439' rpy='-1.34452 0.47634 0.465309'/>
+      <geometry>
+        <box size='0.04 0.135 0.0385'/>
+      </geometry>
+    </visual>
+    <visual name='tof_right_camera_visual'>
+      <origin xyz='0.527 -0.015 0.429' rpy='-1.79707 0.47634 -0.465309'/>
+      <geometry>
+        <mesh filename='meshes/realsense.dae' scale='1 1 1'/>
+      </geometry>
+    </visual>
+    <visual name='tof_right_camera_mount_visual'>
+      <origin xyz='0.5105 -0.01 0.439' rpy='-1.79707 0.47634 -0.465309'/>
+      <geometry>
+        <box size='0.04 0.135 0.0385'/>
+      </geometry>
+    </visual>
+    <visual name='sensor_head_visual'>
+      <origin xyz='0.4379 0 0.54818' rpy='0 -0 0'/>
+      <geometry>
+        <box size='0.1 0.1 0.125'/>
+      </geometry>
+    </visual>
+    <visual name='sensor_tower_support_visual'>
+      <origin xyz='0.4379 0 0.39918' rpy='0 -0 0'/>
+      <geometry>
+        <box size='0.04 0.04 0.25'/>
+      </geometry>
+    </visual>
+    <visual name='vertical_lidar_support_visual'>
+      <origin xyz='0.4029 0 0.44418' rpy='0 -0 0'/>
+      <geometry>
+        <box size='0.2 0.04 0.04'/>
+      </geometry>
+    </visual>
+    <visual name='diagonal_lidar_support_visual'>
+      <origin xyz='0.3779 0 0.36418' rpy='0 0.8854 0'/>
+      <geometry>
+        <box size='0.18 0.04 0.04'/>
+      </geometry>
+    </visual>
+    <visual name='base_link_fixed_joint_lump__velodyne_base_link_visual_10'>
+      <origin xyz='0.4379 0 0.61018' rpy='0 -0 0'/>
+      <geometry>
+        <mesh filename='meshes/VLP16_base_1.dae' scale='1 1 1'/>
+      </geometry>
+    </visual>
+    <visual name='base_link_fixed_joint_lump__velodyne_base_link_visual_11'>
+      <origin xyz='0.4379 0 0.61018' rpy='0 -0 0'/>
+      <geometry>
+        <mesh filename='meshes/VLP16_base_2.dae' scale='1 1 1'/>
+      </geometry>
+    </visual>
+    <visual name='base_link_fixed_joint_lump__velodyne_visual_12'>
+      <origin xyz='0.4379 0 0.61018' rpy='0 -0 0'/>
+      <geometry>
+        <mesh filename='meshes/VLP16_scan.dae' scale='1 1 1'/>
+      </geometry>
+    </visual>
+    <visual name='base_link_fixed_joint_lump__velodyne_base_link_visual_13'>
+      <origin xyz='0.31037 0 0.44818' rpy='3.14159 -1.57079 3.14159'/>
+      <geometry>
+        <mesh filename='meshes/VLP16_base_1.dae' scale='1 1 1'/>
+      </geometry>
+    </visual>
+    <visual name='base_link_fixed_joint_lump__velodyne_base_link_visual_14'>
+      <origin xyz='0.31037 0 0.44818' rpy='3.14159 -1.57079 3.14159'/>
+      <geometry>
+        <mesh filename='meshes/VLP16_base_2.dae' scale='1 1 1'/>
+      </geometry>
+    </visual>
+    <visual name='base_link_fixed_joint_lump__velodyne_visual_15'>
+      <origin xyz='0.31037 0 0.44818' rpy='3.14159 -1.57079 3.14159'/>
+      <geometry>
+        <mesh filename='meshes/VLP16_scan.dae' scale='1 1 1'/>
+      </geometry>
+    </visual>
+    <visual name='camera_front_visual'>
+      <origin xyz='0.5179 0 0.53718' rpy='3.14159 1.57069 3.14159'/>
+      <geometry>
+        <cylinder radius='0.03' length='0.065'/>
+      </geometry>
+    </visual>
+    <visual name='camera_back_visual'>
+      <origin xyz='0.3579 0 0.53718' rpy='3.14159 1.57069 3.14159'/>
+      <geometry>
+        <cylinder radius='0.03' length='0.065'/>
+      </geometry>
+    </visual>
+    <visual name='camera_left_visual'>
+      <origin xyz='0.4379 0.08 0.53718' rpy='1.5709 -0 0'/>
+      <geometry>
+        <cylinder radius='0.03' length='0.065'/>
+      </geometry>
+    </visual>
+    <visual name='camera_right_visual'>
+      <origin xyz='0.4379 -0.08 0.53718' rpy='1.5709 -0 0'/>
+      <geometry>
+        <cylinder radius='0.03' length='0.065'/>
+      </geometry>
+    </visual>
   </link>
-  <sensor name='camera_front' update_rate='30'>
-    <parent link='${robot_namespace}/imu_link'/>
-    <origin xyz='0.468 0 0.36' rpy='0 -0 0'/>
-    <camera>
-      <image width='640' height='480' format='R8G8B8' hfov='1.5184' near='0.01' far='300' />
-    </camera>
-  </sensor>
-  <sensor name='camera_back' update_rate='30'>
-    <parent link='${robot_namespace}/base_link'/>
-    <origin xyz='0.468 0 0.36' rpy='0 -0 0'/>
-    <camera>
-      <image width='640' height='480' format='R8G8B8' hfov='1.5184' near='0.01' far='300' />
-    </camera>
-  </sensor>
-  <sensor name='planar_laser' update_rate='10'>
-    <parent link='${robot_namespace}/base_link'/>
-    <origin xyz='0.474 0 0.127' rpy='0 -0 0'/>
-  </sensor>
-  <sensor name='front_laser' update_rate='20'>
-    <parent link='${robot_namespace}/base_link'/>
-    <origin xyz='0.424 0 0.387' rpy='0 -0 0'/>
-  </sensor>
-  <sensor name='imu_sensor' update_rate='250'>
-    <parent link='${robot_namespace}/base_link'/>
-    <origin xyz='0.4379 0 0.52418' rpy='0 -0 0'/>
+  <sensor name='planar_laser' update_rate='20'>
+    <parent link='${robot_namespace}/base_link'/>
+    <origin xyz='0.485 0 0.166' rpy='0 -0 0'/>
+  </sensor>
+  <sensor name='tof_left' update_rate='10'>
+    <parent link='${robot_namespace}/base_link'/>
+    <origin xyz='0.527 0.015 0.429' rpy='-1.34452 0.47634 0.465309'/>
+    <camera>
+      <image width='224' height='171' format='R8G8B8' hfov='1.0821' near='0.1' far='4' />
+    </camera>
+  </sensor>
+  <sensor name='tof_right' update_rate='10'>
+    <parent link='${robot_namespace}/base_link'/>
+    <origin xyz='0.527 -0.015 0.429' rpy='-1.79707 0.47634 -0.465309'/>
+    <camera>
+      <image width='224' height='171' format='R8G8B8' hfov='1.0821' near='0.1' far='4' />
+    </camera>
+  </sensor>
+  <sensor name='imu_sensor' update_rate='200'>
+    <parent link='${robot_namespace}/base_link'/>
+    <origin xyz='0 0 0' rpy='0 -0 0'/>
+  </sensor>
+  <sensor name='front_laser' update_rate='10'>
+    <parent link='${robot_namespace}/base_link'/>
+    <origin xyz='0.4379 0 0.67018' rpy='0 -0 0'/>
+  </sensor>
+  <sensor name='vert_laser' update_rate='10'>
+    <parent link='${robot_namespace}/base_link'/>
+    <origin xyz='0.31037 0 0.44818' rpy='3.14159 -1.57079 3.14159'/>
+  </sensor>
+  <sensor name='camera_front' update_rate='10'>
+    <parent link='${robot_namespace}/base_link'/>
+    <origin xyz='0.5579 0 0.53718' rpy='0 -0 0'/>
+    <camera>
+      <image width='808' height='608' format='R8G8B8' hfov='1.39626' near='0.01' far='300' />
+    </camera>
+  </sensor>
+  <sensor name='camera_back' update_rate='10'>
+    <parent link='${robot_namespace}/base_link'/>
+    <origin xyz='0.3179 0 0.53718' rpy='0 -0 3.14159'/>
+    <camera>
+      <image width='808' height='608' format='R8G8B8' hfov='1.39626' near='0.01' far='300' />
+    </camera>
+  </sensor>
+  <sensor name='camera_left' update_rate='10'>
+    <parent link='${robot_namespace}/base_link'/>
+    <origin xyz='0.4379 0.12 0.53718' rpy='0 -0 1.5708'/>
+    <camera>
+      <image width='808' height='608' format='R8G8B8' hfov='1.39626' near='0.01' far='300' />
+    </camera>
+  </sensor>
+  <sensor name='camera_right' update_rate='10'>
+    <parent link='${robot_namespace}/base_link'/>
+    <origin xyz='0.4379 -0.12 0.53718' rpy='0 0 -1.5708'/>
+    <camera>
+      <image width='808' height='608' format='R8G8B8' hfov='1.39626' near='0.01' far='300' />
+    </camera>
   </sensor>
   <link name='${robot_namespace}/front_left_wheel_link'>
@@ -195,5 +347,5 @@
       <origin xyz='0 0 0' rpy='0 -0 0'/>
       <geometry>
-        <mesh filename='package://marble_husky_sensor_config_6/meshes/wheel.dae' scale='1 1 1'/>
+        <mesh filename='meshes/wheel.dae' scale='1 1 1'/>
       </geometry>
     </visual>
@@ -214,5 +366,5 @@
       <origin xyz='0 0 0' rpy='0 -0 0'/>
       <geometry>
-        <mesh filename='package://marble_husky_sensor_config_6/meshes/wheel.dae' scale='1 1 1'/>
+        <mesh filename='meshes/wheel.dae' scale='1 1 1'/>
       </geometry>
     </visual>
@@ -233,5 +385,5 @@
       <origin xyz='0 0 0' rpy='0 -0 0'/>
       <geometry>
-        <mesh filename='package://marble_husky_sensor_config_6/meshes/wheel.dae' scale='1 1 1'/>
+        <mesh filename='meshes/wheel.dae' scale='1 1 1'/>
       </geometry>
     </visual>
@@ -252,77 +404,8 @@
       <origin xyz='0 0 0' rpy='0 -0 0'/>
       <geometry>
-        <mesh filename='package://marble_husky_sensor_config_6/meshes/wheel.dae' scale='1 1 1'/>
+        <mesh filename='meshes/wheel.dae' scale='1 1 1'/>
       </geometry>
     </visual>
   </link>
-  <link name='${robot_namespace}/pan_gimbal_link'>
-    <inertial>
-      <origin xyz='0 0 0' rpy='0 -0 0'/>
-      <mass value='0.1'/>
-      <inertia ixx='1' ixy='0' ixz='0' iyy='1' iyz='0' izz='1'/>
-    </inertial>
-    <collision name='pan_gimbal_link_collision'>
-      <origin xyz='0 0 0' rpy='0 -0 0'/>
-      <geometry>
-        <cylinder radius='0.014' length='0.045'/>
-      </geometry>
-    </collision>
-    <visual name='pan_gimbal_link_visual'>
-      <origin xyz='0 0 0' rpy='0 -0 0'/>
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
Commit message: rviz model description now visual properly. Weight updated properly in specifications.md

File: submitted_models/marble_husky_sensor_config_6/urdf/robot_from_sdf.xacro (robot description, xacro)
@@ -120,5 +120,5 @@
       <origin xyz='0 0 0' rpy='0 -0 0'/>
       <geometry>
-        <mesh filename='meshes/base_link.dae' scale='1 1 1'/>
+        <mesh filename='package://marble_husky_sensor_config_6/meshes/base_link.dae' scale='1 1 1'/>
       </geometry>
     </visual>
@@ -126,5 +126,5 @@
       <origin xyz='0.48 0 0.091' rpy='0 -0 0'/>
       <geometry>
-        <mesh filename='meshes/bumper.dae' scale='1 1 1'/>
+        <mesh filename='package://marble_husky_sensor_config_6/meshes/bumper.dae' scale='1 1 1'/>
       </geometry>
     </visual>
@@ -132,5 +132,5 @@
       <origin xyz='-0.48 0 0.091' rpy='0 -0 3.14159'/>
       <geometry>
-        <mesh filename='meshes/bumper.dae' scale='1 1 1'/>
+        <mesh filename='package://marble_husky_sensor_config_6/meshes/bumper.dae' scale='1 1 1'/>
       </geometry>
     </visual>
@@ -138,5 +138,5 @@
       <origin xyz='0 0 0' rpy='0 -0 0'/>
       <geometry>
-        <mesh filename='meshes/top_chassis.dae' scale='1 1 1'/>
+        <mesh filename='package://marble_husky_sensor_config_6/meshes/top_chassis.dae' scale='1 1 1'/>
       </geometry>
     </visual>
@@ -144,5 +144,5 @@
       <origin xyz='0.272 0 0.245' rpy='0 -0 0'/>
       <geometry>
-        <mesh filename='meshes/user_rail.dae' scale='1 1 1'/>
+        <mesh filename='package://marble_husky_sensor_config_6/meshes/user_rail.dae' scale='1 1 1'/>
       </geometry>
     </visual>
@@ -168,5 +168,5 @@
       <origin xyz='0.527 0.015 0.429' rpy='-1.34452 0.47634 0.465309'/>
       <geometry>
-        <mesh filename='meshes/realsense.dae' scale='1 1 1'/>
+        <mesh filename='package://marble_husky_sensor_config_6/meshes/realsense.dae' scale='1 1 1'/>
       </geometry>
     </visual>
@@ -180,5 +180,5 @@
       <origin xyz='0.527 -0.015 0.429' rpy='-1.79707 0.47634 -0.465309'/>
       <geometry>
-        <mesh filename='meshes/realsense.dae' scale='1 1 1'/>
+        <mesh filename='package://marble_husky_sensor_config_6/meshes/realsense.dae' scale='1 1 1'/>
       </geometry>
     </visual>
@@ -216,5 +216,5 @@
       <origin xyz='0.4379 0 0.61018' rpy='0 -0 0'/>
       <geometry>
-        <mesh filename='meshes/VLP16_base_1.dae' scale='1 1 1'/>
+        <mesh filename='package://marble_husky_sensor_config_6/meshes/VLP16_base_1.dae' scale='1 1 1'/>
       </geometry>
     </visual>
@@ -222,5 +222,5 @@
       <origin xyz='0.4379 0 0.61018' rpy='0 -0 0'/>
       <geometry>
-        <mesh filename='meshes/VLP16_base_2.dae' scale='1 1 1'/>
+        <mesh filename='package://marble_husky_sensor_config_6/meshes/VLP16_base_2.dae' scale='1 1 1'/>
       </geometry>
     </visual>
@@ -228,5 +228,5 @@
       <origin xyz='0.4379 0 0.61018' rpy='0 -0 0'/>
       <geometry>
-        <mesh filename='meshes/VLP16_scan.dae' scale='1 1 1'/>
+        <mesh filename='package://marble_husky_sensor_config_6/meshes/VLP16_scan.dae' scale='1 1 1'/>
       </geometry>
     </visual>
@@ -234,5 +234,5 @@
       <origin xyz='0.31037 0 0.44818' rpy='3.14159 -1.57079 3.14159'/>
       <geometry>
-        <mesh filename='meshes/VLP16_base_1.dae' scale='1 1 1'/>
+        <mesh filename='package://marble_husky_sensor_config_6/meshes/VLP16_base_1.dae' scale='1 1 1'/>
       </geometry>
     </visual>
@@ -240,5 +240,5 @@
       <origin xyz='0.31037 0 0.44818' rpy='3.14159 -1.57079 3.14159'/>
       <geometry>
-        <mesh filename='meshes/VLP16_base_2.dae' scale='1 1 1'/>
+        <mesh filename='package://marble_husky_sensor_config_6/meshes/VLP16_base_2.dae' scale='1 1 1'/>
       </geometry>
     </visual>
@@ -246,5 +246,5 @@
       <origin xyz='0.31037 0 0.44818' rpy='3.14159 -1.57079 3.14159'/>
       <geometry>
-        <mesh filename='meshes/VLP16_scan.dae' scale='1 1 1'/>
+        <mesh filename='package://marble_husky_sensor_config_6/meshes/VLP16_scan.dae' scale='1 1 1'/>
       </geometry>
     </visual>
@@ -347,5 +347,5 @@
       <origin xyz='0 0 0' rpy='0 -0 0'/>
       <geometry>
-        <mesh filename='meshes/wheel.dae' scale='1 1 1'/>
+        <mesh filename='package://marble_husky_sensor_config_6/meshes/wheel.dae' scale='1 1 1'/>
       </geometry>
     </visual>
@@ -366,5 +366,5 @@
       <origin xyz='0 0 0' rpy='0 -0 0'/>
       <geometry>
-        <mesh filename='meshes/wheel.dae' scale='1 1 1'/>
+        <mesh filename='package://marble_husky_sensor_config_6/meshes/wheel.dae' scale='1 1 1'/>
       </geometry>
     </visual>
@@ -385,5 +385,5 @@
       <origin xyz='0 0 0' rpy='0 -0 0'/>
       <geometry>
-        <mesh filename='meshes/wheel.dae' scale='1 1 1'/>
+        <mesh filename='package://marble_husky_sensor_config_6/meshes/wheel.dae' scale='1 1 1'/>
       </geometry>
     </visual>
@@ -404,5 +404,5 @@
       <origin xyz='0 0 0' rpy='0 -0 0'/>
       <geometry>
-        <mesh filename='meshes/wheel.dae' scale='1 1 1'/>
+        <mesh filename='package://marble_husky_sensor_config_6/meshes/wheel.dae' scale='1 1 1'/>
       </geometry>
     </visual>
