Commit message: Updated RViz visualization for kloubak sc 3.

File: submitted_models/robotika_kloubak_sensor_config_3/urdf/model.xacro (robot description, xacro)
@@ -58,19 +58,19 @@
     </collision>
     <visual name='visual_chassis'>
-      <origin xyz='-0.34 0 0.03' rpy='0 -0 0'/>
-      <geometry>
-        <mesh filename='meshes/k2.dae' scale='1 1 1'/>
+      <origin xyz='-0.33 0 -0.19' rpy='0 -0 0'/>
+      <geometry>
+        <mesh filename='package://robotika_kloubak_sensor_config_3/meshes/k2.dae' scale='1 1 1'/>
       </geometry>
     </visual>
     <visual name='rs_holder_front'>
-      <origin xyz='0.06 0.015 0.5185' rpy='0 -0 0'/>
-      <geometry>
-        <mesh filename='meshes/rs_holder.dae' scale='1 1 1'/>
+      <origin xyz='0.06 0.015 0.2985' rpy='0 -0 0'/>
+      <geometry>
+        <mesh filename='package://robotika_kloubak_sensor_config_3/meshes/rs_holder.dae' scale='1 1 1'/>
       </geometry>
     </visual>
     <visual name='visual_depth_camera_front_slope'>
-      <origin xyz='0.163 0.012 0.544' rpy='1.91986 0 1.56329'/>
-      <geometry>
-        <mesh filename='meshes/realsense_d435.dae' scale='1 1 1'/>
+      <origin xyz='0.163 0.012 0.324' rpy='1.91986 0 1.56329'/>
+      <geometry>
+        <mesh filename='package://robotika_kloubak_sensor_config_3/meshes/realsense_d435.dae' scale='1 1 1'/>
       </geometry>
     </visual>
@@ -143,20 +143,14 @@
       </geometry>
     </collision>
-    <visual name='visual_chassis'>
-      <origin xyz='-0.01 0 -0.19' rpy='0 -0 0'/>
-      <geometry>
-        <mesh filename='meshes/k2.dae' scale='1 1 1'/>
-      </geometry>
-    </visual>
     <visual name='rs_holder_back'>
-      <origin xyz='-0.44 -0.023 0.375' rpy='0 -0 -3.14159'/>
-      <geometry>
-        <mesh filename='meshes/rs_holder.dae' scale='1 1 1'/>
+      <origin xyz='-0.105 -0.023 0.377' rpy='0 -0 -3.14159'/>
+      <geometry>
+        <mesh filename='package://robotika_kloubak_sensor_config_3/meshes/rs_holder.dae' scale='1 1 1'/>
       </geometry>
     </visual>
     <visual name='visual_depth_camera_back_slope'>
-      <origin xyz='-0.543 0.015 0.401' rpy='-1.91986 -0 1.56329'/>
-      <geometry>
-        <mesh filename='meshes/realsense_d435.dae' scale='1 1 1'/>
+      <origin xyz='-0.208 0.015 0.403' rpy='-1.91986 -0 1.56329'/>
+      <geometry>
+        <mesh filename='package://robotika_kloubak_sensor_config_3/meshes/realsense_d435.dae' scale='1 1 1'/>
       </geometry>
     </visual>
@@ -207,10 +201,4 @@
       </geometry>
     </collision>
-    <visual name='visual'>
-      <origin xyz='-0.0132 0 0' rpy='0 -0 0'/>
-      <geometry>
-        <mesh filename='meshes/k2.dae' scale='1 1 1'/>
-      </geometry>
-    </visual>
   </link>
   <link name='${robot_namespace}/front_left_wheel'>
@@ -226,10 +214,4 @@
       </geometry>
     </collision>
-    <visual name='tire_visual'>
-      <origin xyz='0 0 0' rpy='0 -0 0'/>
-      <geometry>
-        <mesh filename='meshes/k2.dae' scale='1 1 1'/>
-      </geometry>
-    </visual>
   </link>
   <link name='${robot_namespace}/front_right_wheel'>
@@ -245,10 +227,4 @@
       </geometry>
     </collision>
-    <visual name='tire_visual'>
-      <origin xyz='0 0 0' rpy='0 -0 0'/>
-      <geometry>
-        <mesh filename='meshes/k2.dae' scale='1 1 1'/>
-      </geometry>
-    </visual>
   </link>
   <link name='${robot_namespace}/rear_left_wheel'>
@@ -264,10 +240,4 @@
       </geometry>
     </collision>
-    <visual name='tire_visual'>
-      <origin xyz='0 0 0' rpy='0 -0 0'/>
-      <geometry>
-        <mesh filename='meshes/k2.dae' scale='1 1 1'/>
-      </geometry>
-    </visual>
   </link>
   <link name='${robot_namespace}/rear_right_wheel'>
@@ -283,10 +253,4 @@
       </geometry>
     </collision>
-    <visual name='tire_visual'>
-      <origin xyz='0 0 0' rpy='0 -0 0'/>
-      <geometry>
-        <mesh filename='meshes/k2.dae' scale='1 1 1'/>
-      </geometry>
-    </visual>
   </link>
   <joint name='front_left_wheel_joint' type='revolute'>
