Commit message: Rename marble huksy 6 to 5
Signed-off-by: Nate Koenig <nate@openrobotics.org>

File: submitted_models/marble_husky_sensor_config_5/urdf/husky_custom.orig.urdf (robot description, URDF)
Before this commit: robot marble_husky_sensor_config_6, 5 links, 4 joints
Links:
- removed link ${robot_namespace}/base_link
- removed link ${robot_namespace}/front_left_wheel_link
- removed link ${robot_namespace}/front_right_wheel_link
- removed link ${robot_namespace}/rear_left_wheel_link
- removed link ${robot_namespace}/rear_right_wheel_link
- added link base_link, mass 46.064; collision box size=0.0078 0.13 0.0192; collision box size=0.0078 0.13 0.0192
- added link front_left_wheel_link, mass 2.637; collision cylinder length=0.1143 radius=0.1651; visual mesh filename=meshes/wheel.dae scale=1 1 1
- added link front_right_wheel_link, mass 2.637; collision cylinder length=0.1143 radius=0.1651; visual mesh filename=meshes/wheel.dae scale=1 1 1
- added link rear_left_wheel_link, mass 2.637; collision cylinder length=0.1143 radius=0.1651; visual mesh filename=meshes/wheel.dae scale=1 1 1
- added link rear_right_wheel_link, mass 2.637; collision cylinder length=0.1143 radius=0.1651; visual mesh filename=meshes/wheel.dae scale=1 1 1
Joints:
- joint front_left_wheel_joint: child ${robot_namespace}/front_left_wheel_link -> front_left_wheel_link; parent ${robot_namespace}/base_link -> base_link
- joint front_right_wheel_joint: child ${robot_namespace}/front_right_wheel_link -> front_right_wheel_link; parent ${robot_namespace}/base_link -> base_link
- joint rear_left_wheel_joint: child ${robot_namespace}/rear_left_wheel_link -> rear_left_wheel_link; parent ${robot_namespace}/base_link -> base_link
- joint rear_right_wheel_joint: child ${robot_namespace}/rear_right_wheel_link -> rear_right_wheel_link; parent ${robot_namespace}/base_link -> base_link

File: submitted_models/marble_husky_sensor_config_5/urdf/robot_from_sdf.xacro (robot description, xacro)
@@ -1,5 +1,7 @@
 <?xml version='1.0' encoding='utf-8'?>
-<robot name='marble_husky_sensor_config_6'>
-  <link name='base_link'>
+<robot name='marble_husky_sensor_config_5' xmlns:xacro='http://ros.org/wiki/xacro'>
+  <xacro:arg name="name" default="marble_husky_sensor_config_5"/>
+  <xacro:property name="robot_namespace" value="$(arg name)"/>
+  <link name='${robot_namespace}/base_link'>
     <inertial>
       <origin xyz='-0.000543 -0.084945 0.062329' rpy='0 -0 0'/>
@@ -118,5 +120,5 @@
       <origin xyz='0 0 0' rpy='0 -0 0'/>
       <geometry>
-        <mesh filename='meshes/base_link.dae' scale='1 1 1'/>
+        <mesh filename='package://marble_husky_sensor_config_5/meshes/base_link.dae' scale='1 1 1'/>
       </geometry>
     </visual>
@@ -124,5 +126,5 @@
       <origin xyz='0.48 0 0.091' rpy='0 -0 0'/>
       <geometry>
-        <mesh filename='meshes/bumper.dae' scale='1 1 1'/>
+        <mesh filename='package://marble_husky_sensor_config_5/meshes/bumper.dae' scale='1 1 1'/>
       </geometry>
     </visual>
@@ -130,5 +132,5 @@
       <origin xyz='-0.48 0 0.091' rpy='0 -0 3.14159'/>
       <geometry>
-        <mesh filename='meshes/bumper.dae' scale='1 1 1'/>
+        <mesh filename='package://marble_husky_sensor_config_5/meshes/bumper.dae' scale='1 1 1'/>
       </geometry>
     </visual>
@@ -136,5 +138,5 @@
       <origin xyz='0 0 0' rpy='0 -0 0'/>
       <geometry>
-        <mesh filename='meshes/top_chassis.dae' scale='1 1 1'/>
+        <mesh filename='package://marble_husky_sensor_config_5/meshes/top_chassis.dae' scale='1 1 1'/>
       </geometry>
     </visual>
@@ -142,5 +144,5 @@
       <origin xyz='0.272 0 0.245' rpy='0 -0 0'/>
       <geometry>
-        <mesh filename='meshes/user_rail.dae' scale='1 1 1'/>
+        <mesh filename='package://marble_husky_sensor_config_5/meshes/user_rail.dae' scale='1 1 1'/>
       </geometry>
     </visual>
@@ -166,5 +168,5 @@
       <origin xyz='0.527 0.015 0.429' rpy='-1.34452 0.47634 0.465309'/>
       <geometry>
-        <mesh filename='meshes/realsense.dae' scale='1 1 1'/>
+        <mesh filename='package://marble_husky_sensor_config_5/meshes/realsense.dae' scale='1 1 1'/>
       </geometry>
     </visual>
@@ -178,5 +180,5 @@
       <origin xyz='0.527 -0.015 0.429' rpy='-1.79707 0.47634 -0.465309'/>
       <geometry>
-        <mesh filename='meshes/realsense.dae' scale='1 1 1'/>
+        <mesh filename='package://marble_husky_sensor_config_5/meshes/realsense.dae' scale='1 1 1'/>
       </geometry>
     </visual>
@@ -214,5 +216,5 @@
       <origin xyz='0.4379 0 0.61018' rpy='0 -0 0'/>
       <geometry>
-        <mesh filename='meshes/VLP16_base_1.dae' scale='1 1 1'/>
+        <mesh filename='package://marble_husky_sensor_config_5/meshes/VLP16_base_1.dae' scale='1 1 1'/>
       </geometry>
     </visual>
@@ -220,5 +222,5 @@
       <origin xyz='0.4379 0 0.61018' rpy='0 -0 0'/>
       <geometry>
-        <mesh filename='meshes/VLP16_base_2.dae' scale='1 1 1'/>
+        <mesh filename='package://marble_husky_sensor_config_5/meshes/VLP16_base_2.dae' scale='1 1 1'/>
       </geometry>
     </visual>
@@ -226,5 +228,5 @@
       <origin xyz='0.4379 0 0.61018' rpy='0 -0 0'/>
       <geometry>
-        <mesh filename='meshes/VLP16_scan.dae' scale='1 1 1'/>
+        <mesh filename='package://marble_husky_sensor_config_5/meshes/VLP16_scan.dae' scale='1 1 1'/>
       </geometry>
     </visual>
@@ -232,5 +234,5 @@
       <origin xyz='0.31037 0 0.44818' rpy='3.14159 -1.57079 3.14159'/>
       <geometry>
-        <mesh filename='meshes/VLP16_base_1.dae' scale='1 1 1'/>
+        <mesh filename='package://marble_husky_sensor_config_5/meshes/VLP16_base_1.dae' scale='1 1 1'/>
       </geometry>
     </visual>
@@ -238,5 +240,5 @@
       <origin xyz='0.31037 0 0.44818' rpy='3.14159 -1.57079 3.14159'/>
       <geometry>
-        <mesh filename='meshes/VLP16_base_2.dae' scale='1 1 1'/>
+        <mesh filename='package://marble_husky_sensor_config_5/meshes/VLP16_base_2.dae' scale='1 1 1'/>
       </geometry>
     </visual>
@@ -244,5 +246,5 @@
       <origin xyz='0.31037 0 0.44818' rpy='3.14159 -1.57079 3.14159'/>
       <geometry>
-        <mesh filename='meshes/VLP16_scan.dae' scale='1 1 1'/>
+        <mesh filename='package://marble_husky_sensor_config_5/meshes/VLP16_scan.dae' scale='1 1 1'/>
       </geometry>
     </visual>
@@ -273,9 +275,9 @@
   </link>
   <sensor name='planar_laser' update_rate='20'>
-    <parent link='base_link'/>
+    <parent link='${robot_namespace}/base_link'/>
     <origin xyz='0.485 0 0.166' rpy='0 -0 0'/>
   </sensor>
   <sensor name='tof_left' update_rate='10'>
-    <parent link='base_link'/>
+    <parent link='${robot_namespace}/base_link'/>
     <origin xyz='0.527 0.015 0.429' rpy='-1.34452 0.47634 0.465309'/>
     <camera>
@@ -284,5 +286,5 @@
   </sensor>
   <sensor name='tof_right' update_rate='10'>
-    <parent link='base_link'/>
+    <parent link='${robot_namespace}/base_link'/>
     <origin xyz='0.527 -0.015 0.429' rpy='-1.79707 0.47634 -0.465309'/>
     <camera>
@@ -291,17 +293,17 @@
   </sensor>
   <sensor name='imu_sensor' update_rate='200'>
-    <parent link='base_link'/>
+    <parent link='${robot_namespace}/base_link'/>
     <origin xyz='0 0 0' rpy='0 -0 0'/>
   </sensor>
   <sensor name='front_laser' update_rate='10'>
-    <parent link='base_link'/>
+    <parent link='${robot_namespace}/base_link'/>
     <origin xyz='0.4379 0 0.67018' rpy='0 -0 0'/>
   </sensor>
   <sensor name='vert_laser' update_rate='10'>
-    <parent link='base_link'/>
+    <parent link='${robot_namespace}/base_link'/>
     <origin xyz='0.31037 0 0.44818' rpy='3.14159 -1.57079 3.14159'/>
   </sensor>
   <sensor name='camera_front' update_rate='10'>
-    <parent link='base_link'/>
+    <parent link='${robot_namespace}/base_link'/>
     <origin xyz='0.5579 0 0.53718' rpy='0 -0 0'/>
     <camera>
@@ -310,5 +312,5 @@
   </sensor>
   <sensor name='camera_back' update_rate='10'>
-    <parent link='base_link'/>
+    <parent link='${robot_namespace}/base_link'/>
     <origin xyz='0.3179 0 0.53718' rpy='0 -0 3.14159'/>
     <camera>
@@ -317,5 +319,5 @@
   </sensor>
   <sensor name='camera_left' update_rate='10'>
-    <parent link='base_link'/>
+    <parent link='${robot_namespace}/base_link'/>
     <origin xyz='0.4379 0.12 0.53718' rpy='0 -0 1.5708'/>
     <camera>
@@ -324,5 +326,5 @@
   </sensor>
   <sensor name='camera_right' update_rate='10'>
-    <parent link='base_link'/>
+    <parent link='${robot_namespace}/base_link'/>
     <origin xyz='0.4379 -0.12 0.53718' rpy='0 0 -1.5708'/>
     <camera>
@@ -330,5 +332,5 @@
     </camera>
   </sensor>
-  <link name='front_left_wheel_link'>
+  <link name='${robot_namespace}/front_left_wheel_link'>
     <inertial>
       <origin xyz='0 0 0' rpy='0 -0 0'/>
@@ -345,9 +347,9 @@
       <origin xyz='0 0 0' rpy='0 -0 0'/>
       <geometry>
-        <mesh filename='meshes/wheel.dae' scale='1 1 1'/>
+        <mesh filename='package://marble_husky_sensor_config_5/meshes/wheel.dae' scale='1 1 1'/>
       </geometry>
     </visual>
   </link>
-  <link name='front_right_wheel_link'>
+  <link name='${robot_namespace}/front_right_wheel_link'>
     <inertial>
       <origin xyz='0 0 0' rpy='0 -0 0'/>
@@ -364,9 +366,9 @@
       <origin xyz='0 0 0' rpy='0 -0 0'/>
       <geometry>
-        <mesh filename='meshes/wheel.dae' scale='1 1 1'/>
+        <mesh filename='package://marble_husky_sensor_config_5/meshes/wheel.dae' scale='1 1 1'/>
       </geometry>
     </visual>
   </link>
-  <link name='rear_left_wheel_link'>
+  <link name='${robot_namespace}/rear_left_wheel_link'>
     <inertial>
       <origin xyz='0 0 0' rpy='0 -0 0'/>
@@ -383,9 +385,9 @@
       <origin xyz='0 0 0' rpy='0 -0 0'/>
       <geometry>
-        <mesh filename='meshes/wheel.dae' scale='1 1 1'/>
+        <mesh filename='package://marble_husky_sensor_config_5/meshes/wheel.dae' scale='1 1 1'/>
       </geometry>
     </visual>
   </link>
-  <link name='rear_right_wheel_link'>
+  <link name='${robot_namespace}/rear_right_wheel_link'>
     <inertial>
       <origin xyz='0 0 0' rpy='0 -0 0'/>
@@ -402,5 +404,5 @@
       <origin xyz='0 0 0' rpy='0 -0 0'/>
       <geometry>
-        <mesh filename='meshes/wheel.dae' scale='1 1 1'/>
+        <mesh filename='package://marble_husky_sensor_config_5/meshes/wheel.dae' scale='1 1 1'/>
       </geometry>
     </visual>
@@ -408,6 +410,6 @@
   <joint name='front_left_wheel_joint' type='revolute'>
     <origin xyz='0.256 0.2854 0.03282' rpy='0 -0 0'/>
-    <parent link='base_link'/>
-    <child link='front_left_wheel_link'/>
+    <parent link='${robot_namespace}/base_link'/>
+    <child link='${robot_namespace}/front_left_wheel_link'/>
     <dynamics damping='0' friction='0' />
     <axis xyz='0 1 0'/>
@@ -416,6 +418,6 @@
   <joint name='front_right_wheel_joint' type='revolute'>
     <origin xyz='0.256 -0.2854 0.03282' rpy='0 -0 0'/>
-    <parent link='base_link'/>
-    <child link='front_right_wheel_link'/>
+    <parent link='${robot_namespace}/base_link'/>
+    <child link='${robot_namespace}/front_right_wheel_link'/>
     <dynamics damping='0' friction='0' />
     <axis xyz='0 1 0'/>
@@ -424,6 +426,6 @@
   <joint name='rear_left_wheel_joint' type='revolute'>
     <origin xyz='-0.256 0.2854 0.03282' rpy='0 -0 0'/>
-    <parent link='base_link'/>
-    <child link='rear_left_wheel_link'/>
+    <parent link='${robot_namespace}/base_link'/>
+    <child link='${robot_namespace}/rear_left_wheel_link'/>
     <dynamics damping='0' friction='0' />
     <axis xyz='0 1 0'/>
@@ -432,6 +434,6 @@
   <joint name='rear_right_wheel_joint' type='revolute'>
     <origin xyz='-0.256 -0.2854 0.03282' rpy='0 -0 0'/>
-    <parent link='base_link'/>
-    <child link='rear_right_wheel_link'/>
+    <parent link='${robot_namespace}/base_link'/>
+    <child link='${robot_namespace}/rear_right_wheel_link'/>
     <dynamics damping='0' friction='0' />
     <axis xyz='0 1 0'/>
