Commit message: Updates based on validation data and changes in other models

File: submitted_models/coro_mark_sensor_config_1/urdf/model.xacro (robot description, xacro)
@@ -6,6 +6,6 @@
     <inertial>
       <origin xyz='0 0 0' rpy='0 -0 0'/>
-      <mass value='3.461'/>
-      <inertia ixx='0.0324' ixy='0' ixz='0' iyy='0.0324' iyz='0' izz='0.0519'/>
+      <mass value='2.217'/>
+      <inertia ixx='0.0207' ixy='0' ixz='0' iyy='0.0207' iyz='0' izz='0.0333'/>
     </inertial>
     <collision name='base_link_inertia_collision'>
@@ -268,27 +268,8 @@
     <inertial>
       <origin xyz='0 0 0' rpy='0 -0 0'/>
-      <mass value='0.024'/>
-      <inertia ixx='8e-07' ixy='0' ixz='0' iyy='5e-05' iyz='0' izz='5e-05'/>
-    </inertial>
-    <collision name='rotor_0_collision'>
-      <origin xyz='0 0 0' rpy='0 -0 0'/>
-      <geometry>
-        <cylinder radius='0.11' length='0.01'/>
-      </geometry>
-    </collision>
-    <visual name='rotor_0_visual'>
-      <origin xyz='0 0 0' rpy='0 -0 0'/>
-      <geometry>
-        <mesh filename='package://coro_mark_sensor_config_1/meshes/propeller_ccw.dae' scale='0.11 0.11 0.11'/>
-      </geometry>
-    </visual>
-  </link>
-  <link name='${robot_namespace}/rotor_1'>
-    <inertial>
-      <origin xyz='0 0 0' rpy='0 -0 0'/>
       <mass value='0.012'/>
       <inertia ixx='8e-07' ixy='0' ixz='0' iyy='5e-05' iyz='0' izz='5e-05'/>
     </inertial>
-    <collision name='rotor_1_collision'>
+    <collision name='rotor_0_collision'>
       <origin xyz='0 0 0' rpy='0 -0 0'/>
       <geometry>
@@ -296,5 +277,5 @@
       </geometry>
     </collision>
-    <visual name='rotor_1_visual'>
+    <visual name='rotor_0_visual'>
       <origin xyz='0 0 0' rpy='0 -0 0'/>
       <geometry>
@@ -303,5 +284,5 @@
     </visual>
   </link>
-  <link name='${robot_namespace}/rotor_2'>
+  <link name='${robot_namespace}/rotor_1'>
     <inertial>
       <origin xyz='0 0 0' rpy='0 -0 0'/>
@@ -309,4 +290,23 @@
       <inertia ixx='8e-07' ixy='0' ixz='0' iyy='5e-05' iyz='0' izz='5e-05'/>
     </inertial>
+    <collision name='rotor_1_collision'>
+      <origin xyz='0 0 0' rpy='0 -0 0'/>
+      <geometry>
+        <cylinder radius='0.11' length='0.01'/>
+      </geometry>
+    </collision>
+    <visual name='rotor_1_visual'>
+      <origin xyz='0 0 0' rpy='0 -0 0'/>
+      <geometry>
+        <mesh filename='package://coro_mark_sensor_config_1/meshes/propeller_ccw.dae' scale='0.11 0.11 0.11'/>
+      </geometry>
+    </visual>
+  </link>
+  <link name='${robot_namespace}/rotor_2'>
+    <inertial>
+      <origin xyz='0 0 0' rpy='0 -0 0'/>
+      <mass value='0.012'/>
+      <inertia ixx='8e-07' ixy='0' ixz='0' iyy='5e-05' iyz='0' izz='5e-05'/>
+    </inertial>
     <collision name='rotor_2_collision'>
       <origin xyz='0 0 0' rpy='0 -0 0'/>
@@ -325,5 +325,5 @@
     <inertial>
       <origin xyz='0 0 0' rpy='0 -0 0'/>
-      <mass value='0.024'/>
+      <mass value='0.012'/>
       <inertia ixx='8e-07' ixy='0' ixz='0' iyy='5e-05' iyz='0' izz='5e-05'/>
     </inertial>
