Commit message: Fix path to mesh in URDF

File: submitted_models/ctu_cras_norlab_x500_sensor_config_1/urdf/model.xacro (robot description, xacro)
@@ -72,5 +72,5 @@
       <origin xyz='0.082 0 0.034' rpy='-1.5708 0 1.5708'/>
       <geometry>
-        <mesh filename='package://ctu_cras_norlab_x500_sensor_config_1/meshes/realsense.dae' scale='1 1 1'/>
+        <mesh filename='package://ctu_cras_norlab_x500_sensor_config_1/meshes/sensors/realsense.dae' scale='1 1 1'/>
       </geometry>
     </visual>
@@ -78,5 +78,5 @@
       <origin xyz='0.085 0 -0.02' rpy='1.5708 -0 1.5708'/>
       <geometry>
-        <mesh filename='package://ctu_cras_norlab_x500_sensor_config_1/meshes/realsense.dae' scale='1 1 1'/>
+        <mesh filename='package://ctu_cras_norlab_x500_sensor_config_1/meshes/sensors/realsense.dae' scale='1 1 1'/>
       </geometry>
     </visual>

Commit message: changed imu_joint to fixed

File: submitted_models/ctu_cras_norlab_x500_sensor_config_1/urdf/model.xacro (robot description, xacro)
@@ -362,5 +362,5 @@
     </visual>
   </link>
-  <joint name='imu_joint' type='revolute'>
+  <joint name='imu_joint' type='fixed'>
     <origin xyz='0 0 0' rpy='0 -0 0'/>
     <parent link='${robot_namespace}/base_link'/>

Commit message: addded top and bottom lights

File: submitted_models/ctu_cras_norlab_x500_sensor_config_1/urdf/model.xacro (robot description, xacro)
@@ -15,5 +15,17 @@
       </geometry>
     </collision>
-    <collision name='base_link_fixed_joint_lump__front_left_leg_clip_link_collision_1'>
+    <collision name='base_link_fixed_joint_lump__bottom_light_link_collision_1'>
+      <origin xyz='0.03 0 -0.05' rpy='0 -0 0'/>
+      <geometry>
+        <box size='0.01 0.1 0.003'/>
+      </geometry>
+    </collision>
+    <collision name='base_link_fixed_joint_lump__top_light_link_collision_2'>
+      <origin xyz='0.05 0 0.059' rpy='0 -0 0'/>
+      <geometry>
+        <box size='0.01 0.1 0.003'/>
+      </geometry>
+    </collision>
+    <collision name='base_link_fixed_joint_lump__front_left_leg_clip_link_collision_3'>
       <origin xyz='0.162635 0.162635 -0.0785' rpy='0 -0 0'/>
       <geometry>
@@ -21,5 +33,5 @@
       </geometry>
     </collision>
-    <collision name='base_link_fixed_joint_lump__front_left_leg_light_link_collision_2'>
+    <collision name='base_link_fixed_joint_lump__front_left_leg_light_link_collision_4'>
       <origin xyz='0.159099 0.152028 -0.0785' rpy='0 -0 2.35619'/>
       <geometry>
@@ -27,5 +39,5 @@
       </geometry>
     </collision>
-    <collision name='base_link_fixed_joint_lump__front_right_leg_clip_link_collision_3'>
+    <collision name='base_link_fixed_joint_lump__front_right_leg_clip_link_collision_5'>
       <origin xyz='0.162635 -0.162635 -0.0785' rpy='0 0 -1.5708'/>
       <geometry>
@@ -33,5 +45,5 @@
       </geometry>
     </collision>
-    <collision name='base_link_fixed_joint_lump__front_right_leg_light_link_collision_4'>
+    <collision name='base_link_fixed_joint_lump__front_right_leg_light_link_collision_6'>
       <origin xyz='0.159099 -0.152028 -0.0785' rpy='0 -0 0.785398'/>
       <geometry>
@@ -39,5 +51,5 @@
       </geometry>
     </collision>
-    <collision name='base_link_fixed_joint_lump__os_sensor_link_collision_5'>
+    <collision name='base_link_fixed_joint_lump__os_sensor_link_collision_7'>
       <origin xyz='0 0 0.0944' rpy='0 -0 1.5708'/>
       <geometry>
@@ -45,5 +57,5 @@
       </geometry>
     </collision>
-    <collision name='base_link_fixed_joint_lump__rear_left_leg_clip_link_collision_6'>
+    <collision name='base_link_fixed_joint_lump__rear_left_leg_clip_link_collision_8'>
       <origin xyz='-0.162635 0.162635 -0.0785' rpy='0 -0 1.5708'/>
       <geometry>
@@ -51,5 +63,5 @@
       </geometry>
     </collision>
-    <collision name='base_link_fixed_joint_lump__rear_right_leg_clip_link_collision_7'>
+    <collision name='base_link_fixed_joint_lump__rear_right_leg_clip_link_collision_9'>
       <origin xyz='-0.162635 -0.162635 -0.0785' rpy='0 0 -3.14159'/>
       <geometry>
@@ -57,5 +69,5 @@
       </geometry>
     </collision>
-    <collision name='base_link_fixed_joint_lump__rs_up_holder_link_collision_8'>
+    <collision name='base_link_fixed_joint_lump__rs_up_holder_link_collision_10'>
       <origin xyz='0.085 0 0.032' rpy='-1.5708 -0 -1.5708'/>
       <geometry>
@@ -63,5 +75,5 @@
       </geometry>
     </collision>
-    <collision name='base_link_fixed_joint_lump__sensor_holder_link_collision_9'>
+    <collision name='base_link_fixed_joint_lump__sensor_holder_link_collision_11'>
       <origin xyz='0 0 -0.022' rpy='1.5708 0 -1.5708'/>
       <geometry>
@@ -135,5 +147,11 @@
       </geometry>
     </visual>
-    <visual name='base_link_fixed_joint_lump__computer_board_link_visual_11'>
+    <visual name='base_link_fixed_joint_lump__bottom_light_link_visual_11'>
+      <origin xyz='0.03 0 -0.05' rpy='0 -0 0'/>
+      <geometry>
+        <box size='0.01 0.1 0.003'/>
+      </geometry>
+    </visual>
+    <visual name='base_link_fixed_joint_lump__computer_board_link_visual_12'>
       <origin xyz='0 0 0.058' rpy='0 -0 0'/>
       <geometry>
@@ -141,5 +159,11 @@
       </geometry>
     </visual>
-    <visual name='base_link_fixed_joint_lump__front_left_arm_link_visual_12'>
+    <visual name='base_link_fixed_joint_lump__top_light_link_visual_13'>
+      <origin xyz='0.05 0 0.059' rpy='0 -0 0'/>
+      <geometry>
+        <box size='0.01 0.1 0.003'/>
+      </geometry>
+    </visual>
+    <visual name='base_link_fixed_joint_lump__front_left_arm_link_visual_14'>
       <origin xyz='0 0 0' rpy='0 -0 0.785398'/>
       <geometry>
@@ -147,5 +171,5 @@
       </geometry>
     </visual>
-    <visual name='base_link_fixed_joint_lump__front_left_leg_clip_link_visual_13'>
+    <visual name='base_link_fixed_joint_lump__front_left_leg_clip_link_visual_15'>
       <origin xyz='0.162635 0.162635 -0.157' rpy='0 -0 0.785398'/>
       <geometry>
@@ -153,5 +177,5 @@
       </geometry>
     </visual>
-    <visual name='base_link_fixed_joint_lump__front_left_leg_light_link_visual_14'>
+    <visual name='base_link_fixed_joint_lump__front_left_leg_light_link_visual_16'>
       <origin xyz='0.159099 0.152028 -0.0785' rpy='0 -0 2.35619'/>
       <geometry>
@@ -159,5 +183,5 @@
       </geometry>
     </visual>
-    <visual name='base_link_fixed_joint_lump__front_left_rotor_link_visual_15'>
+    <visual name='base_link_fixed_joint_lump__front_left_rotor_link_visual_17'>
       <origin xyz='0.177484 0.177484 0.021' rpy='0 -0 0'/>
       <geometry>
@@ -165,5 +189,5 @@
       </geometry>
     </visual>
-    <visual name='base_link_fixed_joint_lump__front_right_arm_link_visual_16'>
+    <visual name='base_link_fixed_joint_lump__front_right_arm_link_visual_18'>
       <origin xyz='0 0 0' rpy='0 0 -0.785398'/>
       <geometry>
@@ -171,5 +195,5 @@
       </geometry>
     </visual>
-    <visual name='base_link_fixed_joint_lump__front_right_leg_clip_link_visual_17'>
+    <visual name='base_link_fixed_joint_lump__front_right_leg_clip_link_visual_19'>
       <origin xyz='0.162635 -0.162635 -0.157' rpy='0 0 -0.785398'/>
       <geometry>
@@ -177,5 +201,5 @@
       </geometry>
     </visual>
-    <visual name='base_link_fixed_joint_lump__front_right_leg_light_link_visual_18'>
+    <visual name='base_link_fixed_joint_lump__front_right_leg_light_link_visual_20'>
       <origin xyz='0.159099 -0.152028 -0.0785' rpy='0 -0 0.785398'/>
       <geometry>
@@ -183,5 +207,5 @@
       </geometry>
     </visual>
-    <visual name='base_link_fixed_joint_lump__front_right_rotor_link_visual_19'>
+    <visual name='base_link_fixed_joint_lump__front_right_rotor_link_visual_21'>
       <origin xyz='0.177484 -0.177484 0.021' rpy='0 -0 0'/>
       <geometry>
@@ -189,5 +213,5 @@
       </geometry>
     </visual>
-    <visual name='base_link_fixed_joint_lump__left_cover_link_visual_20'>
+    <visual name='base_link_fixed_joint_lump__left_cover_link_visual_22'>
       <origin xyz='0 0.064 0.03' rpy='0 0 -3.14159'/>
       <geometry>
@@ -195,5 +219,5 @@
       </geometry>
     </visual>
-    <visual name='base_link_fixed_joint_lump__os_sensor_link_visual_21'>
+    <visual name='base_link_fixed_joint_lump__os_sensor_link_visual_23'>
       <origin xyz='0 0 0.06' rpy='0 -0 1.5708'/>
       <geometry>
@@ -201,5 +225,5 @@
       </geometry>
     </visual>
-    <visual name='base_link_fixed_joint_lump__os_sensor_window_link_visual_22'>
+    <visual name='base_link_fixed_joint_lump__os_sensor_window_link_visual_24'>
       <origin xyz='0 0 0.0944' rpy='0 -0 0'/>
       <geometry>
@@ -207,5 +231,5 @@
       </geometry>
     </visual>
-    <visual name='base_link_fixed_joint_lump__pc_mount_link_visual_23'>
+    <visual name='base_link_fixed_joint_lump__pc_mount_link_visual_25'>
       <origin xyz='0 0 0' rpy='0 -0 0'/>
       <geometry>
@@ -213,5 +237,5 @@
       </geometry>
     </visual>
-    <visual name='base_link_fixed_joint_lump__pixhawk_link_visual_24'>
+    <visual name='base_link_fixed_joint_lump__pixhawk_link_visual_26'>
       <origin xyz='0 0 0.036' rpy='0 -0 0'/>
       <geometry>
@@ -219,5 +243,5 @@
       </geometry>
     </visual>
-    <visual name='base_link_fixed_joint_lump__rear_left_leg_clip_link_visual_25'>
+    <visual name='base_link_fixed_joint_lump__rear_left_leg_clip_link_visual_27'>
       <origin xyz='-0.162635 0.162635 -0.157' rpy='0 -0 2.35619'/>
       <geometry>
@@ -225,5 +249,5 @@
       </geometry>
     </visual>
-    <visual name='base_link_fixed_joint_lump__rear_right_leg_clip_link_visual_26'>
+    <visual name='base_link_fixed_joint_lump__rear_right_leg_clip_link_visual_28'>
       <origin xyz='-0.162635 -0.162635 -0.157' rpy='0 0 -2.35619'/>
       <geometry>
@@ -231,5 +255,5 @@
       </geometry>
     </visual>
-    <visual name='base_link_fixed_joint_lump__right_cover_link_visual_27'>
+    <visual name='base_link_fixed_joint_lump__right_cover_link_visual_29'>
       <origin xyz='0 -0.064 0.03' rpy='0 -0 0'/>
       <geometry>
@@ -237,5 +261,5 @@
       </geometry>
     </visual>
-    <visual name='base_link_fixed_joint_lump__rs_up_holder_link_visual_28'>
+    <visual name='base_link_fixed_joint_lump__rs_up_holder_link_visual_30'>
       <origin xyz='0.085 0 0.032' rpy='-1.5708 -0 -1.5708'/>
       <geometry>
@@ -243,5 +267,5 @@
       </geometry>
     </visual>
-    <visual name='base_link_fixed_joint_lump__sensor_holder_link_visual_29'>
+    <visual name='base_link_fixed_joint_lump__sensor_holder_link_visual_31'>
       <origin xyz='0 0 -0.022' rpy='1.5708 0 -1.5708'/>
       <geometry>
