Commit message: Fix X500 RViz model

File: submitted_models/ctu_cras_norlab_x500_sensor_config_1/urdf/model.xacro (robot description, xacro)
@@ -72,5 +72,5 @@
       <origin xyz='0.085 0 0.032' rpy='-1.5708 -0 -1.5708'/>
       <geometry>
-        <mesh filename='package://ctu_cras_norlab_x500_sensor_config_1/meshes/holders/holder_rs_up.dae' scale='1 1 1'/>
+        <mesh filename='package://ctu_cras_norlab_x500_sensor_config_1/meshes/holder_rs_up.dae' scale='1 1 1'/>
       </geometry>
     </collision>
@@ -78,5 +78,5 @@
       <origin xyz='0 0 -0.022' rpy='1.5708 0 -1.5708'/>
       <geometry>
-        <mesh filename='package://ctu_cras_norlab_x500_sensor_config_1/meshes/holders/holder_rs_down_bfox.dae' scale='1 1 1'/>
+        <mesh filename='package://ctu_cras_norlab_x500_sensor_config_1/meshes/holder_rs_down_bfox.dae' scale='1 1 1'/>
       </geometry>
     </collision>
@@ -84,5 +84,5 @@
       <origin xyz='0.082 0 0.034' rpy='-1.5708 0 1.5708'/>
       <geometry>
-        <mesh filename='package://ctu_cras_norlab_x500_sensor_config_1/meshes/sensors/realsense.dae' scale='1 1 1'/>
+        <mesh filename='package://ctu_cras_norlab_x500_sensor_config_1/meshes/realsense.dae' scale='1 1 1'/>
       </geometry>
     </visual>
@@ -90,5 +90,5 @@
       <origin xyz='0.085 0 -0.02' rpy='1.5708 -0 1.5708'/>
       <geometry>
-        <mesh filename='package://ctu_cras_norlab_x500_sensor_config_1/meshes/sensors/realsense.dae' scale='1 1 1'/>
+        <mesh filename='package://ctu_cras_norlab_x500_sensor_config_1/meshes/realsense.dae' scale='1 1 1'/>
       </geometry>
     </visual>
@@ -96,5 +96,5 @@
       <origin xyz='0.107 0 0' rpy='0 -0 0'/>
       <geometry>
-        <mesh filename='package://ctu_cras_norlab_x500_sensor_config_1/meshes/sensors/bluefox.dae' scale='1 1 1'/>
+        <mesh filename='package://ctu_cras_norlab_x500_sensor_config_1/meshes/bluefox.dae' scale='1 1 1'/>
       </geometry>
     </visual>
@@ -102,5 +102,5 @@
       <origin xyz='-0.064 0 0.03' rpy='0 -0 1.5708'/>
       <geometry>
-        <mesh filename='package://ctu_cras_norlab_x500_sensor_config_1/meshes/holders/side_mrs.dae' scale='1 1 1'/>
+        <mesh filename='package://ctu_cras_norlab_x500_sensor_config_1/meshes/side_mrs.dae' scale='1 1 1'/>
       </geometry>
     </visual>
@@ -108,5 +108,5 @@
       <origin xyz='0 0 0' rpy='0 -0 2.35619'/>
       <geometry>
-        <mesh filename='package://ctu_cras_norlab_x500_sensor_config_1/meshes/holybro/holybro_x500_arm.dae' scale='1 1 1'/>
+        <mesh filename='package://ctu_cras_norlab_x500_sensor_config_1/meshes/holybro_x500_arm.dae' scale='1 1 1'/>
       </geometry>
     </visual>
@@ -114,5 +114,5 @@
       <origin xyz='-0.177484 0.177484 0.021' rpy='0 -0 0'/>
       <geometry>
-        <mesh filename='package://ctu_cras_norlab_x500_sensor_config_1/meshes/holybro/holybro_x500_motor.dae' scale='1 1 1'/>
+        <mesh filename='package://ctu_cras_norlab_x500_sensor_config_1/meshes/holybro_x500_motor.dae' scale='1 1 1'/>
       </geometry>
     </visual>
@@ -120,5 +120,5 @@
       <origin xyz='0 0 0' rpy='0 0 -2.35619'/>
       <geometry>
-        <mesh filename='package://ctu_cras_norlab_x500_sensor_config_1/meshes/holybro/holybro_x500_arm.dae' scale='1 1 1'/>
+        <mesh filename='package://ctu_cras_norlab_x500_sensor_config_1/meshes/holybro_x500_arm.dae' scale='1 1 1'/>
       </geometry>
     </visual>
@@ -126,5 +126,5 @@
       <origin xyz='-0.177484 -0.177484 0.021' rpy='0 -0 0'/>
       <geometry>
-        <mesh filename='package://ctu_cras_norlab_x500_sensor_config_1/meshes/holybro/holybro_x500_motor.dae' scale='1 1 1'/>
+        <mesh filename='package://ctu_cras_norlab_x500_sensor_config_1/meshes/holybro_x500_motor.dae' scale='1 1 1'/>
       </geometry>
     </visual>
@@ -132,5 +132,5 @@
       <origin xyz='-0.02 0.03 0' rpy='0 -0 0'/>
       <geometry>
-        <mesh filename='package://ctu_cras_norlab_x500_sensor_config_1/meshes/holybro/holybro_x500_battery.dae' scale='1 1 1'/>
+        <mesh filename='package://ctu_cras_norlab_x500_sensor_config_1/meshes/holybro_x500_battery.dae' scale='1 1 1'/>
       </geometry>
     </visual>
@@ -138,5 +138,5 @@
       <origin xyz='-0.02 -0.03 0' rpy='0 -0 0'/>
       <geometry>
-        <mesh filename='package://ctu_cras_norlab_x500_sensor_config_1/meshes/holybro/holybro_x500_battery.dae' scale='1 1 1'/>
+        <mesh filename='package://ctu_cras_norlab_x500_sensor_config_1/meshes/holybro_x500_battery.dae' scale='1 1 1'/>
       </geometry>
     </visual>
@@ -144,5 +144,5 @@
       <origin xyz='0 0 0' rpy='0 -0 0'/>
       <geometry>
-        <mesh filename='package://ctu_cras_norlab_x500_sensor_config_1/meshes/holybro/holybro_x500_bottom_board.dae' scale='1 1 1'/>
+        <mesh filename='package://ctu_cras_norlab_x500_sensor_config_1/meshes/holybro_x500_bottom_board.dae' scale='1 1 1'/>
       </geometry>
     </visual>
@@ -168,5 +168,5 @@
       <origin xyz='0 0 0' rpy='0 -0 0.785398'/>
       <geometry>
-        <mesh filename='package://ctu_cras_norlab_x500_sensor_config_1/meshes/holybro/holybro_x500_arm.dae' scale='1 1 1'/>
+        <mesh filename='package://ctu_cras_norlab_x500_sensor_config_1/meshes/holybro_x500_arm.dae' scale='1 1 1'/>
       </geometry>
     </visual>
@@ -174,5 +174,5 @@
       <origin xyz='0.162635 0.162635 -0.157' rpy='0 -0 0.785398'/>
       <geometry>
-        <mesh filename='package://ctu_cras_norlab_x500_sensor_config_1/meshes/holybro/holybro_x500_leg.dae' scale='1 1 1'/>
+        <mesh filename='package://ctu_cras_norlab_x500_sensor_config_1/meshes/holybro_x500_leg.dae' scale='1 1 1'/>
       </geometry>
     </visual>
@@ -186,5 +186,5 @@
       <origin xyz='0.177484 0.177484 0.021' rpy='0 -0 0'/>
       <geometry>
-        <mesh filename='package://ctu_cras_norlab_x500_sensor_config_1/meshes/holybro/holybro_x500_motor.dae' scale='1 1 1'/>
+        <mesh filename='package://ctu_cras_norlab_x500_sensor_config_1/meshes/holybro_x500_motor.dae' scale='1 1 1'/>
       </geometry>
     </visual>
@@ -192,5 +192,5 @@
       <origin xyz='0 0 0' rpy='0 0 -0.785398'/>
       <geometry>
-        <mesh filename='package://ctu_cras_norlab_x500_sensor_config_1/meshes/holybro/holybro_x500_arm.dae' scale='1 1 1'/>
+        <mesh filename='package://ctu_cras_norlab_x500_sensor_config_1/meshes/holybro_x500_arm.dae' scale='1 1 1'/>
       </geometry>
     </visual>
@@ -198,5 +198,5 @@
       <origin xyz='0.162635 -0.162635 -0.157' rpy='0 0 -0.785398'/>
       <geometry>
-        <mesh filename='package://ctu_cras_norlab_x500_sensor_config_1/meshes/holybro/holybro_x500_leg.dae' scale='1 1 1'/>
+        <mesh filename='package://ctu_cras_norlab_x500_sensor_config_1/meshes/holybro_x500_leg.dae' scale='1 1 1'/>
       </geometry>
     </visual>
@@ -210,5 +210,5 @@
       <origin xyz='0.177484 -0.177484 0.021' rpy='0 -0 0'/>
       <geometry>
-        <mesh filename='package://ctu_cras_norlab_x500_sensor_config_1/meshes/holybro/holybro_x500_motor.dae' scale='1 1 1'/>
+        <mesh filename='package://ctu_cras_norlab_x500_sensor_config_1/meshes/holybro_x500_motor.dae' scale='1 1 1'/>
       </geometry>
     </visual>
@@ -216,5 +216,5 @@
       <origin xyz='0 0.064 0.03' rpy='0 0 -3.14159'/>
       <geometry>
-        <mesh filename='package://ctu_cras_norlab_x500_sensor_config_1/meshes/holders/side_ctu.dae' scale='1 1 1'/>
+        <mesh filename='package://ctu_cras_norlab_x500_sensor_config_1/meshes/side_ctu.dae' scale='1 1 1'/>
       </geometry>
     </visual>
@@ -222,5 +222,5 @@
       <origin xyz='0 0 0.06' rpy='0 -0 1.5708'/>
       <geometry>
-        <mesh filename='package://ctu_cras_norlab_x500_sensor_config_1/meshes/sensors/os1_64.dae' scale='1 1 1'/>
+        <mesh filename='package://ctu_cras_norlab_x500_sensor_config_1/meshes/os1_64.dae' scale='1 1 1'/>
       </geometry>
     </visual>
@@ -234,5 +234,5 @@
       <origin xyz='0 0 0' rpy='0 -0 0'/>
       <geometry>
-        <mesh filename='package://ctu_cras_norlab_x500_sensor_config_1/meshes/holybro/holybro_x500_pc_mount.dae' scale='1 1 1'/>
+        <mesh filename='package://ctu_cras_norlab_x500_sensor_config_1/meshes/holybro_x500_pc_mount.dae' scale='1 1 1'/>
       </geometry>
     </visual>
@@ -240,5 +240,5 @@
       <origin xyz='0 0 0.036' rpy='0 -0 0'/>
       <geometry>
-        <mesh filename='package://ctu_cras_norlab_x500_sensor_config_1/meshes/sensors/pixhawk.dae' scale='1 1 1'/>
+        <mesh filename='package://ctu_cras_norlab_x500_sensor_config_1/meshes/pixhawk.dae' scale='1 1 1'/>
       </geometry>
     </visual>
@@ -246,5 +246,5 @@
       <origin xyz='-0.162635 0.162635 -0.157' rpy='0 -0 2.35619'/>
       <geometry>
-        <mesh filename='package://ctu_cras_norlab_x500_sensor_config_1/meshes/holybro/holybro_x500_leg.dae' scale='1 1 1'/>
+        <mesh filename='package://ctu_cras_norlab_x500_sensor_config_1/meshes/holybro_x500_leg.dae' scale='1 1 1'/>
       </geometry>
     </visual>
@@ -252,5 +252,5 @@
       <origin xyz='-0.162635 -0.162635 -0.157' rpy='0 0 -2.35619'/>
       <geometry>
-        <mesh filename='package://ctu_cras_norlab_x500_sensor_config_1/meshes/holybro/holybro_x500_leg.dae' scale='1 1 1'/>
+        <mesh filename='package://ctu_cras_norlab_x500_sensor_config_1/meshes/holybro_x500_leg.dae' scale='1 1 1'/>
       </geometry>
     </visual>
@@ -258,5 +258,5 @@
       <origin xyz='0 -0.064 0.03' rpy='0 -0 0'/>
       <geometry>
-        <mesh filename='package://ctu_cras_norlab_x500_sensor_config_1/meshes/holders/side_ctu.dae' scale='1 1 1'/>
+        <mesh filename='package://ctu_cras_norlab_x500_sensor_config_1/meshes/side_ctu.dae' scale='1 1 1'/>
       </geometry>
     </visual>
@@ -264,5 +264,5 @@
       <origin xyz='0.085 0 0.032' rpy='-1.5708 -0 -1.5708'/>
       <geometry>
-        <mesh filename='package://ctu_cras_norlab_x500_sensor_config_1/meshes/holders/holder_rs_up.dae' scale='1 1 1'/>
+        <mesh filename='package://ctu_cras_norlab_x500_sensor_config_1/meshes/holder_rs_up.dae' scale='1 1 1'/>
       </geometry>
     </visual>
@@ -270,5 +270,5 @@
       <origin xyz='0 0 -0.022' rpy='1.5708 0 -1.5708'/>
       <geometry>
-        <mesh filename='package://ctu_cras_norlab_x500_sensor_config_1/meshes/holders/holder_rs_down_bfox.dae' scale='1 1 1'/>
+        <mesh filename='package://ctu_cras_norlab_x500_sensor_config_1/meshes/holder_rs_down_bfox.dae' scale='1 1 1'/>
       </geometry>
     </visual>
@@ -312,10 +312,10 @@
   <link name='${robot_namespace}/rotor_0'>
     <inertial>
-      <origin xyz='-0.177484 0.177484 -0.057' rpy='0 -0 0'/>
+      <origin xyz='0 0 0' rpy='0 -0 0'/>
       <mass value='0.005'/>
       <inertia ixx='0.0001' ixy='0' ixz='0' iyy='0.0001' iyz='0' izz='0.0001'/>
     </inertial>
     <collision name='rotor_0_collision'>
-      <origin xyz='-0.177484 0.177484 -0.057' rpy='0 -0 0'/>
+      <origin xyz='0 0 0' rpy='0 -0 0'/>
       <geometry>
         <cylinder radius='0.127' length='0.005'/>
@@ -323,7 +323,7 @@
     </collision>
     <visual name='rotor_0_visual'>
-      <origin xyz='-0.177484 0.177484 -0.057' rpy='0 -0 0'/>
-      <geometry>
-        <mesh filename='package://ctu_cras_norlab_x500_sensor_config_1/meshes/holybro/holybro_x500_prop.dae' scale='1 1 1'/>
+      <origin xyz='0 0 0' rpy='0 -0 0'/>
+      <geometry>
+        <mesh filename='package://ctu_cras_norlab_x500_sensor_config_1/meshes/holybro_x500_prop.dae' scale='1 1 1'/>
       </geometry>
     </visual>
@@ -331,10 +331,10 @@
   <link name='${robot_namespace}/rotor_1'>
     <inertial>
-      <origin xyz='0.177484 -0.177484 -0.057' rpy='0 -0 0'/>
+      <origin xyz='0 0 0' rpy='0 -0 0'/>
       <mass value='0.005'/>
       <inertia ixx='0.0001' ixy='0' ixz='0' iyy='0.0001' iyz='0' izz='0.0001'/>
     </inertial>
     <collision name='rotor_1_collision'>
-      <origin xyz='0.177484 -0.177484 -0.057' rpy='0 -0 0'/>
+      <origin xyz='0 0 0' rpy='0 -0 0'/>
       <geometry>
         <cylinder radius='0.127' length='0.005'/>
@@ -342,7 +342,7 @@
     </collision>
     <visual name='rotor_1_visual'>
-      <origin xyz='0.177484 -0.177484 -0.057' rpy='0 -0 0'/>
-      <geometry>
-        <mesh filename='package://ctu_cras_norlab_x500_sensor_config_1/meshes/holybro/holybro_x500_prop.dae' scale='1 1 1'/>
+      <origin xyz='0 0 0' rpy='0 -0 0'/>
+      <geometry>
+        <mesh filename='package://ctu_cras_norlab_x500_sensor_config_1/meshes/holybro_x500_prop.dae' scale='1 1 1'/>
       </geometry>
     </visual>
@@ -350,10 +350,10 @@
   <link name='${robot_namespace}/rotor_2'>
     <inertial>
-      <origin xyz='-0.177484 -0.177484 -0.057' rpy='0 -0 0'/>
+      <origin xyz='0 0 0' rpy='0 -0 0'/>
       <mass value='0.005'/>
       <inertia ixx='0.0001' ixy='0' ixz='0' iyy='0.0001' iyz='0' izz='0.0001'/>
     </inertial>
     <collision name='rotor_2_collision'>
-      <origin xyz='-0.177484 -0.177484 -0.057' rpy='0 -0 0'/>
+      <origin xyz='0 0 0' rpy='0 -0 0'/>
       <geometry>
         <cylinder radius='0.127' length='0.005'/>
@@ -361,7 +361,7 @@
     </collision>
     <visual name='rotor_2_visual'>
-      <origin xyz='-0.177484 -0.177484 -0.057' rpy='0 -0 0'/>
-      <geometry>
-        <mesh filename='package://ctu_cras_norlab_x500_sensor_config_1/meshes/holybro/holybro_x500_prop.dae' scale='-1 1 1'/>
+      <origin xyz='0 0 0' rpy='0 -0 0'/>
+      <geometry>
+        <mesh filename='package://ctu_cras_norlab_x500_sensor_config_1/meshes/holybro_x500_prop.dae' scale='-1 1 1'/>
       </geometry>
     </visual>
@@ -369,10 +369,10 @@
   <link name='${robot_namespace}/rotor_3'>
     <inertial>
-      <origin xyz='0.177484 0.177484 -0.057' rpy='0 -0 0'/>
+      <origin xyz='0 0 0' rpy='0 -0 0'/>
       <mass value='0.005'/>
       <inertia ixx='0.0001' ixy='0' ixz='0' iyy='0.0001' iyz='0' izz='0.0001'/>
     </inertial>
     <collision name='rotor_3_collision'>
-      <origin xyz='0.177484 0.177484 -0.057' rpy='0 -0 0'/>
+      <origin xyz='0 0 0' rpy='0 -0 0'/>
       <geometry>
         <cylinder radius='0.127' length='0.005'/>
@@ -380,7 +380,7 @@
     </collision>
     <visual name='rotor_3_visual'>
-      <origin xyz='0.177484 0.177484 -0.057' rpy='0 -0 0'/>
-      <geometry>
-        <mesh filename='package://ctu_cras_norlab_x500_sensor_config_1/meshes/holybro/holybro_x500_prop.dae' scale='-1 1 1'/>
+      <origin xyz='0 0 0' rpy='0 -0 0'/>
+      <geometry>
+        <mesh filename='package://ctu_cras_norlab_x500_sensor_config_1/meshes/holybro_x500_prop.dae' scale='-1 1 1'/>
       </geometry>
     </visual>
