Commit message: Corrected permissions on xacros, fixed number of samples for the vlp16, and added payload mass calculation to vlp16 and d435s.

File: submitted_models/explorer_spot_sensor_config_1/urdf/3d_lidar.xacro (robot description, xacro)
@@ -32,9 +32,10 @@
     topic: ROS topic name where the 3D points are published.
   -->
+  <xacro:property name="vlp16_mass" value="1.0" scope="global" />
   <xacro:macro name="velodyne_lidar" params="name
                                              update_rate:=10
                                              vertical_lasers:=16
                                              samples:=1800
-                                             resolution:=0.1
+                                             resolution:=1
                                              min_angle:=${-pi}
                                              max_angle:=${pi}
@@ -45,4 +46,5 @@
                                              robot_namespace:=/
                                              topic:=points">
+    <xacro:property name="vlp16_void" value="${payload_mass.append(vlp16_mass)}" scope="global" />
     <link name="${name}">
       <!--visual name="${name}_visual">>

File: submitted_models/explorer_spot_sensor_config_1/urdf/basler_cameras.xacro (robot description, xacro)
@@ -77,12 +77,20 @@
                             <stddev>0.007</stddev>
                         </noise>
-                        <xacro:if value="${fisheye and '$(arg rendering_target)' == 'gz'}">
-                            <lens>
+                        <lens>
+                            <intrinsics>
+                                <xacro:property name="f" value="${resolution_x / (2 * tan(radians(hfov_deg)/2))}" />
+                                <fx>${f}</fx>
+                                <fy>${f}</fy>
+                                <cx>${(resolution_x - 1) / 2}</cx>
+                                <cy>${(resolution_y - 1) / 2}</cy>
+                                <s>0</s>
+                            </intrinsics>
+                            <xacro:if value="${fisheye and '$(arg rendering_target)' == 'gz'}">
                                 <type>stereographic</type>
                                 <scale_to_hfov>true</scale_to_hfov>
                                 <cutoff_angle>${pi}</cutoff_angle>
                                 <env_texture_size>1024</env_texture_size>
-                            </lens>
-                        </xacro:if>
+                            </xacro:if>
+                        </lens>
                     </camera>
                 </sensor>
@@ -94,5 +102,5 @@
             fisheye="${fisheye}" simulate="${simulate}" visualize="${visualize}"
             camera_length="0.0555" origin_to_camera_front_dist="0.0524" camera_mass="${basler_ace2_pro_mass}"
-            camera_mesh="package://marble_spot_sensor_config_1/meshes/basler_ace2_pro.dae"
+            camera_mesh="package://explorer_spot_sensor_config_1/meshes/basler_ace2_pro.dae"
             lens_length="${lens_length}" lens_back_focal_distance="${lens_back_focal_distance}"
             lens_entrance_pupil_position="${lens_entrance_pupil_position}" lens_mass="${lens_mass}" lens_mesh="${lens_mesh}"
@@ -103,5 +111,5 @@
         <xacro:basler_ace2_pro_link name="${name}" hfov_deg="86.5" simulate="${simulate}" visualize="${visualize}"
             lens_back_focal_distance="0.00809" lens_entrance_pupil_position="0.01066" lens_length="0.03974" lens_mass="${omnicam_lens_mass}"
-            lens_mesh="package://marble_spot_sensor_config_1/meshes/evetar_lens.dae" />
+            lens_mesh="package://explorer_spot_sensor_config_1/meshes/evetar_lens.dae" />
     </xacro:macro>
 </root>

File: submitted_models/explorer_spot_sensor_config_1/urdf/flir_cameras.xacro (robot description, xacro)
@@ -90,5 +90,5 @@
             fisheye="${fisheye}" simulate="${simulate}" visualize="${visualize}"
             camera_length="0.0555" origin_to_camera_front_dist="0.0524" camera_mass="${flir_backly_mass}"
-            camera_mesh="package://marble_spot_sensor_config_1/meshes/basler_ace2_pro.dae"
+            camera_mesh="package://explorer_spot_sensor_config_1/meshes/basler_ace2_pro.dae"
             lens_length="${lens_length}" lens_back_focal_distance="${lens_back_focal_distance}"
             lens_entrance_pupil_position="${lens_entrance_pupil_position}" lens_mass="${lens_mass}" lens_mesh="${lens_mesh}"
@@ -99,5 +99,5 @@
         <xacro:flir_backly_link name="${name}" hfov_deg="80" simulate="${simulate}" visualize="${visualize}"
             lens_back_focal_distance="0.00809" lens_entrance_pupil_position="0.01066" lens_length="0.03974" lens_mass="${lens_mass}"
-            lens_mesh="package://marble_spot_sensor_config_1/meshes/evetar_lens.dae" />
+            lens_mesh="package://explorer_spot_sensor_config_1/meshes/evetar_lens.dae" />
     </xacro:macro>
 </root>

File: submitted_models/explorer_spot_sensor_config_1/urdf/imu.xacro (robot description, xacro)
@@ -20,4 +20,5 @@
                     <always_on>1</always_on>
                     <update_rate>50</update_rate>
+                    <enable_orientation>0</enable_orientation>
                     <imu>
                         <angular_velocity>

File: submitted_models/explorer_spot_sensor_config_1/urdf/mote_deployer.xacro (robot description, xacro)
@@ -9,5 +9,5 @@
             <visual>
                 <geometry>
-                    <mesh filename="package://marble_spot_sensor_config_1/meshes/mote_deployer.dae" />
+                    <mesh filename="package://explorer_spot_sensor_config_1/meshes/mote_deployer.dae" />
                 </geometry>
             </visual>

File: submitted_models/explorer_spot_sensor_config_1/urdf/ouster_lidar.xacro (robot description, xacro)
@@ -7,5 +7,5 @@
             <visual>
                 <geometry>
-                    <mesh filename="package://marble_spot_sensor_config_1/meshes/ouster-os0.dae"/>
+                    <mesh filename="package://explorer_spot_sensor_config_1/meshes/ouster-os0.dae"/>
                 </geometry>
             </visual>

File: submitted_models/explorer_spot_sensor_config_1/urdf/ouster_lidar_alt.xacro (robot description, xacro)
@@ -7,5 +7,5 @@
             <visual>
                 <geometry>
-                    <mesh filename="package://marble_spot_sensor_config_1/meshes/ouster-os0.dae"/>
+                    <mesh filename="package://explorer_spot_sensor_config_1/meshes/ouster-os0.dae"/>
                 </geometry>
             </visual>

File: submitted_models/explorer_spot_sensor_config_1/urdf/rgbd_camera.xacro (robot description, xacro)
@@ -24,4 +24,5 @@
     pointCloudCutoffMax: Maximum distance for points.
   -->
+  <xacro:property name="d435_mass" value="0.5" scope="global" />
   <xacro:macro name="rgbd_camera"
                params="name:=camera
@@ -37,4 +38,5 @@
                        pitch:=0
                        yaw:=0">
+    <xacro:property name="d435_void" value="${payload_mass.append(d435_mass)}" scope="global" />
     <link name="${name}_link">
       <visual>

File: submitted_models/explorer_spot_sensor_config_1/urdf/spot.urdf.xacro (robot description, xacro)
@@ -17,5 +17,4 @@
     <!-- Include the basic Spot URDF -->
     <xacro:include filename="$(find bosdyn_spot)/urdf/spot.urdf.xacro"/>
-    <xacro:include filename="$(find explorer_spot_sensor_config_1)/urdf/3d_lidar.xacro" />
     <!-- Here is place for all custom URDF code for this sensor config. -->
     <!-- Colon-separated list of payload Xacro files to include. Whitespace around is ignored. -->
@@ -28,4 +27,5 @@
       $(find explorer_spot_sensor_config_1)/urdf/flir_cameras.xacro :
       $(find explorer_spot_sensor_config_1)/urdf/rgbd_camera.xacro :
+      $(find explorer_spot_sensor_config_1)/urdf/3d_lidar.xacro :
     " />
     <!-- Append to this list in included payload Xacro files to count their weight to the total robot mass -->
