Commit message: Updated static tf rate, added mapping server relays, removed the lidar visual link in the xacro, added orientation parameter to the IMU, and added an example RViz file.

File: submitted_models/dynamo_x4_sensor_config_1/urdf/model.xacro (robot description, xacro)
@@ -81,10 +81,4 @@
       </geometry>
     </visual>
-    <visual name='laser_visual'>
-      <origin xyz='0.08 0 0.3' rpy='0 -0 0'/>
-      <geometry>
-        <cylinder radius='0.03' length='0.1'/>
-      </geometry>
-    </visual>
   </link>
   <sensor name='imu_sensor' update_rate='250'>
