Commit message: Updated the xacro

File: submitted_models/marble_hd2_sensor_config_1/urdf/robot_from_sdf.xacro (robot description, xacro)
@@ -18,5 +18,5 @@
       <origin xyz='0 0 0.046' rpy='0 -0 0'/>
       <geometry>
-        <box size='0.8 0.5709 0.095'/>
+        <box size='0.8 0.5709 0.2'/>
       </geometry>
     </collision>
@@ -72,9 +72,21 @@
       <origin xyz='0 0 0' rpy='1.57 -0 1.57'/>
       <geometry>
-        <mesh filename='package://marble_hd2_sensor_config_1/meshes/HD2_Urban_Assembly.stl' scale='1 1 1'/>
+        <mesh filename='package://marble_hd2_sensor_config_1/meshes/hd2_chassis.stl' scale='1 1 1'/>
+      </geometry>
+    </visual>
+    <visual name='track_left_visual'>
+      <origin xyz='0 0.2625 0' rpy='1.57 -0 1.57'/>
+      <geometry>
+        <mesh filename='package://marble_hd2_sensor_config_1/meshes/track.stl' scale='1 1 1'/>
+      </geometry>
+    </visual>
+    <visual name='track_right_visual'>
+      <origin xyz='0 -0.2625 0' rpy='1.57 -0 1.57'/>
+      <geometry>
+        <mesh filename='package://marble_hd2_sensor_config_1/meshes/track.stl' scale='1 1 1'/>
       </geometry>
     </visual>
     <visual name='base_link_fixed_joint_lump__camera/camera_link_visual_1'>
-      <origin xyz='0.478 0 0.26' rpy='0 0.5236 0'/>
+      <origin xyz='0.44 0 0.26' rpy='0 0.5236 0'/>
       <geometry>
         <mesh filename='package://marble_hd2_sensor_config_1/meshes/realsense.dae' scale='1 1 1'/>
@@ -82,5 +94,5 @@
     </visual>
     <visual name='base_link_fixed_joint_lump__camera/camera_link_visual_2'>
-      <origin xyz='0.478 0 0.285' rpy='0 -0 0'/>
+      <origin xyz='0.44 0 0.295' rpy='0 -0 0'/>
       <geometry>
         <mesh filename='package://marble_hd2_sensor_config_1/meshes/realsense.dae' scale='1 1 1'/>
@@ -88,5 +100,5 @@
     </visual>
     <visual name='base_link_fixed_joint_lump__velodyne_base_link_visual_10'>
-      <origin xyz='0.424 0 0.327' rpy='0 -0 0'/>
+      <origin xyz='0.354 0 0.327' rpy='0 -0 0'/>
       <geometry>
         <mesh filename='package://marble_hd2_sensor_config_1/meshes/VLP16_base_1.dae' scale='1 1 1'/>
@@ -94,5 +106,5 @@
     </visual>
     <visual name='base_link_fixed_joint_lump__velodyne_base_link_visual_11'>
-      <origin xyz='0.424 0 0.327' rpy='0 -0 0'/>
+      <origin xyz='0.354 0 0.327' rpy='0 -0 0'/>
       <geometry>
         <mesh filename='package://marble_hd2_sensor_config_1/meshes/VLP16_base_2.dae' scale='1 1 1'/>
@@ -100,5 +112,5 @@
     </visual>
     <visual name='base_link_fixed_joint_lump__velodyne_visual_12'>
-      <origin xyz='0.424 0 0.327' rpy='0 -0 0'/>
+      <origin xyz='0.354 0 0.327' rpy='0 -0 0'/>
       <geometry>
         <mesh filename='package://marble_hd2_sensor_config_1/meshes/VLP16_scan.dae' scale='1 1 1'/>
@@ -106,5 +118,5 @@
     </visual>
     <visual name='base_link_fixed_joint_lump__planar_lidar_link_visual_14'>
-      <origin xyz='0.474 0 0.127' rpy='0 -0 0'/>
+      <origin xyz='0.354 0 0.127' rpy='0 -0 0'/>
       <geometry>
         <cylinder radius='0.045' length='0.05'/>
@@ -112,5 +124,5 @@
     </visual>
     <visual name='base_link_fixed_joint_lump__velodyne_gimbal_plate_15'>
-      <origin xyz='0.424 0 0.4' rpy='0 -0 0'/>
+      <origin xyz='0.354 0 0.4' rpy='0 -0 0'/>
       <geometry>
         <box size='0.12 0.12 0.01'/>
@@ -118,19 +130,25 @@
     </visual>
     <visual name='base_link_fixed_joint_lump__sensor_tower_16'>
-      <origin xyz='0.374 0 0.215' rpy='0 -0 0'/>
-      <geometry>
-        <box size='0.2 0.25 0.225'/>
+      <origin xyz='0.354 0 0.19' rpy='0 -0 0'/>
+      <geometry>
+        <box size='0.18 0.25 0.275'/>
       </geometry>
     </visual>
     <visual name='base_link_fixed_joint_lump__computer_block_17'>
-      <origin xyz='0.05 0 0.185' rpy='0 -0 0'/>
+      <origin xyz='0.05 0 0.135' rpy='0 -0 0'/>
       <geometry>
         <box size='0.3 0.355 0.175'/>
       </geometry>
     </visual>
+    <visual name='base_link_fixed_joint_lid_18'>
+      <origin xyz='0 0 0.05' rpy='0 -0 0'/>
+      <geometry>
+        <box size='0.7 0.35 0.02'/>
+      </geometry>
+    </visual>
   </link>
   <sensor name='camera_front' update_rate='30'>
     <parent link='${robot_namespace}/base_link'/>
-    <origin xyz='0.468 0 0.36' rpy='0 -0 0'/>
+    <origin xyz='0.44 0 0.36' rpy='0 -0 0'/>
     <camera>
       <image width='1280' height='720' format='R8G8B8' hfov='1.5184' near='0.01' far='300' />
@@ -139,5 +157,5 @@
   <sensor name='camera_down' update_rate='30'>
     <parent link='${robot_namespace}/base_link'/>
-    <origin xyz='0.473 0 0.335' rpy='0 0.5236 0'/>
+    <origin xyz='0.44 0 0.335' rpy='0 0.5236 0'/>
     <camera>
       <image width='1280' height='720' format='R8G8B8' hfov='1.5184' near='0.01' far='300' />
@@ -146,11 +164,11 @@
   <sensor name='planar_laser' update_rate='10'>
     <parent link='${robot_namespace}/base_link'/>
-    <origin xyz='0.474 0 0.127' rpy='0 -0 0'/>
+    <origin xyz='0.354 0 0.127' rpy='0 -0 0'/>
   </sensor>
   <sensor name='front_laser' update_rate='20'>
     <parent link='${robot_namespace}/base_link'/>
-    <origin xyz='0.424 0 0.402' rpy='0 -0 0'/>
-  </sensor>
-  <sensor name='imu_sensor' update_rate='50'>
+    <origin xyz='0.354 0 0.402' rpy='0 -0 0'/>
+  </sensor>
+  <sensor name='imu_sensor' update_rate='250'>
     <parent link='${robot_namespace}/base_link'/>
     <origin xyz='0 0 0' rpy='0 -0 0'/>
@@ -165,7 +183,70 @@
       <origin xyz='0 0 0' rpy='1.5708 -0 0'/>
       <geometry>
+        <cylinder radius='0.129' length='0.1'/>
+      </geometry>
+    </collision>
+    <visual name='front_left_wheel_link_visual'>
+      <origin xyz='0 0 0' rpy='1.5708 -0 0'/>
+      <geometry>
+        <cylinder radius='0.129' length='0.1'/>
+      </geometry>
+    </visual>
+  </link>
+  <link name='${robot_namespace}/front_middle_left_wheel_link'>
+    <inertial>
+      <origin xyz='0 0 0' rpy='0 -0 0'/>
+      <mass value='2.637'/>
+      <inertia ixx='0.02467' ixy='0' ixz='0' iyy='0.04411' iyz='0' izz='0.02467'/>
+    </inertial>
+    <collision name='front_middle_left_wheel_link_collision'>
+      <origin xyz='0 0 0' rpy='1.5708 -0 0'/>
+      <geometry>
+        <cylinder radius='0.129' length='0.1'/>
+      </geometry>
+    </collision>
+    <visual name='front_middle_left_wheel_link_visual'>
+      <origin xyz='0 0 0' rpy='1.5708 -0 0'/>
+      <geometry>
+        <cylinder radius='0.129' length='0.1'/>
+      </geometry>
+    </visual>
+  </link>
+  <link name='${robot_namespace}/rear_middle_left_wheel_link'>
+    <inertial>
+      <origin xyz='0 0 0' rpy='0 -0 0'/>
+      <mass value='2.637'/>
+      <inertia ixx='0.02467' ixy='0' ixz='0' iyy='0.04411' iyz='0' izz='0.02467'/>
+    </inertial>
+    <collision name='rear_middle_left_wheel_link_collision'>
+      <origin xyz='0 0 0' rpy='1.5708 -0 0'/>
+      <geometry>
+        <cylinder radius='0.129' length='0.1'/>
+      </geometry>
+    </collision>
+    <visual name='rear_middle_left_wheel_link_visual'>
+      <origin xyz='0 0 0' rpy='1.5708 -0 0'/>
+      <geometry>
+        <cylinder radius='0.129' length='0.1'/>
+      </geometry>
+    </visual>
+  </link>
+  <link name='${robot_namespace}/rear_left_wheel_link'>
+    <inertial>
+      <origin xyz='0 0 0' rpy='0 -0 0'/>
+      <mass value='2.637'/>
+      <inertia ixx='0.02467' ixy='0' ixz='0' iyy='0.04411' iyz='0' izz='0.02467'/>
+    </inertial>
+    <collision name='rear_left_wheel_link_collision'>
+      <origin xyz='0 0 0' rpy='1.5708 -0 0'/>
+      <geometry>
         <cylinder radius='0.1651' length='0.1143'/>
       </geometry>
     </collision>
+    <visual name='rear_left_wheel_link_visual'>
+      <origin xyz='0 0 0' rpy='1.5708 -0 0'/>
+      <geometry>
+        <cylinder radius='0.129' length='0.1'/>
+      </geometry>
+    </visual>
   </link>
   <link name='${robot_namespace}/front_right_wheel_link'>
@@ -178,33 +259,70 @@
       <origin xyz='0 0 0' rpy='1.5708 -0 0'/>
       <geometry>
+        <cylinder radius='0.129' length='0.1'/>
+      </geometry>
+    </collision>
+    <visual name='front_right_wheel_link_visual'>
+      <origin xyz='0 0 0' rpy='1.5708 -0 0'/>
+      <geometry>
+        <cylinder radius='0.129' length='0.1'/>
+      </geometry>
+    </visual>
+  </link>
+  <link name='${robot_namespace}/front_middle_right_wheel_link'>
+    <inertial>
+      <origin xyz='0 0 0' rpy='0 -0 0'/>
+      <mass value='2.637'/>
+      <inertia ixx='0.02467' ixy='0' ixz='0' iyy='0.04411' iyz='0' izz='0.02467'/>
+    </inertial>
+    <collision name='front_middle_right_wheel_link_collision'>
+      <origin xyz='0 0 0' rpy='1.5708 -0 0'/>
+      <geometry>
+        <cylinder radius='0.129' length='0.1'/>
+      </geometry>
+    </collision>
+    <visual name='front_middle_right_wheel_link_visual'>
+      <origin xyz='0 0 0' rpy='1.5708 -0 0'/>
+      <geometry>
+        <cylinder radius='0.129' length='0.1'/>
+      </geometry>
+    </visual>
+  </link>
+  <link name='${robot_namespace}/rear_middle_right_wheel_link'>
+    <inertial>
+      <origin xyz='0 0 0' rpy='0 -0 0'/>
+      <mass value='2.637'/>
+      <inertia ixx='0.02467' ixy='0' ixz='0' iyy='0.04411' iyz='0' izz='0.02467'/>
+    </inertial>
+    <collision name='rear_middle_right_wheel_link_collision'>
+      <origin xyz='0 0 0' rpy='1.5708 -0 0'/>
+      <geometry>
+        <cylinder radius='0.129' length='0.1'/>
+      </geometry>
+    </collision>
+    <visual name='rear_middle_right_wheel_link_visual'>
+      <origin xyz='0 0 0' rpy='1.5708 -0 0'/>
+      <geometry>
+        <cylinder radius='0.129' length='0.1'/>
+      </geometry>
+    </visual>
+  </link>
+  <link name='${robot_namespace}/rear_right_wheel_link'>
+    <inertial>
+      <origin xyz='0 0 0' rpy='0 -0 0'/>
+      <mass value='2.637'/>
+      <inertia ixx='0.02467' ixy='0' ixz='0' iyy='0.04411' iyz='0' izz='0.02467'/>
+    </inertial>
+    <collision name='rear_right_wheel_link_collision'>
+      <origin xyz='0 0 0' rpy='1.5708 -0 0'/>
+      <geometry>
         <cylinder radius='0.1651' length='0.1143'/>
       </geometry>
     </collision>
-  </link>
-  <link name='${robot_namespace}/rear_left_wheel_link'>
-    <inertial>
-      <origin xyz='0 0 0' rpy='0 -0 0'/>
-      <mass value='2.637'/>
-      <inertia ixx='0.02467' ixy='0' ixz='0' iyy='0.04411' iyz='0' izz='0.02467'/>
-    </inertial>
-    <collision name='rear_left_wheel_link_collision'>
-      <origin xyz='0 0 0' rpy='1.5708 -0 0'/>
-      <geometry>
-        <cylinder radius='0.1651' length='0.1143'/>
-      </geometry>
-    </collision>
-  </link>
-  <link name='${robot_namespace}/rear_right_wheel_link'>
-    <inertial>
-      <origin xyz='0 0 0' rpy='0 -0 0'/>
-      <mass value='2.637'/>
-      <inertia ixx='0.02467' ixy='0' ixz='0' iyy='0.04411' iyz='0' izz='0.02467'/>
-    </inertial>
-    <collision name='rear_right_wheel_link_collision'>
-      <origin xyz='0 0 0' rpy='1.5708 -0 0'/>
-      <geometry>
-        <cylinder radius='0.1651' length='0.1143'/>
-      </geometry>
-    </collision>
+    <visual name='rear_right_wheel_link_visual'>
+      <origin xyz='0 0 0' rpy='1.5708 -0 0'/>
+      <geometry>
+        <cylinder radius='0.129' length='0.1'/>
+      </geometry>
+    </visual>
   </link>
   <link name='${robot_namespace}/pan_gimbal_link'>
@@ -278,5 +396,5 @@
   </sensor>
   <joint name='front_left_wheel_joint' type='revolute'>
-    <origin xyz='0.256 0.2854 0.03282' rpy='0 -0 0'/>
+    <origin xyz='0.36 0.26 0' rpy='0 -0 0'/>
     <parent link='${robot_namespace}/base_link'/>
     <child link='${robot_namespace}/front_left_wheel_link'/>
@@ -285,6 +403,30 @@
     <limit lower='-1e+16' upper='1e+16' effort='-1' velocity='-1'/>
   </joint>
+  <joint name='front_middle_left_wheel_joint' type='revolute'>
+    <origin xyz='0.12 0.26 0' rpy='0 -0 0'/>
+    <parent link='${robot_namespace}/base_link'/>
+    <child link='${robot_namespace}/front_middle_left_wheel_link'/>
+    <dynamics damping='0' friction='0' />
+    <axis xyz='0 1 0'/>
+    <limit lower='-1e+16' upper='1e+16' effort='-1' velocity='-1'/>
+  </joint>
+  <joint name='rear_middle_left_wheel_joint' type='revolute'>
+    <origin xyz='-0.12 0.26 0' rpy='0 -0 0'/>
+    <parent link='${robot_namespace}/base_link'/>
+    <child link='${robot_namespace}/rear_middle_left_wheel_link'/>
+    <dynamics damping='0' friction='0' />
+    <axis xyz='0 1 0'/>
+    <limit lower='-1e+16' upper='1e+16' effort='-1' velocity='-1'/>
+  </joint>
+  <joint name='rear_left_wheel_joint' type='revolute'>
+    <origin xyz='-0.36 0.26 0' rpy='0 -0 0'/>
+    <parent link='${robot_namespace}/base_link'/>
+    <child link='${robot_namespace}/rear_left_wheel_link'/>
+    <dynamics damping='0' friction='0' />
+    <axis xyz='0 1 0'/>
+    <limit lower='-1e+16' upper='1e+16' effort='-1' velocity='-1'/>
+  </joint>
   <joint name='front_right_wheel_joint' type='revolute'>
-    <origin xyz='0.256 -0.2854 0.03282' rpy='0 -0 0'/>
+    <origin xyz='0.36 -0.26 0' rpy='0 -0 0'/>
     <parent link='${robot_namespace}/base_link'/>
     <child link='${robot_namespace}/front_right_wheel_link'/>
@@ -293,8 +435,16 @@
     <limit lower='-1e+16' upper='1e+16' effort='-1' velocity='-1'/>
   </joint>
-  <joint name='rear_left_wheel_joint' type='revolute'>
-    <origin xyz='-0.256 0.2854 0.03282' rpy='0 -0 0'/>
-    <parent link='${robot_namespace}/base_link'/>
-    <child link='${robot_namespace}/rear_left_wheel_link'/>
+  <joint name='front_middle_right_wheel_joint' type='revolute'>
+    <origin xyz='0.12 -0.26 0' rpy='0 -0 0'/>
+    <parent link='${robot_namespace}/base_link'/>
+    <child link='${robot_namespace}/front_middle_right_wheel_link'/>
+    <dynamics damping='0' friction='0' />
+    <axis xyz='0 1 0'/>
+    <limit lower='-1e+16' upper='1e+16' effort='-1' velocity='-1'/>
+  </joint>
+  <joint name='rear_middle_right_wheel_joint' type='revolute'>
+    <origin xyz='-0.12 -0.26 0' rpy='0 -0 0'/>
+    <parent link='${robot_namespace}/base_link'/>
+    <child link='${robot_namespace}/rear_middle_right_wheel_link'/>
     <dynamics damping='0' friction='0' />
     <axis xyz='0 1 0'/>
@@ -302,5 +452,5 @@
   </joint>
   <joint name='rear_right_wheel_joint' type='revolute'>
-    <origin xyz='-0.256 -0.2854 0.03282' rpy='0 -0 0'/>
+    <origin xyz='-0.36 -0.26 0' rpy='0 -0 0'/>
     <parent link='${robot_namespace}/base_link'/>
     <child link='${robot_namespace}/rear_right_wheel_link'/>
@@ -310,5 +460,5 @@
   </joint>
   <joint name='pan_gimbal_joint' type='revolute'>
-    <origin xyz='0.424 0 0.427' rpy='0 -0 0'/>
+    <origin xyz='0.354 0 0.427' rpy='0 -0 0'/>
     <parent link='${robot_namespace}/base_link'/>
     <child link='${robot_namespace}/pan_gimbal_link'/>
@@ -318,5 +468,5 @@
   </joint>
   <joint name='tilt_gimbal_joint' type='revolute'>
-    <origin xyz='0.424 0 0.46' rpy='0 -0 0'/>
+    <origin xyz='0.354 0 0.46' rpy='0 -0 0'/>
     <parent link='${robot_namespace}/pan_gimbal_link'/>
     <child link='${robot_namespace}/tilt_gimbal_link'/>

Commit message: Fixed urdf and xacro

File: submitted_models/marble_hd2_sensor_config_1/urdf/robot_from_sdf.xacro (robot description, xacro)
@@ -64,7 +64,7 @@
     </collision>
     <collision name='base_link_fixed_joint_lump__computer_block_9'>
-      <origin xyz='0.05 0 0.185' rpy='0 -0 0'/>
-      <geometry>
-        <box size='0.3 0.355 0.175'/>
+      <origin xyz='0.05 0 0.155' rpy='0 -0 0'/>
+      <geometry>
+        <box size='0.3 0.355 0.16'/>
       </geometry>
     </collision>
@@ -126,5 +126,5 @@
       <origin xyz='0.354 0 0.4' rpy='0 -0 0'/>
       <geometry>
-        <box size='0.12 0.12 0.01'/>
+        <box size='0.06 0.06 0.01'/>
       </geometry>
     </visual>
@@ -168,5 +168,5 @@
   <sensor name='front_laser' update_rate='20'>
     <parent link='${robot_namespace}/base_link'/>
-    <origin xyz='0.354 0 0.402' rpy='0 -0 0'/>
+    <origin xyz='0.354 0 0.387' rpy='0 -0 0'/>
   </sensor>
   <sensor name='imu_sensor' update_rate='250'>
