Commit message: CSIRO_OZBOT_ATR: Implemented proper track model.

File: submitted_models/csiro_data61_ozbot_atr_sensor_config_1/urdf/robot_from_sdf.xacro (robot description, xacro)
@@ -228,31 +228,12 @@
     <origin xyz='0 0 0' rpy='0 -0 0'/>
   </sensor>
-  <link name='${robot_namespace}/left_10_wheel'>
+  <link name='${robot_namespace}/left_track'>
     <inertial>
       <origin xyz='0 0 0' rpy='0 -0 0'/>
       <mass value='2'/>
-      <inertia ixx='0.0164667' ixy='0' ixz='0' iyy='0.0164667' iyz='0' izz='0.0196'/>
-    </inertial>
-    <collision name='left_10_wheel_collision'>
-      <origin xyz='0 0 0' rpy='1.5708 -0 0'/>
-      <geometry>
-        <cylinder radius='0.14' length='0.2'/>
-      </geometry>
-    </collision>
-    <visual name='left_10_wheel_visual'>
-      <origin xyz='0 0 0' rpy='1.5708 -0 0'/>
-      <geometry>
-        <cylinder radius='0.14' length='0.2'/>
-      </geometry>
-    </visual>
-  </link>
-  <link name='${robot_namespace}/left_11_wheel'>
-    <inertial>
-      <origin xyz='0 0 0' rpy='0 -0 0'/>
-      <mass value='2'/>
-      <inertia ixx='0.0164667' ixy='0' ixz='0' iyy='0.0164667' iyz='0' izz='0.0196'/>
+      <inertia ixx='0.1467' ixy='0' ixz='0' iyy='2.0754' iyz='0' izz='2.0754'/>
     </inertial>
     <collision name='left_11_wheel_collision'>
-      <origin xyz='0 0 0' rpy='1.5708 -0 0'/>
+      <origin xyz='-0.64 0 0.183' rpy='1.5708 -0 0'/>
       <geometry>
         <cylinder radius='0.14' length='0.2'/>
@@ -260,208 +241,95 @@
     </collision>
     <visual name='left_11_wheel_visual'>
-      <origin xyz='0 0 0' rpy='1.5708 -0 0'/>
-      <geometry>
-        <cylinder radius='0.14' length='0.2'/>
+      <origin xyz='-0.64 0 0.183' rpy='1.5708 -0 0'/>
+      <geometry>
+        <cylinder radius='0.14' length='0.2'/>
+      </geometry>
+    </visual>
+    <collision name='left_1_wheel_collision'>
+      <origin xyz='0.693 0 0.21' rpy='1.5708 -0 0'/>
+      <geometry>
+        <cylinder radius='0.11' length='0.2'/>
+      </geometry>
+    </collision>
+    <visual name='left_1_wheel_visual'>
+      <origin xyz='0.693 0 0.21' rpy='1.5708 -0 0'/>
+      <geometry>
+        <cylinder radius='0.11' length='0.2'/>
+      </geometry>
+    </visual>
+    <collision name='left_3_wheel_collision'>
+      <origin xyz='0.485 0 -0.037758' rpy='1.5708 -0 0'/>
+      <geometry>
+        <cylinder radius='0.14' length='0.2'/>
+      </geometry>
+    </collision>
+    <visual name='left_3_wheel_visual'>
+      <origin xyz='0.485 0 -0.037758' rpy='1.5708 -0 0'/>
+      <geometry>
+        <cylinder radius='0.14' length='0.2'/>
+      </geometry>
+    </visual>
+    <collision name='left_9_wheel_collision'>
+      <origin xyz='-0.56 0 -0.07' rpy='1.5708 -0 0'/>
+      <geometry>
+        <cylinder radius='0.11' length='0.2'/>
+      </geometry>
+    </collision>
+    <visual name='left_9_wheel_visual'>
+      <origin xyz='-0.56 0 -0.07' rpy='1.5708 -0 0'/>
+      <geometry>
+        <cylinder radius='0.11' length='0.2'/>
+      </geometry>
+    </visual>
+    <collision name='left_bottom_box_collision'>
+      <origin xyz='-0.0375 0 -0.068' rpy='0 0 0'/>
+      <geometry>
+        <box size='1.045 0.2 0.22' />
+      </geometry>
+    </collision>
+    <visual name='left_bottom_box_visual'>
+      <origin xyz='-0.0375 0 -0.068' rpy='0 0 0'/>
+      <geometry>
+        <box size='1.045 0.2 0.22' />
+      </geometry>
+    </visual>
+    <collision name='left_rear_box_collision'>
+      <origin xyz='-0.612 0 0.05114' rpy='0 1.15017 0'/>
+      <geometry>
+        <box size='0.285 0.2 0.22' />
+      </geometry>
+    </collision>
+    <visual name='left_rear_box_visual'>
+      <origin xyz='-0.612 0 0.05114' rpy='0 1.15017 0'/>
+      <geometry>
+        <box size='0.285 0.2 0.22' />
+      </geometry>
+    </visual>
+    <collision name='left_front_box_collision'>
+      <origin xyz='0.6 0 0.07898' rpy='0 -0.96517 0'/>
+      <geometry>
+        <box size='0.35 0.2 0.22' />
+      </geometry>
+    </collision>
+    <visual name='left_front_box_visual'>
+      <origin xyz='0.6 0 0.07898' rpy='0 -0.96517 0'/>
+      <geometry>
+        <box size='0.35 0.2 0.22' />
       </geometry>
     </visual>
   </link>
-  <link name='${robot_namespace}/left_1_wheel'>
+  <joint name='left_track_j' type='fixed'>
+    <origin xyz='0 0.269 0' rpy='0 0 0'/>
+    <parent link='${robot_namespace}/base_link'/>
+    <child link='${robot_namespace}/left_track'/>
+  </joint>
+  <link name='${robot_namespace}/right_track'>
     <inertial>
       <origin xyz='0 0 0' rpy='0 -0 0'/>
       <mass value='2'/>
-      <inertia ixx='0.0164667' ixy='0' ixz='0' iyy='0.0164667' iyz='0' izz='0.0196'/>
-    </inertial>
-    <collision name='left_1_wheel_collision'>
-      <origin xyz='0 0 0' rpy='1.5708 -0 0'/>
-      <geometry>
-        <cylinder radius='0.14' length='0.2'/>
-      </geometry>
-    </collision>
-    <visual name='left_1_wheel_visual'>
-      <origin xyz='0 0 0' rpy='1.5708 -0 0'/>
-      <geometry>
-        <cylinder radius='0.14' length='0.2'/>
-      </geometry>
-    </visual>
-  </link>
-  <link name='${robot_namespace}/left_2_wheel'>
-    <inertial>
-      <origin xyz='0 0 0' rpy='0 -0 0'/>
-      <mass value='2'/>
-      <inertia ixx='0.0164667' ixy='0' ixz='0' iyy='0.0164667' iyz='0' izz='0.0196'/>
-    </inertial>
-    <collision name='left_2_wheel_collision'>
-      <origin xyz='0 0 0' rpy='1.5708 -0 0'/>
-      <geometry>
-        <cylinder radius='0.14' length='0.2'/>
-      </geometry>
-    </collision>
-    <visual name='left_2_wheel_visual'>
-      <origin xyz='0 0 0' rpy='1.5708 -0 0'/>
-      <geometry>
-        <cylinder radius='0.14' length='0.2'/>
-      </geometry>
-    </visual>
-  </link>
-  <link name='${robot_namespace}/left_3_wheel'>
-    <inertial>
-      <origin xyz='0 0 0' rpy='0 -0 0'/>
-      <mass value='2'/>
-      <inertia ixx='0.0164667' ixy='0' ixz='0' iyy='0.0164667' iyz='0' izz='0.0196'/>
-    </inertial>
-    <collision name='left_3_wheel_collision'>
-      <origin xyz='0 0 0' rpy='1.5708 -0 0'/>
-      <geometry>
-        <cylinder radius='0.14' length='0.2'/>
-      </geometry>
-    </collision>
-    <visual name='left_3_wheel_visual'>
-      <origin xyz='0 0 0' rpy='1.5708 -0 0'/>
-      <geometry>
-        <cylinder radius='0.14' length='0.2'/>
-      </geometry>
-    </visual>
-  </link>
-  <link name='${robot_namespace}/left_4_wheel'>
-    <inertial>
-      <origin xyz='0 0 0' rpy='0 -0 0'/>
-      <mass value='2'/>
-      <inertia ixx='0.0164667' ixy='0' ixz='0' iyy='0.0164667' iyz='0' izz='0.0196'/>
-    </inertial>
-    <collision name='left_4_wheel_collision'>
-      <origin xyz='0 0 0' rpy='1.5708 -0 0'/>
-      <geometry>
-        <cylinder radius='0.14' length='0.2'/>
-      </geometry>
-    </collision>
-    <visual name='left_4_wheel_visual'>
-      <origin xyz='0 0 0' rpy='1.5708 -0 0'/>
-      <geometry>
-        <cylinder radius='0.14' length='0.2'/>
-      </geometry>
-    </visual>
-  </link>
-  <link name='${robot_namespace}/left_5_wheel'>
-    <inertial>
-      <origin xyz='0 0 0' rpy='0 -0 0'/>
-      <mass value='2'/>
-      <inertia ixx='0.0164667' ixy='0' ixz='0' iyy='0.0164667' iyz='0' izz='0.0196'/>
-    </inertial>
-    <collision name='left_5_wheel_collision'>
-      <origin xyz='0 0 0' rpy='1.5708 -0 0'/>
-      <geometry>
-        <cylinder radius='0.14' length='0.2'/>
-      </geometry>
-    </collision>
-    <visual name='left_5_wheel_visual'>
-      <origin xyz='0 0 0' rpy='1.5708 -0 0'/>
-      <geometry>
-        <cylinder radius='0.14' length='0.2'/>
-      </geometry>
-    </visual>
-  </link>
-  <link name='${robot_namespace}/left_6_wheel'>
-    <inertial>
-      <origin xyz='0 0 0' rpy='0 -0 0'/>
-      <mass value='2'/>
-      <inertia ixx='0.0164667' ixy='0' ixz='0' iyy='0.0164667' iyz='0' izz='0.0196'/>
-    </inertial>
-    <collision name='left_6_wheel_collision'>
-      <origin xyz='0 0 0' rpy='1.5708 -0 0'/>
-      <geometry>
-        <cylinder radius='0.14' length='0.2'/>
-      </geometry>
-    </collision>
-    <visual name='left_6_wheel_visual'>
-      <origin xyz='0 0 0' rpy='1.5708 -0 0'/>
-      <geometry>
-        <cylinder radius='0.14' length='0.2'/>
-      </geometry>
-    </visual>
-  </link>
-  <link name='${robot_namespace}/left_7_wheel'>
-    <inertial>
-      <origin xyz='0 0 0' rpy='0 -0 0'/>
-      <mass value='2'/>
-      <inertia ixx='0.0164667' ixy='0' ixz='0' iyy='0.0164667' iyz='0' izz='0.0196'/>
-    </inertial>
-    <collision name='left_7_wheel_collision'>
-      <origin xyz='0 0 0' rpy='1.5708 -0 0'/>
-      <geometry>
-        <cylinder radius='0.14' length='0.2'/>
-      </geometry>
-    </collision>
-    <visual name='left_7_wheel_visual'>
-      <origin xyz='0 0 0' rpy='1.5708 -0 0'/>
-      <geometry>
-        <cylinder radius='0.14' length='0.2'/>
-      </geometry>
-    </visual>
-  </link>
-  <link name='${robot_namespace}/left_8_wheel'>
-    <inertial>
-      <origin xyz='0 0 0' rpy='0 -0 0'/>
-      <mass value='2'/>
-      <inertia ixx='0.0164667' ixy='0' ixz='0' iyy='0.0164667' iyz='0' izz='0.0196'/>
-    </inertial>
-    <collision name='left_8_wheel_collision'>
-      <origin xyz='0 0 0' rpy='1.5708 -0 0'/>
-      <geometry>
-        <cylinder radius='0.14' length='0.2'/>
-      </geometry>
-    </collision>
-    <visual name='left_8_wheel_visual'>
-      <origin xyz='0 0 0' rpy='1.5708 -0 0'/>
-      <geometry>
-        <cylinder radius='0.14' length='0.2'/>
-      </geometry>
-    </visual>
-  </link>
-  <link name='${robot_namespace}/left_9_wheel'>
-    <inertial>
-      <origin xyz='0 0 0' rpy='0 -0 0'/>
-      <mass value='2'/>
-      <inertia ixx='0.0164667' ixy='0' ixz='0' iyy='0.0164667' iyz='0' izz='0.0196'/>
-    </inertial>
-    <collision name='left_9_wheel_collision'>
-      <origin xyz='0 0 0' rpy='1.5708 -0 0'/>
-      <geometry>
-        <cylinder radius='0.14' length='0.2'/>
-      </geometry>
-    </collision>
-    <visual name='left_9_wheel_visual'>
-      <origin xyz='0 0 0' rpy='1.5708 -0 0'/>
-      <geometry>
-        <cylinder radius='0.14' length='0.2'/>
-      </geometry>
-    </visual>
-  </link>
-  <link name='${robot_namespace}/right_10_wheel'>
-    <inertial>
-      <origin xyz='0 0 0' rpy='0 -0 0'/>
-      <mass value='2'/>
-      <inertia ixx='0.0164667' ixy='0' ixz='0' iyy='0.0164667' iyz='0' izz='0.0196'/>
-    </inertial>
-    <collision name='right_10_wheel_collision'>
-      <origin xyz='0 0 0' rpy='1.5708 -0 0'/>
-      <geometry>
-        <cylinder radius='0.14' length='0.2'/>
-      </geometry>
-    </collision>
-    <visual name='right_10_wheel_visual'>
-      <origin xyz='0 0 0' rpy='1.5708 -0 0'/>
-      <geometry>
-        <cylinder radius='0.14' length='0.2'/>
-      </geometry>
-    </visual>
-  </link>
-  <link name='${robot_namespace}/right_11_wheel'>
-    <inertial>
-      <origin xyz='0 0 0' rpy='0 -0 0'/>
-      <mass value='2'/>
-      <inertia ixx='0.0164667' ixy='0' ixz='0' iyy='0.0164667' iyz='0' izz='0.0196'/>
+      <inertia ixx='0.1467' ixy='0' ixz='0' iyy='2.0754' iyz='0' izz='2.0754'/>
     </inertial>
     <collision name='right_11_wheel_collision'>
-      <origin xyz='0 0 0' rpy='1.5708 -0 0'/>
+      <origin xyz='-0.64 0 0.183' rpy='1.5708 -0 0'/>
       <geometry>
         <cylinder radius='0.14' length='0.2'/>
@@ -469,181 +337,87 @@
     </collision>
     <visual name='right_11_wheel_visual'>
-      <origin xyz='0 0 0' rpy='1.5708 -0 0'/>
-      <geometry>
-        <cylinder radius='0.14' length='0.2'/>
+      <origin xyz='-0.64 0 0.183' rpy='1.5708 -0 0'/>
+      <geometry>
+        <cylinder radius='0.14' length='0.2'/>
+      </geometry>
+    </visual>
+    <collision name='right_1_wheel_collision'>
+      <origin xyz='0.693 0 0.21' rpy='1.5708 -0 0'/>
+      <geometry>
+        <cylinder radius='0.11' length='0.2'/>
+      </geometry>
+    </collision>
+    <visual name='right_1_wheel_visual'>
+      <origin xyz='0.693 0 0.21' rpy='1.5708 -0 0'/>
+      <geometry>
+        <cylinder radius='0.11' length='0.2'/>
+      </geometry>
+    </visual>
+    <collision name='right_3_wheel_collision'>
+      <origin xyz='0.485 0 -0.037758' rpy='1.5708 -0 0'/>
+      <geometry>
+        <cylinder radius='0.14' length='0.2'/>
+      </geometry>
+    </collision>
+    <visual name='right_3_wheel_visual'>
+      <origin xyz='0.485 0 -0.037758' rpy='1.5708 -0 0'/>
+      <geometry>
+        <cylinder radius='0.14' length='0.2'/>
+      </geometry>
+    </visual>
+    <collision name='right_9_wheel_collision'>
+      <origin xyz='-0.56 0 -0.07' rpy='1.5708 -0 0'/>
+      <geometry>
+        <cylinder radius='0.11' length='0.2'/>
+      </geometry>
+    </collision>
+    <visual name='right_9_wheel_visual'>
+      <origin xyz='-0.56 0 -0.07' rpy='1.5708 -0 0'/>
+      <geometry>
+        <cylinder radius='0.11' length='0.2'/>
+      </geometry>
+    </visual>
+    <collision name='right_bottom_box_collision'>
+      <origin xyz='-0.0375 0 -0.068' rpy='0 0 0'/>
+      <geometry>
+        <box size='1.045 0.2 0.22' />
+      </geometry>
+    </collision>
+    <visual name='right_bottom_box_visual'>
+      <origin xyz='-0.0375 0 -0.068' rpy='0 0 0'/>
+      <geometry>
+        <box size='1.045 0.2 0.22' />
+      </geometry>
+    </visual>
+    <collision name='right_rear_box_collision'>
+      <origin xyz='-0.612 0 0.05114' rpy='0 1.15017 0'/>
+      <geometry>
+        <box size='0.285 0.2 0.22' />
+      </geometry>
+    </collision>
+    <visual name='right_rear_box_visual'>
+      <origin xyz='-0.612 0 0.05114' rpy='0 1.15017 0'/>
+      <geometry>
+        <box size='0.285 0.2 0.22' />
+      </geometry>
+    </visual>
+    <collision name='right_front_box_collision'>
+      <origin xyz='0.6 0 0.07898' rpy='0 -0.96517 0'/>
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